Commit message: Clean up after motoman package rename to motoman_config and dx100.
git-svn-id: https://swri-ros-pkg.googlecode.com/svn/branches/stack_reorg@347 076cdf4d-ed99-c8c1-5d01-9bc0d27e81bd

File: motoman_config/cfg/sia10d_mesh.xacro (robot description, xacro)
@@ -1,5 +1,5 @@
 <?xml version="1.0" ?>
 <robot name="sia10d_mesh" xmlns:xacro="http://ros.org/wiki/xacro">
-	<include filename="$(find motoman)/cfg/sia10d_mesh_macro.xacro" />
+	<include filename="$(find motoman_config)/cfg/sia10d_mesh_macro.xacro" />
 	<xacro:sia10d_mesh prefix=""/>
 </robot>

File: motoman_config/cfg/sia10d_mesh_macro.xacro (robot description, xacro)
@@ -6,5 +6,5 @@
 			<visual>
 				<geometry>
-					<mesh filename="package://motoman/meshes/sia10d/visual/MOTOMAN_BASE.stl" />
+					<mesh filename="package://motoman_config/meshes/sia10d/visual/MOTOMAN_BASE.stl" />
 				</geometry>
 				<material name="blue">
@@ -14,5 +14,5 @@
 			<collision>
 				<geometry>
-					<mesh filename="package://motoman/meshes/sia10d/collision/MOTOMAN_BASE.stl" />
+					<mesh filename="package://motoman_config/meshes/sia10d/collision/MOTOMAN_BASE.stl" />
 				</geometry>
 				<material name="yellow">
@@ -24,5 +24,5 @@
 			<visual>
 				<geometry>
-					<mesh filename="package://motoman/meshes/sia10d/visual/MOTOMAN_AXIS_S.stl"/>
+					<mesh filename="package://motoman_config/meshes/sia10d/visual/MOTOMAN_AXIS_S.stl"/>
 				</geometry>
 				<material name="silver">
@@ -32,5 +32,5 @@
 			<collision>
 				<geometry>
-					<mesh filename="package://motoman/meshes/sia10d/collision/MOTOMAN_AXIS_S.stl" />
+					<mesh filename="package://motoman_config/meshes/sia10d/collision/MOTOMAN_AXIS_S.stl" />
 				</geometry>
 				<material name="yellow"/>
@@ -41,5 +41,5 @@
 				<origin rpy="1.57 3.1416 0" xyz="0 0 0"/>
 				<geometry>
-					<mesh filename="package://motoman/meshes/sia10d/visual/MOTOMAN_AXIS_L.stl"/>
+					<mesh filename="package://motoman_config/meshes/sia10d/visual/MOTOMAN_AXIS_L.stl"/>
 				</geometry>
 				<material name="blue"/>
@@ -48,5 +48,5 @@
 				<origin rpy="1.57 3.1416 0" xyz="0 0 0"/>
 				<geometry>
-					<mesh filename="package://motoman/meshes/sia10d/collision/MOTOMAN_AXIS_L.stl" />
+					<mesh filename="package://motoman_config/meshes/sia10d/collision/MOTOMAN_AXIS_L.stl" />
 				</geometry>
 				<material name="yellow"/>
@@ -57,5 +57,5 @@
 				<origin rpy="0 0 3.1415" xyz="0 0 0"/>
 				<geometry>
-					<mesh filename="package://motoman/meshes/sia10d/visual/MOTOMAN_AXIS_E.stl"/>
+					<mesh filename="package://motoman_config/meshes/sia10d/visual/MOTOMAN_AXIS_E.stl"/>
 				</geometry>
 				<material name="silver"/>
@@ -64,5 +64,5 @@
 				<origin rpy="0 0 3.1415" xyz="0 0 0"/>
 				<geometry>
-					<mesh filename="package://motoman/meshes/sia10d/collision/MOTOMAN_AXIS_E.stl" />
+					<mesh filename="package://motoman_config/meshes/sia10d/collision/MOTOMAN_AXIS_E.stl" />
 				</geometry>
 				<material name="yellow"/>
@@ -73,5 +73,5 @@
 				<origin rpy="1.57 -3.1415 0" xyz="0 0 0"/>
 				<geometry>
-					<mesh filename="package://motoman/meshes/sia10d/visual/MOTOMAN_AXIS_U.stl"/>
+					<mesh filename="package://motoman_config/meshes/sia10d/visual/MOTOMAN_AXIS_U.stl"/>
 				</geometry>
 				<material name="blue"/>
@@ -80,5 +80,5 @@
 				<origin rpy="1.57 -3.1415 0" xyz="0 0 0"/>
 				<geometry>
-					<mesh filename="package://motoman/meshes/sia10d/collision/MOTOMAN_AXIS_U.stl" />
+					<mesh filename="package://motoman_config/meshes/sia10d/collision/MOTOMAN_AXIS_U.stl" />
 				</geometry>
 				<material name="yellow"/>
@@ -89,5 +89,5 @@
 				<origin rpy="0 0 3.1416" xyz="0 0 0"/>
 				<geometry>
-					<mesh filename="package://motoman/meshes/sia10d/visual/MOTOMAN_AXIS_R.stl"/>
+					<mesh filename="package://motoman_config/meshes/sia10d/visual/MOTOMAN_AXIS_R.stl"/>
 				</geometry>
 				<material name="silver"/>
@@ -96,5 +96,5 @@
 				<origin rpy="0 0 3.1416" xyz="0 0 0"/>
 				<geometry>
-					<mesh filename="package://motoman/meshes/sia10d/collision/MOTOMAN_AXIS_R.stl" />
+					<mesh filename="package://motoman_config/meshes/sia10d/collision/MOTOMAN_AXIS_R.stl" />
 				</geometry>
 				<material name="yellow"/>
@@ -105,5 +105,5 @@
 				<origin rpy="-1.57 0 3.1416" xyz="0 0 0"/>
 				<geometry>
-					<mesh filename="package://motoman/meshes/sia10d/visual/MOTOMAN_AXIS_B.stl"/>
+					<mesh filename="package://motoman_config/meshes/sia10d/visual/MOTOMAN_AXIS_B.stl"/>
 				</geometry>
 				<material name="blue"/>
@@ -112,5 +112,5 @@
 				<origin rpy="-1.57 0 3.1416" xyz="0 0 0"/>
 				<geometry>
-					<mesh filename="package://motoman/meshes/sia10d/collision/MOTOMAN_AXIS_B.stl" />
+					<mesh filename="package://motoman_config/meshes/sia10d/collision/MOTOMAN_AXIS_B.stl" />
 				</geometry>
 				<material name="yellow"/>
@@ -120,5 +120,5 @@
 			<visual>
 				<geometry>
-					<mesh filename="package://motoman/meshes/sia10d/visual/MOTOMAN_AXIS_T.stl" />
+					<mesh filename="package://motoman_config/meshes/sia10d/visual/MOTOMAN_AXIS_T.stl" />
 				</geometry>
 				<material name="silver"/>
@@ -126,5 +126,5 @@
 			<collision>
 				<geometry>
-					<mesh filename="package://motoman/meshes/sia10d/collision/MOTOMAN_AXIS_T.stl" />
+					<mesh filename="package://motoman_config/meshes/sia10d/collision/MOTOMAN_AXIS_T.stl" />
 				</geometry>
 				<material name="yellow"/>

File: motoman_config/cfg/sia20d_mesh.xacro (robot description, xacro)
@@ -1,5 +1,5 @@
 <?xml version="1.0" ?>
 <robot name="SIA20D_Mesh" xmlns:xacro="http://ros.org/wiki/xacro">
-	<include filename="$(find motoman)/cfg/sia20d_mesh_macro.xacro" />
+	<include filename="$(find motoman_config)/cfg/sia20d_mesh_macro.xacro" />
 	<xacro:sia20d_mesh prefix=""/>
 </robot>

File: motoman_config/cfg/sia20d_mesh_macro.xacro (robot description, xacro)
@@ -5,5 +5,5 @@
 			<visual>
 				<geometry>
-					<mesh filename="package://motoman/meshes/sia20d/visual/MOTOMAN_BASE.stl" />
+					<mesh filename="package://motoman_config/meshes/sia20d/visual/MOTOMAN_BASE.stl" />
 				</geometry>
 				<material name="blue">
@@ -13,5 +13,5 @@
 			<collision>
 				<geometry>
-					<mesh filename="package://motoman/meshes/sia20d/collision/MOTOMAN_BASE.stl" />
+					<mesh filename="package://motoman_config/meshes/sia20d/collision/MOTOMAN_BASE.stl" />
 				</geometry>
 				<material name="yellow">
@@ -24,5 +24,5 @@
 				<origin rpy="0 0 3.1416" xyz="0 0 0"/>
 				<geometry>
-					<mesh filename="package://motoman/meshes/sia20d/visual/MOTOMAN_AXIS_S.stl"/>
+					<mesh filename="package://motoman_config/meshes/sia20d/visual/MOTOMAN_AXIS_S.stl"/>
 				</geometry>
 				<material name="silver">
@@ -33,5 +33,5 @@
 				<origin rpy="0 0 3.1416" xyz="0 0 0"/>
 				<geometry>
-					<mesh filename="package://motoman/meshes/sia20d/collision/MOTOMAN_AXIS_S.stl" />
+					<mesh filename="package://motoman_config/meshes/sia20d/collision/MOTOMAN_AXIS_S.stl" />
 				</geometry>
 				<material name="yellow"/>
@@ -42,5 +42,5 @@
 				<origin rpy="1.57 3.1416 3.1416" xyz="0 0 0"/>
 				<geometry>
-					<mesh filename="package://motoman/meshes/sia20d/visual/MOTOMAN_AXIS_L.stl"/>
+					<mesh filename="package://motoman_config/meshes/sia20d/visual/MOTOMAN_AXIS_L.stl"/>
 				</geometry>
 				<material name="blue"/>
@@ -49,5 +49,5 @@
 				<origin rpy="1.57 3.1416 3.1416" xyz="0 0 0"/>
 				<geometry>
-					<mesh filename="package://motoman/meshes/sia20d/collision/MOTOMAN_AXIS_L.stl"/>
+					<mesh filename="package://motoman_config/meshes/sia20d/collision/MOTOMAN_AXIS_L.stl"/>
 				</geometry>
 				<material name="yellow"/>
@@ -58,5 +58,5 @@
 				<origin rpy="0 0 0" xyz="0 0 0"/>
 				<geometry>
-					<mesh filename="package://motoman/meshes/sia20d/visual/MOTOMAN_AXIS_E.stl"/>
+					<mesh filename="package://motoman_config/meshes/sia20d/visual/MOTOMAN_AXIS_E.stl"/>
 				</geometry>
 				<material name="silver"/>
@@ -65,5 +65,5 @@
 				<origin rpy="0 0 0" xyz="0 0 0"/>
 				<geometry>
-					<mesh filename="package://motoman/meshes/sia20d/collision/MOTOMAN_AXIS_E.stl"/>
+					<mesh filename="package://motoman_config/meshes/sia20d/collision/MOTOMAN_AXIS_E.stl"/>
 				</geometry>
 				<material name="yellow"/>
@@ -74,5 +74,5 @@
 				<origin rpy="1.57 -3.1415 3.1416" xyz="0 0 0"/>
 				<geometry>
-					<mesh filename="package://motoman/meshes/sia20d/visual/MOTOMAN_AXIS_U.stl"/>
+					<mesh filename="package://motoman_config/meshes/sia20d/visual/MOTOMAN_AXIS_U.stl"/>
 				</geometry>
 				<material name="blue"/>
@@ -81,5 +81,5 @@
 				<origin rpy="1.57 -3.1415 3.1416" xyz="0 0 0"/>
 				<geometry>
-					<mesh filename="package://motoman/meshes/sia20d/collision/MOTOMAN_AXIS_U.stl"/>
+					<mesh filename="package://motoman_config/meshes/sia20d/collision/MOTOMAN_AXIS_U.stl"/>
 				</geometry>
 				<material name="yellow"/>
@@ -90,5 +90,5 @@
 				<origin rpy="0 0 0" xyz="0 0 0"/>
 				<geometry>
-					<mesh filename="package://motoman/meshes/sia20d/visual/MOTOMAN_AXIS_R.stl"/>
+					<mesh filename="package://motoman_config/meshes/sia20d/visual/MOTOMAN_AXIS_R.stl"/>
 				</geometry>
 				<material name="silver"/>
@@ -97,5 +97,5 @@
 				<origin rpy="0 0 0" xyz="0 0 0"/>
 				<geometry>
-					<mesh filename="package://motoman/meshes/sia20d/collision/MOTOMAN_AXIS_R.stl"/>
+					<mesh filename="package://motoman_config/meshes/sia20d/collision/MOTOMAN_AXIS_R.stl"/>
 				</geometry>
 				<material name="yellow"/>
@@ -106,5 +106,5 @@
 				<origin rpy="-1.57 0 0" xyz="0 0 0"/>
 				<geometry>
-					<mesh filename="package://motoman/meshes/sia20d/visual/MOTOMAN_AXIS_B.stl"/>
+					<mesh filename="package://motoman_config/meshes/sia20d/visual/MOTOMAN_AXIS_B.stl"/>
 				</geometry>
 				<material name="blue"/>
@@ -113,5 +113,5 @@
 				<origin rpy="-1.57 0 0" xyz="0 0 0"/>
 				<geometry>
-					<mesh filename="package://motoman/meshes/sia20d/collision/MOTOMAN_AXIS_B.stl"/>
+					<mesh filename="package://motoman_config/meshes/sia20d/collision/MOTOMAN_AXIS_B.stl"/>
 				</geometry>
 				<material name="yellow"/>
@@ -121,5 +121,5 @@
 			<visual>
 				<geometry>
-					<mesh filename="package://motoman/meshes/sia20d/visual/MOTOMAN_AXIS_T.stl" />
+					<mesh filename="package://motoman_config/meshes/sia20d/visual/MOTOMAN_AXIS_T.stl" />
 				</geometry>
 				<material name="silver"/>
@@ -127,5 +127,5 @@
 			<collision>
 				<geometry>
-					<mesh filename="package://motoman/meshes/sia20d/collision/MOTOMAN_AXIS_T.stl" />
+					<mesh filename="package://motoman_config/meshes/sia20d/collision/MOTOMAN_AXIS_T.stl" />
 				</geometry>
 				<material name="yellow"/>
