Commit message: moved xacros and meshes for sia5 from non-conformal stack into motoman_config package
git-svn-id: https://swri-ros-pkg.googlecode.com/svn/trunk@1092 076cdf4d-ed99-c8c1-5d01-9bc0d27e81bd

File: motoman_config/cfg/sia5_macro.xacro (robot description, xacro)
@@ -1,11 +1,12 @@
 <?xml version="1.0" ?>
 <robot xmlns:xacro="http://ros.org/wiki/xacro">
-	<include filename="$(find sia5_description)/urdf/properties.xacro"/> <!--contains properties such as pi and deg-->
-	<xacro:macro name="sia5_macro" params="prefix">
+	<property name="pi" value="3.141592654" />
+	<property name="deg" value="0.017453293" /> <!--degrees to radians-->
+	<xacro:macro name="sia5" params="prefix">
   <link name="${prefix}base_link">
     <visual>
       <origin xyz="0 0 0" rpy="0 0 0" />
       <geometry>
-        <mesh filename="package://sia5_description/meshes/visual/base.dae" />
+        <mesh filename="package://motoman_config/meshes/sia5/visual/base.dae" />
       </geometry>
     </visual>
@@ -13,5 +14,5 @@
       <origin xyz="0 0 0" rpy="0 0 0" />
       <geometry>
-        <mesh filename="package://sia5_description/meshes/collision/base.dae" />
+        <mesh filename="package://motoman_config/meshes/sia5/collision/base.dae" />
       </geometry>
     </collision>
@@ -21,5 +22,5 @@
       <origin xyz="0 0 0" rpy="0 0 0" />
       <geometry>
-        <mesh filename="package://sia5_description/meshes/visual/link_s.dae" />
+        <mesh filename="package://motoman_config/meshes/sia5/visual/link_s.dae" />
       </geometry>
     </visual>
@@ -27,5 +28,5 @@
       <origin xyz="0 0 0" rpy="0 0 0" />
       <geometry>
-        <mesh filename="package://sia5_description/meshes/collision/link_s.dae" />
+        <mesh filename="package://motoman_config/meshes/sia5/collision/link_s.dae" />
       </geometry>
     </collision>
@@ -43,5 +44,5 @@
       <origin xyz="0 0 0" rpy="0 0 0" />
       <geometry>
-        <mesh filename="package://sia5_description/meshes/visual/link_l.dae" />
+        <mesh filename="package://motoman_config/meshes/sia5/visual/link_l.dae" />
       </geometry>
     </visual>
@@ -49,5 +50,5 @@
       <origin xyz="0 0 0" rpy="0 0 0" />
       <geometry>
-        <mesh filename="package://sia5_description/meshes/collision/link_l.dae" />
+        <mesh filename="package://motoman_config/meshes/sia5/collision/link_l.dae" />
       </geometry>
     </collision>
@@ -65,5 +66,5 @@
       <origin xyz="0 0 0" rpy="0 0 0" />
       <geometry>
-        <mesh filename="package://sia5_description/meshes/visual/link_e.dae" />
+        <mesh filename="package://motoman_config/meshes/sia5/visual/link_e.dae" />
       </geometry>
     </visual>
@@ -71,5 +72,5 @@
       <origin xyz="0 0 0" rpy="0 0 0" />
       <geometry>
-        <mesh filename="package://sia5_description/meshes/collision/link_e.dae" />
+        <mesh filename="package://motoman_config/meshes/sia5/collision/link_e.dae" />
       </geometry>
     </collision>
@@ -87,5 +88,5 @@
       <origin xyz="0 0 0" rpy="0 0 0" />
       <geometry>
-        <mesh filename="package://sia5_description/meshes/visual/link_u.dae" />
+        <mesh filename="package://motoman_config/meshes/sia5/visual/link_u.dae" />
       </geometry>
     </visual>
@@ -93,5 +94,5 @@
       <origin xyz="0 0 0" rpy="0 0 0" />
       <geometry>
-        <mesh filename="package://sia5_description/meshes/collision/link_u.dae" />
+        <mesh filename="package://motoman_config/meshes/sia5/collision/link_u.dae" />
       </geometry>
     </collision>
@@ -109,5 +110,5 @@
       <origin xyz="0 0 0" rpy="0 0 0" />
       <geometry>
-        <mesh filename="package://sia5_description/meshes/visual/link_r.dae" />
+        <mesh filename="package://motoman_config/meshes/sia5/visual/link_r.dae" />
       </geometry>
     </visual>
@@ -115,5 +116,5 @@
       <origin xyz="0 0 0" rpy="0 0 0" />
       <geometry>
-        <mesh filename="package://sia5_description/meshes/collision/link_r.dae" />
+        <mesh filename="package://motoman_config/meshes/sia5/collision/link_r.dae" />
       </geometry>
     </collision>
@@ -131,5 +132,5 @@
       <origin xyz="0 0 0" rpy="0 0 0" />
       <geometry>
-        <mesh filename="package://sia5_description/meshes/visual/link_b.dae" />
+        <mesh filename="package://motoman_config/meshes/sia5/visual/link_b.dae" />
       </geometry>
     </visual>
@@ -137,5 +138,5 @@
       <origin xyz="0 0 0" rpy="0 0 0" />
       <geometry>
-        <mesh filename="package://sia5_description/meshes/collision/link_b.dae" />
+        <mesh filename="package://motoman_config/meshes/sia5/collision/link_b.dae" />
       </geometry>
     </collision>
@@ -153,5 +154,5 @@
       <origin xyz="0 0 0" rpy="0 0 0" />
       <geometry>
-        <mesh filename="package://sia5_description/meshes/visual/link_t.dae" />
+        <mesh filename="package://motoman_config/meshes/sia5/visual/link_t.dae" />
       </geometry>
     </visual>
@@ -159,5 +160,5 @@
       <origin xyz="0 0 0" rpy="0 0 0" />
       <geometry>
-        <mesh filename="package://sia5_description/meshes/collision/link_t.dae" />
+        <mesh filename="package://motoman_config/meshes/sia5/collision/link_t.dae" />
       </geometry>
     </collision>
