Commit message: manually adjusted the color values in the dae files for the sia20d

File: motoman_config/cfg/sia20d_macro.xacro (robot description, xacro)
@@ -10,5 +10,5 @@
     <collision>
       <geometry>
-        <mesh filename="package://motoman_config/meshes/sia20d/collision/MOTOMAN_BASE_COLLISION.dae" />
+        <mesh filename="package://motoman_config/meshes/sia20d/collision/MOTOMAN_BASE.dae" />
       </geometry>
     </collision>
@@ -24,10 +24,10 @@
     <visual>
       <geometry>
-        <mesh filename="package://motoman_config/meshes/sia20d/visual/MOTOMAN_AXIS_S.dae.dae" />
+        <mesh filename="package://motoman_config/meshes/sia20d/visual/MOTOMAN_AXIS_S.dae" />
       </geometry>
     </visual>
     <collision>
       <geometry>
-        <mesh filename="package://motoman_config/meshes/sia20d/collision/MOTOMAN_AXIS_S_COLLISION.dae" />
+        <mesh filename="package://motoman_config/meshes/sia20d/collision/MOTOMAN_AXIS_S.dae" />
       </geometry>
     </collision>
@@ -48,5 +48,5 @@
     <collision>
       <geometry>
-        <mesh filename="package://motoman_config/meshes/sia20d/collision/MOTOMAN_AXIS_L_COLLISION.dae" />
+        <mesh filename="package://motoman_config/meshes/sia20d/collision/MOTOMAN_AXIS_L.dae" />
       </geometry>
     </collision>
@@ -67,5 +67,5 @@
     <collision>
       <geometry>
-        <mesh filename="package://motoman_config/meshes/sia20d/collision/MOTOMAN_AXIS_E_COLLISION.dae" />
+        <mesh filename="package://motoman_config/meshes/sia20d/collision/MOTOMAN_AXIS_E.dae" />
       </geometry>
     </collision>
@@ -86,5 +86,5 @@
     <collision>
       <geometry>
-        <mesh filename="package://motoman_config/meshes/sia20d/collision/MOTOMAN_AXIS_U_COLLISION.dae" />
+        <mesh filename="package://motoman_config/meshes/sia20d/collision/MOTOMAN_AXIS_U.dae" />
       </geometry>
     </collision>
@@ -105,5 +105,5 @@
     <collision>
       <geometry>
-        <mesh filename="package://motoman_config/meshes/sia20d/collision/MOTOMAN_AXIS_R_COLLISION.dae" />
+        <mesh filename="package://motoman_config/meshes/sia20d/collision/MOTOMAN_AXIS_R.dae" />
       </geometry>
     </collision>
@@ -124,5 +124,5 @@
     <collision>
       <geometry>
-        <mesh filename="package://motoman_config/meshes/sia20d/collision/MOTOMAN_AXIS_B_COLLISION.dae" />
+        <mesh filename="package://motoman_config/meshes/sia20d/collision/MOTOMAN_AXIS_B.dae" />
       </geometry>
     </collision>
@@ -143,5 +143,5 @@
     <collision>
       <geometry>
-        <mesh filename="package://motoman_config/meshes/sia20d/collision/MOTOMAN_AXIS_T_COLLISION.dae" />
+        <mesh filename="package://motoman_config/meshes/sia20d/collision/MOTOMAN_AXIS_T.dae" />
       </geometry>
     </collision>
