Commit message: Corrected motoman robot name (added motoman prefix)

File: motoman_sia20d_support/urdf/sia20d.xacro (robot description, xacro)
@@ -1,5 +1,5 @@
 <?xml version="1.0" ?>
-<robot name="sia20d" xmlns:xacro="http://ros.org/wiki/xacro">
+<robot name="motoman_sia20d" xmlns:xacro="http://ros.org/wiki/xacro">
 	<xacro:include filename="$(find motoman_sia20d_support)/urdf/sia20d_macro.xacro" />
-	<xacro:sia20d prefix=""/>
+	<xacro:motoman_sia20d prefix=""/>
 </robot>

File: motoman_sia20d_support/urdf/sia20d_macro.xacro (robot description, xacro)
@@ -1,5 +1,5 @@
 <?xml version="1.0" ?>
 <robot xmlns:xacro="http://ros.org/wiki/xacro">
-	<xacro:macro name="sia20d" params="prefix">
+	<xacro:macro name="motoman_sia20d" params="prefix">
 		<!-- link list -->
 		<link name="${prefix}base_link">
