Commit message: sia20: don't round PI in joint_t-tool0 transform. Fix #106.
Leads to incorrect 'base->tool0' transform orientations.

File: motoman_sia20d_support/urdf/sia20d_macro.xacro (robot description, xacro)
@@ -186,5 +186,5 @@
 		</joint>
     <joint name="${prefix}link_t-tool0" type="fixed" >
-      <origin xyz="0 0 0.0" rpy="0 0 -3.1416"/>
+      <origin xyz="0 0 0.0" rpy="0 0 -3.1415926535"/>
       <parent link="${prefix}link_t" />
       <child link="${prefix}tool0" />
