Commit message: Added tool0 to sia20.  Matches motoman tool0

File: motoman_sia20d_support/urdf/sia20d.urdf (robot description, URDF)
Before this commit: robot sia20d, 8 links, 7 joints
Links:
- added link tool0
Joints:
- added joint link_t-tool0: type fixed, parent link_t, child tool0, origin xyz=0 0 0.0 rpy=0 0 -3.1416

File: motoman_sia20d_support/urdf/sia20d_macro.xacro (robot description, xacro)
@@ -133,4 +133,5 @@
 			</collision>
 		</link>
+    <link name="${prefix}tool0" />
 		<!-- end of link list -->
 		<!-- joint list -->
@@ -184,4 +185,9 @@
 			<limit lower="-3.1416" upper="3.1416" effort="100" velocity="6.97" />
 		</joint>
+    <joint name="${prefix}link_t-tool0" type="fixed" >
+      <origin xyz="0 0 0.0" rpy="0 0 -3.1416"/>
+      <parent link="${prefix}link_t" />
+      <child link="${prefix}tool0" />
+    </joint>
 		<!-- end of joint list -->
 	</xacro:macro>

Commit message: sia20d: fix joint limits S, R & T. Fix #102.
This floors PI, instead of rounding. This makes the joint limits slightly
stricter than what is specced, but will avoid OOB errors on the controller.

File: motoman_sia20d_support/urdf/sia20d.urdf (robot description, URDF)
Before this commit: robot motoman_sia20d, 9 links, 8 joints
Joints:
- joint joint_r: limit lower=-3.1416 upper=3.1416 effort=100 velocity=3.48 -> lower=-3.1415 upper=3.1415 effort=100 velocity=3.48
- joint joint_s: limit lower=-3.1416 upper=3.1416 effort=100 velocity=2.26 -> lower=-3.1415 upper=3.1415 effort=100 velocity=2.26
- joint joint_t: limit lower=-3.1416 upper=3.1416 effort=100 velocity=6.97 -> lower=-3.1415 upper=3.1415 effort=100 velocity=6.97

File: motoman_sia20d_support/urdf/sia20d_macro.xacro (robot description, xacro)
@@ -141,5 +141,5 @@
 			<origin xyz="0 0 0.41" rpy="0 0 0"/>
 			<axis xyz="0 0 1" />
-			<limit lower="-3.1416" upper="3.1416" effort="100" velocity="2.26" />
+			<limit lower="-3.1415" upper="3.1415" effort="100" velocity="2.26" />
 		</joint>
 		<joint name="${prefix}joint_l" type="revolute">
@@ -169,5 +169,5 @@
 			<origin xyz="0 0 0.420" rpy="0 0 0"/>
 			<axis xyz="0 0 -1" />
-			<limit lower="-3.1416" upper="3.1416" effort="100" velocity="3.48" />
+			<limit lower="-3.1415" upper="3.1415" effort="100" velocity="3.48" />
 		</joint>
 		<joint name="${prefix}joint_b" type="revolute">
@@ -183,5 +183,5 @@
 			<origin xyz="0 0 0.18" rpy="0 0 0"/>
 			<axis xyz="0 0 -1" />
-			<limit lower="-3.1416" upper="3.1416" effort="100" velocity="6.97" />
+			<limit lower="-3.1415" upper="3.1415" effort="100" velocity="6.97" />
 		</joint>
     <joint name="${prefix}link_t-tool0" type="fixed" >

Commit message: sia20d: make all joint limits correspond to specsheet.
All values truncated after the 4th digit.

File: motoman_sia20d_support/urdf/sia20d.urdf (robot description, URDF)
Before this commit: robot motoman_sia20d, 9 links, 8 joints
Joints:
- joint joint_b: limit lower=-1.91 upper=1.91 effort=100 velocity=3.48 -> lower=-1.9198 upper=1.9198 effort=100 velocity=3.4906
- joint joint_e: limit lower=-2.96 upper=2.96 effort=100 velocity=2.96 -> lower=-2.9670 upper=2.9670 effort=100 velocity=2.9670
- joint joint_l: limit lower=-1.91 upper=1.91 effort=100 velocity=2.26 -> lower=-1.9198 upper=1.9198 effort=100 velocity=2.2689
- joint joint_r: limit lower=-3.1415 upper=3.1415 effort=100 velocity=3.48 -> lower=-3.1415 upper=3.1415 effort=100 velocity=3.4906
- joint joint_s: limit lower=-3.1415 upper=3.1415 effort=100 velocity=2.26 -> lower=-3.1415 upper=3.1415 effort=100 velocity=2.2689
- joint joint_t: limit lower=-3.1415 upper=3.1415 effort=100 velocity=6.97 -> lower=-3.1415 upper=3.1415 effort=100 velocity=6.9813
- joint joint_u: limit lower=-2.26 upper=2.26 effort=100 velocity=2.96 -> lower=-2.2689 upper=2.2689 effort=100 velocity=2.9670

File: motoman_sia20d_support/urdf/sia20d_macro.xacro (robot description, xacro)
@@ -141,5 +141,5 @@
 			<origin xyz="0 0 0.41" rpy="0 0 0"/>
 			<axis xyz="0 0 1" />
-			<limit lower="-3.1415" upper="3.1415" effort="100" velocity="2.26" />
+			<limit lower="-3.1415" upper="3.1415" effort="100" velocity="2.2689" />
 		</joint>
 		<joint name="${prefix}joint_l" type="revolute">
@@ -148,5 +148,5 @@
 			<origin xyz="0 0 0" rpy="0 0 0"/>
 			<axis xyz="0 1 0" />
-			<limit lower="-1.91" upper="1.91" effort="100" velocity="2.26" />
+			<limit lower="-1.9198" upper="1.9198" effort="100" velocity="2.2689" />
 		</joint>
 		<joint name="${prefix}joint_e" type="revolute">
@@ -155,5 +155,5 @@
 			<origin xyz="0 0 0.49" rpy="0 0 0"/>
 			<axis xyz="0 0 1" />
-			<limit lower="-2.96" upper="2.96" effort="100" velocity="2.96" />
+			<limit lower="-2.9670" upper="2.9670" effort="100" velocity="2.9670" />
 		</joint>
 		<joint name="${prefix}joint_u" type="revolute">
@@ -162,5 +162,5 @@
 			<origin xyz="0 0 0" rpy="0 0 0"/>
 			<axis xyz="0 -1 0" />
-			<limit lower="-2.26" upper="2.26" effort="100" velocity="2.96" />
+			<limit lower="-2.2689" upper="2.2689" effort="100" velocity="2.9670" />
 		</joint>
 		<joint name="${prefix}joint_r" type="revolute">
@@ -169,5 +169,5 @@
 			<origin xyz="0 0 0.420" rpy="0 0 0"/>
 			<axis xyz="0 0 -1" />
-			<limit lower="-3.1415" upper="3.1415" effort="100" velocity="3.48" />
+			<limit lower="-3.1415" upper="3.1415" effort="100" velocity="3.4906" />
 		</joint>
 		<joint name="${prefix}joint_b" type="revolute">
@@ -176,5 +176,5 @@
 			<origin xyz="0 0 0" rpy="0 0 0"/>
 			<axis xyz="0 -1 0" />
-			<limit lower="-1.91" upper="1.91" effort="100" velocity="3.48" />
+			<limit lower="-1.9198" upper="1.9198" effort="100" velocity="3.4906" />
 		</joint>
 		<joint name="${prefix}joint_t" type="revolute">
@@ -183,5 +183,5 @@
 			<origin xyz="0 0 0.18" rpy="0 0 0"/>
 			<axis xyz="0 0 -1" />
-			<limit lower="-3.1415" upper="3.1415" effort="100" velocity="6.97" />
+			<limit lower="-3.1415" upper="3.1415" effort="100" velocity="6.9813" />
 		</joint>
     <joint name="${prefix}link_t-tool0" type="fixed" >

Commit message: Fix for issue #102: fix incorrect joint limits in SIA20 urdf/xacro (#109)
* sia20d: fix joint limits S, R & T. Fix #102.

This floors PI, instead of rounding. This makes the joint limits slightly
stricter than what is specced, but will avoid OOB errors on the controller.

* sia20d: make all joint limits correspond to specsheet.

All values truncated after the 4th digit.

File: motoman_sia20d_support/urdf/sia20d.urdf (robot description, URDF)
Before this commit: robot motoman_sia20d, 9 links, 8 joints
Joints:
- joint joint_b: limit lower=-1.91 upper=1.91 effort=100 velocity=3.48 -> lower=-1.9198 upper=1.9198 effort=100 velocity=3.4906
- joint joint_e: limit lower=-2.96 upper=2.96 effort=100 velocity=2.96 -> lower=-2.9670 upper=2.9670 effort=100 velocity=2.9670
- joint joint_l: limit lower=-1.91 upper=1.91 effort=100 velocity=2.26 -> lower=-1.9198 upper=1.9198 effort=100 velocity=2.2689
- joint joint_r: limit lower=-3.1416 upper=3.1416 effort=100 velocity=3.48 -> lower=-3.1415 upper=3.1415 effort=100 velocity=3.4906
- joint joint_s: limit lower=-3.1416 upper=3.1416 effort=100 velocity=2.26 -> lower=-3.1415 upper=3.1415 effort=100 velocity=2.2689
- joint joint_t: limit lower=-3.1416 upper=3.1416 effort=100 velocity=6.97 -> lower=-3.1415 upper=3.1415 effort=100 velocity=6.9813
- joint joint_u: limit lower=-2.26 upper=2.26 effort=100 velocity=2.96 -> lower=-2.2689 upper=2.2689 effort=100 velocity=2.9670

File: motoman_sia20d_support/urdf/sia20d_macro.xacro (robot description, xacro)
@@ -141,5 +141,5 @@
 			<origin xyz="0 0 0.41" rpy="0 0 0"/>
 			<axis xyz="0 0 1" />
-			<limit lower="-3.1416" upper="3.1416" effort="100" velocity="2.26" />
+			<limit lower="-3.1415" upper="3.1415" effort="100" velocity="2.2689" />
 		</joint>
 		<joint name="${prefix}joint_l" type="revolute">
@@ -148,5 +148,5 @@
 			<origin xyz="0 0 0" rpy="0 0 0"/>
 			<axis xyz="0 1 0" />
-			<limit lower="-1.91" upper="1.91" effort="100" velocity="2.26" />
+			<limit lower="-1.9198" upper="1.9198" effort="100" velocity="2.2689" />
 		</joint>
 		<joint name="${prefix}joint_e" type="revolute">
@@ -155,5 +155,5 @@
 			<origin xyz="0 0 0.49" rpy="0 0 0"/>
 			<axis xyz="0 0 1" />
-			<limit lower="-2.96" upper="2.96" effort="100" velocity="2.96" />
+			<limit lower="-2.9670" upper="2.9670" effort="100" velocity="2.9670" />
 		</joint>
 		<joint name="${prefix}joint_u" type="revolute">
@@ -162,5 +162,5 @@
 			<origin xyz="0 0 0" rpy="0 0 0"/>
 			<axis xyz="0 -1 0" />
-			<limit lower="-2.26" upper="2.26" effort="100" velocity="2.96" />
+			<limit lower="-2.2689" upper="2.2689" effort="100" velocity="2.9670" />
 		</joint>
 		<joint name="${prefix}joint_r" type="revolute">
@@ -169,5 +169,5 @@
 			<origin xyz="0 0 0.420" rpy="0 0 0"/>
 			<axis xyz="0 0 -1" />
-			<limit lower="-3.1416" upper="3.1416" effort="100" velocity="3.48" />
+			<limit lower="-3.1415" upper="3.1415" effort="100" velocity="3.4906" />
 		</joint>
 		<joint name="${prefix}joint_b" type="revolute">
@@ -176,5 +176,5 @@
 			<origin xyz="0 0 0" rpy="0 0 0"/>
 			<axis xyz="0 -1 0" />
-			<limit lower="-1.91" upper="1.91" effort="100" velocity="3.48" />
+			<limit lower="-1.9198" upper="1.9198" effort="100" velocity="3.4906" />
 		</joint>
 		<joint name="${prefix}joint_t" type="revolute">
@@ -183,5 +183,5 @@
 			<origin xyz="0 0 0.18" rpy="0 0 0"/>
 			<axis xyz="0 0 -1" />
-			<limit lower="-3.1416" upper="3.1416" effort="100" velocity="6.97" />
+			<limit lower="-3.1415" upper="3.1415" effort="100" velocity="6.9813" />
 		</joint>
     <joint name="${prefix}link_t-tool0" type="fixed" >
