Commit message: Update to allow for use in simulation
Added mass properties and other Gazebo tags

File: motoman_sia10d_support/urdf/sia10d.urdf (robot description, URDF)
Before this commit: robot motoman_sia10d, 8 links, 7 joints
Links:
- added link world
- link base_link: mass None -> 400
- link link_b: mass None -> 2.3902999
- link link_e: mass None -> 4.7092004
- link link_l: mass None -> 5.227999
- link link_r: mass None -> 3.0270943
- link link_s: mass None -> 13.746057
- link link_t: mass None -> 0.63670412
- link link_u: mass None -> 3.1488649
Joints:
- added joint world-base: type fixed, parent world, child base_link, origin xyz=0 0 0 rpy=0 0 0

Commit message: sia10: fix joint limits S, R & T. Fix #104.
This floors PI, instead of rounding. This makes the joint limits slightly
stricter than what is specced, but will avoid OOB errors on the controller.

File: motoman_sia10d_support/urdf/sia10d.urdf (robot description, URDF)
Before this commit: robot motoman_sia10d, 9 links, 8 joints
Joints:
- joint joint_r: limit lower=-3.1416 upper=3.1416 effort=100 velocity=3.48 -> lower=-3.1415 upper=3.1415 effort=100 velocity=3.48
- joint joint_s: limit lower=-3.1416 upper=3.1416 effort=100 velocity=2.96 -> lower=-3.1415 upper=3.1415 effort=100 velocity=2.96
- joint joint_t: limit lower=-3.1416 upper=3.1416 effort=100 velocity=6.97 -> lower=-3.1415 upper=3.1415 effort=100 velocity=6.97

File: motoman_sia10d_support/urdf/sia10d_macro.xacro (robot description, xacro)
@@ -225,5 +225,5 @@
 			<origin xyz="0 0 0.36" rpy="0 0 0"/>
 			<axis xyz="0 0 1" />
-			<limit lower="-3.1416" upper="3.1416" effort="100" velocity="2.96" />
+			<limit lower="-3.1415" upper="3.1415" effort="100" velocity="2.96" />
 		</joint>
 		<joint name="${prefix}joint_l" type="revolute">
@@ -253,5 +253,5 @@
 			<origin xyz="0 0 0.360" rpy="0 0 0"/>
 			<axis xyz="0 0 -1" />
-			<limit lower="-3.1416" upper="3.1416" effort="100" velocity="3.48" />
+			<limit lower="-3.1415" upper="3.1415" effort="100" velocity="3.48" />
 		</joint>
 		<joint name="${prefix}joint_b" type="revolute">
@@ -267,5 +267,5 @@
 			<origin xyz="0 0 0.155" rpy="0 0 0"/>
 			<axis xyz="0 0 -1" />
-			<limit lower="-3.1416" upper="3.1416" effort="100" velocity="6.97" />
+			<limit lower="-3.1415" upper="3.1415" effort="100" velocity="6.97" />
 		</joint>
 		<!-- end of joint list -->

File: motoman_sia10f_support/urdf/sia10f.urdf (robot description, URDF)
Before this commit: robot motoman_sia10f, 8 links, 7 joints
Joints:
- joint joint_r: limit lower=-3.1416 upper=3.1416 effort=100 velocity=3.48 -> lower=-3.1415 upper=3.1415 effort=100 velocity=3.48
- joint joint_s: limit lower=-3.1416 upper=3.1416 effort=100 velocity=2.96 -> lower=-3.1415 upper=3.1415 effort=100 velocity=2.96
- joint joint_t: limit lower=-3.1416 upper=3.1416 effort=100 velocity=6.97 -> lower=-3.1415 upper=3.1415 effort=100 velocity=6.97

File: motoman_sia10f_support/urdf/sia10f_macro.xacro (robot description, xacro)
@@ -139,5 +139,5 @@
 			<origin xyz="0 0 0.36" rpy="0 0 0"/>
 			<axis xyz="0 0 1" />
-			<limit lower="-3.1416" upper="3.1416" effort="0" velocity="2.96" />
+			<limit lower="-3.1415" upper="3.1415" effort="0" velocity="2.96" />
 		</joint>
 		<joint name="${prefix}joint_2_l" type="revolute">
@@ -167,5 +167,5 @@
 			<origin xyz="0 0 0.360" rpy="0 0 0"/>
 			<axis xyz="0 0 -1" />
-			<limit lower="-3.1416" upper="3.1416" effort="0" velocity="3.48" />
+			<limit lower="-3.1415" upper="3.1415" effort="0" velocity="3.48" />
 		</joint>
 		<joint name="${prefix}joint_6_b" type="revolute">
@@ -181,5 +181,5 @@
 			<origin xyz="0 0 0.155" rpy="0 0 0"/>
 			<axis xyz="0 0 -1" />
-			<limit lower="-3.1416" upper="3.1416" effort="0" velocity="6.97" />
+			<limit lower="-3.1415" upper="3.1415" effort="0" velocity="6.97" />
 		</joint>
     <joint name="${prefix}joint_tool0" type="fixed" >

Commit message: sia10: make all joint limits correspond to specsheet.
All values truncated after the 4th digit.

File: motoman_sia10d_support/urdf/sia10d.urdf (robot description, URDF)
Before this commit: robot motoman_sia10d, 9 links, 8 joints
Joints:
- joint joint_b: limit lower=-1.91 upper=1.91 effort=100 velocity=3.48 -> lower=-1.9198 upper=1.9198 effort=100 velocity=3.4906
- joint joint_e: limit lower=-2.96 upper=2.96 effort=100 velocity=2.96 -> lower=-2.9670 upper=2.9670 effort=100 velocity=2.9670
- joint joint_l: limit lower=-1.91 upper=1.91 effort=100 velocity=2.96 -> lower=-1.9198 upper=1.9198 effort=100 velocity=2.9670
- joint joint_r: limit lower=-3.1415 upper=3.1415 effort=100 velocity=3.48 -> lower=-3.1415 upper=3.1415 effort=100 velocity=3.4906
- joint joint_s: limit lower=-3.1415 upper=3.1415 effort=100 velocity=2.96 -> lower=-3.1415 upper=3.1415 effort=100 velocity=2.9670
- joint joint_t: limit lower=-3.1415 upper=3.1415 effort=100 velocity=6.97 -> lower=-3.1415 upper=3.1415 effort=100 velocity=6.9813
- joint joint_u: limit lower=-2.35 upper=2.35 effort=100 velocity=2.96 -> lower=-2.3561 upper=2.3561 effort=100 velocity=2.9670

File: motoman_sia10d_support/urdf/sia10d_macro.xacro (robot description, xacro)
@@ -225,5 +225,5 @@
 			<origin xyz="0 0 0.36" rpy="0 0 0"/>
 			<axis xyz="0 0 1" />
-			<limit lower="-3.1415" upper="3.1415" effort="100" velocity="2.96" />
+			<limit lower="-3.1415" upper="3.1415" effort="100" velocity="2.9670" />
 		</joint>
 		<joint name="${prefix}joint_l" type="revolute">
@@ -232,5 +232,5 @@
 			<origin xyz="0 0 0" rpy="0 0 0"/>
 			<axis xyz="0 1 0" />
-			<limit lower="-1.91" upper="1.91" effort="100" velocity="2.96" />
+			<limit lower="-1.9198" upper="1.9198" effort="100" velocity="2.9670" />
 		</joint>
 		<joint name="${prefix}joint_e" type="revolute">
@@ -239,5 +239,5 @@
 			<origin xyz="0 0 0.36" rpy="0 0 0"/>
 			<axis xyz="0 0 1" />
-			<limit lower="-2.96" upper="2.96" effort="100" velocity="2.96" />
+			<limit lower="-2.9670" upper="2.9670" effort="100" velocity="2.9670" />
 		</joint>
 		<joint name="${prefix}joint_u" type="revolute">
@@ -246,5 +246,5 @@
 			<origin xyz="0 0 0" rpy="0 0 0"/>
 			<axis xyz="0 -1 0" />
-			<limit lower="-2.35" upper="2.35" effort="100" velocity="2.96" />
+			<limit lower="-2.3561" upper="2.3561" effort="100" velocity="2.9670" />
 		</joint>
 		<joint name="${prefix}joint_r" type="revolute">
@@ -253,5 +253,5 @@
 			<origin xyz="0 0 0.360" rpy="0 0 0"/>
 			<axis xyz="0 0 -1" />
-			<limit lower="-3.1415" upper="3.1415" effort="100" velocity="3.48" />
+			<limit lower="-3.1415" upper="3.1415" effort="100" velocity="3.4906" />
 		</joint>
 		<joint name="${prefix}joint_b" type="revolute">
@@ -260,5 +260,5 @@
 			<origin xyz="0 0 0" rpy="0 0 0"/>
 			<axis xyz="0 -1 0" />
-			<limit lower="-1.91" upper="1.91" effort="100" velocity="3.48" />
+			<limit lower="-1.9198" upper="1.9198" effort="100" velocity="3.4906" />
 		</joint>
 		<joint name="${prefix}joint_t" type="revolute">
@@ -267,5 +267,5 @@
 			<origin xyz="0 0 0.155" rpy="0 0 0"/>
 			<axis xyz="0 0 -1" />
-			<limit lower="-3.1415" upper="3.1415" effort="100" velocity="6.97" />
+			<limit lower="-3.1415" upper="3.1415" effort="100" velocity="6.9813" />
 		</joint>
 		<!-- end of joint list -->

File: motoman_sia10f_support/urdf/sia10f.urdf (robot description, URDF)
Before this commit: robot motoman_sia10f, 8 links, 7 joints
Joints:
- joint joint_b: limit lower=-1.91 upper=1.91 effort=100 velocity=3.48 -> lower=-1.9198 upper=1.9198 effort=100 velocity=3.4906
- joint joint_e: limit lower=-2.96 upper=2.96 effort=100 velocity=2.96 -> lower=-2.9670 upper=2.9670 effort=100 velocity=2.9670
- joint joint_l: limit lower=-1.91 upper=1.91 effort=100 velocity=2.96 -> lower=-1.9198 upper=1.9198 effort=100 velocity=2.9670
- joint joint_r: limit lower=-3.1415 upper=3.1415 effort=100 velocity=3.48 -> lower=-3.1415 upper=3.1415 effort=100 velocity=3.4906
- joint joint_s: limit lower=-3.1415 upper=3.1415 effort=100 velocity=2.96 -> lower=-3.1415 upper=3.1415 effort=100 velocity=2.9670
- joint joint_t: limit lower=-3.1415 upper=3.1415 effort=100 velocity=6.97 -> lower=-3.1415 upper=3.1415 effort=100 velocity=6.9813
- joint joint_u: limit lower=-2.35 upper=2.35 effort=100 velocity=2.96 -> lower=-2.3561 upper=2.3561 effort=100 velocity=2.9670

File: motoman_sia10f_support/urdf/sia10f_macro.xacro (robot description, xacro)
@@ -139,5 +139,5 @@
 			<origin xyz="0 0 0.36" rpy="0 0 0"/>
 			<axis xyz="0 0 1" />
-			<limit lower="-3.1415" upper="3.1415" effort="0" velocity="2.96" />
+			<limit lower="-3.1415" upper="3.1415" effort="0" velocity="2.9670" />
 		</joint>
 		<joint name="${prefix}joint_2_l" type="revolute">
@@ -146,5 +146,5 @@
 			<origin xyz="0 0 0" rpy="0 0 0"/>
 			<axis xyz="0 1 0" />
-			<limit lower="-1.91" upper="1.91" effort="0" velocity="2.96" />
+			<limit lower="-1.9198" upper="1.9198" effort="0" velocity="2.9670" />
 		</joint>
 		<joint name="${prefix}joint_3_e" type="revolute">
@@ -153,5 +153,5 @@
 			<origin xyz="0 0 0.36" rpy="0 0 0"/>
 			<axis xyz="0 0 1" />
-			<limit lower="-2.96" upper="2.96" effort="0" velocity="2.96" />
+			<limit lower="-2.9670" upper="2.9670" effort="0" velocity="2.9670" />
 		</joint>
 		<joint name="${prefix}joint_4_u" type="revolute">
@@ -160,5 +160,5 @@
 			<origin xyz="0 0 0" rpy="0 0 0"/>
 			<axis xyz="0 -1 0" />
-			<limit lower="-2.35" upper="2.35" effort="0" velocity="2.96" />
+			<limit lower="-2.3561" upper="2.3561" effort="0" velocity="2.9670" />
 		</joint>
 		<joint name="${prefix}joint_5_r" type="revolute">
@@ -167,5 +167,5 @@
 			<origin xyz="0 0 0.360" rpy="0 0 0"/>
 			<axis xyz="0 0 -1" />
-			<limit lower="-3.1415" upper="3.1415" effort="0" velocity="3.48" />
+			<limit lower="-3.1415" upper="3.1415" effort="0" velocity="3.4906" />
 		</joint>
 		<joint name="${prefix}joint_6_b" type="revolute">
@@ -174,5 +174,5 @@
 			<origin xyz="0 0 0" rpy="0 0 0"/>
 			<axis xyz="0 -1 0" />
-			<limit lower="-1.91" upper="1.91" effort="0" velocity="3.48" />
+			<limit lower="-1.9198" upper="1.9198" effort="0" velocity="3.4906" />
 		</joint>
 		<joint name="${prefix}joint_7_t" type="revolute">
@@ -181,5 +181,5 @@
 			<origin xyz="0 0 0.155" rpy="0 0 0"/>
 			<axis xyz="0 0 -1" />
-			<limit lower="-3.1415" upper="3.1415" effort="0" velocity="6.97" />
+			<limit lower="-3.1415" upper="3.1415" effort="0" velocity="6.9813" />
 		</joint>
     <joint name="${prefix}joint_tool0" type="fixed" >

Commit message: Fix for issue #104: fix incorrect joint limits in SIA10 urdf/xacro (#108)
* sia10: fix joint limits S, R & T. Fix #104.

This floors PI, instead of rounding. This makes the joint limits slightly
stricter than what is specced, but will avoid OOB errors on the controller.

* sia10: make all joint limits correspond to specsheet.

All values truncated after the 4th digit.

File: motoman_sia10d_support/urdf/sia10d.urdf (robot description, URDF)
Before this commit: robot motoman_sia10d, 9 links, 8 joints
Joints:
- joint joint_b: limit lower=-1.91 upper=1.91 effort=100 velocity=3.48 -> lower=-1.9198 upper=1.9198 effort=100 velocity=3.4906
- joint joint_e: limit lower=-2.96 upper=2.96 effort=100 velocity=2.96 -> lower=-2.9670 upper=2.9670 effort=100 velocity=2.9670
- joint joint_l: limit lower=-1.91 upper=1.91 effort=100 velocity=2.96 -> lower=-1.9198 upper=1.9198 effort=100 velocity=2.9670
- joint joint_r: limit lower=-3.1416 upper=3.1416 effort=100 velocity=3.48 -> lower=-3.1415 upper=3.1415 effort=100 velocity=3.4906
- joint joint_s: limit lower=-3.1416 upper=3.1416 effort=100 velocity=2.96 -> lower=-3.1415 upper=3.1415 effort=100 velocity=2.9670
- joint joint_t: limit lower=-3.1416 upper=3.1416 effort=100 velocity=6.97 -> lower=-3.1415 upper=3.1415 effort=100 velocity=6.9813
- joint joint_u: limit lower=-2.35 upper=2.35 effort=100 velocity=2.96 -> lower=-2.3561 upper=2.3561 effort=100 velocity=2.9670

File: motoman_sia10d_support/urdf/sia10d_macro.xacro (robot description, xacro)
@@ -225,5 +225,5 @@
 			<origin xyz="0 0 0.36" rpy="0 0 0"/>
 			<axis xyz="0 0 1" />
-			<limit lower="-3.1416" upper="3.1416" effort="100" velocity="2.96" />
+			<limit lower="-3.1415" upper="3.1415" effort="100" velocity="2.9670" />
 		</joint>
 		<joint name="${prefix}joint_l" type="revolute">
@@ -232,5 +232,5 @@
 			<origin xyz="0 0 0" rpy="0 0 0"/>
 			<axis xyz="0 1 0" />
-			<limit lower="-1.91" upper="1.91" effort="100" velocity="2.96" />
+			<limit lower="-1.9198" upper="1.9198" effort="100" velocity="2.9670" />
 		</joint>
 		<joint name="${prefix}joint_e" type="revolute">
@@ -239,5 +239,5 @@
 			<origin xyz="0 0 0.36" rpy="0 0 0"/>
 			<axis xyz="0 0 1" />
-			<limit lower="-2.96" upper="2.96" effort="100" velocity="2.96" />
+			<limit lower="-2.9670" upper="2.9670" effort="100" velocity="2.9670" />
 		</joint>
 		<joint name="${prefix}joint_u" type="revolute">
@@ -246,5 +246,5 @@
 			<origin xyz="0 0 0" rpy="0 0 0"/>
 			<axis xyz="0 -1 0" />
-			<limit lower="-2.35" upper="2.35" effort="100" velocity="2.96" />
+			<limit lower="-2.3561" upper="2.3561" effort="100" velocity="2.9670" />
 		</joint>
 		<joint name="${prefix}joint_r" type="revolute">
@@ -253,5 +253,5 @@
 			<origin xyz="0 0 0.360" rpy="0 0 0"/>
 			<axis xyz="0 0 -1" />
-			<limit lower="-3.1416" upper="3.1416" effort="100" velocity="3.48" />
+			<limit lower="-3.1415" upper="3.1415" effort="100" velocity="3.4906" />
 		</joint>
 		<joint name="${prefix}joint_b" type="revolute">
@@ -260,5 +260,5 @@
 			<origin xyz="0 0 0" rpy="0 0 0"/>
 			<axis xyz="0 -1 0" />
-			<limit lower="-1.91" upper="1.91" effort="100" velocity="3.48" />
+			<limit lower="-1.9198" upper="1.9198" effort="100" velocity="3.4906" />
 		</joint>
 		<joint name="${prefix}joint_t" type="revolute">
@@ -267,5 +267,5 @@
 			<origin xyz="0 0 0.155" rpy="0 0 0"/>
 			<axis xyz="0 0 -1" />
-			<limit lower="-3.1416" upper="3.1416" effort="100" velocity="6.97" />
+			<limit lower="-3.1415" upper="3.1415" effort="100" velocity="6.9813" />
 		</joint>
 		<!-- end of joint list -->

File: motoman_sia10f_support/urdf/sia10f.urdf (robot description, URDF)
Before this commit: robot motoman_sia10f, 8 links, 7 joints
Joints:
- joint joint_b: limit lower=-1.91 upper=1.91 effort=100 velocity=3.48 -> lower=-1.9198 upper=1.9198 effort=100 velocity=3.4906
- joint joint_e: limit lower=-2.96 upper=2.96 effort=100 velocity=2.96 -> lower=-2.9670 upper=2.9670 effort=100 velocity=2.9670
- joint joint_l: limit lower=-1.91 upper=1.91 effort=100 velocity=2.96 -> lower=-1.9198 upper=1.9198 effort=100 velocity=2.9670
- joint joint_r: limit lower=-3.1416 upper=3.1416 effort=100 velocity=3.48 -> lower=-3.1415 upper=3.1415 effort=100 velocity=3.4906
- joint joint_s: limit lower=-3.1416 upper=3.1416 effort=100 velocity=2.96 -> lower=-3.1415 upper=3.1415 effort=100 velocity=2.9670
- joint joint_t: limit lower=-3.1416 upper=3.1416 effort=100 velocity=6.97 -> lower=-3.1415 upper=3.1415 effort=100 velocity=6.9813
- joint joint_u: limit lower=-2.35 upper=2.35 effort=100 velocity=2.96 -> lower=-2.3561 upper=2.3561 effort=100 velocity=2.9670

File: motoman_sia10f_support/urdf/sia10f_macro.xacro (robot description, xacro)
@@ -139,5 +139,5 @@
 			<origin xyz="0 0 0.36" rpy="0 0 0"/>
 			<axis xyz="0 0 1" />
-			<limit lower="-3.1416" upper="3.1416" effort="0" velocity="2.96" />
+			<limit lower="-3.1415" upper="3.1415" effort="0" velocity="2.9670" />
 		</joint>
 		<joint name="${prefix}joint_2_l" type="revolute">
@@ -146,5 +146,5 @@
 			<origin xyz="0 0 0" rpy="0 0 0"/>
 			<axis xyz="0 1 0" />
-			<limit lower="-1.91" upper="1.91" effort="0" velocity="2.96" />
+			<limit lower="-1.9198" upper="1.9198" effort="0" velocity="2.9670" />
 		</joint>
 		<joint name="${prefix}joint_3_e" type="revolute">
@@ -153,5 +153,5 @@
 			<origin xyz="0 0 0.36" rpy="0 0 0"/>
 			<axis xyz="0 0 1" />
-			<limit lower="-2.96" upper="2.96" effort="0" velocity="2.96" />
+			<limit lower="-2.9670" upper="2.9670" effort="0" velocity="2.9670" />
 		</joint>
 		<joint name="${prefix}joint_4_u" type="revolute">
@@ -160,5 +160,5 @@
 			<origin xyz="0 0 0" rpy="0 0 0"/>
 			<axis xyz="0 -1 0" />
-			<limit lower="-2.35" upper="2.35" effort="0" velocity="2.96" />
+			<limit lower="-2.3561" upper="2.3561" effort="0" velocity="2.9670" />
 		</joint>
 		<joint name="${prefix}joint_5_r" type="revolute">
@@ -167,5 +167,5 @@
 			<origin xyz="0 0 0.360" rpy="0 0 0"/>
 			<axis xyz="0 0 -1" />
-			<limit lower="-3.1416" upper="3.1416" effort="0" velocity="3.48" />
+			<limit lower="-3.1415" upper="3.1415" effort="0" velocity="3.4906" />
 		</joint>
 		<joint name="${prefix}joint_6_b" type="revolute">
@@ -174,5 +174,5 @@
 			<origin xyz="0 0 0" rpy="0 0 0"/>
 			<axis xyz="0 -1 0" />
-			<limit lower="-1.91" upper="1.91" effort="0" velocity="3.48" />
+			<limit lower="-1.9198" upper="1.9198" effort="0" velocity="3.4906" />
 		</joint>
 		<joint name="${prefix}joint_7_t" type="revolute">
@@ -181,5 +181,5 @@
 			<origin xyz="0 0 0.155" rpy="0 0 0"/>
 			<axis xyz="0 0 -1" />
-			<limit lower="-3.1416" upper="3.1416" effort="0" velocity="6.97" />
+			<limit lower="-3.1415" upper="3.1415" effort="0" velocity="6.9813" />
 		</joint>
     <joint name="${prefix}joint_tool0" type="fixed" >
