Commit message: Adds changes to the sia name

File: motoman_sia10f_support/urdf/sia10f.urdf (robot description, URDF)
Before this commit: robot motoman_sia10d, 8 links, 7 joints
Links:
- link base_link: geometry collision mesh filename=package://motoman_sia10f_support/meshes/sia10f/collision/MO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; visual mesh filename=package://motoman_sia10f_support/meshes/sia10f/visual/MOTOM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
- link link_b: geometry collision mesh filename=package://motoman_sia10f_support/meshes/sia10f/collision/MO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; visual mesh filename=package://motoman_sia10f_support/meshes/sia10f/visual/MOTOM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
- link link_e: geometry collision mesh filename=package://motoman_sia10f_support/meshes/sia10f/collision/MO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; visual mesh filename=package://motoman_sia10f_support/meshes/sia10f/visual/MOTOM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
- link link_l: geometry collision mesh filename=package://motoman_sia10f_support/meshes/sia10f/collision/MO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; visual mesh filename=package://motoman_sia10f_support/meshes/sia10f/visual/MOTOM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
- link link_r: geometry collision mesh filename=package://motoman_sia10f_support/meshes/sia10f/collision/MO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; visual mesh filename=package://motoman_sia10f_support/meshes/sia10f/visual/MOTOM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
- link link_s: geometry collision mesh filename=package://motoman_sia10f_support/meshes/sia10f/collision/MO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; visual mesh filename=package://motoman_sia10f_support/meshes/sia10f/visual/MOTOM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
- link link_t: geometry collision mesh filename=package://motoman_sia10f_support/meshes/sia10f/collision/MO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; visual mesh filename=package://motoman_sia10f_support/meshes/sia10f/visual/MOTOM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
- link link_u: geometry collision mesh filename=package://motoman_sia10f_support/meshes/sia10f/collision/MO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; visual mesh filename=package://motoman_sia10f_support/meshes/sia10f/visual/MOTOM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

File: motoman_sia10f_support/urdf/sia10f.xacro (robot description, xacro)
@@ -1,5 +1,5 @@
 <?xml version="1.0" ?>
-<robot name="motoman_sia10d" xmlns:xacro="http://ros.org/wiki/xacro">
-	<xacro:include filename="$(find motoman_sia10d_support)/urdf/sia10d_macro.xacro" />
-	<xacro:motoman_sia10d prefix=""/>
+<robot name="motoman_sia10f" xmlns:xacro="http://ros.org/wiki/xacro">
+	<xacro:include filename="$(find motoman_sia10f_support)/urdf/sia10f_macro.xacro" />
+	<xacro:motoman_sia10f prefix=""/>
 </robot>

File: motoman_sia10f_support/urdf/sia10f_macro.xacro (robot description, xacro)
@@ -6,5 +6,5 @@
 			<visual>
 				<geometry>
-					<mesh filename="package://motoman_sia10d_support/meshes/sia10d/visual/MOTOMAN_BASE.stl" />
+					<mesh filename="package://motoman_sia10f_support/meshes/sia10f/visual/MOTOMAN_BASE.stl" />
 				</geometry>
 				<material name="blue">
@@ -14,5 +14,5 @@
 			<collision>
 				<geometry>
-					<mesh filename="package://motoman_sia10d_support/meshes/sia10d/collision/MOTOMAN_BASE.stl" />
+					<mesh filename="package://motoman_sia10f_support/meshes/sia10f/collision/MOTOMAN_BASE.stl" />
 				</geometry>
 				<material name="yellow">
@@ -24,5 +24,5 @@
 			<visual>
 				<geometry>
-					<mesh filename="package://motoman_sia10d_support/meshes/sia10d/visual/MOTOMAN_AXIS_S.stl"/>
+					<mesh filename="package://motoman_sia10f_support/meshes/sia10f/visual/MOTOMAN_AXIS_S.stl"/>
 				</geometry>
 				<material name="silver">
@@ -32,5 +32,5 @@
 			<collision>
 				<geometry>
-					<mesh filename="package://motoman_sia10d_support/meshes/sia10d/collision/MOTOMAN_AXIS_S.stl" />
+					<mesh filename="package://motoman_sia10f_support/meshes/sia10f/collision/MOTOMAN_AXIS_S.stl" />
 				</geometry>
 				<material name="yellow"/>
@@ -41,5 +41,5 @@
 				<origin rpy="1.57 3.1416 0" xyz="0 0 0"/>
 				<geometry>
-					<mesh filename="package://motoman_sia10d_support/meshes/sia10d/visual/MOTOMAN_AXIS_L.stl"/>
+					<mesh filename="package://motoman_sia10f_support/meshes/sia10f/visual/MOTOMAN_AXIS_L.stl"/>
 				</geometry>
 				<material name="blue"/>
@@ -48,5 +48,5 @@
 				<origin rpy="1.57 3.1416 0" xyz="0 0 0"/>
 				<geometry>
-					<mesh filename="package://motoman_sia10d_support/meshes/sia10d/collision/MOTOMAN_AXIS_L.stl" />
+					<mesh filename="package://motoman_sia10f_support/meshes/sia10f/collision/MOTOMAN_AXIS_L.stl" />
 				</geometry>
 				<material name="yellow"/>
@@ -57,5 +57,5 @@
 				<origin rpy="0 0 3.1415" xyz="0 0 0"/>
 				<geometry>
-					<mesh filename="package://motoman_sia10d_support/meshes/sia10d/visual/MOTOMAN_AXIS_E.stl"/>
+					<mesh filename="package://motoman_sia10f_support/meshes/sia10f/visual/MOTOMAN_AXIS_E.stl"/>
 				</geometry>
 				<material name="silver"/>
@@ -64,5 +64,5 @@
 				<origin rpy="0 0 3.1415" xyz="0 0 0"/>
 				<geometry>
-					<mesh filename="package://motoman_sia10d_support/meshes/sia10d/collision/MOTOMAN_AXIS_E.stl" />
+					<mesh filename="package://motoman_sia10f_support/meshes/sia10f/collision/MOTOMAN_AXIS_E.stl" />
 				</geometry>
 				<material name="yellow"/>
@@ -73,5 +73,5 @@
 				<origin rpy="1.57 -3.1415 0" xyz="0 0 0"/>
 				<geometry>
-					<mesh filename="package://motoman_sia10d_support/meshes/sia10d/visual/MOTOMAN_AXIS_U.stl"/>
+					<mesh filename="package://motoman_sia10f_support/meshes/sia10f/visual/MOTOMAN_AXIS_U.stl"/>
 				</geometry>
 				<material name="blue"/>
@@ -80,5 +80,5 @@
 				<origin rpy="1.57 -3.1415 0" xyz="0 0 0"/>
 				<geometry>
-					<mesh filename="package://motoman_sia10d_support/meshes/sia10d/collision/MOTOMAN_AXIS_U.stl" />
+					<mesh filename="package://motoman_sia10f_support/meshes/sia10f/collision/MOTOMAN_AXIS_U.stl" />
 				</geometry>
 				<material name="yellow"/>
@@ -89,5 +89,5 @@
 				<origin rpy="0 0 3.1416" xyz="0 0 0"/>
 				<geometry>
-					<mesh filename="package://motoman_sia10d_support/meshes/sia10d/visual/MOTOMAN_AXIS_R.stl"/>
+					<mesh filename="package://motoman_sia10f_support/meshes/sia10f/visual/MOTOMAN_AXIS_R.stl"/>
 				</geometry>
 				<material name="silver"/>
@@ -96,5 +96,5 @@
 				<origin rpy="0 0 3.1416" xyz="0 0 0"/>
 				<geometry>
-					<mesh filename="package://motoman_sia10d_support/meshes/sia10d/collision/MOTOMAN_AXIS_R.stl" />
+					<mesh filename="package://motoman_sia10f_support/meshes/sia10f/collision/MOTOMAN_AXIS_R.stl" />
 				</geometry>
 				<material name="yellow"/>
@@ -105,5 +105,5 @@
 				<origin rpy="-1.57 0 3.1416" xyz="0 0 0"/>
 				<geometry>
-					<mesh filename="package://motoman_sia10d_support/meshes/sia10d/visual/MOTOMAN_AXIS_B.stl"/>
+					<mesh filename="package://motoman_sia10f_support/meshes/sia10f/visual/MOTOMAN_AXIS_B.stl"/>
 				</geometry>
 				<material name="blue"/>
@@ -112,5 +112,5 @@
 				<origin rpy="-1.57 0 3.1416" xyz="0 0 0"/>
 				<geometry>
-					<mesh filename="package://motoman_sia10d_support/meshes/sia10d/collision/MOTOMAN_AXIS_B.stl" />
+					<mesh filename="package://motoman_sia10f_support/meshes/sia10f/collision/MOTOMAN_AXIS_B.stl" />
 				</geometry>
 				<material name="yellow"/>
@@ -120,5 +120,5 @@
 			<visual>
 				<geometry>
-					<mesh filename="package://motoman_sia10d_support/meshes/sia10d/visual/MOTOMAN_AXIS_T.stl" />
+					<mesh filename="package://motoman_sia10f_support/meshes/sia10f/visual/MOTOMAN_AXIS_T.stl" />
 				</geometry>
 				<material name="silver"/>
@@ -126,5 +126,5 @@
 			<collision>
 				<geometry>
-					<mesh filename="package://motoman_sia10d_support/meshes/sia10d/collision/MOTOMAN_AXIS_T.stl" />
+					<mesh filename="package://motoman_sia10f_support/meshes/sia10f/collision/MOTOMAN_AXIS_T.stl" />
 				</geometry>
 				<material name="yellow"/>

Commit message: Lower-cased sia10f.urdf stl file references, to match stl file names.

File: motoman_sia10f_support/urdf/sia10f.urdf (robot description, URDF)
Before this commit: robot motoman_sia10f, 8 links, 7 joints
Links:
- link base_link: geometry collision mesh filename=package://motoman_sia10f_support/meshes/sia10f/collision/mo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; visual mesh filename=package://motoman_sia10f_support/meshes/sia10f/visual/motom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
- link link_b: geometry collision mesh filename=package://motoman_sia10f_support/meshes/sia10f/collision/mo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; visual mesh filename=package://motoman_sia10f_support/meshes/sia10f/visual/motom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
- link link_e: geometry collision mesh filename=package://motoman_sia10f_support/meshes/sia10f/collision/mo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; visual mesh filename=package://motoman_sia10f_support/meshes/sia10f/visual/motom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
- link link_l: geometry collision mesh filename=package://motoman_sia10f_support/meshes/sia10f/collision/mo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; visual mesh filename=package://motoman_sia10f_support/meshes/sia10f/visual/motom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
- link link_r: geometry collision mesh filename=package://motoman_sia10f_support/meshes/sia10f/collision/mo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; visual mesh filename=package://motoman_sia10f_support/meshes/sia10f/visual/motom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
- link link_s: geometry collision mesh filename=package://motoman_sia10f_support/meshes/sia10f/collision/mo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; visual mesh filename=package://motoman_sia10f_support/meshes/sia10f/visual/motom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
- link link_t: geometry collision mesh filename=package://motoman_sia10f_support/meshes/sia10f/collision/mo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; visual mesh filename=package://motoman_sia10f_support/meshes/sia10f/visual/motom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
- link link_u: geometry collision mesh filename=package://motoman_sia10f_support/meshes/sia10f/collision/mo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; visual mesh filename=package://motoman_sia10f_support/meshes/sia10f/visual/motom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
