Commit message: fixed motoman_sia10f macro name

File: motoman_sia10f_support/urdf/sia10f_macro.xacro (robot description, xacro)
@@ -1,5 +1,5 @@
 <?xml version="1.0" ?>
 <robot xmlns:xacro="http://ros.org/wiki/xacro">
-	<xacro:macro name="motoman_sia10d" params="prefix">
+	<xacro:macro name="motoman_sia10f" params="prefix">
 		<!-- link list -->
 		<link name="${prefix}base_link">

Commit message: rename joints to be sorted alphabetically

File: motoman_sia10f_support/urdf/sia10f_macro.xacro (robot description, xacro)
@@ -21,5 +21,5 @@
 			</collision>
 		</link>
-		<link name="${prefix}link_s">
+		<link name="${prefix}link_1_s">
 			<visual>
 				<geometry>
@@ -37,5 +37,5 @@
 			</collision>
 		</link>
-		<link name="${prefix}link_l">
+		<link name="${prefix}link_2_l">
 			<visual>
 				<origin rpy="1.57 3.1416 0" xyz="0 0 0"/>
@@ -53,5 +53,5 @@
 			</collision>
 		</link>
-		<link name="${prefix}link_e">
+		<link name="${prefix}link_3_e">
 			<visual>
 				<origin rpy="0 0 3.1415" xyz="0 0 0"/>
@@ -69,5 +69,5 @@
 			</collision>
 		</link>
-		<link name="${prefix}link_u">
+		<link name="${prefix}link_4_u">
 			<visual>
 				<origin rpy="1.57 -3.1415 0" xyz="0 0 0"/>
@@ -85,5 +85,5 @@
 			</collision>
 		</link>
-		<link name="${prefix}link_r">
+		<link name="${prefix}link_5_r">
 			<visual>
 				<origin rpy="0 0 3.1416" xyz="0 0 0"/>
@@ -101,5 +101,5 @@
 			</collision>
 		</link>
-		<link name="${prefix}link_b">
+		<link name="${prefix}link_6_b">
 			<visual>
 				<origin rpy="-1.57 0 3.1416" xyz="0 0 0"/>
@@ -117,5 +117,5 @@
 			</collision>
 		</link>
-		<link name="${prefix}link_t">
+		<link name="${prefix}link_7_t">
 			<visual>
 				<geometry>
@@ -133,49 +133,49 @@
 		<!-- end of link list -->
 		<!-- joint list -->
-		<joint name="${prefix}joint_s" type="revolute">
+		<joint name="${prefix}joint_1_s" type="revolute">
 			<parent link="${prefix}base_link"/>
-			<child link="${prefix}link_s"/>
+			<child link="${prefix}link_1_s"/>
 			<origin xyz="0 0 0.36" rpy="0 0 0"/>
 			<axis xyz="0 0 1" />
 			<limit lower="-3.1416" upper="3.1416" effort="100" velocity="2.96" />
 		</joint>
-		<joint name="${prefix}joint_l" type="revolute">
-			<parent link="${prefix}link_s"/>
-			<child link="${prefix}link_l"/>
+		<joint name="${prefix}joint_2_l" type="revolute">
+			<parent link="${prefix}link_1_s"/>
+			<child link="${prefix}link_2_l"/>
 			<origin xyz="0 0 0" rpy="0 0 0"/>
 			<axis xyz="0 1 0" />
 			<limit lower="-1.91" upper="1.91" effort="100" velocity="2.96" />
 		</joint>
-		<joint name="${prefix}joint_e" type="revolute">
-			<parent link="${prefix}link_l"/>
-			<child link="${prefix}link_e"/>
+		<joint name="${prefix}joint_3_e" type="revolute">
+			<parent link="${prefix}link_2_l"/>
+			<child link="${prefix}link_3_e"/>
 			<origin xyz="0 0 0.36" rpy="0 0 0"/>
 			<axis xyz="0 0 1" />
 			<limit lower="-2.96" upper="2.96" effort="100" velocity="2.96" />
 		</joint>
-		<joint name="${prefix}joint_u" type="revolute">
-			<parent link="${prefix}link_e"/>
-			<child link="${prefix}link_u"/>
+		<joint name="${prefix}joint_4_u" type="revolute">
+			<parent link="${prefix}link_3_e"/>
+			<child link="${prefix}link_4_u"/>
 			<origin xyz="0 0 0" rpy="0 0 0"/>
 			<axis xyz="0 -1 0" />
 			<limit lower="-2.35" upper="2.35" effort="100" velocity="2.96" />
 		</joint>
-		<joint name="${prefix}joint_r" type="revolute">
-			<parent link="${prefix}link_u"/>
-			<child link="${prefix}link_r"/>
+		<joint name="${prefix}joint_5_r" type="revolute">
+			<parent link="${prefix}link_4_u"/>
+			<child link="${prefix}link_5_r"/>
 			<origin xyz="0 0 0.360" rpy="0 0 0"/>
 			<axis xyz="0 0 -1" />
 			<limit lower="-3.1416" upper="3.1416" effort="100" velocity="3.48" />
 		</joint>
-		<joint name="${prefix}joint_b" type="revolute">
-			<parent link="${prefix}link_r"/>
-			<child link="${prefix}link_b"/>
+		<joint name="${prefix}joint_6_b" type="revolute">
+			<parent link="${prefix}link_5_r"/>
+			<child link="${prefix}link_6_b"/>
 			<origin xyz="0 0 0" rpy="0 0 0"/>
 			<axis xyz="0 -1 0" />
 			<limit lower="-1.91" upper="1.91" effort="100" velocity="3.48" />
 		</joint>
-		<joint name="${prefix}joint_t" type="revolute">
-			<parent link="${prefix}link_b"/>
-			<child link="${prefix}link_t"/>
+		<joint name="${prefix}joint_7_t" type="revolute">
+			<parent link="${prefix}link_6_b"/>
+			<child link="${prefix}link_7_t"/>
 			<origin xyz="0 0 0.155" rpy="0 0 0"/>
 			<axis xyz="0 0 -1" />

Commit message: Smaller lines to make roslint happier and case fixes for the urdf

File: motoman_sia10f_support/urdf/sia10f_macro.xacro (robot description, xacro)
@@ -6,5 +6,5 @@
 			<visual>
 				<geometry>
-					<mesh filename="package://motoman_sia10f_support/meshes/sia10f/visual/MOTOMAN_BASE.stl" />
+					<mesh filename="package://motoman_sia10f_support/meshes/sia10f/visual/motoman_base.stl" />
 				</geometry>
 				<material name="blue">
@@ -14,5 +14,5 @@
 			<collision>
 				<geometry>
-					<mesh filename="package://motoman_sia10f_support/meshes/sia10f/collision/MOTOMAN_BASE.stl" />
+					<mesh filename="package://motoman_sia10f_support/meshes/sia10f/collision/motoman_base.stl" />
 				</geometry>
 				<material name="yellow">
@@ -24,5 +24,5 @@
 			<visual>
 				<geometry>
-					<mesh filename="package://motoman_sia10f_support/meshes/sia10f/visual/MOTOMAN_AXIS_S.stl"/>
+					<mesh filename="package://motoman_sia10f_support/meshes/sia10f/visual/motoman_axis_s.stl"/>
 				</geometry>
 				<material name="silver">
@@ -32,5 +32,5 @@
 			<collision>
 				<geometry>
-					<mesh filename="package://motoman_sia10f_support/meshes/sia10f/collision/MOTOMAN_AXIS_S.stl" />
+					<mesh filename="package://motoman_sia10f_support/meshes/sia10f/collision/motoman_axis_s.stl" />
 				</geometry>
 				<material name="yellow"/>
@@ -41,5 +41,5 @@
 				<origin rpy="1.57 3.1416 0" xyz="0 0 0"/>
 				<geometry>
-					<mesh filename="package://motoman_sia10f_support/meshes/sia10f/visual/MOTOMAN_AXIS_L.stl"/>
+					<mesh filename="package://motoman_sia10f_support/meshes/sia10f/visual/motoman_axis_l.stl"/>
 				</geometry>
 				<material name="blue"/>
@@ -48,5 +48,5 @@
 				<origin rpy="1.57 3.1416 0" xyz="0 0 0"/>
 				<geometry>
-					<mesh filename="package://motoman_sia10f_support/meshes/sia10f/collision/MOTOMAN_AXIS_L.stl" />
+					<mesh filename="package://motoman_sia10f_support/meshes/sia10f/collision/motoman_axis_l.stl" />
 				</geometry>
 				<material name="yellow"/>
@@ -57,5 +57,5 @@
 				<origin rpy="0 0 3.1415" xyz="0 0 0"/>
 				<geometry>
-					<mesh filename="package://motoman_sia10f_support/meshes/sia10f/visual/MOTOMAN_AXIS_E.stl"/>
+					<mesh filename="package://motoman_sia10f_support/meshes/sia10f/visual/motoman_axis_e.stl"/>
 				</geometry>
 				<material name="silver"/>
@@ -64,5 +64,5 @@
 				<origin rpy="0 0 3.1415" xyz="0 0 0"/>
 				<geometry>
-					<mesh filename="package://motoman_sia10f_support/meshes/sia10f/collision/MOTOMAN_AXIS_E.stl" />
+					<mesh filename="package://motoman_sia10f_support/meshes/sia10f/collision/motoman_axis_e.stl" />
 				</geometry>
 				<material name="yellow"/>
@@ -73,5 +73,5 @@
 				<origin rpy="1.57 -3.1415 0" xyz="0 0 0"/>
 				<geometry>
-					<mesh filename="package://motoman_sia10f_support/meshes/sia10f/visual/MOTOMAN_AXIS_U.stl"/>
+					<mesh filename="package://motoman_sia10f_support/meshes/sia10f/visual/motoman_axis_u.stl"/>
 				</geometry>
 				<material name="blue"/>
@@ -80,5 +80,5 @@
 				<origin rpy="1.57 -3.1415 0" xyz="0 0 0"/>
 				<geometry>
-					<mesh filename="package://motoman_sia10f_support/meshes/sia10f/collision/MOTOMAN_AXIS_U.stl" />
+					<mesh filename="package://motoman_sia10f_support/meshes/sia10f/collision/motoman_axis_u.stl" />
 				</geometry>
 				<material name="yellow"/>
@@ -89,5 +89,5 @@
 				<origin rpy="0 0 3.1416" xyz="0 0 0"/>
 				<geometry>
-					<mesh filename="package://motoman_sia10f_support/meshes/sia10f/visual/MOTOMAN_AXIS_R.stl"/>
+					<mesh filename="package://motoman_sia10f_support/meshes/sia10f/visual/motoman_axis_r.stl"/>
 				</geometry>
 				<material name="silver"/>
@@ -96,5 +96,5 @@
 				<origin rpy="0 0 3.1416" xyz="0 0 0"/>
 				<geometry>
-					<mesh filename="package://motoman_sia10f_support/meshes/sia10f/collision/MOTOMAN_AXIS_R.stl" />
+					<mesh filename="package://motoman_sia10f_support/meshes/sia10f/collision/motoman_axis_r.stl" />
 				</geometry>
 				<material name="yellow"/>
@@ -105,5 +105,5 @@
 				<origin rpy="-1.57 0 3.1416" xyz="0 0 0"/>
 				<geometry>
-					<mesh filename="package://motoman_sia10f_support/meshes/sia10f/visual/MOTOMAN_AXIS_B.stl"/>
+					<mesh filename="package://motoman_sia10f_support/meshes/sia10f/visual/motoman_axis_b.stl"/>
 				</geometry>
 				<material name="blue"/>
@@ -112,5 +112,5 @@
 				<origin rpy="-1.57 0 3.1416" xyz="0 0 0"/>
 				<geometry>
-					<mesh filename="package://motoman_sia10f_support/meshes/sia10f/collision/MOTOMAN_AXIS_B.stl" />
+					<mesh filename="package://motoman_sia10f_support/meshes/sia10f/collision/motoman_axis_b.stl" />
 				</geometry>
 				<material name="yellow"/>
@@ -120,5 +120,5 @@
 			<visual>
 				<geometry>
-					<mesh filename="package://motoman_sia10f_support/meshes/sia10f/visual/MOTOMAN_AXIS_T.stl" />
+					<mesh filename="package://motoman_sia10f_support/meshes/sia10f/visual/motoman_axis_t.stl" />
 				</geometry>
 				<material name="silver"/>
@@ -126,5 +126,5 @@
 			<collision>
 				<geometry>
-					<mesh filename="package://motoman_sia10f_support/meshes/sia10f/collision/MOTOMAN_AXIS_T.stl" />
+					<mesh filename="package://motoman_sia10f_support/meshes/sia10f/collision/motoman_axis_t.stl" />
 				</geometry>
 				<material name="yellow"/>
@@ -138,5 +138,5 @@
 			<origin xyz="0 0 0.36" rpy="0 0 0"/>
 			<axis xyz="0 0 1" />
-			<limit lower="-3.1416" upper="3.1416" effort="100" velocity="2.96" />
+			<limit lower="-3.1416" upper="3.1416" effort="0" velocity="2.96" />
 		</joint>
 		<joint name="${prefix}joint_2_l" type="revolute">
@@ -145,5 +145,5 @@
 			<origin xyz="0 0 0" rpy="0 0 0"/>
 			<axis xyz="0 1 0" />
-			<limit lower="-1.91" upper="1.91" effort="100" velocity="2.96" />
+			<limit lower="-1.91" upper="1.91" effort="0" velocity="2.96" />
 		</joint>
 		<joint name="${prefix}joint_3_e" type="revolute">
@@ -152,5 +152,5 @@
 			<origin xyz="0 0 0.36" rpy="0 0 0"/>
 			<axis xyz="0 0 1" />
-			<limit lower="-2.96" upper="2.96" effort="100" velocity="2.96" />
+			<limit lower="-2.96" upper="2.96" effort="0" velocity="2.96" />
 		</joint>
 		<joint name="${prefix}joint_4_u" type="revolute">
@@ -159,5 +159,5 @@
 			<origin xyz="0 0 0" rpy="0 0 0"/>
 			<axis xyz="0 -1 0" />
-			<limit lower="-2.35" upper="2.35" effort="100" velocity="2.96" />
+			<limit lower="-2.35" upper="2.35" effort="0" velocity="2.96" />
 		</joint>
 		<joint name="${prefix}joint_5_r" type="revolute">
@@ -166,5 +166,5 @@
 			<origin xyz="0 0 0.360" rpy="0 0 0"/>
 			<axis xyz="0 0 -1" />
-			<limit lower="-3.1416" upper="3.1416" effort="100" velocity="3.48" />
+			<limit lower="-3.1416" upper="3.1416" effort="0" velocity="3.48" />
 		</joint>
 		<joint name="${prefix}joint_6_b" type="revolute">
@@ -173,5 +173,5 @@
 			<origin xyz="0 0 0" rpy="0 0 0"/>
 			<axis xyz="0 -1 0" />
-			<limit lower="-1.91" upper="1.91" effort="100" velocity="3.48" />
+			<limit lower="-1.91" upper="1.91" effort="0" velocity="3.48" />
 		</joint>
 		<joint name="${prefix}joint_7_t" type="revolute">
@@ -180,5 +180,5 @@
 			<origin xyz="0 0 0.155" rpy="0 0 0"/>
 			<axis xyz="0 0 -1" />
-			<limit lower="-3.1416" upper="3.1416" effort="100" velocity="6.97" />
+			<limit lower="-3.1416" upper="3.1416" effort="0" velocity="6.97" />
 		</joint>
 		<!-- end of joint list -->

Commit message: Added tool0 for sia10f

File: motoman_sia10f_support/urdf/sia10f_macro.xacro (robot description, xacro)
@@ -131,4 +131,5 @@
 			</collision>
 		</link>
+		<link name="${prefix}link_tool0" />
 		<!-- end of link list -->
 		<!-- joint list -->
@@ -182,4 +183,9 @@
 			<limit lower="-3.1416" upper="3.1416" effort="0" velocity="6.97" />
 		</joint>
+		    <joint name="${prefix}joint_tool0" type="fixed" >
+      <origin xyz="0 0 0.0" rpy="0 0 -3.1416"/>
+      <parent link="${prefix}link_7_t" />
+      <child link="${prefix}link_tool0" />
+    </joint>
 		<!-- end of joint list -->
 	</xacro:macro>

Commit message: ident

File: motoman_sia10f_support/urdf/sia10f_macro.xacro (robot description, xacro)
@@ -183,5 +183,5 @@
 			<limit lower="-3.1416" upper="3.1416" effort="0" velocity="6.97" />
 		</joint>
-		    <joint name="${prefix}joint_tool0" type="fixed" >
+    <joint name="${prefix}joint_tool0" type="fixed" >
       <origin xyz="0 0 0.0" rpy="0 0 -3.1416"/>
       <parent link="${prefix}link_7_t" />

Commit message: sia10f: don't round PI in joint_t-tool0 transform.
Leads to incorrect 'base->tool0' transform orientations.

File: motoman_sia10f_support/urdf/sia10f_macro.xacro (robot description, xacro)
@@ -184,5 +184,5 @@
 		</joint>
     <joint name="${prefix}joint_tool0" type="fixed" >
-      <origin xyz="0 0 0.0" rpy="0 0 -3.1416"/>
+      <origin xyz="0 0 0.0" rpy="0 0 -3.1415926535"/>
       <parent link="${prefix}link_7_t" />
       <child link="${prefix}link_tool0" />

Commit message: Fix for issue #106: use full-precision PI for tool0 transform (#110)
* sia10f: don't round PI in joint_t-tool0 transform.

Leads to incorrect 'base->tool0' transform orientations.

* sia20: don't round PI in joint_t-tool0 transform. Fix #106.

Leads to incorrect 'base->tool0' transform orientations.

File: motoman_sia10f_support/urdf/sia10f_macro.xacro (robot description, xacro)
@@ -184,5 +184,5 @@
 		</joint>
     <joint name="${prefix}joint_tool0" type="fixed" >
-      <origin xyz="0 0 0.0" rpy="0 0 -3.1416"/>
+      <origin xyz="0 0 0.0" rpy="0 0 -3.1415926535"/>
       <parent link="${prefix}link_7_t" />
       <child link="${prefix}link_tool0" />

File: motoman_sia20d_support/urdf/sia20d_macro.xacro (robot description, xacro)
@@ -186,5 +186,5 @@
 		</joint>
     <joint name="${prefix}link_t-tool0" type="fixed" >
-      <origin xyz="0 0 0.0" rpy="0 0 -3.1416"/>
+      <origin xyz="0 0 0.0" rpy="0 0 -3.1415926535"/>
       <parent link="${prefix}link_t" />
       <child link="${prefix}tool0" />
