Commit message: Fix B axis orientation at position 0.

File: motoman_mh6_support/urdf/mh6.urdf (robot description, URDF)
Before this commit: robot motoman_mh6, 7 links, 6 joints
Joints:
- joint joint_t: axis -1 0 0 -> 0 0 1; origin xyz=0.095 0 0 -> xyz=0 0 -0.095

File: motoman_mh6_support/urdf/mh6_macro.xacro (robot description, xacro)
@@ -149,6 +149,6 @@
 			<parent link="${prefix}link_b"/>
 			<child link="${prefix}link_t"/>
-			<origin xyz="0.095 0 0" />
-			<axis xyz="-1 0 0" />
+			<origin xyz="0 0 -0.095" />
+			<axis xyz="0 0 1" />
 			<limit lower="${-360 * pi / 180}" upper="${360 * pi / 180}" effort="100" velocity="${610 * pi / 180}" />
 		</joint>
