Commit message: mpl_support: update pkg references in files.

File: motoman_mpl_support/urdf/mpl80.xacro (robot description, xacro)
@@ -1,5 +1,5 @@
 <?xml version="1.0" ?>
 <robot name="motoman_mpl80" xmlns:xacro="http://ros.org/wiki/xacro">
-  <xacro:include filename="$(find motoman_mpl80_support)/urdf/mpl80_macro.xacro"/>
+  <xacro:include filename="$(find motoman_mpl_support)/urdf/mpl80_macro.xacro"/>
   <xacro:motoman_mpl80 prefix=""/>
 </robot>

File: motoman_mpl_support/urdf/mpl80_macro.xacro (robot description, xacro)
@@ -7,5 +7,5 @@
       <origin xyz="-0.407 -0.287 0" rpy="0 0 0"/>
       <geometry>
-        <mesh filename="package://motoman_mpl80_support/meshes/mpl80/visual/base_link.stl"/>
+        <mesh filename="package://motoman_mpl_support/meshes/mpl80/visual/base_link.stl"/>
       </geometry>
       <material name="blue">
@@ -16,5 +16,5 @@
       <origin xyz="-0.407 -0.287 0" rpy="0 0 0"/>
       <geometry>
-        <mesh filename="package://motoman_mpl80_support/meshes/mpl80/collision/base_link.stl"/>
+        <mesh filename="package://motoman_mpl_support/meshes/mpl80/collision/base_link.stl"/>
       </geometry>
       <material name="collision_material">
@@ -27,5 +27,5 @@
       <origin xyz="-0.407 -0.287 -0.540" rpy="0 0 0"/>
       <geometry>
-        <mesh filename="package://motoman_mpl80_support/meshes/mpl80/visual/link_s.stl"/>
+        <mesh filename="package://motoman_mpl_support/meshes/mpl80/visual/link_s.stl"/>
       </geometry>
       <material name="blue"/>
@@ -34,5 +34,5 @@
       <origin xyz="-0.407 -0.287 -0.540" rpy="0 0 0"/>
       <geometry>
-        <mesh filename="package://motoman_mpl80_support/meshes/mpl80/collision/link_s.stl"/>
+        <mesh filename="package://motoman_mpl_support/meshes/mpl80/collision/link_s.stl"/>
       </geometry>
       <material name="collision_material"/>
@@ -43,5 +43,5 @@
       <origin xyz="-0.552 -0.287 -0.540" rpy="0 0 0"/>
       <geometry>
-        <mesh filename="package://motoman_mpl80_support/meshes/mpl80/visual/link_l.stl"/>
+        <mesh filename="package://motoman_mpl_support/meshes/mpl80/visual/link_l.stl"/>
       </geometry>
       <material name="blue"/>
@@ -50,5 +50,5 @@
       <origin xyz="-0.552 -0.287 -0.540" rpy="0 0 0"/>
       <geometry>
-        <mesh filename="package://motoman_mpl80_support/meshes/mpl80/collision/link_l.stl"/>
+        <mesh filename="package://motoman_mpl_support/meshes/mpl80/collision/link_l.stl"/>
       </geometry>
       <material name="collision_material"/>
@@ -59,5 +59,5 @@
       <origin xyz="-0.546 -0.287 -1.411" rpy="0 0 0"/>
       <geometry>
-        <mesh filename="package://motoman_mpl80_support/meshes/mpl80/visual/link_u.stl"/>
+        <mesh filename="package://motoman_mpl_support/meshes/mpl80/visual/link_u.stl"/>
       </geometry>
       <material name="blue"/>
@@ -66,5 +66,5 @@
       <origin xyz="-0.546 -0.287 -1.411" rpy="0 0 0"/>
       <geometry>
-        <mesh filename="package://motoman_mpl80_support/meshes/mpl80/collision/link_u.stl"/>
+        <mesh filename="package://motoman_mpl_support/meshes/mpl80/collision/link_u.stl"/>
       </geometry>
       <material name="collision_material"/>
@@ -75,5 +75,5 @@
       <origin xyz="-0.546 -0.287 -1.621" rpy="0 0 0"/>
       <geometry>
-        <mesh filename="package://motoman_mpl80_support/meshes/mpl80/visual/link_r.stl"/>
+        <mesh filename="package://motoman_mpl_support/meshes/mpl80/visual/link_r.stl"/>
       </geometry>
       <material name="blue"/>
@@ -82,5 +82,5 @@
       <origin xyz="-0.546 -0.287 -1.621" rpy="0 0 0"/>
       <geometry>
-        <mesh filename="package://motoman_mpl80_support/meshes/mpl80/collision/link_r.stl"/>
+        <mesh filename="package://motoman_mpl_support/meshes/mpl80/collision/link_r.stl"/>
       </geometry>
       <material name="collision_material"/>
@@ -91,5 +91,5 @@
       <origin xyz="-1.571 -0.291 -1.621" rpy="0 0 0"/>
       <geometry>
-        <mesh filename="package://motoman_mpl80_support/meshes/mpl80/visual/link_b.stl"/>
+        <mesh filename="package://motoman_mpl_support/meshes/mpl80/visual/link_b.stl"/>
       </geometry>
       <material name="blue"/>
@@ -98,5 +98,5 @@
       <origin xyz="-1.571 -0.291 -1.621" rpy="0 0 0"/>
       <geometry>
-        <mesh filename="package://motoman_mpl80_support/meshes/mpl80/collision/link_b.stl"/>
+        <mesh filename="package://motoman_mpl_support/meshes/mpl80/collision/link_b.stl"/>
       </geometry>
       <material name="collision_material"/>
@@ -107,5 +107,5 @@
       <origin xyz="-1.571 -0.291 -1.446" rpy="0 0 0"/>
       <geometry>
-        <mesh filename="package://motoman_mpl80_support/meshes/mpl80/visual/link_t.stl"/>
+        <mesh filename="package://motoman_mpl_support/meshes/mpl80/visual/link_t.stl"/>
       </geometry>
       <material name="blue"/>
@@ -114,5 +114,5 @@
       <origin xyz="-1.571 -0.291 -1.446" rpy="0 0 0"/>
       <geometry>
-        <mesh filename="package://motoman_mpl80_support/meshes/mpl80/collision/link_t.stl"/>
+        <mesh filename="package://motoman_mpl_support/meshes/mpl80/collision/link_t.stl"/>
       </geometry>
       <material name="collision_material"/>
