Commit message: mpl80: give all meshes link-local origins.

File: motoman_mpl_support/urdf/mpl80_macro.xacro (robot description, xacro)
@@ -5,5 +5,5 @@
   <link name="${prefix}base_link">
     <visual>
-      <origin xyz="-0.407 -0.287 0" rpy="0 0 0"/>
+      <origin xyz="0 0 0" rpy="0 0 0"/>
       <geometry>
         <mesh filename="package://motoman_mpl_support/meshes/mpl80/visual/base_link.stl"/>
@@ -14,5 +14,5 @@
     </visual>
     <collision>
-      <origin xyz="-0.407 -0.287 0" rpy="0 0 0"/>
+      <origin xyz="0 0 0" rpy="0 0 0"/>
       <geometry>
         <mesh filename="package://motoman_mpl_support/meshes/mpl80/collision/base_link.stl"/>
@@ -25,5 +25,5 @@
   <link name="${prefix}link_s">
     <visual>
-      <origin xyz="-0.407 -0.287 -0.540" rpy="0 0 0"/>
+      <origin xyz="0 0 0" rpy="0 0 0"/>
       <geometry>
         <mesh filename="package://motoman_mpl_support/meshes/mpl80/visual/link_s.stl"/>
@@ -32,5 +32,5 @@
     </visual>
     <collision>
-      <origin xyz="-0.407 -0.287 -0.540" rpy="0 0 0"/>
+      <origin xyz="0 0 0" rpy="0 0 0"/>
       <geometry>
         <mesh filename="package://motoman_mpl_support/meshes/mpl80/collision/link_s.stl"/>
@@ -41,5 +41,5 @@
   <link name="${prefix}link_l">
     <visual>
-      <origin xyz="-0.552 -0.287 -0.540" rpy="0 0 0"/>
+      <origin xyz="0 0 0" rpy="0 0 0"/>
       <geometry>
         <mesh filename="package://motoman_mpl_support/meshes/mpl80/visual/link_l.stl"/>
@@ -48,5 +48,5 @@
     </visual>
     <collision>
-      <origin xyz="-0.552 -0.287 -0.540" rpy="0 0 0"/>
+      <origin xyz="0 0 0" rpy="0 0 0"/>
       <geometry>
         <mesh filename="package://motoman_mpl_support/meshes/mpl80/collision/link_l.stl"/>
@@ -57,5 +57,5 @@
   <link name="${prefix}link_u">
     <visual>
-      <origin xyz="-0.546 -0.287 -1.411" rpy="0 0 0"/>
+      <origin xyz="0 0 0" rpy="0 0 0"/>
       <geometry>
         <mesh filename="package://motoman_mpl_support/meshes/mpl80/visual/link_u.stl"/>
@@ -64,5 +64,5 @@
     </visual>
     <collision>
-      <origin xyz="-0.546 -0.287 -1.411" rpy="0 0 0"/>
+      <origin xyz="0 0 0" rpy="0 0 0"/>
       <geometry>
         <mesh filename="package://motoman_mpl_support/meshes/mpl80/collision/link_u.stl"/>
@@ -73,5 +73,5 @@
   <link name="${prefix}link_r">
     <visual>
-      <origin xyz="-0.546 -0.287 -1.621" rpy="0 0 0"/>
+      <origin xyz="0 0 0" rpy="0 0 0"/>
       <geometry>
         <mesh filename="package://motoman_mpl_support/meshes/mpl80/visual/link_r.stl"/>
@@ -80,5 +80,5 @@
     </visual>
     <collision>
-      <origin xyz="-0.546 -0.287 -1.621" rpy="0 0 0"/>
+      <origin xyz="0 0 0" rpy="0 0 0"/>
       <geometry>
         <mesh filename="package://motoman_mpl_support/meshes/mpl80/collision/link_r.stl"/>
@@ -89,5 +89,5 @@
   <link name="${prefix}link_b">
     <visual>
-      <origin xyz="-1.571 -0.291 -1.621" rpy="0 0 0"/>
+      <origin xyz="0 0 0" rpy="0 0 0"/>
       <geometry>
         <mesh filename="package://motoman_mpl_support/meshes/mpl80/visual/link_b.stl"/>
@@ -96,5 +96,5 @@
     </visual>
     <collision>
-      <origin xyz="-1.571 -0.291 -1.621" rpy="0 0 0"/>
+      <origin xyz="0 0 0" rpy="0 0 0"/>
       <geometry>
         <mesh filename="package://motoman_mpl_support/meshes/mpl80/collision/link_b.stl"/>
@@ -105,5 +105,5 @@
   <link name="${prefix}link_t">
     <visual>
-      <origin xyz="-1.571 -0.291 -1.446" rpy="0 0 0"/>
+      <origin xyz="0 0 0" rpy="0 0 0"/>
       <geometry>
         <mesh filename="package://motoman_mpl_support/meshes/mpl80/visual/link_t.stl"/>
@@ -112,5 +112,5 @@
     </visual>
     <collision>
-      <origin xyz="-1.571 -0.291 -1.446" rpy="0 0 0"/>
+      <origin xyz="0 0 0" rpy="0 0 0"/>
       <geometry>
         <mesh filename="package://motoman_mpl_support/meshes/mpl80/collision/link_t.stl"/>

Commit message: Removed none standard robot position b10deg from MoveIt package Correction of the "base" frame in the xacro file to correspond to the manufacturer standard coordinate system.

File: motoman_mpl_support/urdf/mpl80_macro.xacro (robot description, xacro)
@@ -171,5 +171,5 @@
   <link name="${prefix}base" />
   <joint name="${prefix}base_link-base" type="fixed">
-    <origin xyz="0 0 0" rpy="0 0 0"/>
+    <origin xyz="0 0 0.540" rpy="0 0 0"/>
     <parent link="${prefix}base_link"/>
     <child link="${prefix}base"/>
