Commit message: Modified version of the urdf

File: motoman_sda10f_support/urdf/sda10f_macro.xacro (robot description, xacro)
@@ -1,417 +1,13 @@
 <?xml version="1.0" ?>
-<robot xmlns:xacro="http://ros.org/wiki/xacro">
-	<xacro:macro name="motoman_sda10f" params="prefix">
-		<!-- link list -->
-		<link name="${prefix}base_link">
-			<visual>
-				<geometry>
-					<mesh filename="package://motoman_sda10f_support/meshes/sda10f/visual/motoman_base.stl" />
-				</geometry>
-				<material name="blue">
-					<color rgba="0 0 1 1"/>
-				</material>
-			</visual>
-			<collision>
-				<geometry>
-					<mesh filename="package://motoman_sda10f_support/meshes/sda10f/collision/motoman_base.stl" />
-				</geometry>
-				<material name="yellow">
-					<color rgba="0 1 1 1"/>
-				</material>
-			</collision>
-		</link>
-		<link name="${prefix}link_x_b1">
-			<visual>
-				<origin rpy="0 0 0" xyz="0 0 0"/>
-				<geometry>
-					<mesh filename="package://motoman_sda10f_support/meshes/sda10f/visual/motoman_axis_b1.stl"/>
-				</geometry>
-				<material name="silver">
-					<color rgba="0.8 0.8 0.8 1"/>
-				</material>
-			</visual>
-			<collision>
-				<origin rpy="0 0 0" xyz="0 0 0"/>
-				<geometry>
-					<mesh filename="package://motoman_sda10f_support/meshes/sda10f/collision/motoman_axis_b1.stl" />
-				</geometry>
-				<material name="yellow"/>
-			</collision>
-		</link>
-		<link name="${prefix}link_x_b2">
-			<visual>
-				<origin rpy="0 0 0" xyz="0 0 0"/>
-				<geometry>
-					<mesh filename="package://motoman_sda10f_support/meshes/sda10f/visual/motoman_axis_b1.stl"/>
-				</geometry>
-				<material name="silver">
-					<color rgba="0.8 0.8 0.8 1"/>
-				</material>
-			</visual>
-			<collision>
-				<origin rpy="0 0 0" xyz="0 0 0"/>
-				<geometry>
-					<mesh filename="package://motoman_sda10f_support/meshes/sda10f/collision/motoman_axis_b1.stl" />
-				</geometry>
-				<material name="yellow"/>
-			</collision>
-		</link>
-		<!-- R1 Group -->
-		<link name="${prefix}link_r1_1_s">
-			<visual>
-				<origin rpy="0 0 0" xyz="0 0 0"/>
-				<geometry>
-					<mesh filename="package://motoman_sda10f_support/meshes/sda10f/visual/motoman_axis_r1_s.stl"/>
-				</geometry>
-				<material name="blue">
-					<color rgba="0.8 0.8 0.8 1"/>
-				</material>
-			</visual>
-			<collision>
-				<origin rpy="0 0 0" xyz="0 0 0"/>
-				<geometry>
-					<mesh filename="package://motoman_sda10f_support/meshes/sda10f/collision/motoman_axis_r1_s.stl" />
-				</geometry>
-				<material name="yellow"/>
-			</collision>
-		</link>
-		<link name="${prefix}link_r1_2_l">
-			<visual>
-				<origin rpy="0 0 0" xyz="0 0 0"/>
-				<geometry>
-					<mesh filename="package://motoman_sda10f_support/meshes/sda10f/visual/motoman_axis_r1_l.stl"/>
-				</geometry>
-				<material name="silver"/>
-			</visual>
-			<collision>
-				<origin rpy="0 0 0" xyz="0 0 0"/>
-				<geometry>
-					<mesh filename="package://motoman_sda10f_support/meshes/sda10f/collision/motoman_axis_r1_l.stl"/>
-				</geometry>
-				<material name="yellow"/>
-			</collision>
-		</link>
-		<link name="${prefix}link_r1_3_e">
-			<visual>
-				<origin rpy="0 0 0" xyz="0 0 0"/>
-				<geometry>
-					<mesh filename="package://motoman_sda10f_support/meshes/sda10f/visual/motoman_axis_r1_e.stl"/>
-				</geometry>
-				<material name="blue"/>
-			</visual>
-			<collision>
-				<origin rpy="0 0 0" xyz="0 0 0"/>
-				<geometry>
-					<mesh filename="package://motoman_sda10f_support/meshes/sda10f/collision/motoman_axis_r1_e.stl"/>
-				</geometry>
-				<material name="yellow"/>
-			</collision>
-		</link>
-		<link name="${prefix}link_r1_4_u">
-			<visual>
-				<origin rpy="0 0 0" xyz="0 0 0"/>
-				<geometry>
-					<mesh filename="package://motoman_sda10f_support/meshes/sda10f/visual/motoman_axis_r1_u.stl"/>
-				</geometry>
-				<material name="silver"/>
-			</visual>
-			<collision>
-				<origin rpy="0 0 0" xyz="0 0 0"/>
-				<geometry>
-					<mesh filename="package://motoman_sda10f_support/meshes/sda10f/collision/motoman_axis_r1_u.stl"/>
-				</geometry>
-				<material name="yellow"/>
-			</collision>
-		</link>
-		<link name="${prefix}link_r1_5_r">
-			<visual>
-				<origin rpy="0 0 0" xyz="0 0 0"/>
-				<geometry>
-					<mesh filename="package://motoman_sda10f_support/meshes/sda10f/visual/motoman_axis_r1_r.stl"/>
-				</geometry>
-				<material name="blue"/>
-			</visual>
-			<collision>
-				<origin rpy="0 0 0" xyz="0 0 0"/>
-				<geometry>
-					<mesh filename="package://motoman_sda10f_support/meshes/sda10f/collision/motoman_axis_r1_r.stl"/>
-				</geometry>
-				<material name="yellow"/>
-			</collision>
-		</link>
-		<link name="${prefix}link_r1_6_b">
-			<visual>
-				<origin rpy="0 0 0" xyz="0 0 0"/>
-				<geometry>
-					<mesh filename="package://motoman_sda10f_support/meshes/sda10f/visual/motoman_axis_r1_b.stl"/>
-				</geometry>
-				<material name="silver"/>
-			</visual>
-			<collision>
-				<origin rpy="0 0 0" xyz="0 0 0"/>
-				<geometry>
-					<mesh filename="package://motoman_sda10f_support/meshes/sda10f/collision/motoman_axis_r1_b.stl"/>
-				</geometry>
-				<material name="yellow"/>
-			</collision>
-		</link>
-		<link name="${prefix}link_r1_7_t">
-			<visual>
-				<geometry>
-					<mesh filename="package://motoman_sda10f_support/meshes/sda10f/visual/motoman_axis_r1_t.stl" />
-				</geometry>
-				<material name="blue"/>
-			</visual>
-			<collision>
-				<geometry>
-					<mesh filename="package://motoman_sda10f_support/meshes/sda10f/collision/motoman_axis_r1_t.stl" />
-				</geometry>
-				<material name="yellow"/>
-			</collision>
-		</link>
-	    <link name="${prefix}r1_tool0" />
-		<!-- R2 Group -->
-		<link name="${prefix}link_r2_1_s">
-			<visual>
-				<origin rpy="0 0 0" xyz="0 0 0"/>
-				<geometry>
-					<mesh filename="package://motoman_sda10f_support/meshes/sda10f/visual/motoman_axis_r2_s.stl"/>
-				</geometry>
-				<material name="blue">
-					<color rgba="0.8 0.8 0.8 1"/>
-				</material>
-			</visual>
-			<collision>
-				<origin rpy="0 0 0" xyz="0 0 0"/>
-				<geometry>
-					<mesh filename="package://motoman_sda10f_support/meshes/sda10f/collision/motoman_axis_r2_s.stl" />
-				</geometry>
-				<material name="yellow"/>
-			</collision>
-		</link>
-		<link name="${prefix}link_r2_2_l">
-			<visual>
-				<origin rpy="0 0 0" xyz="0 0 0"/>
-				<geometry>
-					<mesh filename="package://motoman_sda10f_support/meshes/sda10f/visual/motoman_axis_r2_l.stl"/>
-				</geometry>
-				<material name="silver"/>
-			</visual>
-			<collision>
-				<origin rpy="0 0 0" xyz="0 0 0"/>
-				<geometry>
-					<mesh filename="package://motoman_sda10f_support/meshes/sda10f/collision/motoman_axis_r2_l.stl"/>
-				</geometry>
-				<material name="yellow"/>
-			</collision>
-		</link>
-		<link name="${prefix}link_r2_3_e">
-			<visual>
-				<origin rpy="0 0 0" xyz="0 0 0"/>
-				<geometry>
-					<mesh filename="package://motoman_sda10f_support/meshes/sda10f/visual/motoman_axis_r2_e.stl"/>
-				</geometry>
-				<material name="blue"/>
-			</visual>
-			<collision>
-				<origin rpy="0 0 0" xyz="0 0 0"/>
-				<geometry>
-					<mesh filename="package://motoman_sda10f_support/meshes/sda10f/collision/motoman_axis_r2_e.stl"/>
-				</geometry>
-				<material name="yellow"/>
-			</collision>
-		</link>
-		<link name="${prefix}link_r2_4_u">
-			<visual>
-				<origin rpy="0 0 0" xyz="0 0 0"/>
-				<geometry>
-					<mesh filename="package://motoman_sda10f_support/meshes/sda10f/visual/motoman_axis_r2_u.stl"/>
-				</geometry>
-				<material name="silver"/>
-			</visual>
-			<collision>
-				<origin rpy="0 0 0" xyz="0 0 0"/>
-				<geometry>
-					<mesh filename="package://motoman_sda10f_support/meshes/sda10f/collision/motoman_axis_r2_u.stl"/>
-				</geometry>
-				<material name="yellow"/>
-			</collision>
-		</link>
-		<link name="${prefix}link_r2_5_r">
-			<visual>
-				<origin rpy="0 0 0" xyz="0 0 0"/>
-				<geometry>
-					<mesh filename="package://motoman_sda10f_support/meshes/sda10f/visual/motoman_axis_r2_r.stl"/>
-				</geometry>
-				<material name="blue"/>
-			</visual>
-			<collision>
-				<origin rpy="0 0 0" xyz="0 0 0"/>
-				<geometry>
-					<mesh filename="package://motoman_sda10f_support/meshes/sda10f/collision/motoman_axis_r2_r.stl"/>
-				</geometry>
-				<material name="yellow"/>
-			</collision>
-		</link>
-		<link name="${prefix}link_r2_6_b">
-			<visual>
-				<origin rpy="0 0 0" xyz="0 0 0"/>
-				<geometry>
-					<mesh filename="package://motoman_sda10f_support/meshes/sda10f/visual/motoman_axis_r2_b.stl"/>
-				</geometry>
-				<material name="silver"/>
-			</visual>
-			<collision>
-				<origin rpy="0 0 0" xyz="0 0 0"/>
-				<geometry>
-					<mesh filename="package://motoman_sda10f_support/meshes/sda10f/collision/motoman_axis_r2_b.stl"/>
-				</geometry>
-				<material name="yellow"/>
-			</collision>
-		</link>
-		<link name="${prefix}link_r2_7_t">
-			<visual>
-				<geometry>
-					<mesh filename="package://motoman_sda10f_support/meshes/sda10f/visual/motoman_axis_r2_t.stl" />
-				</geometry>
-				<material name="blue"/>
-			</visual>
-			<collision>
-				<geometry>
-					<mesh filename="package://motoman_sda10f_support/meshes/sda10f/collision/motoman_axis_r2_t.stl" />
-				</geometry>
-				<material name="yellow"/>
-			</collision>
-		</link>
-    <link name="${prefix}r2_tool0" />
-		<!-- end of link list -->
-		<!-- joint list -->
-		<joint name="${prefix}joint_x_b1" type="revolute">
-			<parent link="${prefix}base_link"/>
-			<child link="${prefix}link_x_b1"/>
-			<origin xyz="0.09257 0 0.8835" rpy="0 0 0"/>
-			<axis xyz="0 0 1" />
-			<limit lower="-2.9570" upper="2.9570" effort="100" velocity="2.26" />
-		</joint>
-		<joint name="${prefix}joint_x_b2" type="revolute">
-			<parent link="${prefix}base_link"/>
-			<child link="${prefix}link_x_b2"/>
-			<origin xyz="0.09257 0 0.8835" rpy="0 0 0"/>
-			<axis xyz="0 0 1" />
-			<limit lower="-2.9570" upper="2.9570" effort="100" velocity="2.26" />
-			<mimic joint="${prefix}joint_x_b1" multiplier="1" offset="0"/>
-		</joint>
-		<!-- R1 -->
-		<joint name="${prefix}joint_r1_1_s" type="revolute">
-			<parent link="${prefix}link_x_b1"/>
-			<child link="${prefix}link_r1_1_s"/>
-			<origin xyz="0.09996 0.0275 0.32214" rpy="1.57 0 0"/>
-			<axis xyz="0 0 -1" />
-			<limit lower="-3.13" upper="3.13" effort="100" velocity="2.95" />
-		</joint>
-		<joint name="${prefix}joint_r1_2_l" type="revolute">
-			<parent link="${prefix}link_r1_1_s"/>
-			<child link="${prefix}link_r1_2_l"/>
-			<origin xyz="0 0.0577 -0.2255" rpy="-1.57 0 0"/>
-			<axis xyz="0 0 -1" />
-			<limit lower="-1.90" upper="1.90" effort="100" velocity="2.95" />
-		</joint>
-		<joint name="${prefix}joint_r1_3_e" type="revolute">
-			<parent link="${prefix}link_r1_2_l"/>
-			<child link="${prefix}link_r1_3_e"/>
-			<origin xyz="0 0.1690 -0.0454" rpy="1.57 0 0"/>
-			<axis xyz="0 0 -1" />
-			<limit lower="-2.95" upper="2.95" effort="100" velocity="2.95" />
-		</joint>
-		<joint name="${prefix}joint_r1_4_u" type="revolute">
-			<parent link="${prefix}link_r1_3_e"/>
-			<child link="${prefix}link_r1_4_u"/>
-			<origin xyz="0 -0.0085 -0.181" rpy="-1.57 0 0"/>
-			<axis xyz="0 0 1" />
-			<limit lower="-2.36" upper="2.36" effort="100" velocity="2.95" />
-		</joint>
-		<joint name="${prefix}joint_r1_5_r" type="revolute">
-			<parent link="${prefix}link_r1_4_u"/>
-			<child link="${prefix}link_r1_5_r"/>
-			<origin xyz="0 0.1936 0.0155" rpy="1.57 0 0"/>
-			<axis xyz="0 0 1" />
-			<limit lower="-3.13" upper="3.13" effort="100" velocity="3.48" />
-		</joint>
-		<joint name="${prefix}joint_r1_6_b" type="revolute">
-			<parent link="${prefix}link_r1_5_r"/>
-			<child link="${prefix}link_r1_6_b"/>
-			<origin xyz="0 0.0080 -0.155" rpy="-1.57 0 0"/>
-			<axis xyz="0 0 1" />
-			<limit lower="-1.90" upper="1.90" effort="100" velocity="3.48" />
-		</joint>
-		<joint name="${prefix}joint_r1_7_t" type="revolute">
-			<parent link="${prefix}link_r1_6_b"/>
-			<child link="${prefix}link_r1_7_t"/>
-			<origin xyz="0 0.168 -0.015" rpy="1.57 0 0"/>
-			<axis xyz="0 0 1" />
-			<limit lower="-3.13" upper="3.13" effort="100" velocity="6.97" />
-		</joint>
-    <joint name="${prefix}link_r1_7_t-tool0" type="fixed" >
-      <origin xyz="0 0 0.0" rpy="0 0 -3.13"/>
-      <parent link="${prefix}link_r1_7_t" />
-      <child link="${prefix}r1_tool0" />
-    </joint>
-		<!-- end of joint list -->
-		<!-- R2 -->
-		<joint name="${prefix}joint_r2_1_s" type="revolute">
-			<parent link="${prefix}link_x_b1"/>
-			<child link="${prefix}link_r2_1_s"/>
-			<origin xyz="0.09996 -0.0275 0.32214" rpy="1.57 0 0"/>
-			<axis xyz="0 0 -1" />
-			<limit lower="-3.13" upper="3.13" effort="100" velocity="2.95" />
-		</joint>
-		<joint name="${prefix}joint_r2_2_l" type="revolute">
-			<parent link="${prefix}link_r2_1_s"/>
-			<child link="${prefix}link_r2_2_l"/>
-			<origin xyz="0 0.0577 0.2255" rpy="-1.57 0 0"/>
-			<axis xyz="0 0 1" />
-			<limit lower="-1.90" upper="1.90" effort="100" velocity="2.95" />
-		</joint>
-		<joint name="${prefix}joint_r2_3_e" type="revolute">
-			<parent link="${prefix}link_r2_2_l"/>
-			<child link="${prefix}link_r2_3_e"/>
-			<origin xyz="0 -0.1690 -0.0454" rpy="1.57 0 0"/>
-			<axis xyz="0 0 -1" />
-			<limit lower="-2.95" upper="2.95" effort="100" velocity="2.95" />
-		</joint>
-		<joint name="${prefix}joint_r2_4_u" type="revolute">
-			<parent link="${prefix}link_r2_3_e"/>
-			<child link="${prefix}link_r2_4_u"/>
-			<origin xyz="0 -0.0085 0.181" rpy="-1.57 0 0"/>
-			<axis xyz="0 0 -1" />
-			<limit lower="-2.36" upper="2.36" effort="100" velocity="2.95" />
-		</joint>
-		<joint name="${prefix}joint_r2_5_r" type="revolute">
-			<parent link="${prefix}link_r2_4_u"/>
-			<child link="${prefix}link_r2_5_r"/>
-			<origin xyz="0 -0.1936 0.0155" rpy="1.57 0 0"/>
-			<axis xyz="0 0 1" />
-			<limit lower="-3.13" upper="3.13" effort="100" velocity="3.48" />
-		</joint>
-		<joint name="${prefix}joint_r2_6_b" type="revolute">
-			<parent link="${prefix}link_r2_5_r"/>
-			<child link="${prefix}link_r2_6_b"/>
-			<origin xyz="0 0.0080 0.155" rpy="-1.57 0 0"/>
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
Commit message: Patch for issue #166

File: motoman_sda10f_support/urdf/sda10f_macro.xacro (robot description, xacro)
@@ -1,13 +1,19 @@
 <?xml version="1.0" ?>
-<robot xmlns:xacro="http://ros.org/wiki/xacro"
-    name="sda10f">
-        <xacro:include filename="$(find motoman_sda10f_support)/urdf/common_torso_macro.xacro" />
-        <xacro:include filename="$(find motoman_sda10f_support)/urdf/arm_macro.xacro" />
-        <xacro:torso name="torso" prefix="torso_"/>
-        <xacro:motoman_arm name="arm_left" prefix="arm_left_" parent="torso_link_b1" reflect="1">
+<robot xmlns:xacro="http://ros.org/wiki/xacro">
+     <xacro:include filename="$(find motoman_sda10f_support)/urdf/common_torso_macro.xacro" />
+     <xacro:include filename="$(find motoman_sda10f_support)/urdf/arm_macro.xacro" />
+     <xacro:macro name="motoman_sda10f" params="prefix">
+        <xacro:torso name="torso" prefix="${prefix}torso_"/>
+        <xacro:motoman_arm name="${prefix}arm_left" prefix="${prefix}arm_left_" parent="${prefix}torso_link_b1" reflect="1">
             <origin xyz="0.09996 0.0275 0.32214" rpy="1.57 0 0" />
         </xacro:motoman_arm>
-        <xacro:motoman_arm name="arm_right" prefix="arm_right_" parent="torso_link_b1" reflect="-1">
+        <xacro:motoman_arm name="${prefix}arm_right" prefix="${prefix}arm_right_" parent="${prefix}torso_link_b1" reflect="-1">
             <origin xyz="0.09996 -0.0275 0.32214" rpy="1.57 0 0" />
         </xacro:motoman_arm>
+     </xacro:macro>
+<!-- The following xacro is kept for backwards compatibility, it should not be used -->
+<!-- see: https://github.com/ros-industrial/motoman/issues/166 -->
+     <xacro:macro name="sda10f">
+          <xacro:motoman_sda10f prefix=""/>
+     </xacro:macro>
 </robot>
