Commit message: Some rotating directions fixed when testing with the real robot

File: motoman_sda10f_support/urdf/arm_macro.xacro (robot description, xacro)
@@ -121,5 +121,5 @@
 			<child link="${prefix}link_1"/>
 			<origin xyz="0.09996 ${reflect*0.0275} 0.32214" rpy="1.57 0 ${(reflect-1)*1.57}"/>
-			<axis xyz="0 0 -1" />
+			<axis xyz="0 0 ${-reflect}" />
 			<limit lower="-3.13" upper="3.13" effort="100" velocity="2.95" />
 		</joint>
@@ -135,5 +135,5 @@
 			<child link="${prefix}link_3"/>
 			<origin xyz="0 0.1690 -0.0454" rpy="1.57 0 0"/>
-			<axis xyz="0 0 1" />
+			<axis xyz="0 0 ${-reflect}" />
 			<limit lower="-2.95" upper="2.95" effort="100" velocity="2.95" />
 		</joint>
@@ -149,5 +149,5 @@
 			<child link="${prefix}link_5"/>
 			<origin xyz="0 0.1936 0.0155" rpy="1.57 0 0"/>
-			<axis xyz="0 0 1" />
+			<axis xyz="0 0 ${reflect}" />
 			<limit lower="-3.13" upper="3.13" effort="100" velocity="3.48" />
 		</joint>
@@ -163,5 +163,5 @@
 			<child link="${prefix}link_7"/>
 			<origin xyz="0 0.168 -0.015" rpy="1.57 0 0"/>
-			<axis xyz="0 0 1" />
+			<axis xyz="0 0 ${-reflect}" />
 			<limit lower="-3.13" upper="3.13" effort="100" velocity="6.97" />
 		</joint>

Commit message: Multiple changes on URDF

File: motoman_sda10f_support/urdf/arm_macro.xacro (robot description, xacro)
@@ -7,5 +7,5 @@
 				<origin rpy="0 0 0" xyz="0 0 0"/>
 				<geometry>
-					<mesh filename="package://motoman_sda10f_support/meshes/sda10f/visual/motoman_axis_r1_s.stl"/>
+					<mesh filename="package://motoman_sda10f_support/meshes/sda10f/visual/motoman_axis_s.stl"/>
 				</geometry>
 				<material name="blue">
@@ -16,5 +16,5 @@
 				<origin rpy="0 0 0" xyz="0 0 0"/>
 				<geometry>
-					<mesh filename="package://motoman_sda10f_support/meshes/sda10f/collision/motoman_axis_r1_s.stl" />
+					<mesh filename="package://motoman_sda10f_support/meshes/sda10f/collision/motoman_axis_s.stl" />
 				</geometry>
 				<material name="yellow"/>
@@ -25,5 +25,5 @@
 				<origin rpy="0 0 0" xyz="0 0 0"/>
 				<geometry>
-					<mesh filename="package://motoman_sda10f_support/meshes/sda10f/visual/motoman_axis_r1_l.stl"/>
+					<mesh filename="package://motoman_sda10f_support/meshes/sda10f/visual/motoman_axis_l.stl"/>
 				</geometry>
 				<material name="silver"/>
@@ -32,5 +32,5 @@
 				<origin rpy="0 0 0" xyz="0 0 0"/>
 				<geometry>
-					<mesh filename="package://motoman_sda10f_support/meshes/sda10f/collision/motoman_axis_r1_l.stl"/>
+					<mesh filename="package://motoman_sda10f_support/meshes/sda10f/collision/motoman_axis_l.stl"/>
 				</geometry>
 				<material name="yellow"/>
@@ -41,5 +41,5 @@
 				<origin rpy="0 0 0" xyz="0 0 0"/>
 				<geometry>
-					<mesh filename="package://motoman_sda10f_support/meshes/sda10f/visual/motoman_axis_r1_e.stl"/>
+					<mesh filename="package://motoman_sda10f_support/meshes/sda10f/visual/motoman_axis_e.stl"/>
 				</geometry>
 				<material name="blue"/>
@@ -48,5 +48,5 @@
 				<origin rpy="0 0 0" xyz="0 0 0"/>
 				<geometry>
-					<mesh filename="package://motoman_sda10f_support/meshes/sda10f/collision/motoman_axis_r1_e.stl"/>
+					<mesh filename="package://motoman_sda10f_support/meshes/sda10f/collision/motoman_axis_e.stl"/>
 				</geometry>
 				<material name="yellow"/>
@@ -57,5 +57,5 @@
 				<origin rpy="0 0 0" xyz="0 0 0"/>
 				<geometry>
-					<mesh filename="package://motoman_sda10f_support/meshes/sda10f/visual/motoman_axis_r1_u.stl"/>
+					<mesh filename="package://motoman_sda10f_support/meshes/sda10f/visual/motoman_axis_u.stl"/>
 				</geometry>
 				<material name="silver"/>
@@ -64,5 +64,5 @@
 				<origin rpy="0 0 0" xyz="0 0 0"/>
 				<geometry>
-					<mesh filename="package://motoman_sda10f_support/meshes/sda10f/collision/motoman_axis_r1_u.stl"/>
+					<mesh filename="package://motoman_sda10f_support/meshes/sda10f/collision/motoman_axis_u.stl"/>
 				</geometry>
 				<material name="yellow"/>
@@ -73,5 +73,5 @@
 				<origin rpy="0 0 0" xyz="0 0 0"/>
 				<geometry>
-					<mesh filename="package://motoman_sda10f_support/meshes/sda10f/visual/motoman_axis_r1_r.stl"/>
+					<mesh filename="package://motoman_sda10f_support/meshes/sda10f/visual/motoman_axis_r.stl"/>
 				</geometry>
 				<material name="blue"/>
@@ -80,5 +80,5 @@
 				<origin rpy="0 0 0" xyz="0 0 0"/>
 				<geometry>
-					<mesh filename="package://motoman_sda10f_support/meshes/sda10f/collision/motoman_axis_r1_r.stl"/>
+					<mesh filename="package://motoman_sda10f_support/meshes/sda10f/collision/motoman_axis_r.stl"/>
 				</geometry>
 				<material name="yellow"/>
@@ -89,5 +89,5 @@
 				<origin rpy="0 0 0" xyz="0 0 0"/>
 				<geometry>
-					<mesh filename="package://motoman_sda10f_support/meshes/sda10f/visual/motoman_axis_r1_b.stl"/>
+					<mesh filename="package://motoman_sda10f_support/meshes/sda10f/visual/motoman_axis_b.stl"/>
 				</geometry>
 				<material name="silver"/>
@@ -96,5 +96,5 @@
 				<origin rpy="0 0 0" xyz="0 0 0"/>
 				<geometry>
-					<mesh filename="package://motoman_sda10f_support/meshes/sda10f/collision/motoman_axis_r1_b.stl"/>
+					<mesh filename="package://motoman_sda10f_support/meshes/sda10f/collision/motoman_axis_b.stl"/>
 				</geometry>
 				<material name="yellow"/>
@@ -104,5 +104,5 @@
 			<visual>
 				<geometry>
-					<mesh filename="package://motoman_sda10f_support/meshes/sda10f/visual/motoman_axis_r1_t.stl" />
+					<mesh filename="package://motoman_sda10f_support/meshes/sda10f/visual/motoman_axis_t.stl" />
 				</geometry>
 				<material name="blue"/>
@@ -110,5 +110,5 @@
 			<collision>
 				<geometry>
-					<mesh filename="package://motoman_sda10f_support/meshes/sda10f/collision/motoman_axis_r1_t.stl" />
+					<mesh filename="package://motoman_sda10f_support/meshes/sda10f/collision/motoman_axis_t.stl" />
 				</geometry>
 				<material name="yellow"/>
@@ -122,5 +122,5 @@
 			<origin xyz="0.09996 ${reflect*0.0275} 0.32214" rpy="1.57 0 ${(reflect-1)*1.57}"/>
 			<axis xyz="0 0 ${-reflect}" />
-			<limit lower="-3.13" upper="3.13" effort="100" velocity="2.95" />
+			<limit lower="-3.13" upper="3.13" effort="0" velocity="2.95" />
 		</joint>
 		<joint name="${prefix}joint_2" type="revolute">
@@ -129,5 +129,5 @@
 			<origin xyz="0 0.0577 -0.2255" rpy="-1.57 0 0"/>
 			<axis xyz="0 0 ${-reflect}" />
-			<limit lower="-1.90" upper="1.90" effort="100" velocity="2.95" />
+			<limit lower="-1.90" upper="1.90" effort="0" velocity="2.95" />
 		</joint>
 		<joint name="${prefix}joint_3" type="revolute">
@@ -136,5 +136,5 @@
 			<origin xyz="0 0.1690 -0.0454" rpy="1.57 0 0"/>
 			<axis xyz="0 0 ${-reflect}" />
-			<limit lower="-2.95" upper="2.95" effort="100" velocity="2.95" />
+			<limit lower="-2.95" upper="2.95" effort="0" velocity="2.95" />
 		</joint>
 		<joint name="${prefix}joint_4" type="revolute">
@@ -143,5 +143,5 @@
 			<origin xyz="0 -0.0085 -0.181" rpy="-1.57 0 0"/>
 			<axis xyz="0 0 ${reflect}" />
-			<limit lower="-2.36" upper="2.36" effort="100" velocity="2.95" />
+			<limit lower="-2.36" upper="2.36" effort="0" velocity="2.95" />
 		</joint>
 		<joint name="${prefix}joint_5" type="revolute">
@@ -150,5 +150,5 @@
 			<origin xyz="0 0.1936 0.0155" rpy="1.57 0 0"/>
 			<axis xyz="0 0 ${reflect}" />
-			<limit lower="-3.13" upper="3.13" effort="100" velocity="3.48" />
+			<limit lower="-3.13" upper="3.13" effort="0" velocity="3.48" />
 		</joint>
 		<joint name="${prefix}joint_6" type="revolute">
@@ -157,5 +157,5 @@
 			<origin xyz="0 0.0080 -0.155" rpy="-1.57 0 0"/>
 			<axis xyz="0 0 ${reflect}" />
-			<limit lower="-1.90" upper="1.90" effort="100" velocity="3.48" />
+			<limit lower="-1.90" upper="1.90" effort="0" velocity="3.48" />
 		</joint>
 		<joint name="${prefix}joint_7" type="revolute">
@@ -164,5 +164,5 @@
 			<origin xyz="0 0.168 -0.015" rpy="1.57 0 0"/>
 			<axis xyz="0 0 ${-reflect}" />
-			<limit lower="-3.13" upper="3.13" effort="100" velocity="6.97" />
+			<limit lower="-3.13" upper="3.13" effort="0" velocity="6.97" />
 		</joint>
     <joint name="${prefix}joint_tool0" type="fixed" >

Commit message: Trying to get moveit running again

File: motoman_sda10f_support/urdf/arm_macro.xacro (robot description, xacro)
@@ -2,6 +2,5 @@
 <robot xmlns:xacro="http://ros.org/wiki/xacro">
 	<xacro:macro name="motoman_arm" params="name prefix parent *origin reflect">
-		<!-- R Group -->
-		<link name="${prefix}link_1">
+		<link name="${prefix}link_1_s">
 			<visual>
 				<origin rpy="0 0 0" xyz="0 0 0"/>
@@ -21,5 +20,5 @@
 			</collision>
 		</link>
-		<link name="${prefix}link_2">
+		<link name="${prefix}link_2_l">
 			<visual>
 				<origin rpy="0 0 0" xyz="0 0 0"/>
@@ -37,5 +36,5 @@
 			</collision>
 		</link>
-		<link name="${prefix}link_3">
+		<link name="${prefix}link_3_e">
 			<visual>
 				<origin rpy="0 0 0" xyz="0 0 0"/>
@@ -53,5 +52,5 @@
 			</collision>
 		</link>
-		<link name="${prefix}link_4">
+		<link name="${prefix}link_4_u">
 			<visual>
 				<origin rpy="0 0 0" xyz="0 0 0"/>
@@ -69,5 +68,5 @@
 			</collision>
 		</link>
-		<link name="${prefix}link_5">
+		<link name="${prefix}link_5_r">
 			<visual>
 				<origin rpy="0 0 0" xyz="0 0 0"/>
@@ -85,5 +84,5 @@
 			</collision>
 		</link>
-		<link name="${prefix}link_6">
+		<link name="${prefix}link_6_b">
 			<visual>
 				<origin rpy="0 0 0" xyz="0 0 0"/>
@@ -101,5 +100,5 @@
 			</collision>
 		</link>
-		<link name="${prefix}link_7">
+		<link name="${prefix}link_7_t">
 			<visual>
 				<geometry>
@@ -116,57 +115,56 @@
 		</link>
 	    <link name="${prefix}link_tool0" />
-		<!-- R -->
-		<joint name="${prefix}joint_1" type="revolute">
+		<joint name="${prefix}joint_1_s" type="revolute">
 			<parent link="torso_link_b1"/>
-			<child link="${prefix}link_1"/>
+			<child link="${prefix}link_1_s"/>
 			<origin xyz="0.09996 ${reflect*0.0275} 0.32214" rpy="1.57 0 ${(reflect-1)*1.57}"/>
 			<axis xyz="0 0 ${-reflect}" />
 			<limit lower="-3.13" upper="3.13" effort="0" velocity="2.95" />
 		</joint>
-		<joint name="${prefix}joint_2" type="revolute">
-			<parent link="${prefix}link_1"/>
-			<child link="${prefix}link_2"/>
+		<joint name="${prefix}joint_2_l" type="revolute">
+			<parent link="${prefix}link_1_s"/>
+			<child link="${prefix}link_2_l"/>
 			<origin xyz="0 0.0577 -0.2255" rpy="-1.57 0 0"/>
 			<axis xyz="0 0 ${-reflect}" />
 			<limit lower="-1.90" upper="1.90" effort="0" velocity="2.95" />
 		</joint>
-		<joint name="${prefix}joint_3" type="revolute">
-			<parent link="${prefix}link_2"/>
-			<child link="${prefix}link_3"/>
+		<joint name="${prefix}joint_3_e" type="revolute">
+			<parent link="${prefix}link_2_l"/>
+			<child link="${prefix}link_3_e"/>
 			<origin xyz="0 0.1690 -0.0454" rpy="1.57 0 0"/>
 			<axis xyz="0 0 ${-reflect}" />
 			<limit lower="-2.95" upper="2.95" effort="0" velocity="2.95" />
 		</joint>
-		<joint name="${prefix}joint_4" type="revolute">
-			<parent link="${prefix}link_3"/>
-			<child link="${prefix}link_4"/>
+		<joint name="${prefix}joint_4_u" type="revolute">
+			<parent link="${prefix}link_3_e"/>
+			<child link="${prefix}link_4_u"/>
 			<origin xyz="0 -0.0085 -0.181" rpy="-1.57 0 0"/>
 			<axis xyz="0 0 ${reflect}" />
 			<limit lower="-2.36" upper="2.36" effort="0" velocity="2.95" />
 		</joint>
-		<joint name="${prefix}joint_5" type="revolute">
-			<parent link="${prefix}link_4"/>
-			<child link="${prefix}link_5"/>
+		<joint name="${prefix}joint_5_r" type="revolute">
+			<parent link="${prefix}link_4_u"/>
+			<child link="${prefix}link_5_r"/>
 			<origin xyz="0 0.1936 0.0155" rpy="1.57 0 0"/>
 			<axis xyz="0 0 ${reflect}" />
 			<limit lower="-3.13" upper="3.13" effort="0" velocity="3.48" />
 		</joint>
-		<joint name="${prefix}joint_6" type="revolute">
-			<parent link="${prefix}link_5"/>
-			<child link="${prefix}link_6"/>
+		<joint name="${prefix}joint_6_b" type="revolute">
+			<parent link="${prefix}link_5_r"/>
+			<child link="${prefix}link_6_b"/>
 			<origin xyz="0 0.0080 -0.155" rpy="-1.57 0 0"/>
 			<axis xyz="0 0 ${reflect}" />
 			<limit lower="-1.90" upper="1.90" effort="0" velocity="3.48" />
 		</joint>
-		<joint name="${prefix}joint_7" type="revolute">
-			<parent link="${prefix}link_6"/>
-			<child link="${prefix}link_7"/>
+		<joint name="${prefix}joint_7_t" type="revolute">
+			<parent link="${prefix}link_6_b"/>
+			<child link="${prefix}link_7_t"/>
 			<origin xyz="0 0.168 -0.015" rpy="1.57 0 0"/>
 			<axis xyz="0 0 ${-reflect}" />
 			<limit lower="-3.13" upper="3.13" effort="0" velocity="6.97" />
 		</joint>
-    <joint name="${prefix}joint_tool0" type="fixed" >
+    <joint name="${prefix}joint_7_tool0" type="fixed" >
       <origin xyz="0 0 0.0" rpy="0 0 -3.13"/>
-      <parent link="${prefix}link_7" />
+      <parent link="${prefix}link_7_t" />
       <child link="${prefix}link_tool0" />
     </joint>

Commit message: Moveit config and everything working on the real hardware

File: motoman_sda10f_support/urdf/arm_macro.xacro (robot description, xacro)
@@ -164,5 +164,5 @@
 			<limit lower="-3.13" upper="3.13" effort="0" velocity="6.97" />
 		</joint>
-    <joint name="${prefix}joint_7_tool0" type="fixed" >
+    <joint name="${prefix}joint_tool0" type="fixed" >
       <origin xyz="0 0 0.0" rpy="0 0 -3.13"/>
       <parent link="${prefix}link_7_t" />

File: motoman_sda10f_support/urdf/common_torso_macro.xacro (robot description, xacro)
@@ -3,5 +3,5 @@
 	<xacro:macro name="torso" params="name prefix">
 		<!-- link list -->
-		<link name="${prefix}base_link">
+		<link name="base_link">
 			<visual>
 				<geometry>
@@ -21,5 +21,5 @@
 			</collision>
 		</link>
-		<link name="${prefix}torso_link_b1">
+		<link name="${prefix}link_b1">
 			<visual>
 				<origin rpy="0 0 0" xyz="0 0 0"/>
@@ -39,5 +39,5 @@
 			</collision>
 		</link>
-		<link name="${prefix}torso_link_b2">
+		<link name="${prefix}link_b2">
 			<visual>
 				<origin rpy="0 0 0" xyz="0 0 0"/>
@@ -58,18 +58,18 @@
 		</link>
 		<!-- joint list -->
-		<joint name="${prefix}torso_joint_b1" type="revolute">
-			<parent link="${prefix}base_link"/>
-			<child link="${prefix}torso_link_b1"/>
+		<joint name="${prefix}joint_b1" type="revolute">
+			<parent link="base_link"/>
+			<child link="${prefix}link_b1"/>
 			<origin xyz="0.09257 0 0.8835" rpy="0 0 0"/>
 			<axis xyz="0 0 1" />
 			<limit lower="-2.9570" upper="2.9570" effort="100" velocity="2.26" />
 		</joint>
-		<joint name="${prefix}torso_joint_b2" type="revolute">
-			<parent link="${prefix}base_link"/>
-			<child link="${prefix}torso_link_b2"/>
+		<joint name="${prefix}joint_b2" type="revolute">
+			<parent link="base_link"/>
+			<child link="${prefix}link_b2"/>
 			<origin xyz="0.09257 0 0.8835" rpy="0 0 0"/>
 			<axis xyz="0 0 1" />
 			<limit lower="-2.9570" upper="2.9570" effort="100" velocity="2.26" />
-			<mimic joint="${prefix}torso_joint_b1" multiplier="1" offset="0"/>
+			<mimic joint="${prefix}joint_b1" multiplier="1" offset="0"/>
 		</joint>
 		<!-- end of joint list -->

File: motoman_sda10f_support/urdf/sda10f_macro.xacro (robot description, xacro)
@@ -4,5 +4,5 @@
         <xacro:include filename="$(find motoman_sda10f_support)/urdf/common_torso_macro.xacro" />
         <xacro:include filename="$(find motoman_sda10f_support)/urdf/arm_macro.xacro" />
-        <xacro:torso name="torso" prefix=""/>
+        <xacro:torso name="torso" prefix="torso_"/>
         <xacro:motoman_arm name="arm_left" prefix="arm_left_" parent="torso_link_b1" reflect="1">
             <origin xyz="0.09996 0.0275 0.32214" rpy="1.57 0 0" />

Commit message: update URDF with official 3D CAD model dimensiones

File: motoman_sda10f_support/urdf/arm_macro.xacro (robot description, xacro)
@@ -118,5 +118,5 @@
 			<parent link="${parent}"/>
 			<child link="${prefix}link_1_s"/>
-			<origin xyz="0.09996 ${reflect*0.0275} 0.32214" rpy="1.57 0 ${(reflect-1)*1.57}"/>
+			<origin xyz="0.100 ${reflect*0.0275} 0.3114" rpy="1.57 0 ${(reflect-1)*1.57}"/>
 			<axis xyz="0 0 ${-reflect}" />
 			<limit lower="-3.13" upper="3.13" effort="0" velocity="2.95" />
@@ -125,5 +125,5 @@
 			<parent link="${prefix}link_1_s"/>
 			<child link="${prefix}link_2_l"/>
-			<origin xyz="0 0.0577 -0.2255" rpy="-1.57 0 0"/>
+			<origin xyz="0 0.0539 -0.2375" rpy="-1.57 0 0"/>
 			<axis xyz="0 0 ${-reflect}" />
 			<limit lower="-1.90" upper="1.90" effort="0" velocity="2.95" />
@@ -132,5 +132,5 @@
 			<parent link="${prefix}link_2_l"/>
 			<child link="${prefix}link_3_e"/>
-			<origin xyz="0 0.1690 -0.0454" rpy="1.57 0 0"/>
+			<origin xyz="0 0.211 -0.0539" rpy="1.57 0 0"/>
 			<axis xyz="0 0 ${-reflect}" />
 			<limit lower="-2.95" upper="2.95" effort="0" velocity="2.95" />
@@ -139,5 +139,5 @@
 			<parent link="${prefix}link_3_e"/>
 			<child link="${prefix}link_4_u"/>
-			<origin xyz="0 -0.0085 -0.181" rpy="-1.57 0 0"/>
+			<origin xyz="0 -0.0375 -0.149" rpy="-1.57 0 0"/>
 			<axis xyz="0 0 ${reflect}" />
 			<limit lower="-2.36" upper="2.36" effort="0" velocity="2.95" />
@@ -146,5 +146,5 @@
 			<parent link="${prefix}link_4_u"/>
 			<child link="${prefix}link_5_r"/>
-			<origin xyz="0 0.1936 0.0155" rpy="1.57 0 0"/>
+			<origin xyz="0 0.233 0.0375" rpy="1.57 0 0"/>
 			<axis xyz="0 0 ${reflect}" />
 			<limit lower="-3.13" upper="3.13" effort="0" velocity="3.48" />
@@ -153,5 +153,5 @@
 			<parent link="${prefix}link_5_r"/>
 			<child link="${prefix}link_6_b"/>
-			<origin xyz="0 0.0080 -0.155" rpy="-1.57 0 0"/>
+			<origin xyz="0 0.0335 -0.127" rpy="-1.57 0 0"/>
 			<axis xyz="0 0 ${reflect}" />
 			<limit lower="-1.90" upper="1.90" effort="0" velocity="3.48" />
@@ -160,5 +160,5 @@
 			<parent link="${prefix}link_6_b"/>
 			<child link="${prefix}link_7_t"/>
-			<origin xyz="0 0.168 -0.015" rpy="1.57 0 0"/>
+			<origin xyz="0 0.155 -0.0335" rpy="1.57 0 0"/>
 			<axis xyz="0 0 ${-reflect}" />
 			<limit lower="-3.13" upper="3.13" effort="0" velocity="6.97" />

File: motoman_sda10f_support/urdf/sda10f_macro.xacro (robot description, xacro)
@@ -5,9 +5,9 @@
      <xacro:macro name="motoman_sda10f" params="prefix">
         <xacro:torso name="${prefix}torso" prefix="${prefix}torso_"/>
-        <xacro:motoman_arm name="${prefix}arm_left" prefix="${prefix}arm_left_" parent="${prefix}torso_link_b1" reflect="1">
-            <origin xyz="0.09996 0.0275 0.32214" rpy="1.57 0 0" />
+        <xacro:motoman_arm name="${prefix}arm_left" prefix="${prefix}arm_left_" parent="${prefix}torso_link_b1" reflect="1" joint_limited="false">
+            <origin xyz="0.100 0.0275 0.3114" rpy="1.57 0 0" />
         </xacro:motoman_arm>
-        <xacro:motoman_arm name="${prefix}arm_right" prefix="${prefix}arm_right_" parent="${prefix}torso_link_b1" reflect="-1">
-            <origin xyz="0.09996 -0.0275 0.32214" rpy="1.57 0 0" />
+        <xacro:motoman_arm name="${prefix}arm_right" prefix="${prefix}arm_right_" parent="${prefix}torso_link_b1" reflect="-1" joint_limited="false">
+            <origin xyz="0.100 -0.0275 0.3114" rpy="1.57 0 0" />
         </xacro:motoman_arm>
      </xacro:macro>

Commit message: invert rotation sign of sda10f joint_7t

File: motoman_sda10f_support/urdf/arm_macro.xacro (robot description, xacro)
@@ -160,5 +160,5 @@
 			<parent link="${prefix}link_6_b"/>
 			<child link="${prefix}link_7_t"/>
-			<origin xyz="0 0.155 -0.0335" rpy="1.57 0 0"/>
+			<origin xyz="0 0.155 -0.0335" rpy="-1.57 0 0"/>
 			<axis xyz="0 0 ${-reflect}" />
 			<limit lower="-3.13" upper="3.13" effort="0" velocity="6.97" />
