Commit message: SDA10F Support Package Update
Restructured kinematic model to match standard Yaskawa model
Relocation position of mesh origin
Update of B and E axis models

File: motoman_sda10f_support/urdf/arm_macro.xacro (robot description, xacro)
@@ -118,54 +118,54 @@
 			<parent link="${parent}"/>
 			<child link="${prefix}link_1_s"/>
-			<origin xyz="0.09996 ${reflect*0.0275} 0.32214" rpy="1.57 0 ${(reflect-1)*1.57}"/>
+                        <origin xyz="0.100 ${reflect*0.265} 0.0" rpy="${radians(90)} 0.0 ${(reflect-1)*${radians(90)}}"/>
 			<axis xyz="0 0 ${-reflect}" />
-			<limit lower="-3.13" upper="3.13" effort="0" velocity="2.95" />
+			<limit lower="${radians(-180)}" upper="${radians(180)}" effort="0" velocity="${radians(170)}" />
 		</joint>
 		<joint name="${prefix}joint_2_l" type="revolute">
 			<parent link="${prefix}link_1_s"/>
 			<child link="${prefix}link_2_l"/>
-			<origin xyz="0 0.0577 -0.2255" rpy="-1.57 0 0"/>
+                        <origin xyz="0.0 0.0 0.0" rpy="${radians(-90)} 0.0 0.0"/>
 			<axis xyz="0 0 ${-reflect}" />
-			<limit lower="-1.90" upper="1.90" effort="0" velocity="2.95" />
+			<limit lower="${radians(-110)}" upper="${radians(110)}" effort="0" velocity="${radians(170)}" />
 		</joint>
 		<joint name="${prefix}joint_3_e" type="revolute">
 			<parent link="${prefix}link_2_l"/>
 			<child link="${prefix}link_3_e"/>
-			<origin xyz="0 0.1690 -0.0454" rpy="1.57 0 0"/>
+                        <origin xyz="0.0 0.360 0.0" rpy="${radians(90)} 0.0 0.0"/>
 			<axis xyz="0 0 ${-reflect}" />
-			<limit lower="-2.95" upper="2.95" effort="0" velocity="2.95" />
+			<limit lower="${radians(-170)}" upper="${radians(170)}" effort="0" velocity="${radians(170)}" />
 		</joint>
 		<joint name="${prefix}joint_4_u" type="revolute">
 			<parent link="${prefix}link_3_e"/>
 			<child link="${prefix}link_4_u"/>
-			<origin xyz="0 -0.0085 -0.181" rpy="-1.57 0 0"/>
+                        <origin xyz="0.0 0.0 0.0" rpy="${radians(-90)} 0.0 0.0"/>
 			<axis xyz="0 0 ${reflect}" />
-			<limit lower="-2.36" upper="2.36" effort="0" velocity="2.95" />
+			<limit lower="${radians(-135)}" upper="${radians(135)}" effort="0" velocity="${radians(170)}" />
 		</joint>
 		<joint name="${prefix}joint_5_r" type="revolute">
 			<parent link="${prefix}link_4_u"/>
 			<child link="${prefix}link_5_r"/>
-			<origin xyz="0 0.1936 0.0155" rpy="1.57 0 0"/>
+                        <origin xyz="0.0 0.360 0.0" rpy="${radians(90)} 0.0 0.0"/>
 			<axis xyz="0 0 ${reflect}" />
-			<limit lower="-3.13" upper="3.13" effort="0" velocity="3.48" />
+			<limit lower="${radians(-180)}" upper="${radians(180)}" effort="0" velocity="${radians(200)}" />
 		</joint>
 		<joint name="${prefix}joint_6_b" type="revolute">
 			<parent link="${prefix}link_5_r"/>
 			<child link="${prefix}link_6_b"/>
-			<origin xyz="0 0.0080 -0.155" rpy="-1.57 0 0"/>
+                        <origin xyz="0.0 0.0 0.0" rpy="${radians(-90)} 0.0 0.0"/>
 			<axis xyz="0 0 ${reflect}" />
-			<limit lower="-1.90" upper="1.90" effort="0" velocity="3.48" />
+			<limit lower="${radians(-110)}" upper="${radians(110)}" effort="0" velocity="${radians(200)}" />
 		</joint>
 		<joint name="${prefix}joint_7_t" type="revolute">
 			<parent link="${prefix}link_6_b"/>
 			<child link="${prefix}link_7_t"/>
-			<origin xyz="0 0.168 -0.015" rpy="1.57 0 0"/>
-			<axis xyz="0 0 ${-reflect}" />
-			<limit lower="-3.13" upper="3.13" effort="0" velocity="6.97" />
+                        <origin xyz="0.0 0.155 0.0" rpy="${radians(-90)} 0.0 0.0"/>
+                        <axis xyz="0 0 ${-reflect}" />
+			<limit lower="${radians(-180)}" upper="${radians(180)}" effort="0" velocity="${radians(400)}" />
 		</joint>
     <joint name="${prefix}joint_tool0" type="fixed" >
-      <origin xyz="0 0 0.0" rpy="0 0 -3.13"/>
       <parent link="${prefix}link_7_t" />
       <child link="${prefix}link_tool0" />
+      <origin xyz="0 0 0" rpy="0 0 0"/>
     </joint>
 		<!-- end of joint list -->

File: motoman_sda10f_support/urdf/common_torso_macro.xacro (robot description, xacro)
@@ -61,14 +61,14 @@
 			<parent link="${prefix}base_link"/>
 			<child link="${prefix}link_b1"/>
-			<origin xyz="0.09257 0 0.8835" rpy="0 0 0"/>
+                        <origin xyz="0 0 0" rpy="0 0 0"/>
 			<axis xyz="0 0 1" />
-			<limit lower="-2.9570" upper="2.9570" effort="100" velocity="2.26" />
+			<limit lower="${radians(-170)}" upper="${radians(170)}" effort="100" velocity="${radians(130)}" />
 		</joint>
 		<joint name="${prefix}joint_b2" type="revolute">
 			<parent link="${prefix}base_link"/>
 			<child link="${prefix}link_b2"/>
-			<origin xyz="0.09257 0 0.8835" rpy="0 0 0"/>
+                        <origin xyz="0 0 0" rpy="0 0 0"/>
 			<axis xyz="0 0 1" />
-			<limit lower="-2.9570" upper="2.9570" effort="100" velocity="2.26" />
+			<limit lower="${radians(-170)}" upper="${radians(170)}" effort="100" velocity="${radians(130)}" />
 			<mimic joint="${prefix}joint_b1" multiplier="1" offset="0"/>
 		</joint>

File: motoman_sda10f_support/urdf/sda10f_macro.xacro (robot description, xacro)
@@ -6,9 +6,18 @@
         <xacro:torso name="${prefix}torso" prefix="${prefix}torso_"/>
         <xacro:motoman_arm name="${prefix}arm_left" prefix="${prefix}arm_left_" parent="${prefix}torso_link_b1" reflect="1">
-            <origin xyz="0.09996 0.0275 0.32214" rpy="1.57 0 0" />
+            <origin xyz="0 0 0" rpy="0 0 0" />
         </xacro:motoman_arm>
         <xacro:motoman_arm name="${prefix}arm_right" prefix="${prefix}arm_right_" parent="${prefix}torso_link_b1" reflect="-1">
-            <origin xyz="0.09996 -0.0275 0.32214" rpy="1.57 0 0" />
+            <origin xyz="0 0 0" rpy="0 0 0" />
         </xacro:motoman_arm>
+        <!-- link list -->
+        <link name="${prefix}base_link">
+        </link>
+        <!-- joint list -->
+        <joint name="${prefix}base_link_torso" type="fixed">
+                <parent link="${prefix}base_link"/>
+                <child link="${prefix}torso_base_link"/>
+                <origin xyz="0 0 1.2" rpy="0 0 0"/>
+        </joint>
      </xacro:macro>
 <!-- The following xacro is kept for backwards compatibility, it should not be used -->

Commit message: SDA10F Support Package Update
Correction of error in arm-macro preventing build
Correction of tool0 orienation to match Yaskawa default orientation

File: motoman_sda10f_support/urdf/arm_macro.xacro (robot description, xacro)
@@ -118,5 +118,5 @@
 			<parent link="${parent}"/>
 			<child link="${prefix}link_1_s"/>
-                        <origin xyz="0.100 ${reflect*0.265} 0.0" rpy="${radians(90)} 0.0 ${(reflect-1)*${radians(90)}}"/>
+                        <origin xyz="0.100 ${reflect*0.265} 0.0" rpy="${radians(90)} 0.0 ${(reflect-1)*radians(90)}"/>
 			<axis xyz="0 0 ${-reflect}" />
 			<limit lower="${radians(-180)}" upper="${radians(180)}" effort="0" velocity="${radians(170)}" />
@@ -167,5 +167,5 @@
       <parent link="${prefix}link_7_t" />
       <child link="${prefix}link_tool0" />
-      <origin xyz="0 0 0" rpy="0 0 0"/>
+      <origin xyz="0 0 0" rpy="0 0 ${radians(180)}"/>
     </joint>
 		<!-- end of joint list -->

Commit message: Fix mesh filenames.
Don't repeat mfg prefix. There is no need.

File: motoman_sda10f_support/urdf/arm_macro.xacro (robot description, xacro)
@@ -6,5 +6,5 @@
 				<origin rpy="0 0 0" xyz="0 0 0"/>
 				<geometry>
-					<mesh filename="package://motoman_sda10f_support/meshes/sda10f/visual/motoman_axis_s.stl"/>
+					<mesh filename="package://motoman_sda10f_support/meshes/sda10f/visual/link_s.stl"/>
 				</geometry>
 				<material name="blue">
@@ -15,5 +15,5 @@
 				<origin rpy="0 0 0" xyz="0 0 0"/>
 				<geometry>
-					<mesh filename="package://motoman_sda10f_support/meshes/sda10f/collision/motoman_axis_s.stl" />
+					<mesh filename="package://motoman_sda10f_support/meshes/sda10f/collision/link_s.stl" />
 				</geometry>
 				<material name="yellow"/>
@@ -24,5 +24,5 @@
 				<origin rpy="0 0 0" xyz="0 0 0"/>
 				<geometry>
-					<mesh filename="package://motoman_sda10f_support/meshes/sda10f/visual/motoman_axis_l.stl"/>
+					<mesh filename="package://motoman_sda10f_support/meshes/sda10f/visual/link_l.stl"/>
 				</geometry>
 				<material name="silver"/>
@@ -31,5 +31,5 @@
 				<origin rpy="0 0 0" xyz="0 0 0"/>
 				<geometry>
-					<mesh filename="package://motoman_sda10f_support/meshes/sda10f/collision/motoman_axis_l.stl"/>
+					<mesh filename="package://motoman_sda10f_support/meshes/sda10f/collision/link_l.stl"/>
 				</geometry>
 				<material name="yellow"/>
@@ -40,5 +40,5 @@
 				<origin rpy="0 0 0" xyz="0 0 0"/>
 				<geometry>
-					<mesh filename="package://motoman_sda10f_support/meshes/sda10f/visual/motoman_axis_e.stl"/>
+					<mesh filename="package://motoman_sda10f_support/meshes/sda10f/visual/link_e.stl"/>
 				</geometry>
 				<material name="blue"/>
@@ -47,5 +47,5 @@
 				<origin rpy="0 0 0" xyz="0 0 0"/>
 				<geometry>
-					<mesh filename="package://motoman_sda10f_support/meshes/sda10f/collision/motoman_axis_e.stl"/>
+					<mesh filename="package://motoman_sda10f_support/meshes/sda10f/collision/link_e.stl"/>
 				</geometry>
 				<material name="yellow"/>
@@ -56,5 +56,5 @@
 				<origin rpy="0 0 0" xyz="0 0 0"/>
 				<geometry>
-					<mesh filename="package://motoman_sda10f_support/meshes/sda10f/visual/motoman_axis_u.stl"/>
+					<mesh filename="package://motoman_sda10f_support/meshes/sda10f/visual/link_u.stl"/>
 				</geometry>
 				<material name="silver"/>
@@ -63,5 +63,5 @@
 				<origin rpy="0 0 0" xyz="0 0 0"/>
 				<geometry>
-					<mesh filename="package://motoman_sda10f_support/meshes/sda10f/collision/motoman_axis_u.stl"/>
+					<mesh filename="package://motoman_sda10f_support/meshes/sda10f/collision/link_u.stl"/>
 				</geometry>
 				<material name="yellow"/>
@@ -72,5 +72,5 @@
 				<origin rpy="0 0 0" xyz="0 0 0"/>
 				<geometry>
-					<mesh filename="package://motoman_sda10f_support/meshes/sda10f/visual/motoman_axis_r.stl"/>
+					<mesh filename="package://motoman_sda10f_support/meshes/sda10f/visual/link_r.stl"/>
 				</geometry>
 				<material name="blue"/>
@@ -79,5 +79,5 @@
 				<origin rpy="0 0 0" xyz="0 0 0"/>
 				<geometry>
-					<mesh filename="package://motoman_sda10f_support/meshes/sda10f/collision/motoman_axis_r.stl"/>
+					<mesh filename="package://motoman_sda10f_support/meshes/sda10f/collision/link_r.stl"/>
 				</geometry>
 				<material name="yellow"/>
@@ -88,5 +88,5 @@
 				<origin rpy="0 0 0" xyz="0 0 0"/>
 				<geometry>
-					<mesh filename="package://motoman_sda10f_support/meshes/sda10f/visual/motoman_axis_b.stl"/>
+					<mesh filename="package://motoman_sda10f_support/meshes/sda10f/visual/link_b.stl"/>
 				</geometry>
 				<material name="silver"/>
@@ -95,5 +95,5 @@
 				<origin rpy="0 0 0" xyz="0 0 0"/>
 				<geometry>
-					<mesh filename="package://motoman_sda10f_support/meshes/sda10f/collision/motoman_axis_b.stl"/>
+					<mesh filename="package://motoman_sda10f_support/meshes/sda10f/collision/link_b.stl"/>
 				</geometry>
 				<material name="yellow"/>
@@ -103,5 +103,5 @@
 			<visual>
 				<geometry>
-					<mesh filename="package://motoman_sda10f_support/meshes/sda10f/visual/motoman_axis_t.stl" />
+					<mesh filename="package://motoman_sda10f_support/meshes/sda10f/visual/link_t.stl" />
 				</geometry>
 				<material name="blue"/>
@@ -109,5 +109,5 @@
 			<collision>
 				<geometry>
-					<mesh filename="package://motoman_sda10f_support/meshes/sda10f/collision/motoman_axis_t.stl" />
+					<mesh filename="package://motoman_sda10f_support/meshes/sda10f/collision/link_t.stl" />
 				</geometry>
 				<material name="yellow"/>

File: motoman_sda10f_support/urdf/common_torso_macro.xacro (robot description, xacro)
@@ -6,5 +6,5 @@
 			<visual>
 				<geometry>
-					<mesh filename="package://motoman_sda10f_support/meshes/sda10f/visual/motoman_base.stl" />
+					<mesh filename="package://motoman_sda10f_support/meshes/sda10f/visual/base.stl" />
 				</geometry>
 				<material name="blue">
@@ -14,5 +14,5 @@
 			<collision>
 				<geometry>
-					<mesh filename="package://motoman_sda10f_support/meshes/sda10f/collision/motoman_base.stl" />
+					<mesh filename="package://motoman_sda10f_support/meshes/sda10f/collision/base.stl" />
 				</geometry>
 				<material name="yellow">
@@ -25,5 +25,5 @@
 				<origin rpy="0 0 0" xyz="0 0 0"/>
 				<geometry>
-					<mesh filename="package://motoman_sda10f_support/meshes/sda10f/visual/motoman_axis_b1.stl"/>
+					<mesh filename="package://motoman_sda10f_support/meshes/sda10f/visual/link_b1.stl"/>
 				</geometry>
 				<material name="silver">
@@ -34,5 +34,5 @@
 				<origin rpy="0 0 0" xyz="0 0 0"/>
 				<geometry>
-					<mesh filename="package://motoman_sda10f_support/meshes/sda10f/collision/motoman_axis_b1.stl" />
+					<mesh filename="package://motoman_sda10f_support/meshes/sda10f/collision/link_b1.stl" />
 				</geometry>
 				<material name="yellow"/>
@@ -43,5 +43,5 @@
 				<origin rpy="0 0 0" xyz="0 0 0"/>
 				<geometry>
-					<mesh filename="package://motoman_sda10f_support/meshes/sda10f/visual/motoman_axis_b1.stl"/>
+					<mesh filename="package://motoman_sda10f_support/meshes/sda10f/visual/link_b1.stl"/>
 				</geometry>
 				<material name="silver">
@@ -52,5 +52,5 @@
 				<origin rpy="0 0 0" xyz="0 0 0"/>
 				<geometry>
-					<mesh filename="package://motoman_sda10f_support/meshes/sda10f/collision/motoman_axis_b1.stl" />
+					<mesh filename="package://motoman_sda10f_support/meshes/sda10f/collision/link_b1.stl" />
 				</geometry>
 				<material name="yellow"/>
