Commit message: Cleanup formatting and layout of xacros.

File: motoman_sda10f_support/urdf/arm_macro.xacro (robot description, xacro)
@@ -1,167 +1,167 @@
 <?xml version="1.0" ?>
 <robot xmlns:xacro="http://ros.org/wiki/xacro">
-	<xacro:macro name="motoman_arm" params="name prefix parent *origin reflect">
-		<link name="${prefix}link_1_s">
-			<visual>
-				<origin rpy="0 0 0" xyz="0 0 0"/>
-				<geometry>
-					<mesh filename="package://motoman_sda10f_support/meshes/sda10f/visual/link_s.stl"/>
-				</geometry>
-				<material name="blue">
-					<color rgba="0.8 0.8 0.8 1"/>
-				</material>
-			</visual>
-			<collision>
-				<origin rpy="0 0 0" xyz="0 0 0"/>
-				<geometry>
-					<mesh filename="package://motoman_sda10f_support/meshes/sda10f/collision/link_s.stl" />
-				</geometry>
-				<material name="yellow"/>
-			</collision>
-		</link>
-		<link name="${prefix}link_2_l">
-			<visual>
-				<origin rpy="0 0 0" xyz="0 0 0"/>
-				<geometry>
-					<mesh filename="package://motoman_sda10f_support/meshes/sda10f/visual/link_l.stl"/>
-				</geometry>
-				<material name="silver"/>
-			</visual>
-			<collision>
-				<origin rpy="0 0 0" xyz="0 0 0"/>
-				<geometry>
-					<mesh filename="package://motoman_sda10f_support/meshes/sda10f/collision/link_l.stl"/>
-				</geometry>
-				<material name="yellow"/>
-			</collision>
-		</link>
-		<link name="${prefix}link_3_e">
-			<visual>
-				<origin rpy="0 0 0" xyz="0 0 0"/>
-				<geometry>
-					<mesh filename="package://motoman_sda10f_support/meshes/sda10f/visual/link_e.stl"/>
-				</geometry>
-				<material name="blue"/>
-			</visual>
-			<collision>
-				<origin rpy="0 0 0" xyz="0 0 0"/>
-				<geometry>
-					<mesh filename="package://motoman_sda10f_support/meshes/sda10f/collision/link_e.stl"/>
-				</geometry>
-				<material name="yellow"/>
-			</collision>
-		</link>
-		<link name="${prefix}link_4_u">
-			<visual>
-				<origin rpy="0 0 0" xyz="0 0 0"/>
-				<geometry>
-					<mesh filename="package://motoman_sda10f_support/meshes/sda10f/visual/link_u.stl"/>
-				</geometry>
-				<material name="silver"/>
-			</visual>
-			<collision>
-				<origin rpy="0 0 0" xyz="0 0 0"/>
-				<geometry>
-					<mesh filename="package://motoman_sda10f_support/meshes/sda10f/collision/link_u.stl"/>
-				</geometry>
-				<material name="yellow"/>
-			</collision>
-		</link>
-		<link name="${prefix}link_5_r">
-			<visual>
-				<origin rpy="0 0 0" xyz="0 0 0"/>
-				<geometry>
-					<mesh filename="package://motoman_sda10f_support/meshes/sda10f/visual/link_r.stl"/>
-				</geometry>
-				<material name="blue"/>
-			</visual>
-			<collision>
-				<origin rpy="0 0 0" xyz="0 0 0"/>
-				<geometry>
-					<mesh filename="package://motoman_sda10f_support/meshes/sda10f/collision/link_r.stl"/>
-				</geometry>
-				<material name="yellow"/>
-			</collision>
-		</link>
-		<link name="${prefix}link_6_b">
-			<visual>
-				<origin rpy="0 0 0" xyz="0 0 0"/>
-				<geometry>
-					<mesh filename="package://motoman_sda10f_support/meshes/sda10f/visual/link_b.stl"/>
-				</geometry>
-				<material name="silver"/>
-			</visual>
-			<collision>
-				<origin rpy="0 0 0" xyz="0 0 0"/>
-				<geometry>
-					<mesh filename="package://motoman_sda10f_support/meshes/sda10f/collision/link_b.stl"/>
-				</geometry>
-				<material name="yellow"/>
-			</collision>
-		</link>
-		<link name="${prefix}link_7_t">
-			<visual>
-				<geometry>
-					<mesh filename="package://motoman_sda10f_support/meshes/sda10f/visual/link_t.stl" />
-				</geometry>
-				<material name="blue"/>
-			</visual>
-			<collision>
-				<geometry>
-					<mesh filename="package://motoman_sda10f_support/meshes/sda10f/collision/link_t.stl" />
-				</geometry>
-				<material name="yellow"/>
-			</collision>
-		</link>
-	    <link name="${prefix}link_tool0" />
-		<joint name="${prefix}joint_1_s" type="revolute">
-			<parent link="${parent}"/>
-			<child link="${prefix}link_1_s"/>
-                        <origin xyz="0.100 ${reflect*0.265} 0.0" rpy="${radians(90)} 0.0 ${(reflect-1)*radians(90)}"/>
-			<axis xyz="0 0 ${-reflect}" />
-			<limit lower="${radians(-180)}" upper="${radians(180)}" effort="0" velocity="${radians(170)}" />
-		</joint>
-		<joint name="${prefix}joint_2_l" type="revolute">
-			<parent link="${prefix}link_1_s"/>
-			<child link="${prefix}link_2_l"/>
-                        <origin xyz="0.0 0.0 0.0" rpy="${radians(-90)} 0.0 0.0"/>
-			<axis xyz="0 0 ${-reflect}" />
-			<limit lower="${radians(-110)}" upper="${radians(110)}" effort="0" velocity="${radians(170)}" />
-		</joint>
-		<joint name="${prefix}joint_3_e" type="revolute">
-			<parent link="${prefix}link_2_l"/>
-			<child link="${prefix}link_3_e"/>
-                        <origin xyz="0.0 0.360 0.0" rpy="${radians(90)} 0.0 0.0"/>
-			<axis xyz="0 0 ${-reflect}" />
-			<limit lower="${radians(-170)}" upper="${radians(170)}" effort="0" velocity="${radians(170)}" />
-		</joint>
-		<joint name="${prefix}joint_4_u" type="revolute">
-			<parent link="${prefix}link_3_e"/>
-			<child link="${prefix}link_4_u"/>
-                        <origin xyz="0.0 0.0 0.0" rpy="${radians(-90)} 0.0 0.0"/>
-			<axis xyz="0 0 ${reflect}" />
-			<limit lower="${radians(-135)}" upper="${radians(135)}" effort="0" velocity="${radians(170)}" />
-		</joint>
-		<joint name="${prefix}joint_5_r" type="revolute">
-			<parent link="${prefix}link_4_u"/>
-			<child link="${prefix}link_5_r"/>
-                        <origin xyz="0.0 0.360 0.0" rpy="${radians(90)} 0.0 0.0"/>
-			<axis xyz="0 0 ${reflect}" />
-			<limit lower="${radians(-180)}" upper="${radians(180)}" effort="0" velocity="${radians(200)}" />
-		</joint>
-		<joint name="${prefix}joint_6_b" type="revolute">
-			<parent link="${prefix}link_5_r"/>
-			<child link="${prefix}link_6_b"/>
-                        <origin xyz="0.0 0.0 0.0" rpy="${radians(-90)} 0.0 0.0"/>
-			<axis xyz="0 0 ${reflect}" />
-			<limit lower="${radians(-110)}" upper="${radians(110)}" effort="0" velocity="${radians(200)}" />
-		</joint>
-		<joint name="${prefix}joint_7_t" type="revolute">
-			<parent link="${prefix}link_6_b"/>
-			<child link="${prefix}link_7_t"/>
-                        <origin xyz="0.0 0.155 0.0" rpy="${radians(-90)} 0.0 0.0"/>
-                        <axis xyz="0 0 ${-reflect}" />
-			<limit lower="${radians(-180)}" upper="${radians(180)}" effort="0" velocity="${radians(400)}" />
-		</joint>
+  <xacro:macro name="motoman_arm" params="name prefix parent *origin reflect">
+    <link name="${prefix}link_1_s">
+      <visual>
+        <origin rpy="0 0 0" xyz="0 0 0"/>
+        <geometry>
+          <mesh filename="package://motoman_sda10f_support/meshes/sda10f/visual/link_s.stl"/>
+        </geometry>
+        <material name="blue">
+          <color rgba="0.8 0.8 0.8 1"/>
+        </material>
+      </visual>
+      <collision>
+        <origin rpy="0 0 0" xyz="0 0 0"/>
+        <geometry>
+          <mesh filename="package://motoman_sda10f_support/meshes/sda10f/collision/link_s.stl" />
+        </geometry>
+        <material name="yellow"/>
+      </collision>
+    </link>
+    <link name="${prefix}link_2_l">
+      <visual>
+        <origin rpy="0 0 0" xyz="0 0 0"/>
+        <geometry>
+          <mesh filename="package://motoman_sda10f_support/meshes/sda10f/visual/link_l.stl"/>
+        </geometry>
+        <material name="silver"/>
+      </visual>
+      <collision>
+        <origin rpy="0 0 0" xyz="0 0 0"/>
+        <geometry>
+          <mesh filename="package://motoman_sda10f_support/meshes/sda10f/collision/link_l.stl"/>
+        </geometry>
+        <material name="yellow"/>
+      </collision>
+    </link>
+    <link name="${prefix}link_3_e">
+      <visual>
+        <origin rpy="0 0 0" xyz="0 0 0"/>
+        <geometry>
+          <mesh filename="package://motoman_sda10f_support/meshes/sda10f/visual/link_e.stl"/>
+        </geometry>
+        <material name="blue"/>
+      </visual>
+      <collision>
+        <origin rpy="0 0 0" xyz="0 0 0"/>
+        <geometry>
+          <mesh filename="package://motoman_sda10f_support/meshes/sda10f/collision/link_e.stl"/>
+        </geometry>
+        <material name="yellow"/>
+      </collision>
+    </link>
+    <link name="${prefix}link_4_u">
+      <visual>
+        <origin rpy="0 0 0" xyz="0 0 0"/>
+        <geometry>
+          <mesh filename="package://motoman_sda10f_support/meshes/sda10f/visual/link_u.stl"/>
+        </geometry>
+        <material name="silver"/>
+      </visual>
+      <collision>
+        <origin rpy="0 0 0" xyz="0 0 0"/>
+        <geometry>
+          <mesh filename="package://motoman_sda10f_support/meshes/sda10f/collision/link_u.stl"/>
+        </geometry>
+        <material name="yellow"/>
+      </collision>
+    </link>
+    <link name="${prefix}link_5_r">
+      <visual>
+        <origin rpy="0 0 0" xyz="0 0 0"/>
+        <geometry>
+          <mesh filename="package://motoman_sda10f_support/meshes/sda10f/visual/link_r.stl"/>
+        </geometry>
+        <material name="blue"/>
+      </visual>
+      <collision>
+        <origin rpy="0 0 0" xyz="0 0 0"/>
+        <geometry>
+          <mesh filename="package://motoman_sda10f_support/meshes/sda10f/collision/link_r.stl"/>
+        </geometry>
+        <material name="yellow"/>
+      </collision>
+    </link>
+    <link name="${prefix}link_6_b">
+      <visual>
+        <origin rpy="0 0 0" xyz="0 0 0"/>
+        <geometry>
+          <mesh filename="package://motoman_sda10f_support/meshes/sda10f/visual/link_b.stl"/>
+        </geometry>
+        <material name="silver"/>
+      </visual>
+      <collision>
+        <origin rpy="0 0 0" xyz="0 0 0"/>
+        <geometry>
+          <mesh filename="package://motoman_sda10f_support/meshes/sda10f/collision/link_b.stl"/>
+        </geometry>
+        <material name="yellow"/>
+      </collision>
+    </link>
+    <link name="${prefix}link_7_t">
+      <visual>
+        <geometry>
+          <mesh filename="package://motoman_sda10f_support/meshes/sda10f/visual/link_t.stl" />
+        </geometry>
+        <material name="blue"/>
+      </visual>
+      <collision>
+        <geometry>
+          <mesh filename="package://motoman_sda10f_support/meshes/sda10f/collision/link_t.stl" />
+        </geometry>
+        <material name="yellow"/>
+      </collision>
+    </link>
+    <link name="${prefix}link_tool0" />
+    <joint name="${prefix}joint_1_s" type="revolute">
+      <parent link="${parent}"/>
+      <child link="${prefix}link_1_s"/>
+      <origin xyz="0.100 ${reflect*0.265} 0.0" rpy="${radians(90)} 0.0 ${(reflect-1)*radians(90)}"/>
+      <axis xyz="0 0 ${-reflect}" />
+      <limit lower="${radians(-180)}" upper="${radians(180)}" effort="0" velocity="${radians(170)}" />
+    </joint>
+    <joint name="${prefix}joint_2_l" type="revolute">
+      <parent link="${prefix}link_1_s"/>
+      <child link="${prefix}link_2_l"/>
+      <origin xyz="0.0 0.0 0.0" rpy="${radians(-90)} 0.0 0.0"/>
+      <axis xyz="0 0 ${-reflect}" />
+      <limit lower="${radians(-110)}" upper="${radians(110)}" effort="0" velocity="${radians(170)}" />
+    </joint>
+    <joint name="${prefix}joint_3_e" type="revolute">
+      <parent link="${prefix}link_2_l"/>
+      <child link="${prefix}link_3_e"/>
+      <origin xyz="0.0 0.360 0.0" rpy="${radians(90)} 0.0 0.0"/>
+      <axis xyz="0 0 ${-reflect}" />
+      <limit lower="${radians(-170)}" upper="${radians(170)}" effort="0" velocity="${radians(170)}" />
+    </joint>
+    <joint name="${prefix}joint_4_u" type="revolute">
+      <parent link="${prefix}link_3_e"/>
+      <child link="${prefix}link_4_u"/>
+      <origin xyz="0.0 0.0 0.0" rpy="${radians(-90)} 0.0 0.0"/>
+      <axis xyz="0 0 ${reflect}" />
+      <limit lower="${radians(-135)}" upper="${radians(135)}" effort="0" velocity="${radians(170)}" />
+    </joint>
+    <joint name="${prefix}joint_5_r" type="revolute">
+      <parent link="${prefix}link_4_u"/>
+      <child link="${prefix}link_5_r"/>
+      <origin xyz="0.0 0.360 0.0" rpy="${radians(90)} 0.0 0.0"/>
+      <axis xyz="0 0 ${reflect}" />
+      <limit lower="${radians(-180)}" upper="${radians(180)}" effort="0" velocity="${radians(200)}" />
+    </joint>
+    <joint name="${prefix}joint_6_b" type="revolute">
+      <parent link="${prefix}link_5_r"/>
+      <child link="${prefix}link_6_b"/>
+      <origin xyz="0.0 0.0 0.0" rpy="${radians(-90)} 0.0 0.0"/>
+      <axis xyz="0 0 ${reflect}" />
+      <limit lower="${radians(-110)}" upper="${radians(110)}" effort="0" velocity="${radians(200)}" />
+    </joint>
+    <joint name="${prefix}joint_7_t" type="revolute">
+      <parent link="${prefix}link_6_b"/>
+      <child link="${prefix}link_7_t"/>
+      <origin xyz="0.0 0.155 0.0" rpy="${radians(-90)} 0.0 0.0"/>
+      <axis xyz="0 0 ${-reflect}" />
+      <limit lower="${radians(-180)}" upper="${radians(180)}" effort="0" velocity="${radians(400)}" />
+    </joint>
     <joint name="${prefix}joint_tool0" type="fixed" >
       <parent link="${prefix}link_7_t" />
@@ -169,5 +169,5 @@
       <origin xyz="0 0 0" rpy="0 0 ${radians(180)}"/>
     </joint>
-		<!-- end of joint list -->
-	</xacro:macro>
+    <!-- end of joint list -->
+  </xacro:macro>
 </robot>

File: motoman_sda10f_support/urdf/common_torso_macro.xacro (robot description, xacro)
@@ -1,77 +1,77 @@
 <?xml version="1.0" ?>
 <robot xmlns:xacro="http://ros.org/wiki/xacro">
-	<xacro:macro name="torso" params="name prefix">
-		<!-- link list -->
-		<link name="${prefix}base_link">
-			<visual>
-				<geometry>
-					<mesh filename="package://motoman_sda10f_support/meshes/sda10f/visual/base.stl" />
-				</geometry>
-				<material name="blue">
-					<color rgba="0 0 1 1"/>
-				</material>
-			</visual>
-			<collision>
-				<geometry>
-					<mesh filename="package://motoman_sda10f_support/meshes/sda10f/collision/base.stl" />
-				</geometry>
-				<material name="yellow">
-					<color rgba="0 1 1 1"/>
-				</material>
-			</collision>
-		</link>
-		<link name="${prefix}link_b1">
-			<visual>
-				<origin rpy="0 0 0" xyz="0 0 0"/>
-				<geometry>
-					<mesh filename="package://motoman_sda10f_support/meshes/sda10f/visual/link_b1.stl"/>
-				</geometry>
-				<material name="silver">
-					<color rgba="0.8 0.8 0.8 1"/>
-				</material>
-			</visual>
-			<collision>
-				<origin rpy="0 0 0" xyz="0 0 0"/>
-				<geometry>
-					<mesh filename="package://motoman_sda10f_support/meshes/sda10f/collision/link_b1.stl" />
-				</geometry>
-				<material name="yellow"/>
-			</collision>
-		</link>
-		<link name="${prefix}link_b2">
-			<visual>
-				<origin rpy="0 0 0" xyz="0 0 0"/>
-				<geometry>
-					<mesh filename="package://motoman_sda10f_support/meshes/sda10f/visual/link_b1.stl"/>
-				</geometry>
-				<material name="silver">
-					<color rgba="0.8 0.8 0.8 1"/>
-				</material>
-			</visual>
-			<collision>
-				<origin rpy="0 0 0" xyz="0 0 0"/>
-				<geometry>
-					<mesh filename="package://motoman_sda10f_support/meshes/sda10f/collision/link_b1.stl" />
-				</geometry>
-				<material name="yellow"/>
-			</collision>
-		</link>
-		<!-- joint list -->
-		<joint name="${prefix}joint_b1" type="revolute">
-			<parent link="${prefix}base_link"/>
-			<child link="${prefix}link_b1"/>
-                        <origin xyz="0 0 0" rpy="0 0 0"/>
-			<axis xyz="0 0 1" />
-			<limit lower="${radians(-170)}" upper="${radians(170)}" effort="100" velocity="${radians(130)}" />
-		</joint>
-		<joint name="${prefix}joint_b2" type="revolute">
-			<parent link="${prefix}base_link"/>
-			<child link="${prefix}link_b2"/>
-                        <origin xyz="0 0 0" rpy="0 0 0"/>
-			<axis xyz="0 0 1" />
-			<limit lower="${radians(-170)}" upper="${radians(170)}" effort="100" velocity="${radians(130)}" />
-			<mimic joint="${prefix}joint_b1" multiplier="1" offset="0"/>
-		</joint>
-		<!-- end of joint list -->
-	</xacro:macro>
+  <xacro:macro name="torso" params="name prefix">
+    <!-- link list -->
+    <link name="${prefix}base_link">
+      <visual>
+        <geometry>
+          <mesh filename="package://motoman_sda10f_support/meshes/sda10f/visual/base.stl" />
+        </geometry>
+        <material name="blue">
+          <color rgba="0 0 1 1"/>
+        </material>
+      </visual>
+      <collision>
+        <geometry>
+          <mesh filename="package://motoman_sda10f_support/meshes/sda10f/collision/base.stl" />
+        </geometry>
+        <material name="yellow">
+          <color rgba="0 1 1 1"/>
+        </material>
+      </collision>
+    </link>
+    <link name="${prefix}link_b1">
+      <visual>
+        <origin rpy="0 0 0" xyz="0 0 0"/>
+        <geometry>
+          <mesh filename="package://motoman_sda10f_support/meshes/sda10f/visual/link_b1.stl"/>
+        </geometry>
+        <material name="silver">
+          <color rgba="0.8 0.8 0.8 1"/>
+        </material>
+      </visual>
+      <collision>
+        <origin rpy="0 0 0" xyz="0 0 0"/>
+        <geometry>
+          <mesh filename="package://motoman_sda10f_support/meshes/sda10f/collision/link_b1.stl" />
+        </geometry>
+        <material name="yellow"/>
+      </collision>
+    </link>
+    <link name="${prefix}link_b2">
+      <visual>
+        <origin rpy="0 0 0" xyz="0 0 0"/>
+        <geometry>
+          <mesh filename="package://motoman_sda10f_support/meshes/sda10f/visual/link_b1.stl"/>
+        </geometry>
+        <material name="silver">
+          <color rgba="0.8 0.8 0.8 1"/>
+        </material>
+      </visual>
+      <collision>
+        <origin rpy="0 0 0" xyz="0 0 0"/>
+        <geometry>
+          <mesh filename="package://motoman_sda10f_support/meshes/sda10f/collision/link_b1.stl" />
+        </geometry>
+        <material name="yellow"/>
+      </collision>
+    </link>
+    <!-- joint list -->
+    <joint name="${prefix}joint_b1" type="revolute">
+      <parent link="${prefix}base_link"/>
+      <child link="${prefix}link_b1"/>
+      <origin xyz="0 0 0" rpy="0 0 0"/>
+      <axis xyz="0 0 1" />
+      <limit lower="${radians(-170)}" upper="${radians(170)}" effort="100" velocity="${radians(130)}" />
+    </joint>
+    <joint name="${prefix}joint_b2" type="revolute">
+      <parent link="${prefix}base_link"/>
+      <child link="${prefix}link_b2"/>
+      <origin xyz="0 0 0" rpy="0 0 0"/>
+      <axis xyz="0 0 1" />
+      <limit lower="${radians(-170)}" upper="${radians(170)}" effort="100" velocity="${radians(130)}" />
+      <mimic joint="${prefix}joint_b1" multiplier="1" offset="0"/>
+    </joint>
+    <!-- end of joint list -->
+  </xacro:macro>
 </robot>

File: motoman_sda10f_support/urdf/sda10f_macro.xacro (robot description, xacro)
@@ -1,28 +1,27 @@
 <?xml version="1.0" ?>
 <robot xmlns:xacro="http://ros.org/wiki/xacro">
-     <xacro:include filename="$(find motoman_sda10f_support)/urdf/common_torso_macro.xacro" />
-     <xacro:include filename="$(find motoman_sda10f_support)/urdf/arm_macro.xacro" />
-     <xacro:macro name="motoman_sda10f" params="prefix">
-        <xacro:torso name="${prefix}torso" prefix="${prefix}torso_"/>
-        <xacro:motoman_arm name="${prefix}arm_left" prefix="${prefix}arm_left_" parent="${prefix}torso_link_b1" reflect="1">
-            <origin xyz="0 0 0" rpy="0 0 0" />
-        </xacro:motoman_arm>
-        <xacro:motoman_arm name="${prefix}arm_right" prefix="${prefix}arm_right_" parent="${prefix}torso_link_b1" reflect="-1">
-            <origin xyz="0 0 0" rpy="0 0 0" />
-        </xacro:motoman_arm>
-        <!-- link list -->
-        <link name="${prefix}base_link">
-        </link>
-        <!-- joint list -->
-        <joint name="${prefix}base_link_torso" type="fixed">
-                <parent link="${prefix}base_link"/>
-                <child link="${prefix}torso_base_link"/>
-                <origin xyz="0 0 1.2" rpy="0 0 0"/>
-        </joint>
-     </xacro:macro>
-<!-- The following xacro is kept for backwards compatibility, it should not be used -->
-<!-- see: https://github.com/ros-industrial/motoman/issues/166 -->
-     <xacro:macro name="sda10f">
-          <xacro:motoman_sda10f prefix=""/>
-     </xacro:macro>
+  <xacro:include filename="$(find motoman_sda10f_support)/urdf/common_torso_macro.xacro" />
+  <xacro:include filename="$(find motoman_sda10f_support)/urdf/arm_macro.xacro" />
+  <xacro:macro name="motoman_sda10f" params="prefix">
+    <xacro:torso name="${prefix}torso" prefix="${prefix}torso_"/>
+    <xacro:motoman_arm name="${prefix}arm_left" prefix="${prefix}arm_left_" parent="${prefix}torso_link_b1" reflect="1">
+      <origin xyz="0 0 0" rpy="0 0 0" />
+    </xacro:motoman_arm>
+    <xacro:motoman_arm name="${prefix}arm_right" prefix="${prefix}arm_right_" parent="${prefix}torso_link_b1" reflect="-1">
+      <origin xyz="0 0 0" rpy="0 0 0" />
+    </xacro:motoman_arm>
+    <!-- link list -->
+    <link name="${prefix}base_link" />
+    <!-- joint list -->
+    <joint name="${prefix}base_link_torso" type="fixed">
+      <parent link="${prefix}base_link"/>
+      <child link="${prefix}torso_base_link"/>
+      <origin xyz="0 0 1.2" rpy="0 0 0"/>
+    </joint>
+  </xacro:macro>
+  <!-- The following xacro is kept for backwards compatibility, it should not be used -->
+  <!-- see: https://github.com/ros-industrial/motoman/issues/166 -->
+  <xacro:macro name="sda10f">
+    <xacro:motoman_sda10f prefix=""/>
+  </xacro:macro>
 </robot>
