Commit message: Collision geometry takes its colour from visual geometry.
The 'yellow' colour is never used.

Nor does it make sense.

File: motoman_sda10f_support/urdf/arm_macro.xacro (robot description, xacro)
@@ -17,5 +17,4 @@
           <mesh filename="package://motoman_sda10f_support/meshes/sda10f/collision/link_s.stl" />
         </geometry>
-        <material name="yellow"/>
       </collision>
     </link>
@@ -33,5 +32,4 @@
           <mesh filename="package://motoman_sda10f_support/meshes/sda10f/collision/link_l.stl"/>
         </geometry>
-        <material name="yellow"/>
       </collision>
     </link>
@@ -49,5 +47,4 @@
           <mesh filename="package://motoman_sda10f_support/meshes/sda10f/collision/link_e.stl"/>
         </geometry>
-        <material name="yellow"/>
       </collision>
     </link>
@@ -65,5 +62,4 @@
           <mesh filename="package://motoman_sda10f_support/meshes/sda10f/collision/link_u.stl"/>
         </geometry>
-        <material name="yellow"/>
       </collision>
     </link>
@@ -81,5 +77,4 @@
           <mesh filename="package://motoman_sda10f_support/meshes/sda10f/collision/link_r.stl"/>
         </geometry>
-        <material name="yellow"/>
       </collision>
     </link>
@@ -97,5 +92,4 @@
           <mesh filename="package://motoman_sda10f_support/meshes/sda10f/collision/link_b.stl"/>
         </geometry>
-        <material name="yellow"/>
       </collision>
     </link>
@@ -111,5 +105,4 @@
           <mesh filename="package://motoman_sda10f_support/meshes/sda10f/collision/link_t.stl" />
         </geometry>
-        <material name="yellow"/>
       </collision>
     </link>

File: motoman_sda10f_support/urdf/common_torso_macro.xacro (robot description, xacro)
@@ -16,7 +16,4 @@
           <mesh filename="package://motoman_sda10f_support/meshes/sda10f/collision/base.stl" />
         </geometry>
-        <material name="yellow">
-          <color rgba="0 1 1 1"/>
-        </material>
       </collision>
     </link>
@@ -36,5 +33,4 @@
           <mesh filename="package://motoman_sda10f_support/meshes/sda10f/collision/link_b1.stl" />
         </geometry>
-        <material name="yellow"/>
       </collision>
     </link>
@@ -54,5 +50,4 @@
           <mesh filename="package://motoman_sda10f_support/meshes/sda10f/collision/link_b1.stl" />
         </geometry>
-        <material name="yellow"/>
       </collision>
     </link>
