Commit message: Replaced tabs with spaces in sda10f_test.xacro file

File: motoman_sda10f_support/test/sda10f_test.xacro (robot description, xacro)
@@ -1,10 +1,10 @@
 <?xml version="1.0" ?>
 <robot name="motoman_sda10f_test" xmlns:xacro="http://ros.org/wiki/xacro">
-	<xacro:include filename="$(find motoman_sda10f_support)/urdf/sda10f_macro.xacro" />
-	<xacro:motoman_sda10f prefix=""/>
-	<!-- xacro below should not be used, use form above-->
-	<!--xacro:sda10f/-->
-	<xacro:motoman_sda10f prefix="my_prefix_"/>
-	<joint name="base_link_joint" type="fixed" >
+  <xacro:include filename="$(find motoman_sda10f_support)/urdf/sda10f_macro.xacro" />
+  <xacro:motoman_sda10f prefix=""/>
+  <!-- xacro below should not be used, use form above-->
+  <!--xacro:sda10f/-->
+  <xacro:motoman_sda10f prefix="my_prefix_"/>
+  <joint name="base_link_joint" type="fixed" >
     <origin xyz="1.0 0 0"/>
     <parent link="torso_base_link" />
