Commit message: sia5d: use meshes in support pkg. Fix #81.
Stop using those in the config package. That has been deprecated since 2014.

File: motoman_sia5d_support/urdf/sia5d.urdf (robot description, URDF)
Before this commit: robot motoman_sia5d, 9 links, 8 joints
Links:
- link base_link: geometry collision mesh filename=package://motoman_sia5d_support/meshes/sia5d/collision/base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; visual mesh filename=package://motoman_sia5d_support/meshes/sia5d/visual/base.dae
- link link_b: geometry collision mesh filename=package://motoman_sia5d_support/meshes/sia5d/collision/link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; visual mesh filename=package://motoman_sia5d_support/meshes/sia5d/visual/link_b.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
- link link_e: geometry collision mesh filename=package://motoman_sia5d_support/meshes/sia5d/collision/link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; visual mesh filename=package://motoman_sia5d_support/meshes/sia5d/visual/link_e.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
- link link_l: geometry collision mesh filename=package://motoman_sia5d_support/meshes/sia5d/collision/link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; visual mesh filename=package://motoman_sia5d_support/meshes/sia5d/visual/link_l.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
- link link_r: geometry collision mesh filename=package://motoman_sia5d_support/meshes/sia5d/collision/link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; visual mesh filename=package://motoman_sia5d_support/meshes/sia5d/visual/link_r.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
- link link_s: geometry collision mesh filename=package://motoman_sia5d_support/meshes/sia5d/collision/link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; visual mesh filename=package://motoman_sia5d_support/meshes/sia5d/visual/link_s.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
- link link_t: geometry collision mesh filename=package://motoman_sia5d_support/meshes/sia5d/collision/link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; visual mesh filename=package://motoman_sia5d_support/meshes/sia5d/visual/link_t.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
- link link_u: geometry collision mesh filename=package://motoman_sia5d_support/meshes/sia5d/collision/link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; visual mesh filename=package://motoman_sia5d_support/meshes/sia5d/visual/link_u.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

File: motoman_sia5d_support/urdf/sia5d_macro.xacro (robot description, xacro)
@@ -8,5 +8,5 @@
       <origin xyz="0 0 0" rpy="0 0 0" />
       <geometry>
-        <mesh filename="package://motoman_config/meshes/sia5/visual/base.dae" />
+        <mesh filename="package://motoman_sia5d_support/meshes/sia5d/visual/base.dae" />
       </geometry>
     </visual>
@@ -14,5 +14,5 @@
       <origin xyz="0 0 0" rpy="0 0 0" />
       <geometry>
-        <mesh filename="package://motoman_config/meshes/sia5/collision/base.dae" />
+        <mesh filename="package://motoman_sia5d_support/meshes/sia5d/collision/base.dae" />
       </geometry>
     </collision>
@@ -22,5 +22,5 @@
       <origin xyz="0 0 0" rpy="0 0 0" />
       <geometry>
-        <mesh filename="package://motoman_config/meshes/sia5/visual/link_s.dae" />
+        <mesh filename="package://motoman_sia5d_support/meshes/sia5d/visual/link_s.dae" />
       </geometry>
     </visual>
@@ -28,5 +28,5 @@
       <origin xyz="0 0 0" rpy="0 0 0" />
       <geometry>
-        <mesh filename="package://motoman_config/meshes/sia5/collision/link_s.dae" />
+        <mesh filename="package://motoman_sia5d_support/meshes/sia5d/collision/link_s.dae" />
       </geometry>
     </collision>
@@ -43,5 +43,5 @@
       <origin xyz="0 0 0" rpy="0 0 0" />
       <geometry>
-        <mesh filename="package://motoman_config/meshes/sia5/visual/link_l.dae" />
+        <mesh filename="package://motoman_sia5d_support/meshes/sia5d/visual/link_l.dae" />
       </geometry>
     </visual>
@@ -49,5 +49,5 @@
       <origin xyz="0 0 0" rpy="0 0 0" />
       <geometry>
-        <mesh filename="package://motoman_config/meshes/sia5/collision/link_l.dae" />
+        <mesh filename="package://motoman_sia5d_support/meshes/sia5d/collision/link_l.dae" />
       </geometry>
     </collision>
@@ -64,5 +64,5 @@
       <origin xyz="0 0 0" rpy="0 0 0" />
       <geometry>
-        <mesh filename="package://motoman_config/meshes/sia5/visual/link_e.dae" />
+        <mesh filename="package://motoman_sia5d_support/meshes/sia5d/visual/link_e.dae" />
       </geometry>
     </visual>
@@ -70,5 +70,5 @@
       <origin xyz="0 0 0" rpy="0 0 0" />
       <geometry>
-        <mesh filename="package://motoman_config/meshes/sia5/collision/link_e.dae" />
+        <mesh filename="package://motoman_sia5d_support/meshes/sia5d/collision/link_e.dae" />
       </geometry>
     </collision>
@@ -85,5 +85,5 @@
       <origin xyz="0 0 0" rpy="0 0 0" />
       <geometry>
-        <mesh filename="package://motoman_config/meshes/sia5/visual/link_u.dae" />
+        <mesh filename="package://motoman_sia5d_support/meshes/sia5d/visual/link_u.dae" />
       </geometry>
     </visual>
@@ -91,5 +91,5 @@
       <origin xyz="0 0 0" rpy="0 0 0" />
       <geometry>
-        <mesh filename="package://motoman_config/meshes/sia5/collision/link_u.dae" />
+        <mesh filename="package://motoman_sia5d_support/meshes/sia5d/collision/link_u.dae" />
       </geometry>
     </collision>
@@ -106,5 +106,5 @@
       <origin xyz="0 0 0" rpy="0 0 0" />
       <geometry>
-        <mesh filename="package://motoman_config/meshes/sia5/visual/link_r.dae" />
+        <mesh filename="package://motoman_sia5d_support/meshes/sia5d/visual/link_r.dae" />
       </geometry>
     </visual>
@@ -112,5 +112,5 @@
       <origin xyz="0 0 0" rpy="0 0 0" />
       <geometry>
-        <mesh filename="package://motoman_config/meshes/sia5/collision/link_r.dae" />
+        <mesh filename="package://motoman_sia5d_support/meshes/sia5d/collision/link_r.dae" />
       </geometry>
     </collision>
@@ -127,5 +127,5 @@
       <origin xyz="0 0 0" rpy="0 0 0" />
       <geometry>
-        <mesh filename="package://motoman_config/meshes/sia5/visual/link_b.dae" />
+        <mesh filename="package://motoman_sia5d_support/meshes/sia5d/visual/link_b.dae" />
       </geometry>
     </visual>
@@ -133,5 +133,5 @@
       <origin xyz="0 0 0" rpy="0 0 0" />
       <geometry>
-        <mesh filename="package://motoman_config/meshes/sia5/collision/link_b.dae" />
+        <mesh filename="package://motoman_sia5d_support/meshes/sia5d/collision/link_b.dae" />
       </geometry>
     </collision>
@@ -148,5 +148,5 @@
       <origin xyz="0 0 0" rpy="0 0 0" />
       <geometry>
-        <mesh filename="package://motoman_config/meshes/sia5/visual/link_t.dae" />
+        <mesh filename="package://motoman_sia5d_support/meshes/sia5d/visual/link_t.dae" />
       </geometry>
     </visual>
@@ -154,5 +154,5 @@
       <origin xyz="0 0 0" rpy="0 0 0" />
       <geometry>
-        <mesh filename="package://motoman_config/meshes/sia5/collision/link_t.dae" />
+        <mesh filename="package://motoman_sia5d_support/meshes/sia5d/collision/link_t.dae" />
       </geometry>
     </collision>

Commit message: sia: fix ros-i base frame parent.
Same location as link_l, but not connected to it (otherwise it rotates).

File: motoman_sia5d_support/urdf/sia5d.urdf (robot description, URDF)
Before this commit: robot motoman_sia5d, 10 links, 9 joints
Joints:
- removed joint link_l-base
- added joint base_link-base: type fixed, parent base_link, child base, origin xyz=0 0 0.310 rpy=0 0 0

File: motoman_sia5d_support/urdf/sia5d_macro.xacro (robot description, xacro)
@@ -170,9 +170,9 @@
     <child link="${prefix}tool0" />
   </joint>
-    <!-- ROS base_link (via link_l) to Motoman Robot (not Base) Frame transform -->
+    <!-- ROS base_link (via base_link) to Motoman Robot (not Base) Frame transform -->
     <link name="${prefix}base" />
-    <joint name="${prefix}link_l-base" type="fixed">
-      <origin xyz="0 0 0" rpy="0 0 0"/>
-      <parent link="${prefix}link_l"/>
+    <joint name="${prefix}base_link-base" type="fixed">
+      <origin xyz="0 0 0.310" rpy="0 0 0"/>
+      <parent link="${prefix}base_link"/>
       <child link="${prefix}base"/>
     </joint>
