Commit message: mini: don't add mini prefix to mesh filenames.
It's already clear for which robot these meshes are, no need to repeat the prefix in the filenames again.

File: motoman_mini_support/urdf/mini_macro.xacro (robot description, xacro)
@@ -10,5 +10,5 @@
         <visual>
             <geometry>
-                <mesh filename="package://motoman_mini_support/meshes/visual/mini_base_link.stl"/>
+                <mesh filename="package://motoman_mini_support/meshes/visual/base_link.stl"/>
             </geometry>
             <material name="yaskawa_blue"/>
@@ -16,5 +16,5 @@
         <collision>
             <geometry>
-                <mesh filename="package://motoman_mini_support/meshes/collision/mini_base_link.stl"/>
+                <mesh filename="package://motoman_mini_support/meshes/collision/base_link.stl"/>
             </geometry>
         </collision>
@@ -23,5 +23,5 @@
         <visual>
             <geometry>
-                <mesh filename="package://motoman_mini_support/meshes/visual/mini_link_1_s.stl"/>
+                <mesh filename="package://motoman_mini_support/meshes/visual/link_1_s.stl"/>
             </geometry>
             <material name="yaskawa_blue"/>
@@ -29,5 +29,5 @@
         <collision>
             <geometry>
-                <mesh filename="package://motoman_mini_support/meshes/collision/mini_link_1_s.stl"/>
+                <mesh filename="package://motoman_mini_support/meshes/collision/link_1_s.stl"/>
             </geometry>
         </collision>
@@ -36,5 +36,5 @@
         <visual>
             <geometry>
-                <mesh filename="package://motoman_mini_support/meshes/visual/mini_link_2_l.stl"/>
+                <mesh filename="package://motoman_mini_support/meshes/visual/link_2_l.stl"/>
             </geometry>
             <material name="yaskawa_blue"/>
@@ -42,5 +42,5 @@
         <collision>
             <geometry>
-                <mesh filename="package://motoman_mini_support/meshes/collision/mini_link_2_l.stl"/>
+                <mesh filename="package://motoman_mini_support/meshes/collision/link_2_l.stl"/>
             </geometry>
         </collision>
@@ -49,5 +49,5 @@
         <visual>
             <geometry>
-                <mesh filename="package://motoman_mini_support/meshes/visual/mini_link_3_u.stl"/>
+                <mesh filename="package://motoman_mini_support/meshes/visual/link_3_u.stl"/>
             </geometry>
             <material name="yaskawa_blue"/>
@@ -55,5 +55,5 @@
         <collision>
             <geometry>
-                <mesh filename="package://motoman_mini_support/meshes/collision/mini_link_3_u.stl"/>
+                <mesh filename="package://motoman_mini_support/meshes/collision/link_3_u.stl"/>
             </geometry>
         </collision>
@@ -62,5 +62,5 @@
         <visual>
             <geometry>
-                <mesh filename="package://motoman_mini_support/meshes/visual/mini_link_4_r.stl"/>
+                <mesh filename="package://motoman_mini_support/meshes/visual/link_4_r.stl"/>
             </geometry>
             <material name="yaskawa_blue"/>
@@ -68,5 +68,5 @@
         <collision>
             <geometry>
-                <mesh filename="package://motoman_mini_support/meshes/collision/mini_link_4_r.stl"/>
+                <mesh filename="package://motoman_mini_support/meshes/collision/link_4_r.stl"/>
             </geometry>
         </collision>
@@ -75,5 +75,5 @@
         <visual>
             <geometry>
-                <mesh filename="package://motoman_mini_support/meshes/visual/mini_link_5_b.stl"/>
+                <mesh filename="package://motoman_mini_support/meshes/visual/link_5_b.stl"/>
             </geometry>
             <material name="yaskawa_blue"/>
@@ -81,5 +81,5 @@
         <collision>
             <geometry>
-                <mesh filename="package://motoman_mini_support/meshes/collision/mini_link_5_b.stl"/>
+                <mesh filename="package://motoman_mini_support/meshes/collision/link_5_b.stl"/>
             </geometry>
         </collision>
@@ -88,5 +88,5 @@
         <visual>
             <geometry>
-                <mesh filename="package://motoman_mini_support/meshes/visual/mini_link_6_t.stl"/>
+                <mesh filename="package://motoman_mini_support/meshes/visual/link_6_t.stl"/>
             </geometry>
             <material name="yaskawa_blue"/>
@@ -94,5 +94,5 @@
         <collision>
             <geometry>
-                <mesh filename="package://motoman_mini_support/meshes/collision/mini_link_6_t.stl"/>
+                <mesh filename="package://motoman_mini_support/meshes/collision/link_6_t.stl"/>
             </geometry>
         </collision>

Commit message: mini: place meshes in variant sub dir.

File: motoman_mini_support/urdf/mini_macro.xacro (robot description, xacro)
@@ -10,5 +10,5 @@
         <visual>
             <geometry>
-                <mesh filename="package://motoman_mini_support/meshes/visual/base_link.stl"/>
+                <mesh filename="package://motoman_mini_support/meshes/mini/visual/base_link.stl"/>
             </geometry>
             <material name="yaskawa_blue"/>
@@ -16,5 +16,5 @@
         <collision>
             <geometry>
-                <mesh filename="package://motoman_mini_support/meshes/collision/base_link.stl"/>
+                <mesh filename="package://motoman_mini_support/meshes/mini/collision/base_link.stl"/>
             </geometry>
         </collision>
@@ -23,5 +23,5 @@
         <visual>
             <geometry>
-                <mesh filename="package://motoman_mini_support/meshes/visual/link_1_s.stl"/>
+                <mesh filename="package://motoman_mini_support/meshes/mini/visual/link_1_s.stl"/>
             </geometry>
             <material name="yaskawa_blue"/>
@@ -29,5 +29,5 @@
         <collision>
             <geometry>
-                <mesh filename="package://motoman_mini_support/meshes/collision/link_1_s.stl"/>
+                <mesh filename="package://motoman_mini_support/meshes/mini/collision/link_1_s.stl"/>
             </geometry>
         </collision>
@@ -36,5 +36,5 @@
         <visual>
             <geometry>
-                <mesh filename="package://motoman_mini_support/meshes/visual/link_2_l.stl"/>
+                <mesh filename="package://motoman_mini_support/meshes/mini/visual/link_2_l.stl"/>
             </geometry>
             <material name="yaskawa_blue"/>
@@ -42,5 +42,5 @@
         <collision>
             <geometry>
-                <mesh filename="package://motoman_mini_support/meshes/collision/link_2_l.stl"/>
+                <mesh filename="package://motoman_mini_support/meshes/mini/collision/link_2_l.stl"/>
             </geometry>
         </collision>
@@ -49,5 +49,5 @@
         <visual>
             <geometry>
-                <mesh filename="package://motoman_mini_support/meshes/visual/link_3_u.stl"/>
+                <mesh filename="package://motoman_mini_support/meshes/mini/visual/link_3_u.stl"/>
             </geometry>
             <material name="yaskawa_blue"/>
@@ -55,5 +55,5 @@
         <collision>
             <geometry>
-                <mesh filename="package://motoman_mini_support/meshes/collision/link_3_u.stl"/>
+                <mesh filename="package://motoman_mini_support/meshes/mini/collision/link_3_u.stl"/>
             </geometry>
         </collision>
@@ -62,5 +62,5 @@
         <visual>
             <geometry>
-                <mesh filename="package://motoman_mini_support/meshes/visual/link_4_r.stl"/>
+                <mesh filename="package://motoman_mini_support/meshes/mini/visual/link_4_r.stl"/>
             </geometry>
             <material name="yaskawa_blue"/>
@@ -68,5 +68,5 @@
         <collision>
             <geometry>
-                <mesh filename="package://motoman_mini_support/meshes/collision/link_4_r.stl"/>
+                <mesh filename="package://motoman_mini_support/meshes/mini/collision/link_4_r.stl"/>
             </geometry>
         </collision>
@@ -75,5 +75,5 @@
         <visual>
             <geometry>
-                <mesh filename="package://motoman_mini_support/meshes/visual/link_5_b.stl"/>
+                <mesh filename="package://motoman_mini_support/meshes/mini/visual/link_5_b.stl"/>
             </geometry>
             <material name="yaskawa_blue"/>
@@ -81,5 +81,5 @@
         <collision>
             <geometry>
-                <mesh filename="package://motoman_mini_support/meshes/collision/link_5_b.stl"/>
+                <mesh filename="package://motoman_mini_support/meshes/mini/collision/link_5_b.stl"/>
             </geometry>
         </collision>
@@ -88,5 +88,5 @@
         <visual>
             <geometry>
-                <mesh filename="package://motoman_mini_support/meshes/visual/link_6_t.stl"/>
+                <mesh filename="package://motoman_mini_support/meshes/mini/visual/link_6_t.stl"/>
             </geometry>
             <material name="yaskawa_blue"/>
@@ -94,5 +94,5 @@
         <collision>
             <geometry>
-                <mesh filename="package://motoman_mini_support/meshes/collision/link_6_t.stl"/>
+                <mesh filename="package://motoman_mini_support/meshes/mini/collision/link_6_t.stl"/>
             </geometry>
         </collision>
