Commit message: mini: cleanup xacros.
Use 'pi' constant and indent with 2 spaces everywhere.

File: motoman_mini_support/urdf/mini.xacro (robot description, xacro)
@@ -1,5 +1,5 @@
 <?xml version="1.0" ?>
 <robot name="motoman_mini" xmlns:xacro="http://ros.org/wiki/xacro">
-	<xacro:include filename="$(find motoman_mini_support)/urdf/mini_macro.xacro" />
-	<xacro:motoman_mini prefix=""/>
+  <xacro:include filename="$(find motoman_mini_support)/urdf/mini_macro.xacro" />
+  <xacro:motoman_mini prefix=""/>
 </robot>

File: motoman_mini_support/urdf/mini_macro.xacro (robot description, xacro)
@@ -2,158 +2,158 @@
 <robot xmlns:xacro="http://ros.org/wiki/xacro">
 <xacro:macro name="motoman_mini" params="prefix">
-    <!-- Properties -->
-    <material name="yaskawa_blue">
-          <color rgba="0.12941 0.14902 0.74902 1" />
-    </material>
-    <!-- link list -->
-    <link name="${prefix}base_link">
-        <visual>
-            <geometry>
-                <mesh filename="package://motoman_mini_support/meshes/mini/visual/base_link.stl"/>
-            </geometry>
-            <material name="yaskawa_blue"/>
-        </visual>
-        <collision>
-            <geometry>
-                <mesh filename="package://motoman_mini_support/meshes/mini/collision/base_link.stl"/>
-            </geometry>
-        </collision>
-    </link>
-    <link name="${prefix}link_1_s">
-        <visual>
-            <geometry>
-                <mesh filename="package://motoman_mini_support/meshes/mini/visual/link_1_s.stl"/>
-            </geometry>
-            <material name="yaskawa_blue"/>
-        </visual>
-        <collision>
-            <geometry>
-                <mesh filename="package://motoman_mini_support/meshes/mini/collision/link_1_s.stl"/>
-            </geometry>
-        </collision>
-    </link>
-    <link name="${prefix}link_2_l">
-        <visual>
-            <geometry>
-                <mesh filename="package://motoman_mini_support/meshes/mini/visual/link_2_l.stl"/>
-            </geometry>
-            <material name="yaskawa_blue"/>
-        </visual>
-        <collision>
-            <geometry>
-                <mesh filename="package://motoman_mini_support/meshes/mini/collision/link_2_l.stl"/>
-            </geometry>
-        </collision>
-    </link>
-    <link name="${prefix}link_3_u">
-        <visual>
-            <geometry>
-                <mesh filename="package://motoman_mini_support/meshes/mini/visual/link_3_u.stl"/>
-            </geometry>
-            <material name="yaskawa_blue"/>
-        </visual>
-        <collision>
-            <geometry>
-                <mesh filename="package://motoman_mini_support/meshes/mini/collision/link_3_u.stl"/>
-            </geometry>
-        </collision>
-    </link>
-    <link name="${prefix}link_4_r">
-        <visual>
-            <geometry>
-                <mesh filename="package://motoman_mini_support/meshes/mini/visual/link_4_r.stl"/>
-            </geometry>
-            <material name="yaskawa_blue"/>
-        </visual>
-        <collision>
-            <geometry>
-                <mesh filename="package://motoman_mini_support/meshes/mini/collision/link_4_r.stl"/>
-            </geometry>
-        </collision>
-    </link>
-    <link name="${prefix}link_5_b">
-        <visual>
-            <geometry>
-                <mesh filename="package://motoman_mini_support/meshes/mini/visual/link_5_b.stl"/>
-            </geometry>
-            <material name="yaskawa_blue"/>
-        </visual>
-        <collision>
-            <geometry>
-                <mesh filename="package://motoman_mini_support/meshes/mini/collision/link_5_b.stl"/>
-            </geometry>
-        </collision>
-    </link>
-    <link name="${prefix}link_6_t">
-        <visual>
-            <geometry>
-                <mesh filename="package://motoman_mini_support/meshes/mini/visual/link_6_t.stl"/>
-            </geometry>
-            <material name="yaskawa_blue"/>
-        </visual>
-        <collision>
-            <geometry>
-                <mesh filename="package://motoman_mini_support/meshes/mini/collision/link_6_t.stl"/>
-            </geometry>
-        </collision>
-    </link>
-    <link name="${prefix}tool0"/>
-    <!-- end of link list -->
-    <!-- joint list -->
-    <joint name="${prefix}joint_1_s" type="revolute">
-        <parent link="${prefix}base_link"/>
-        <child link="${prefix}link_1_s"/>
-        <origin xyz="0 0 0.103" rpy="0 0 0" />
-        <axis xyz="0 0 1" />
-        <limit lower="-2.9670" upper="2.9670" effort="0.12" velocity="5.4977"/>
-    </joint>
-    <joint name="${prefix}joint_2_l" type="revolute">
-        <parent link="${prefix}link_1_s"/>
-        <child link="${prefix}link_2_l"/>
-        <origin xyz="0.020 0 0" rpy="0 0 0" />
-        <axis xyz="0 1 0" />
-        <limit lower="-1.4835" upper="1.5707" effort="0.12" velocity="5.4977"/>
-    </joint>
-    <joint name="${prefix}joint_3_u" type="revolute">
-        <parent link="${prefix}link_2_l"/>
-        <child link="${prefix}link_3_u"/>
-        <origin xyz="0 0 0.165" rpy="0 0 0" />
-        <axis xyz="0 -1 0" />
-        <limit lower="-0.8726" upper="1.5707" effort="0.12" velocity="7.3304"/>
-    </joint>
-    <joint name="${prefix}joint_4_r" type="revolute">
-        <parent link="${prefix}link_3_u"/>
-        <child link="${prefix}link_4_r"/>
-        <origin xyz="0.165 0 0" rpy="0 0 0" />
-        <axis xyz="-1 0 0" />
-        <limit lower="-2.4434" upper="2.4434" effort="0.07" velocity="10.4719"/>
-    </joint>
-    <joint name="${prefix}joint_5_b" type="revolute">
-        <parent link="${prefix}link_4_r"/>
-        <child link="${prefix}link_5_b"/>
-        <origin xyz="0 0 0" rpy="0 0 0" />
-        <axis xyz="0 -1 0" />
-        <limit lower="-0.5235" upper="3.6651" effort="0.07" velocity="10.4719"/>
-    </joint>
-    <joint name="${prefix}joint_6_t" type="revolute">
-        <parent link="${prefix}link_5_b"/>
-        <child link="${prefix}link_6_t"/>
-        <origin xyz="0 0 0" rpy="0 0 0" />
-        <axis xyz="0 0 1" />
-        <limit lower="-6.2831" upper="6.2831" effort="0.07" velocity="10.4719"/>
-    </joint>
-    <joint name="${prefix}joint_6_t-tool0" type="fixed">
-        <origin xyz="0 0 -0.040 " rpy="3.1415926 0 0"/>
-        <parent link="${prefix}link_6_t"/>
-        <child link="${prefix}tool0"/>
-    </joint>
-    <!-- end of joint list -->
-    <!-- ROS base_link to Robot Manufacturer World Coordinates transform -->
-    <link name="${prefix}base" />
-    <joint name="${prefix}base_link-base" type="fixed">
-        <origin xyz="0 0 0.103" rpy="0 0 0"/>
-        <parent link="${prefix}base_link"/>
-        <child link="${prefix}base"/>
-    </joint>
-    </xacro:macro>
+  <!-- Properties -->
+  <material name="yaskawa_blue">
+      <color rgba="0.12941 0.14902 0.74902 1" />
+  </material>
+  <!-- link list -->
+  <link name="${prefix}base_link">
+    <visual>
+      <geometry>
+        <mesh filename="package://motoman_mini_support/meshes/mini/visual/base_link.stl"/>
+      </geometry>
+      <material name="yaskawa_blue"/>
+    </visual>
+    <collision>
+      <geometry>
+        <mesh filename="package://motoman_mini_support/meshes/mini/collision/base_link.stl"/>
+      </geometry>
+    </collision>
+  </link>
+  <link name="${prefix}link_1_s">
+    <visual>
+      <geometry>
+        <mesh filename="package://motoman_mini_support/meshes/mini/visual/link_1_s.stl"/>
+      </geometry>
+      <material name="yaskawa_blue"/>
+    </visual>
+    <collision>
+      <geometry>
+        <mesh filename="package://motoman_mini_support/meshes/mini/collision/link_1_s.stl"/>
+      </geometry>
+    </collision>
+  </link>
+  <link name="${prefix}link_2_l">
+    <visual>
+      <geometry>
+        <mesh filename="package://motoman_mini_support/meshes/mini/visual/link_2_l.stl"/>
+      </geometry>
+      <material name="yaskawa_blue"/>
+    </visual>
+    <collision>
+      <geometry>
+        <mesh filename="package://motoman_mini_support/meshes/mini/collision/link_2_l.stl"/>
+      </geometry>
+    </collision>
+  </link>
+  <link name="${prefix}link_3_u">
+    <visual>
+      <geometry>
+        <mesh filename="package://motoman_mini_support/meshes/mini/visual/link_3_u.stl"/>
+      </geometry>
+      <material name="yaskawa_blue"/>
+    </visual>
+    <collision>
+      <geometry>
+        <mesh filename="package://motoman_mini_support/meshes/mini/collision/link_3_u.stl"/>
+      </geometry>
+    </collision>
+  </link>
+  <link name="${prefix}link_4_r">
+    <visual>
+      <geometry>
+        <mesh filename="package://motoman_mini_support/meshes/mini/visual/link_4_r.stl"/>
+      </geometry>
+      <material name="yaskawa_blue"/>
+    </visual>
+    <collision>
+      <geometry>
+        <mesh filename="package://motoman_mini_support/meshes/mini/collision/link_4_r.stl"/>
+      </geometry>
+    </collision>
+  </link>
+  <link name="${prefix}link_5_b">
+    <visual>
+      <geometry>
+        <mesh filename="package://motoman_mini_support/meshes/mini/visual/link_5_b.stl"/>
+      </geometry>
+      <material name="yaskawa_blue"/>
+    </visual>
+    <collision>
+      <geometry>
+        <mesh filename="package://motoman_mini_support/meshes/mini/collision/link_5_b.stl"/>
+      </geometry>
+    </collision>
+  </link>
+  <link name="${prefix}link_6_t">
+    <visual>
+      <geometry>
+        <mesh filename="package://motoman_mini_support/meshes/mini/visual/link_6_t.stl"/>
+      </geometry>
+      <material name="yaskawa_blue"/>
+    </visual>
+    <collision>
+      <geometry>
+        <mesh filename="package://motoman_mini_support/meshes/mini/collision/link_6_t.stl"/>
+      </geometry>
+    </collision>
+  </link>
+  <link name="${prefix}tool0"/>
+  <!-- end of link list -->
+  <!-- joint list -->
+  <joint name="${prefix}joint_1_s" type="revolute">
+    <parent link="${prefix}base_link"/>
+    <child link="${prefix}link_1_s"/>
+    <origin xyz="0 0 0.103" rpy="0 0 0" />
+    <axis xyz="0 0 1" />
+    <limit lower="-2.9670" upper="2.9670" effort="0.12" velocity="5.4977"/>
+  </joint>
+  <joint name="${prefix}joint_2_l" type="revolute">
+    <parent link="${prefix}link_1_s"/>
+    <child link="${prefix}link_2_l"/>
+    <origin xyz="0.020 0 0" rpy="0 0 0" />
+    <axis xyz="0 1 0" />
+    <limit lower="-1.4835" upper="1.5707" effort="0.12" velocity="5.4977"/>
+  </joint>
+  <joint name="${prefix}joint_3_u" type="revolute">
+    <parent link="${prefix}link_2_l"/>
+    <child link="${prefix}link_3_u"/>
+    <origin xyz="0 0 0.165" rpy="0 0 0" />
+    <axis xyz="0 -1 0" />
+    <limit lower="-0.8726" upper="1.5707" effort="0.12" velocity="7.3304"/>
+  </joint>
+  <joint name="${prefix}joint_4_r" type="revolute">
+    <parent link="${prefix}link_3_u"/>
+    <child link="${prefix}link_4_r"/>
+    <origin xyz="0.165 0 0" rpy="0 0 0" />
+    <axis xyz="-1 0 0" />
+    <limit lower="-2.4434" upper="2.4434" effort="0.07" velocity="10.4719"/>
+  </joint>
+  <joint name="${prefix}joint_5_b" type="revolute">
+    <parent link="${prefix}link_4_r"/>
+    <child link="${prefix}link_5_b"/>
+    <origin xyz="0 0 0" rpy="0 0 0" />
+    <axis xyz="0 -1 0" />
+    <limit lower="-0.5235" upper="3.6651" effort="0.07" velocity="10.4719"/>
+  </joint>
+  <joint name="${prefix}joint_6_t" type="revolute">
+    <parent link="${prefix}link_5_b"/>
+    <child link="${prefix}link_6_t"/>
+    <origin xyz="0 0 0" rpy="0 0 0" />
+    <axis xyz="0 0 1" />
+    <limit lower="-6.2831" upper="6.2831" effort="0.07" velocity="10.4719"/>
+  </joint>
+  <joint name="${prefix}joint_6_t-tool0" type="fixed">
+    <origin xyz="0 0 -0.040 " rpy="${pi} 0 0"/>
+    <parent link="${prefix}link_6_t"/>
+    <child link="${prefix}tool0"/>
+  </joint>
+  <!-- end of joint list -->
+  <!-- ROS base_link to Robot Manufacturer World Coordinates transform -->
+  <link name="${prefix}base" />
+  <joint name="${prefix}base_link-base" type="fixed">
+    <origin xyz="0 0 0.103" rpy="0 0 0"/>
+    <parent link="${prefix}base_link"/>
+    <child link="${prefix}base"/>
+  </joint>
+  </xacro:macro>
 </robot>
