Commit message: correction of tool0 coordinate system orientation to be the same as Yaskawa controller flange coordinate system

File: motoman_gp180_120_support/urdf/gp180_120_macro.xacro (robot description, xacro)
@@ -113,4 +113,5 @@
         </collision>
     </link>
+    <!-- corresponds to Yaskawa controller flange coordinate system; Z+ out from the flange, X+ up when robot is in basic position -->
     <link name="${prefix}tool0"/>
     <!-- end of link list -->
@@ -159,5 +160,5 @@
     </joint>
     <joint name="${prefix}joint_6_t-tool0" type="fixed">
-        <origin xyz="-0.0255 0 0" rpy="${DEG2RAD * 180} ${-DEG2RAD * 180} 0"/>
+        <origin xyz="-0.0255 0 0" rpy="0 ${-DEG2RAD * 90} 0"/>
         <parent link="${prefix}link_6_t"/>
         <child link="${prefix}tool0"/>
@@ -165,4 +166,5 @@
     <!-- end of joint list -->
     <!-- ROS base_link to Robot Manufacturer World Coordinates transform -->
+    <!-- corresponds to Yaskawa controller robot coordinate system -->
     <link name="${prefix}base" />
     <joint name="${prefix}base_link-base" type="fixed">
