Commit message: changed package name to motoman_gp180_support in all places (GP180 is robot series, 120 is variant of this series); moved meshes to subdirectory for GP180-120 variant; renamed meshes to lowercase

File: motoman_gp180_support/urdf/gp180_120.xacro (robot description, xacro)
@@ -1,5 +1,5 @@
 <?xml version="1.0" ?>
 <robot name="motoman_gp180_120" xmlns:xacro="http://ros.org/wiki/xacro">
-    <xacro:include filename="$(find motoman_gp180_120_support)/urdf/gp180_120_macro.xacro" />
+    <xacro:include filename="$(find motoman_gp180_support)/urdf/gp180_120_macro.xacro" />
     <xacro:motoman_gp180_120 prefix=""/>
 </robot>

File: motoman_gp180_support/urdf/gp180_120_macro.xacro (robot description, xacro)
@@ -12,5 +12,5 @@
             <origin rpy="${DEG2RAD * 90} 0 0" />
             <geometry>
-                <mesh filename="package://motoman_gp180_120_support/meshes/visual/BASE_AXIS.stl" scale="0.001 0.001 0.001"/>
+                <mesh filename="package://motoman_gp180_support/meshes/gp180_120/visual/base_axis.stl" scale="0.001 0.001 0.001"/>
             </geometry>
             <material name="yaskawa_blue"/>
@@ -19,5 +19,5 @@
             <origin rpy="${DEG2RAD * 90} 0 0" />
             <geometry>
-                <mesh filename="package://motoman_gp180_120_support/meshes/collision/BASE_AXIS.stl" scale="0.001 0.001 0.001"/>
+                <mesh filename="package://motoman_gp180_support/meshes/gp180_120/collision/base_axis.stl" scale="0.001 0.001 0.001"/>
             </geometry>
         </collision>
@@ -27,5 +27,5 @@
             <origin xyz="0 0 -0.317" rpy="${DEG2RAD * 90} 0 0" />
             <geometry>
-                <mesh filename="package://motoman_gp180_120_support/meshes/visual/S_AXIS.stl" scale="0.001 0.001 0.001"/>
+                <mesh filename="package://motoman_gp180_support/meshes/gp180_120/visual/s_axis.stl" scale="0.001 0.001 0.001"/>
             </geometry>
             <material name="yaskawa_blue"/>
@@ -34,5 +34,5 @@
             <origin xyz="0 0 -0.317" rpy="${DEG2RAD * 90} 0 0" />
             <geometry>
-                <mesh filename="package://motoman_gp180_120_support/meshes/collision/S_AXIS.stl" scale="0.001 0.001 0.001"/>
+                <mesh filename="package://motoman_gp180_support/meshes/gp180_120/collision/s_axis.stl" scale="0.001 0.001 0.001"/>
             </geometry>
         </collision>
@@ -42,5 +42,5 @@
             <origin xyz="0.325 0.07 -0.650" rpy="${DEG2RAD * 90} 0 0" />
             <geometry>
-                <mesh filename="package://motoman_gp180_120_support/meshes/visual/L_AXIS.stl" scale="0.001 0.001 0.001"/>
+                <mesh filename="package://motoman_gp180_support/meshes/gp180_120/visual/l_axis.stl" scale="0.001 0.001 0.001"/>
             </geometry>
             <material name="yaskawa_blue"/>
@@ -49,5 +49,5 @@
             <origin xyz="0.325 0.07 -0.650" rpy="${DEG2RAD * 90} 0 0" />
             <geometry>
-                <mesh filename="package://motoman_gp180_120_support/meshes/collision/L_AXIS.stl" scale="0.001 0.001 0.001"/>
+                <mesh filename="package://motoman_gp180_support/meshes/gp180_120/collision/l_axis.stl" scale="0.001 0.001 0.001"/>
             </geometry>
         </collision>
@@ -57,5 +57,5 @@
             <origin xyz="0.325 0.0415 -1.800" rpy="${DEG2RAD * 90} 0 0" />
             <geometry>
-                <mesh filename="package://motoman_gp180_120_support/meshes/visual/U_AXIS.stl" scale="0.001 0.001 0.001"/>
+                <mesh filename="package://motoman_gp180_support/meshes/gp180_120/visual/u_axis.stl" scale="0.001 0.001 0.001"/>
             </geometry>
             <material name="yaskawa_blue"/>
@@ -64,5 +64,5 @@
             <origin xyz="0.325 0.0415 -1.800" rpy="${DEG2RAD * 90} 0 0" />
             <geometry>
-                <mesh filename="package://motoman_gp180_120_support/meshes/collision/U_AXIS.stl" scale="0.001 0.001 0.001"/>
+                <mesh filename="package://motoman_gp180_support/meshes/gp180_120/collision/u_axis.stl" scale="0.001 0.001 0.001"/>
             </geometry>
         </collision>
@@ -72,5 +72,5 @@
             <origin xyz="1.723 0 -2.100" rpy="${DEG2RAD * 90} 0 0" />
             <geometry>
-                <mesh filename="package://motoman_gp180_120_support/meshes/visual/R_AXIS.stl" scale="0.001 0.001 0.001"/>
+                <mesh filename="package://motoman_gp180_support/meshes/gp180_120/visual/r_axis.stl" scale="0.001 0.001 0.001"/>
             </geometry>
             <material name="yaskawa_blue"/>
@@ -79,5 +79,5 @@
             <origin xyz="1.723 0 -2.100" rpy="${DEG2RAD * 90} 0 0" />
             <geometry>
-                <mesh filename="package://motoman_gp180_120_support/meshes/collision/R_AXIS.stl" scale="0.001 0.001 0.001"/>
+                <mesh filename="package://motoman_gp180_support/meshes/gp180_120/collision/r_axis.stl" scale="0.001 0.001 0.001"/>
             </geometry>
         </collision>
@@ -87,5 +87,5 @@
             <origin xyz="1.915 -0.082 -2.100" rpy="${DEG2RAD * 90} 0 0" />
             <geometry>
-                <mesh filename="package://motoman_gp180_120_support/meshes/visual/B_AXIS.stl" scale="0.001 0.001 0.001"/>
+                <mesh filename="package://motoman_gp180_support/meshes/gp180_120/visual/b_axis.stl" scale="0.001 0.001 0.001"/>
             </geometry>
             <material name="yaskawa_blue"/>
@@ -94,5 +94,5 @@
             <origin xyz="1.915 -0.082 -2.100" rpy="${DEG2RAD * 90} 0 0" />
             <geometry>
-                <mesh filename="package://motoman_gp180_120_support/meshes/collision/B_AXIS.stl" scale="0.001 0.001 0.001"/>
+                <mesh filename="package://motoman_gp180_support/meshes/gp180_120/collision/b_axis.stl" scale="0.001 0.001 0.001"/>
             </geometry>
         </collision>
@@ -102,5 +102,5 @@
             <origin xyz="2.1145 0 -2.100" rpy="${DEG2RAD * 90} 0 0" />
             <geometry>
-                <mesh filename="package://motoman_gp180_120_support/meshes/visual/T_AXIS.stl" scale="0.001 0.001 0.001"/>
+                <mesh filename="package://motoman_gp180_support/meshes/gp180_120/visual/t_axis.stl" scale="0.001 0.001 0.001"/>
             </geometry>
             <material name="yaskawa_blue"/>
@@ -109,5 +109,5 @@
             <origin xyz="2.1145 0 -2.100" rpy="${DEG2RAD * 90} 0 0" />
             <geometry>
-                <mesh filename="package://motoman_gp180_120_support/meshes/collision/T_AXIS.stl" scale="0.001 0.001 0.001"/>
+                <mesh filename="package://motoman_gp180_support/meshes/gp180_120/collision/t_axis.stl" scale="0.001 0.001 0.001"/>
             </geometry>
         </collision>
