Commit message: removed DEG2RAD and used Python expressions in xacro instead

File: motoman_gp180_support/urdf/gp180_120_macro.xacro (robot description, xacro)
@@ -6,9 +6,8 @@
           <color rgba="0.12941 0.14902 0.74902 1" />
     </material>
-    <property name="DEG2RAD" value="0.017453292519943295" />
     <!-- link list -->
     <link name="${prefix}base_link">
         <visual>
-            <origin rpy="${DEG2RAD * 90} 0 0" />
+            <origin rpy="${radians(90)} 0 0" />
             <geometry>
                 <mesh filename="package://motoman_gp180_support/meshes/gp180_120/visual/base_axis.stl" scale="0.001 0.001 0.001"/>
@@ -17,5 +16,5 @@
         </visual>
         <collision>
-            <origin rpy="${DEG2RAD * 90} 0 0" />
+            <origin rpy="${radians(90)} 0 0" />
             <geometry>
                 <mesh filename="package://motoman_gp180_support/meshes/gp180_120/collision/base_axis.stl" scale="0.001 0.001 0.001"/>
@@ -25,5 +24,5 @@
     <link name="${prefix}link_1_s">
         <visual>
-            <origin xyz="0 0 -0.317" rpy="${DEG2RAD * 90} 0 0" />
+            <origin xyz="0 0 -0.317" rpy="${radians(90)} 0 0" />
             <geometry>
                 <mesh filename="package://motoman_gp180_support/meshes/gp180_120/visual/s_axis.stl" scale="0.001 0.001 0.001"/>
@@ -32,5 +31,5 @@
         </visual>
         <collision>
-            <origin xyz="0 0 -0.317" rpy="${DEG2RAD * 90} 0 0" />
+            <origin xyz="0 0 -0.317" rpy="${radians(90)} 0 0" />
             <geometry>
                 <mesh filename="package://motoman_gp180_support/meshes/gp180_120/collision/s_axis.stl" scale="0.001 0.001 0.001"/>
@@ -40,5 +39,5 @@
     <link name="${prefix}link_2_l">
         <visual>
-            <origin xyz="0.325 0.07 -0.650" rpy="${DEG2RAD * 90} 0 0" />
+            <origin xyz="0.325 0.07 -0.650" rpy="${radians(90)} 0 0" />
             <geometry>
                 <mesh filename="package://motoman_gp180_support/meshes/gp180_120/visual/l_axis.stl" scale="0.001 0.001 0.001"/>
@@ -47,5 +46,5 @@
         </visual>
         <collision>
-            <origin xyz="0.325 0.07 -0.650" rpy="${DEG2RAD * 90} 0 0" />
+            <origin xyz="0.325 0.07 -0.650" rpy="${radians(90)} 0 0" />
             <geometry>
                 <mesh filename="package://motoman_gp180_support/meshes/gp180_120/collision/l_axis.stl" scale="0.001 0.001 0.001"/>
@@ -55,5 +54,5 @@
     <link name="${prefix}link_3_u">
         <visual>
-            <origin xyz="0.325 0.0415 -1.800" rpy="${DEG2RAD * 90} 0 0" />
+            <origin xyz="0.325 0.0415 -1.800" rpy="${radians(90)} 0 0" />
             <geometry>
                 <mesh filename="package://motoman_gp180_support/meshes/gp180_120/visual/u_axis.stl" scale="0.001 0.001 0.001"/>
@@ -62,5 +61,5 @@
         </visual>
         <collision>
-            <origin xyz="0.325 0.0415 -1.800" rpy="${DEG2RAD * 90} 0 0" />
+            <origin xyz="0.325 0.0415 -1.800" rpy="${radians(90)} 0 0" />
             <geometry>
                 <mesh filename="package://motoman_gp180_support/meshes/gp180_120/collision/u_axis.stl" scale="0.001 0.001 0.001"/>
@@ -70,5 +69,5 @@
     <link name="${prefix}link_4_r">
         <visual>
-            <origin xyz="1.723 0 -2.100" rpy="${DEG2RAD * 90} 0 0" />
+            <origin xyz="1.723 0 -2.100" rpy="${radians(90)} 0 0" />
             <geometry>
                 <mesh filename="package://motoman_gp180_support/meshes/gp180_120/visual/r_axis.stl" scale="0.001 0.001 0.001"/>
@@ -77,5 +76,5 @@
         </visual>
         <collision>
-            <origin xyz="1.723 0 -2.100" rpy="${DEG2RAD * 90} 0 0" />
+            <origin xyz="1.723 0 -2.100" rpy="${radians(90)} 0 0" />
             <geometry>
                 <mesh filename="package://motoman_gp180_support/meshes/gp180_120/collision/r_axis.stl" scale="0.001 0.001 0.001"/>
@@ -85,5 +84,5 @@
     <link name="${prefix}link_5_b">
         <visual>
-            <origin xyz="1.915 -0.082 -2.100" rpy="${DEG2RAD * 90} 0 0" />
+            <origin xyz="1.915 -0.082 -2.100" rpy="${radians(90)} 0 0" />
             <geometry>
                 <mesh filename="package://motoman_gp180_support/meshes/gp180_120/visual/b_axis.stl" scale="0.001 0.001 0.001"/>
@@ -92,5 +91,5 @@
         </visual>
         <collision>
-            <origin xyz="1.915 -0.082 -2.100" rpy="${DEG2RAD * 90} 0 0" />
+            <origin xyz="1.915 -0.082 -2.100" rpy="${radians(90)} 0 0" />
             <geometry>
                 <mesh filename="package://motoman_gp180_support/meshes/gp180_120/collision/b_axis.stl" scale="0.001 0.001 0.001"/>
@@ -100,5 +99,5 @@
     <link name="${prefix}link_6_t">
         <visual>
-            <origin xyz="2.1145 0 -2.100" rpy="${DEG2RAD * 90} 0 0" />
+            <origin xyz="2.1145 0 -2.100" rpy="${radians(90)} 0 0" />
             <geometry>
                 <mesh filename="package://motoman_gp180_support/meshes/gp180_120/visual/t_axis.stl" scale="0.001 0.001 0.001"/>
@@ -107,5 +106,5 @@
         </visual>
         <collision>
-            <origin xyz="2.1145 0 -2.100" rpy="${DEG2RAD * 90} 0 0" />
+            <origin xyz="2.1145 0 -2.100" rpy="${radians(90)} 0 0" />
             <geometry>
                 <mesh filename="package://motoman_gp180_support/meshes/gp180_120/collision/t_axis.stl" scale="0.001 0.001 0.001"/>
@@ -122,5 +121,5 @@
         <origin xyz="0 0 0.317" rpy="0 0 0" />
         <axis xyz="0 0 1" />
-        <limit lower="${-DEG2RAD * 180}" upper="${DEG2RAD * 180}" effort="1300" velocity="${DEG2RAD * 125}"/>
+        <limit lower="${radians(-180)}" upper="${radians(180)}" effort="1300" velocity="${radians(125)}"/>
     </joint>
     <joint name="${prefix}joint_2_l" type="revolute">
@@ -129,5 +128,5 @@
         <origin xyz="-0.325 -0.07 0.333" rpy="0 0 0" />
         <axis xyz="0 -1 0" />
-        <limit lower="${-DEG2RAD * 60}" upper="${DEG2RAD * 76}" effort="1100" velocity="${DEG2RAD * 115}"/>
+        <limit lower="${radians(-60)}" upper="${radians(76)}" effort="1100" velocity="${radians(115)}"/>
     </joint>
     <joint name="${prefix}joint_3_u" type="revolute">
@@ -136,5 +135,5 @@
         <origin xyz="0 0.0285 1.150" rpy="0 0 0" />
         <axis xyz="0 -1 0" />
-        <limit lower="${-DEG2RAD * 86}" upper="${DEG2RAD * 90}" effort="900" velocity="${DEG2RAD * 125}"/>
+        <limit lower="${radians(-86)}" upper="${radians(90)}" effort="900" velocity="${radians(125)}"/>
     </joint>
     <joint name="${prefix}joint_4_r" type="revolute">
@@ -143,5 +142,5 @@
         <origin xyz="-1.398 0.0415 0.300" rpy="0 0 0" />
         <axis xyz="-1 0 0" />
-        <limit lower="${-DEG2RAD * 360}" upper="${DEG2RAD * 360}" effort="883" velocity="${DEG2RAD * 182}"/>
+        <limit lower="${radians(-360)}" upper="${radians(360)}" effort="883" velocity="${radians(182)}"/>
     </joint>
     <joint name="${prefix}joint_5_b" type="revolute">
@@ -150,5 +149,5 @@
         <origin xyz="-0.192 0.082 0" rpy="0 0 0" />
         <axis xyz="0 -1 0" />
-        <limit lower="${-DEG2RAD * 130}" upper="${DEG2RAD * 130}" effort="883" velocity="${DEG2RAD * 175}"/>
+        <limit lower="${radians(-130)}" upper="${radians(130)}" effort="883" velocity="${radians(175)}"/>
     </joint>
     <joint name="${prefix}joint_6_t" type="revolute">
@@ -157,8 +156,8 @@
         <origin xyz="-0.1995 -0.082 0" rpy="0 0 0" />
         <axis xyz="-1 0 0" />
-        <limit lower="${-DEG2RAD * 360}" upper="${DEG2RAD * 360}" effort="520" velocity="${DEG2RAD * 265}"/>
+        <limit lower="${radians(-360)}" upper="${radians(360)}" effort="520" velocity="${radians(265)}"/>
     </joint>
     <joint name="${prefix}joint_6_t-tool0" type="fixed">
-        <origin xyz="-0.0255 0 0" rpy="0 ${-DEG2RAD * 90} 0"/>
+        <origin xyz="-0.0255 0 0" rpy="0 ${radians(-90)} 0"/>
         <parent link="${prefix}link_6_t"/>
         <child link="${prefix}tool0"/>

Commit message: further renamed meshes to have same names as links in URDF

File: motoman_gp180_support/urdf/gp180_120_macro.xacro (robot description, xacro)
@@ -11,5 +11,5 @@
             <origin rpy="${radians(90)} 0 0" />
             <geometry>
-                <mesh filename="package://motoman_gp180_support/meshes/gp180_120/visual/base_axis.stl" scale="0.001 0.001 0.001"/>
+                <mesh filename="package://motoman_gp180_support/meshes/gp180_120/visual/base_link.stl" scale="0.001 0.001 0.001"/>
             </geometry>
             <material name="yaskawa_blue"/>
@@ -18,5 +18,5 @@
             <origin rpy="${radians(90)} 0 0" />
             <geometry>
-                <mesh filename="package://motoman_gp180_support/meshes/gp180_120/collision/base_axis.stl" scale="0.001 0.001 0.001"/>
+                <mesh filename="package://motoman_gp180_support/meshes/gp180_120/collision/base_link.stl" scale="0.001 0.001 0.001"/>
             </geometry>
         </collision>
@@ -26,5 +26,5 @@
             <origin xyz="0 0 -0.317" rpy="${radians(90)} 0 0" />
             <geometry>
-                <mesh filename="package://motoman_gp180_support/meshes/gp180_120/visual/s_axis.stl" scale="0.001 0.001 0.001"/>
+                <mesh filename="package://motoman_gp180_support/meshes/gp180_120/visual/link_1_s.stl" scale="0.001 0.001 0.001"/>
             </geometry>
             <material name="yaskawa_blue"/>
@@ -33,5 +33,5 @@
             <origin xyz="0 0 -0.317" rpy="${radians(90)} 0 0" />
             <geometry>
-                <mesh filename="package://motoman_gp180_support/meshes/gp180_120/collision/s_axis.stl" scale="0.001 0.001 0.001"/>
+                <mesh filename="package://motoman_gp180_support/meshes/gp180_120/collision/link_1_s.stl" scale="0.001 0.001 0.001"/>
             </geometry>
         </collision>
@@ -41,5 +41,5 @@
             <origin xyz="0.325 0.07 -0.650" rpy="${radians(90)} 0 0" />
             <geometry>
-                <mesh filename="package://motoman_gp180_support/meshes/gp180_120/visual/l_axis.stl" scale="0.001 0.001 0.001"/>
+                <mesh filename="package://motoman_gp180_support/meshes/gp180_120/visual/link_2_l.stl" scale="0.001 0.001 0.001"/>
             </geometry>
             <material name="yaskawa_blue"/>
@@ -48,5 +48,5 @@
             <origin xyz="0.325 0.07 -0.650" rpy="${radians(90)} 0 0" />
             <geometry>
-                <mesh filename="package://motoman_gp180_support/meshes/gp180_120/collision/l_axis.stl" scale="0.001 0.001 0.001"/>
+                <mesh filename="package://motoman_gp180_support/meshes/gp180_120/collision/link_2_l.stl" scale="0.001 0.001 0.001"/>
             </geometry>
         </collision>
@@ -56,5 +56,5 @@
             <origin xyz="0.325 0.0415 -1.800" rpy="${radians(90)} 0 0" />
             <geometry>
-                <mesh filename="package://motoman_gp180_support/meshes/gp180_120/visual/u_axis.stl" scale="0.001 0.001 0.001"/>
+                <mesh filename="package://motoman_gp180_support/meshes/gp180_120/visual/link_3_u.stl" scale="0.001 0.001 0.001"/>
             </geometry>
             <material name="yaskawa_blue"/>
@@ -63,5 +63,5 @@
             <origin xyz="0.325 0.0415 -1.800" rpy="${radians(90)} 0 0" />
             <geometry>
-                <mesh filename="package://motoman_gp180_support/meshes/gp180_120/collision/u_axis.stl" scale="0.001 0.001 0.001"/>
+                <mesh filename="package://motoman_gp180_support/meshes/gp180_120/collision/link_3_u.stl" scale="0.001 0.001 0.001"/>
             </geometry>
         </collision>
@@ -71,5 +71,5 @@
             <origin xyz="1.723 0 -2.100" rpy="${radians(90)} 0 0" />
             <geometry>
-                <mesh filename="package://motoman_gp180_support/meshes/gp180_120/visual/r_axis.stl" scale="0.001 0.001 0.001"/>
+                <mesh filename="package://motoman_gp180_support/meshes/gp180_120/visual/link_4_r.stl" scale="0.001 0.001 0.001"/>
             </geometry>
             <material name="yaskawa_blue"/>
@@ -78,5 +78,5 @@
             <origin xyz="1.723 0 -2.100" rpy="${radians(90)} 0 0" />
             <geometry>
-                <mesh filename="package://motoman_gp180_support/meshes/gp180_120/collision/r_axis.stl" scale="0.001 0.001 0.001"/>
+                <mesh filename="package://motoman_gp180_support/meshes/gp180_120/collision/link_4_r.stl" scale="0.001 0.001 0.001"/>
             </geometry>
         </collision>
@@ -86,5 +86,5 @@
             <origin xyz="1.915 -0.082 -2.100" rpy="${radians(90)} 0 0" />
             <geometry>
-                <mesh filename="package://motoman_gp180_support/meshes/gp180_120/visual/b_axis.stl" scale="0.001 0.001 0.001"/>
+                <mesh filename="package://motoman_gp180_support/meshes/gp180_120/visual/link_5_b.stl" scale="0.001 0.001 0.001"/>
             </geometry>
             <material name="yaskawa_blue"/>
@@ -93,5 +93,5 @@
             <origin xyz="1.915 -0.082 -2.100" rpy="${radians(90)} 0 0" />
             <geometry>
-                <mesh filename="package://motoman_gp180_support/meshes/gp180_120/collision/b_axis.stl" scale="0.001 0.001 0.001"/>
+                <mesh filename="package://motoman_gp180_support/meshes/gp180_120/collision/link_5_b.stl" scale="0.001 0.001 0.001"/>
             </geometry>
         </collision>
@@ -101,5 +101,5 @@
             <origin xyz="2.1145 0 -2.100" rpy="${radians(90)} 0 0" />
             <geometry>
-                <mesh filename="package://motoman_gp180_support/meshes/gp180_120/visual/t_axis.stl" scale="0.001 0.001 0.001"/>
+                <mesh filename="package://motoman_gp180_support/meshes/gp180_120/visual/link_6_t.stl" scale="0.001 0.001 0.001"/>
             </geometry>
             <material name="yaskawa_blue"/>
@@ -108,5 +108,5 @@
             <origin xyz="2.1145 0 -2.100" rpy="${radians(90)} 0 0" />
             <geometry>
-                <mesh filename="package://motoman_gp180_support/meshes/gp180_120/collision/t_axis.stl" scale="0.001 0.001 0.001"/>
+                <mesh filename="package://motoman_gp180_support/meshes/gp180_120/collision/link_6_t.stl" scale="0.001 0.001 0.001"/>
             </geometry>
         </collision>

Commit message: scaled and rotated meshes, with origin points translated to correct location; scaling, rotating and translating origin point in URDF no longer needed; added tools directory with script and README file describing automation of the processing of the source meshes (derived from Yaskawa 3D model STEP file)

File: motoman_gp180_support/urdf/gp180_120_macro.xacro (robot description, xacro)
@@ -4,19 +4,18 @@
     <!-- Properties -->
     <material name="yaskawa_blue">
-          <color rgba="0.12941 0.14902 0.74902 1" />
+<!--          <color rgba="0.12941 0.14902 0.74902 1" />-->
+        <color rgba="0 0.35546875 0.671875 1" />
     </material>
     <!-- link list -->
     <link name="${prefix}base_link">
         <visual>
-            <origin rpy="${radians(90)} 0 0" />
             <geometry>
-                <mesh filename="package://motoman_gp180_support/meshes/gp180_120/visual/base_link.stl" scale="0.001 0.001 0.001"/>
+                <mesh filename="package://motoman_gp180_support/meshes/gp180_120/visual/base_link.stl"/>
             </geometry>
             <material name="yaskawa_blue"/>
         </visual>
         <collision>
-            <origin rpy="${radians(90)} 0 0" />
             <geometry>
-                <mesh filename="package://motoman_gp180_support/meshes/gp180_120/collision/base_link.stl" scale="0.001 0.001 0.001"/>
+                <mesh filename="package://motoman_gp180_support/meshes/gp180_120/collision/base_link.stl"/>
             </geometry>
         </collision>
@@ -24,14 +23,12 @@
     <link name="${prefix}link_1_s">
         <visual>
-            <origin xyz="0 0 -0.317" rpy="${radians(90)} 0 0" />
             <geometry>
-                <mesh filename="package://motoman_gp180_support/meshes/gp180_120/visual/link_1_s.stl" scale="0.001 0.001 0.001"/>
+                <mesh filename="package://motoman_gp180_support/meshes/gp180_120/visual/link_1_s.stl"/>
             </geometry>
             <material name="yaskawa_blue"/>
         </visual>
         <collision>
-            <origin xyz="0 0 -0.317" rpy="${radians(90)} 0 0" />
             <geometry>
-                <mesh filename="package://motoman_gp180_support/meshes/gp180_120/collision/link_1_s.stl" scale="0.001 0.001 0.001"/>
+                <mesh filename="package://motoman_gp180_support/meshes/gp180_120/collision/link_1_s.stl"/>
             </geometry>
         </collision>
@@ -39,14 +36,12 @@
     <link name="${prefix}link_2_l">
         <visual>
-            <origin xyz="0.325 0.07 -0.650" rpy="${radians(90)} 0 0" />
             <geometry>
-                <mesh filename="package://motoman_gp180_support/meshes/gp180_120/visual/link_2_l.stl" scale="0.001 0.001 0.001"/>
+                <mesh filename="package://motoman_gp180_support/meshes/gp180_120/visual/link_2_l.stl"/>
             </geometry>
             <material name="yaskawa_blue"/>
         </visual>
         <collision>
-            <origin xyz="0.325 0.07 -0.650" rpy="${radians(90)} 0 0" />
             <geometry>
-                <mesh filename="package://motoman_gp180_support/meshes/gp180_120/collision/link_2_l.stl" scale="0.001 0.001 0.001"/>
+                <mesh filename="package://motoman_gp180_support/meshes/gp180_120/collision/link_2_l.stl"/>
             </geometry>
         </collision>
@@ -54,14 +49,12 @@
     <link name="${prefix}link_3_u">
         <visual>
-            <origin xyz="0.325 0.0415 -1.800" rpy="${radians(90)} 0 0" />
             <geometry>
-                <mesh filename="package://motoman_gp180_support/meshes/gp180_120/visual/link_3_u.stl" scale="0.001 0.001 0.001"/>
+                <mesh filename="package://motoman_gp180_support/meshes/gp180_120/visual/link_3_u.stl"/>
             </geometry>
             <material name="yaskawa_blue"/>
         </visual>
         <collision>
-            <origin xyz="0.325 0.0415 -1.800" rpy="${radians(90)} 0 0" />
             <geometry>
-                <mesh filename="package://motoman_gp180_support/meshes/gp180_120/collision/link_3_u.stl" scale="0.001 0.001 0.001"/>
+                <mesh filename="package://motoman_gp180_support/meshes/gp180_120/collision/link_3_u.stl"/>
             </geometry>
         </collision>
@@ -69,14 +62,12 @@
     <link name="${prefix}link_4_r">
         <visual>
-            <origin xyz="1.723 0 -2.100" rpy="${radians(90)} 0 0" />
             <geometry>
-                <mesh filename="package://motoman_gp180_support/meshes/gp180_120/visual/link_4_r.stl" scale="0.001 0.001 0.001"/>
+                <mesh filename="package://motoman_gp180_support/meshes/gp180_120/visual/link_4_r.stl"/>
             </geometry>
             <material name="yaskawa_blue"/>
         </visual>
         <collision>
-            <origin xyz="1.723 0 -2.100" rpy="${radians(90)} 0 0" />
             <geometry>
-                <mesh filename="package://motoman_gp180_support/meshes/gp180_120/collision/link_4_r.stl" scale="0.001 0.001 0.001"/>
+                <mesh filename="package://motoman_gp180_support/meshes/gp180_120/collision/link_4_r.stl"/>
             </geometry>
         </collision>
@@ -84,14 +75,12 @@
     <link name="${prefix}link_5_b">
         <visual>
-            <origin xyz="1.915 -0.082 -2.100" rpy="${radians(90)} 0 0" />
             <geometry>
-                <mesh filename="package://motoman_gp180_support/meshes/gp180_120/visual/link_5_b.stl" scale="0.001 0.001 0.001"/>
+                <mesh filename="package://motoman_gp180_support/meshes/gp180_120/visual/link_5_b.stl"/>
             </geometry>
             <material name="yaskawa_blue"/>
         </visual>
         <collision>
-            <origin xyz="1.915 -0.082 -2.100" rpy="${radians(90)} 0 0" />
             <geometry>
-                <mesh filename="package://motoman_gp180_support/meshes/gp180_120/collision/link_5_b.stl" scale="0.001 0.001 0.001"/>
+                <mesh filename="package://motoman_gp180_support/meshes/gp180_120/collision/link_5_b.stl"/>
             </geometry>
         </collision>
@@ -99,14 +88,12 @@
     <link name="${prefix}link_6_t">
         <visual>
-            <origin xyz="2.1145 0 -2.100" rpy="${radians(90)} 0 0" />
             <geometry>
-                <mesh filename="package://motoman_gp180_support/meshes/gp180_120/visual/link_6_t.stl" scale="0.001 0.001 0.001"/>
+                <mesh filename="package://motoman_gp180_support/meshes/gp180_120/visual/link_6_t.stl"/>
             </geometry>
             <material name="yaskawa_blue"/>
         </visual>
         <collision>
-            <origin xyz="2.1145 0 -2.100" rpy="${radians(90)} 0 0" />
             <geometry>
-                <mesh filename="package://motoman_gp180_support/meshes/gp180_120/collision/link_6_t.stl" scale="0.001 0.001 0.001"/>
+                <mesh filename="package://motoman_gp180_support/meshes/gp180_120/collision/link_6_t.stl"/>
             </geometry>
         </collision>
