Commit message: shifted meshes origin points and joints origin translations so that the joints are "in line" with only one axis translation between two neighboring joints (exception is link_3_u for upper arm, there is 2-axis translation)

File: motoman_gp180_support/urdf/gp180_120_macro.xacro (robot description, xacro)
@@ -106,5 +106,5 @@
         <parent link="${prefix}base_link"/>
         <child link="${prefix}link_1_s"/>
-        <origin xyz="0 0 0.317" rpy="0 0 0" />
+        <origin xyz="0 0 0.650" rpy="0 0 0" />
         <axis xyz="0 0 1" />
         <limit lower="${radians(-180)}" upper="${radians(180)}" effort="1300" velocity="${radians(125)}"/>
@@ -113,5 +113,5 @@
         <parent link="${prefix}link_1_s"/>
         <child link="${prefix}link_2_l"/>
-        <origin xyz="-0.325 -0.07 0.333" rpy="0 0 0" />
+        <origin xyz="-0.325 0 0" rpy="0 0 0" />
         <axis xyz="0 -1 0" />
         <limit lower="${radians(-60)}" upper="${radians(76)}" effort="1100" velocity="${radians(115)}"/>
@@ -120,5 +120,5 @@
         <parent link="${prefix}link_2_l"/>
         <child link="${prefix}link_3_u"/>
-        <origin xyz="0 0.0285 1.150" rpy="0 0 0" />
+        <origin xyz="0 0 1.150" rpy="0 0 0" />
         <axis xyz="0 -1 0" />
         <limit lower="${radians(-86)}" upper="${radians(90)}" effort="900" velocity="${radians(125)}"/>
@@ -127,5 +127,5 @@
         <parent link="${prefix}link_3_u"/>
         <child link="${prefix}link_4_r"/>
-        <origin xyz="-1.398 0.0415 0.300" rpy="0 0 0" />
+        <origin xyz="-1.398 0 0.300" rpy="0 0 0" />
         <axis xyz="-1 0 0" />
         <limit lower="${radians(-360)}" upper="${radians(360)}" effort="883" velocity="${radians(182)}"/>
@@ -134,5 +134,5 @@
         <parent link="${prefix}link_4_r"/>
         <child link="${prefix}link_5_b"/>
-        <origin xyz="-0.192 0.082 0" rpy="0 0 0" />
+        <origin xyz="-0.192 0 0" rpy="0 0 0" />
         <axis xyz="0 -1 0" />
         <limit lower="${radians(-130)}" upper="${radians(130)}" effort="883" velocity="${radians(175)}"/>
@@ -141,5 +141,5 @@
         <parent link="${prefix}link_5_b"/>
         <child link="${prefix}link_6_t"/>
-        <origin xyz="-0.1995 -0.082 0" rpy="0 0 0" />
+        <origin xyz="-0.1995 0 0" rpy="0 0 0" />
         <axis xyz="-1 0 0" />
         <limit lower="${radians(-360)}" upper="${radians(360)}" effort="520" velocity="${radians(265)}"/>

Commit message: Correction on urdf and model orientation and direction of motion.
The URDF was changed to rotate the whole model so that the X-axis point forward and kinematic model adjusted to match the standard Yaskawa model and dimensions.  The mesh were then adjusted to realign properly with the new kinematic model.  The direction of motion for each axis was also corrected to match the real robot motion.  Finally, the visual meshes were reduce by 50% to reduce the display processing.

File: motoman_gp180_support/urdf/gp180_120_macro.xacro (robot description, xacro)
@@ -113,6 +113,6 @@
         <parent link="${prefix}link_1_s"/>
         <child link="${prefix}link_2_l"/>
-        <origin xyz="-0.325 0 0" rpy="0 0 0" />
-        <axis xyz="0 -1 0" />
+        <origin xyz="0.325 0 0" rpy="0 0 0" />
+        <axis xyz="0 1 0" />
         <limit lower="${radians(-60)}" upper="${radians(76)}" effort="1100" velocity="${radians(115)}"/>
     </joint>
@@ -127,5 +127,5 @@
         <parent link="${prefix}link_3_u"/>
         <child link="${prefix}link_4_r"/>
-        <origin xyz="-1.398 0 0.300" rpy="0 0 0" />
+        <origin xyz="1.590 0 0.300" rpy="0 0 0" />
         <axis xyz="-1 0 0" />
         <limit lower="${radians(-360)}" upper="${radians(360)}" effort="883" velocity="${radians(182)}"/>
@@ -134,5 +134,5 @@
         <parent link="${prefix}link_4_r"/>
         <child link="${prefix}link_5_b"/>
-        <origin xyz="-0.192 0 0" rpy="0 0 0" />
+        <origin xyz="0 0 0" rpy="0 0 0" />
         <axis xyz="0 -1 0" />
         <limit lower="${radians(-130)}" upper="${radians(130)}" effort="883" velocity="${radians(175)}"/>
@@ -141,10 +141,10 @@
         <parent link="${prefix}link_5_b"/>
         <child link="${prefix}link_6_t"/>
-        <origin xyz="-0.1995 0 0" rpy="0 0 0" />
+        <origin xyz="0 0 0" rpy="0 0 0" />
         <axis xyz="-1 0 0" />
         <limit lower="${radians(-360)}" upper="${radians(360)}" effort="520" velocity="${radians(265)}"/>
     </joint>
     <joint name="${prefix}joint_6_t-tool0" type="fixed">
-        <origin xyz="-0.0255 0 0" rpy="0 ${radians(-90)} 0"/>
+        <origin xyz="0.225 0 0" rpy="${radians(180)} ${radians(-90)} 0"/>
         <parent link="${prefix}link_6_t"/>
         <child link="${prefix}tool0"/>
@@ -155,5 +155,5 @@
     <link name="${prefix}base" />
     <joint name="${prefix}base_link-base" type="fixed">
-        <origin xyz="0 0 0.317" rpy="0 0 0"/>
+        <origin xyz="0 0 0.650" rpy="0 0 0"/>
         <parent link="${prefix}base_link"/>
         <child link="${prefix}base"/>

Commit message: updated effort limits to Max Acc/Dec Torque [Nm] values from spreadsheet provided by Eric Marcil

File: motoman_gp180_support/urdf/gp180_120_macro.xacro (robot description, xacro)
@@ -4,5 +4,4 @@
     <!-- Properties -->
     <material name="yaskawa_blue">
-<!--          <color rgba="0.12941 0.14902 0.74902 1" />-->
         <color rgba="0 0.35546875 0.671875 1" />
     </material>
@@ -108,5 +107,5 @@
         <origin xyz="0 0 0.650" rpy="0 0 0" />
         <axis xyz="0 0 1" />
-        <limit lower="${radians(-180)}" upper="${radians(180)}" effort="1300" velocity="${radians(125)}"/>
+        <limit lower="${radians(-180)}" upper="${radians(180)}" effort="9414.38" velocity="${radians(125)}"/>
     </joint>
     <joint name="${prefix}joint_2_l" type="revolute">
@@ -115,5 +114,5 @@
         <origin xyz="0.325 0 0" rpy="0 0 0" />
         <axis xyz="0 1 0" />
-        <limit lower="${radians(-60)}" upper="${radians(76)}" effort="1100" velocity="${radians(115)}"/>
+        <limit lower="${radians(-60)}" upper="${radians(76)}" effort="11645.4" velocity="${radians(115)}"/>
     </joint>
     <joint name="${prefix}joint_3_u" type="revolute">
@@ -122,5 +121,5 @@
         <origin xyz="0 0 1.150" rpy="0 0 0" />
         <axis xyz="0 -1 0" />
-        <limit lower="${radians(-86)}" upper="${radians(90)}" effort="900" velocity="${radians(125)}"/>
+        <limit lower="${radians(-86)}" upper="${radians(90)}" effort="7060.79" velocity="${radians(125)}"/>
     </joint>
     <joint name="${prefix}joint_4_r" type="revolute">
@@ -129,5 +128,5 @@
         <origin xyz="1.590 0 0.300" rpy="0 0 0" />
         <axis xyz="-1 0 0" />
-        <limit lower="${radians(-360)}" upper="${radians(360)}" effort="883" velocity="${radians(182)}"/>
+        <limit lower="${radians(-360)}" upper="${radians(360)}" effort="1392.54" velocity="${radians(182)}"/>
     </joint>
     <joint name="${prefix}joint_5_b" type="revolute">
@@ -136,5 +135,5 @@
         <origin xyz="0 0 0" rpy="0 0 0" />
         <axis xyz="0 -1 0" />
-        <limit lower="${radians(-130)}" upper="${radians(130)}" effort="883" velocity="${radians(175)}"/>
+        <limit lower="${radians(-130)}" upper="${radians(130)}" effort="1863.26" velocity="${radians(175)}"/>
     </joint>
     <joint name="${prefix}joint_6_t" type="revolute">
@@ -143,5 +142,5 @@
         <origin xyz="0 0 0" rpy="0 0 0" />
         <axis xyz="-1 0 0" />
-        <limit lower="${radians(-360)}" upper="${radians(360)}" effort="520" velocity="${radians(265)}"/>
+        <limit lower="${radians(-360)}" upper="${radians(360)}" effort="926.73" velocity="${radians(265)}"/>
     </joint>
     <joint name="${prefix}joint_6_t-tool0" type="fixed">

Commit message: Split J4->J5 transform into two.
This avoids translations in two dimensions for 'joint_4_r'.

File: motoman_gp180_support/urdf/gp180_120_macro.xacro (robot description, xacro)
@@ -125,5 +125,5 @@
         <parent link="${prefix}link_3_u"/>
         <child link="${prefix}link_4_r"/>
-        <origin xyz="1.590 0 0.300" rpy="0 0 0" />
+        <origin xyz="0 0 0.300" rpy="0 0 0" />
         <axis xyz="-1 0 0" />
         <limit lower="${radians(-360)}" upper="${radians(360)}" effort="1392.54" velocity="${radians(182)}"/>
@@ -132,5 +132,5 @@
         <parent link="${prefix}link_4_r"/>
         <child link="${prefix}link_5_b"/>
-        <origin xyz="0 0 0" rpy="0 0 0" />
+        <origin xyz="1.590 0 0" rpy="0 0 0" />
         <axis xyz="0 -1 0" />
         <limit lower="${radians(-130)}" upper="${radians(130)}" effort="1863.26" velocity="${radians(175)}"/>

Commit message: Place tool0 on flange.
So move final translation (from J5->J6) and make J6->tool0 transform identity.

File: motoman_gp180_support/urdf/gp180_120_macro.xacro (robot description, xacro)
@@ -139,10 +139,10 @@
         <parent link="${prefix}link_5_b"/>
         <child link="${prefix}link_6_t"/>
-        <origin xyz="0 0 0" rpy="0 0 0" />
+        <origin xyz="0.225 0 0" rpy="0 0 0" />
         <axis xyz="-1 0 0" />
         <limit lower="${radians(-360)}" upper="${radians(360)}" effort="926.73" velocity="${radians(265)}"/>
     </joint>
     <joint name="${prefix}joint_6_t-tool0" type="fixed">
-        <origin xyz="0.225 0 0" rpy="${radians(180)} ${radians(-90)} 0"/>
+        <origin xyz="0 0 0" rpy="${radians(180)} ${radians(-90)} 0"/>
         <parent link="${prefix}link_6_t"/>
         <child link="${prefix}tool0"/>
