Commit message: Changed GP180 to use motoman_resources. Made gp180 test use joint_state_publisher_gui.

File: motoman_gp180_support/urdf/gp180_macro.xacro (robot description, xacro)
@@ -2,8 +2,5 @@
 <robot xmlns:xacro="http://ros.org/wiki/xacro">
 <xacro:macro name="motoman_gp180" params="prefix">
-    <!-- Properties -->
-    <material name="yaskawa_blue">
-        <color rgba="0 0.35546875 0.671875 1" />
-    </material>
+    <xacro:include filename="$(find motoman_resources)/urdf/common_materials.xacro"/>
     <!-- link list -->
     <link name="${prefix}base_link">
@@ -12,5 +9,5 @@
                 <mesh filename="package://motoman_gp180_support/meshes/gp180_120/visual/base_link.stl"/>
             </geometry>
-            <material name="yaskawa_blue"/>
+            <xacro:material_yaskawa_blue/>
         </visual>
         <collision>
@@ -25,5 +22,5 @@
                 <mesh filename="package://motoman_gp180_support/meshes/gp180_120/visual/link_1_s.stl"/>
             </geometry>
-            <material name="yaskawa_blue"/>
+            <xacro:material_yaskawa_blue/>
         </visual>
         <collision>
@@ -38,5 +35,5 @@
                 <mesh filename="package://motoman_gp180_support/meshes/gp180_120/visual/link_2_l.stl"/>
             </geometry>
-            <material name="yaskawa_blue"/>
+            <xacro:material_yaskawa_blue/>
         </visual>
         <collision>
@@ -51,5 +48,5 @@
                 <mesh filename="package://motoman_gp180_support/meshes/gp180/visual/link_3_u.stl"/>
             </geometry>
-            <material name="yaskawa_blue"/>
+            <xacro:material_yaskawa_blue/>
         </visual>
         <collision>
@@ -64,5 +61,5 @@
                 <mesh filename="package://motoman_gp180_support/meshes/gp180/visual/link_4_r.stl"/>
             </geometry>
-            <material name="yaskawa_blue"/>
+            <xacro:material_yaskawa_blue/>
         </visual>
         <collision>
@@ -77,5 +74,5 @@
                 <mesh filename="package://motoman_gp180_support/meshes/gp180_120/visual/link_5_b.stl"/>
             </geometry>
-            <material name="yaskawa_blue"/>
+            <xacro:material_yaskawa_blue/>
         </visual>
         <collision>
@@ -90,5 +87,5 @@
                 <mesh filename="package://motoman_gp180_support/meshes/gp180_120/visual/link_6_t.stl"/>
             </geometry>
-            <material name="yaskawa_blue"/>
+            <xacro:material_yaskawa_blue/>
         </visual>
         <collision>

Commit message: Modified GP180 to more closely match RoboDK

File: motoman_gp180_support/urdf/gp180_macro.xacro (robot description, xacro)
@@ -62,5 +62,5 @@
     <link name="${prefix}link_4_r">
         <visual>
-            <origin rpy="${radians(0)} ${radians(90)} ${radians(0)}" />
+            <origin rpy="${radians(0)} ${radians(90)} ${radians(0)}" xyz="0 0 1.225"/>
             <geometry>
                 <mesh filename="package://motoman_gp180_support/meshes/gp180/visual/link_4_r.stl"/>
@@ -131,5 +131,5 @@
         <parent link="${prefix}link_3_u"/>
         <child link="${prefix}link_4_r"/>
-        <origin xyz="0.300 0 0" rpy="${radians(-90)} 0 0" />
+        <origin xyz="0.300 -1.225 0" rpy="${radians(-90)} 0 0" />
         <axis xyz="0 0 1" />
         <limit lower="${radians(-360)}" upper="${radians(360)}" effort="1671.05" velocity="${radians(182)}"/>
@@ -138,5 +138,5 @@
         <parent link="${prefix}link_4_r"/>
         <child link="${prefix}link_5_b"/>
-        <origin xyz="0 0 -1.225" rpy="${radians(90)} 0 0" />
+        <origin xyz="0 0 0" rpy="${radians(90)} 0 0" />
         <axis xyz="0 0 1" />
         <limit lower="${radians(-130)}" upper="${radians(130)}" effort="1081.18" velocity="${radians(175)}"/>

Commit message: Fixed bug with GP180 collision model.

File: motoman_gp180_support/urdf/gp180_macro.xacro (robot description, xacro)
@@ -69,5 +69,5 @@
         </visual>
         <collision>
-            <origin rpy="${radians(0)} ${radians(90)} ${radians(0)}" />
+            <origin rpy="${radians(0)} ${radians(90)} ${radians(0)}" xyz="0 0 1.225"/>
             <geometry>
                 <mesh filename="package://motoman_gp180_support/meshes/gp180/collision/link_4_r.stl"/>
