Commit message: WIP - Add combined ma1440 and d500 packages This adds a new package in motoman representing a combined robotic system with an ma1440 arm along with a d500 positioner. In its current state still needs some work to define the world link and where the components are relative to the world, currently just hardcoded values

File: motoman_ma1440_support/urdf/cam_mount/cam_mount.xacro (robot description, xacro)
@@ -3,10 +3,4 @@
   <!-- Constants for robot dimensions -->
   <xacro:property name="M_PI" value="3.1415926535897931"/>
-<!--  <joint name="joint_cam_mount" type="fixed">-->
-<!--    <origin xyz="0 0 -0.0735" rpy="${M_PI} 0 ${M_PI/2}" />-->
-<!--    <parent link="t_link" />-->
-<!--    <child link="cam_mount_link" />-->
-<!--    <axis xyz="0 0 0" />-->
-<!--  </joint>-->
   <link name="cam_mount_link">
     <visual>

File: motoman_ma1440_support/urdf/ma1440/ma1440.xacro (robot description, xacro)
@@ -1,5 +1,5 @@
 <?xml version="1.0" ?>
 <robot name="motoman_ma1440" xmlns:xacro="http://ros.org/wiki/xacro">
-    <xacro:arg name="cam_mount" default="true"/>
+    <xacro:arg name="cam_mount" default="false"/>
     <xacro:include filename="$(find motoman_ma1440_support)/urdf/ma1440/ma1440_macro.xacro" />
     <xacro:motoman_ma1440 prefix=""/>

File: motoman_ma1440_support/urdf/ma1440/ma1440_macro.xacro (robot description, xacro)
@@ -236,8 +236,8 @@
         <!-- end of link list -->
         <!-- joint list -->
-        <joint name="world-base" type="fixed">
+        <joint name="${prefix}world-base" type="fixed">
             <origin xyz="0 0 0" rpy="0 0 0"/>
             <parent link="world" />
-            <child link="base_link"/>
+            <child link="${prefix}base_link"/>
         </joint>
         <joint name="${prefix}joint_s" type="revolute">

File: motoman_motopos_d500_support/urdf/motopos_d500_macro.xacro (robot description, xacro)
@@ -45,4 +45,9 @@
   <!-- end of link list -->
   <!-- joint list -->
+  <joint name="${prefix}world-base" type="fixed">
+      <origin xyz="1 0 0" rpy="0 0 0"/>
+      <parent link="world" />
+      <child link="${prefix}base_link"/>
+  </joint>
   <joint name="joint_1" type="revolute">
     <parent link="${prefix}base_link"/>
@@ -69,5 +74,5 @@
   <!-- ROS base_link to Robot Manufacturer World Coordinates transform -->
   <link name="${prefix}base" />
-  <joint name="base_link-base" type="fixed">
+  <joint name="${prefix}base_link-base" type="fixed">
     <origin xyz="0 0 0.380" rpy="0 0 0"/>
     <parent link="${prefix}base_link"/>
