Commit message: FR-195 FR-309 WIP testing the mh185 stuff. Changed name/moved table top stls into separate folder.

File: motoman_motopos_mh185_vertical_support/urdf/motopos_mh185_vertical.xacro (robot description, xacro)
@@ -2,10 +2,16 @@
 <robot name="motoman_motopos_mh185_vertical" xmlns:xacro="http://ros.org/wiki/xacro">
   <!-- Properties -->
-  <material name="yaskawa_blue">
-      <color rgba="0.12941 0.14902 0.74902 1" />
-  </material>
+<!--  <material name="yaskawa_blue">-->
+<!--      <color rgba="0.12941 0.14902 0.74902 1" />-->
+<!--  </material>-->
+<!--  <xacro:property name="M_PI" value="3.1415926535897931"/>-->
+<!--  <xacro:property name="world_base_xyz" value="0 0 0"/>-->
+<!--  <xacro:property name="world_base_rpy" value="0 0 0"/>-->
   <xacro:include filename="$(find motoman_motopos_mh185_vertical_support)/urdf/motopos_mh185_vertical.transmission.xacro" />
   <xacro:include filename="$(find motoman_motopos_mh185_vertical_support)/urdf/motopos_mh185_vertical_macro.xacro" />
   <xacro:macro name="load_motoman_motopos_mh185_vertical" params="prefix:=mh185_vertical_ world_base_xyz world_base_rpy">
+    <material name="yaskawa_blue">
+      <color rgba="0.12941 0.14902 0.74902 1" />
+    </material>
     <xacro:motoman_motopos_mh185_vertical prefix="${prefix}" world_base_xyz="${world_base_xyz}" world_base_rpy="${world_base_rpy}"/>
   </xacro:macro>

File: motoman_motopos_mh185_vertical_support/urdf/motopos_mh185_vertical_macro.xacro (robot description, xacro)
@@ -18,4 +18,5 @@
     </visual>
     <collision>
+      <origin xyz="-0.083 -0.0245 -.32" rpy="0 ${-90*M_PI/180} 0 " />
       <geometry>
         <mesh filename="package://motoman_motopos_mh185_vertical_support/meshes/mh185_vertical/collision/Full_Assembly.stl"/>
@@ -33,8 +34,8 @@
   </link>
   <!-- this is here to set a base link in the URDF to link the "positioner/base" frame to for scanning -->
-  <link name="positioner_base_dummy_link"/>
+<!--  <link name="positioner_base_dummy_link"/>-->
   <!-- this is here to set a base link in the URDF to link the "positioner/center" frame to for scanning. this is equivalent to the tool frame
   in this case, but we define this so that the naming is consistent across positioner setups -->
-  <link name="positioner_center_dummy_link"/>
+<!--  <link name="positioner_center_dummy_link"/>  -->
   <!-- end of link list -->
   <!-- joint list -->
@@ -61,5 +62,5 @@
     <visual>
       <geometry>
-        <mesh filename="package://motoman_motopos_mh185_vertical_support/meshes/mh185_vertical/visual/Vertical_Table_Top.stl" scale="0.001 0.001 0.001"/>
+        <mesh filename="package://motoman_motopos_mh185_vertical_support/meshes/table_top/visual/table_top.stl" scale="0.001 0.001 0.001"/>
       </geometry>
       <origin xyz="0 0 0" rpy="0 0 0 " />
@@ -70,5 +71,5 @@
     <collision>
       <geometry>
-        <mesh filename="package://motoman_motopos_mh185_vertical_support/meshes/mh185_vertical/collision/Vertical_Table_Top.stl" scale="0.001 0.001 0.001"/>
+        <mesh filename="package://motoman_motopos_mh185_vertical_support/meshes/table_top/collision/table_top.stl" scale="0.001 0.001 0.001"/>
       </geometry>
     </collision>
@@ -80,14 +81,14 @@
   </joint>
   <!--  TODO: Not sure what these are-->
-  <joint name="positioner_base_dummy_joint" type="fixed">
-    <origin xyz="0 0 0" rpy="0 0 0"/>
-    <parent link="${prefix}link_1"/>
-    <child link="positioner_base_dummy_link"/>
-  </joint>
-  <joint name="positioner_center_dummy_joint" type="fixed">
-    <origin xyz="0 0 0" rpy="0 0 0"/>
-    <parent link="${prefix}tool0"/>
-    <child link="positioner_center_dummy_link"/>
-  </joint>
+<!--  <joint name="positioner_base_dummy_joint" type="fixed">-->
+<!--    <origin xyz="0 0 0" rpy="0 0 0"/>-->
+<!--    <parent link="${prefix}link_1"/>-->
+<!--    <child link="positioner_base_dummy_link"/>-->
+<!--  </joint>-->
+<!--  <joint name="positioner_center_dummy_joint" type="fixed">-->
+<!--    <origin xyz="0 0 0" rpy="0 0 0"/>-->
+<!--    <parent link="${prefix}tool0"/>-->
+<!--    <child link="positioner_center_dummy_link"/>-->
+<!--  </joint>    -->
   <!-- end of joint list -->
   <!-- ROS base_link to Robot Manufacturer World Coordinates transform -->
