Commit message: FR-195 FR-309 FR-310 FR-311 Bugfixes and setting changes. Mostly naming issues (d500 -> mh185_vertical). Removed dummy links on mh185 xacro, changed it to make the positioner center/base links directly.

File: motoman_ma1440_mh185_vertical_support/test/ma1440_mh185_vertical_test.xacro (robot description, xacro)
@@ -1,4 +1,4 @@
 <?xml version="1.0" ?>
-<robot name="motoman_ma1440_d500_test" xmlns:xacro="http://ros.org/wiki/xacro">
+<robot name="motoman_ma1440_mh185_vertical_test" xmlns:xacro="http://ros.org/wiki/xacro">
   <xacro:include filename="$(find motoman_ma1440_mh185_vertical_support)/urdf/ma1440_mh185_vertical_macro.xacro" />
   <xacro:motoman_ma1440_mh185_vertical prefix="arm"/>

File: motoman_motopos_mh185_vertical_support/urdf/motopos_mh185_vertical_macro.xacro (robot description, xacro)
@@ -31,8 +31,8 @@
   </link>
   <!-- this is here to set a base link in the URDF to link the "positioner/base" frame to for scanning -->
-<!--  <link name="positioner_base_dummy_link"/>-->
+  <link name="positioner/base_link"/>
   <!-- this is here to set a base link in the URDF to link the "positioner/center" frame to for scanning. this is equivalent to the tool frame
   in this case, but we define this so that the naming is consistent across positioner setups -->
-<!--  <link name="positioner_center_dummy_link"/>  -->
+  <link name="positioner/center_link"/>
   <!-- end of link list -->
   <!-- joint list -->
@@ -77,15 +77,15 @@
     <child link="${prefix}table"/>
   </joint>
-  <!--  TODO: Not sure what these are-->
-<!--  <joint name="positioner_base_dummy_joint" type="fixed">-->
-<!--    <origin xyz="0 0 0" rpy="0 0 0"/>-->
-<!--    <parent link="${prefix}link_1"/>-->
-<!--    <child link="positioner_base_dummy_link"/>-->
-<!--  </joint>-->
-<!--  <joint name="positioner_center_dummy_joint" type="fixed">-->
-<!--    <origin xyz="0 0 0" rpy="0 0 0"/>-->
-<!--    <parent link="${prefix}tool0"/>-->
-<!--    <child link="positioner_center_dummy_link"/>-->
-<!--  </joint>    -->
+  <joint name="positioner/center" type="fixed">
+    <origin xyz="0 0 0" rpy="0 0 0"/>
+    <parent link="${prefix}table"/>
+    <child link="positioner/base_link"/>
+  </joint>
+<!--  TODO: Make this offset more dynamic. Two args added together maybe? -->
+  <joint name="positioner/base" type="fixed">
+    <origin xyz="0 0 0.5295" rpy="0 0 0"/>
+    <parent link="${prefix}base_link"/>
+    <child link="positioner/center_link"/>
+  </joint>
   <!-- end of joint list -->
   <!-- ROS base_link to Robot Manufacturer World Coordinates transform -->
