Commit message: FR-338 Can now specify ma1440 joint offsets for vertical positioner.

File: motoman_ma1440_d500_support/urdf/ma1440_d500_macro.xacro (robot description, xacro)
@@ -10,5 +10,6 @@
           table_thickness
           using_cam_mount
-          offsets_file_path">
+          offsets_file_path"
+  >
     <xacro:include filename="$(find motoman_ma1440_support)/urdf/ma1440/ma1440.xacro"/>
     <xacro:load_motoman_ma1440

File: motoman_ma1440_mh185_vertical_support/urdf/ma1440_mh185_vertical.xacro (robot description, xacro)
@@ -1,10 +1,18 @@
 <?xml version="1.0" ?>
  <robot name="motoman_ma1440_mh185_vertical" xmlns:xacro="http://ros.org/wiki/xacro">
-	<xacro:property name="ma1440_xyz" value="$(arg ma1440_xyz)"/>
-	<xacro:property name="ma1440_rpy" value="$(arg ma1440_rpy)"/>
-	<xacro:property name="mh185_vertical_xyz" value="$(arg mh185_vertical_xyz)"/>
-	<xacro:property name="mh185_vertical_rpy" value="$(arg mh185_vertical_rpy)"/>
-	<xacro:property name="using_cam_mount" value="$(arg using_cam_mount)"/>
+	<xacro:arg name="ma1440_xyz" default=""/>
+	<xacro:arg name="ma1440_rpy" default=""/>
+	<xacro:arg name="mh185_vertical_xyz" default=""/>
+	<xacro:arg name="mh185_vertical_rpy" default=""/>
+	<xacro:arg name="using_cam_mount" default=""/>
+	<xacro:arg name="offsets_file_path" default=""/>
 	<xacro:include filename="$(find motoman_ma1440_mh185_vertical_support)/urdf/ma1440_mh185_vertical_macro.xacro" />
-	<xacro:motoman_ma1440_mh185_vertical/>
+	<xacro:motoman_ma1440_mh185_vertical
+			ma1440_xyz="$(arg ma1440_xyz)"
+			ma1440_rpy="$(arg ma1440_rpy)"
+			mh185_vertical_xyz="$(arg mh185_vertical_xyz)"
+			mh185_vertical_rpy="$(arg mh185_vertical_rpy)"
+			using_cam_mount="$(arg using_cam_mount)"
+			offsets_file_path="$(arg offsets_file_path)"
+	/>
 </robot>

File: motoman_ma1440_mh185_vertical_support/urdf/ma1440_mh185_vertical_macro.xacro (robot description, xacro)
@@ -1,7 +1,21 @@
 <?xml version="1.0" ?>
 <robot name="motoman_ma1440_mh185_vertical" xmlns:xacro="http://ros.org/wiki/xacro">
-  <xacro:macro name="motoman_ma1440_mh185_vertical" params="ma1440_xyz:=^ ma1440_rpy:=^ mh185_vertical_xyz:=^ mh185_vertical_rpy:=^ using_cam_mount:=^">
+  <xacro:macro
+      name="motoman_ma1440_mh185_vertical"
+      params=
+          "ma1440_xyz
+          ma1440_rpy
+          mh185_vertical_xyz
+          mh185_vertical_rpy
+          using_cam_mount
+          offsets_file_path"
+  >
     <xacro:include filename="$(find motoman_ma1440_support)/urdf/ma1440/ma1440.xacro"/>
-    <xacro:load_motoman_ma1440 world_base_xyz="${ma1440_xyz}" world_base_rpy="${ma1440_rpy}" using_cam_mount="${using_cam_mount}"/>
+    <xacro:load_motoman_ma1440
+        world_base_xyz="${ma1440_xyz}"
+        world_base_rpy="${ma1440_rpy}"
+        using_cam_mount="${using_cam_mount}"
+        offsets_file_path="${offsets_file_path}"
+    />
     <xacro:include filename="$(find motoman_motopos_mh185_vertical_support)/urdf/motopos_mh185_vertical.xacro" />
     <xacro:load_motoman_motopos_mh185_vertical world_base_xyz="${mh185_vertical_xyz}" world_base_rpy="${mh185_vertical_rpy}"/>

Commit message: FR-338 Added workflow to positioners to load joint offsets. Does not currently use the offsets anywhere.

File: motoman_ma1440_d500_support/urdf/ma1440_d500_macro.xacro (robot description, xacro)
@@ -20,5 +20,10 @@
     />
     <xacro:include filename="$(find motoman_motopos_d500_support)/urdf/motopos_d500.xacro"/>
-    <xacro:load_motoman_motopos_d500 world_base_xyz="${d500_xyz}" world_base_rpy="${d500_rpy}" table_thickness="${table_thickness}"/>
+    <xacro:load_motoman_motopos_d500
+        world_base_xyz="${d500_xyz}"
+        world_base_rpy="${d500_rpy}"
+        table_thickness="${table_thickness}"
+        offsets_file_path="${offsets_file_path}"
+    />
   </xacro:macro>
 </robot>

File: motoman_ma1440_mh185_vertical_support/urdf/ma1440_mh185_vertical_macro.xacro (robot description, xacro)
@@ -19,5 +19,9 @@
     />
     <xacro:include filename="$(find motoman_motopos_mh185_vertical_support)/urdf/motopos_mh185_vertical.xacro" />
-    <xacro:load_motoman_motopos_mh185_vertical world_base_xyz="${mh185_vertical_xyz}" world_base_rpy="${mh185_vertical_rpy}"/>
+    <xacro:load_motoman_motopos_mh185_vertical
+        world_base_xyz="${mh185_vertical_xyz}"
+        world_base_rpy="${mh185_vertical_rpy}"
+        offsets_file_path="${offsets_file_path}"
+    />
   </xacro:macro>
 </robot>

File: motoman_ma1440_support/urdf/ma1440/ma1440.xacro (robot description, xacro)
@@ -9,6 +9,5 @@
             world_base_rpy
             using_cam_mount:=false
-            offsets_file_path:='$(find motoman_ma1440_support)/config/robot_calibration_offsets.yaml'"
-    >
+            offsets_file_path:='$(find motoman_ma1440_support)/config/robot_calibration_offsets.yaml'">
         <xacro:unless value="${offsets_file_path == ''}">
             <xacro:motoman_ma1440

File: motoman_motopos_d500_support/urdf/motopos_d500.xacro (robot description, xacro)
@@ -1,12 +1,36 @@
 <?xml version="1.0" ?>
 <robot name="motoman_motopos_d500" xmlns:xacro="http://ros.org/wiki/xacro">
-  <!-- Properties -->
-  <material name="yaskawa_blue">
-      <color rgba="0.12941 0.14902 0.74902 1" />
-  </material>
   <xacro:include filename="$(find motoman_motopos_d500_support)/urdf/motopos_d500.transmission.xacro" />
   <xacro:include filename="$(find motoman_motopos_d500_support)/urdf/motopos_d500_macro.xacro" />
-  <xacro:macro name="load_motoman_motopos_d500" params="prefix:=d500_ world_base_xyz world_base_rpy table_thickness">
-    <xacro:motoman_motopos_d500 prefix="${prefix}" world_base_xyz="${world_base_xyz}" world_base_rpy="${world_base_rpy}" table_thickness="${table_thickness}"/>
+  <xacro:macro
+      name="load_motoman_motopos_d500"
+      params=
+          "prefix:=d500_
+          world_base_xyz
+          world_base_rpy
+          table_thickness
+          offsets_file_path:='$(find motoman_motopos_d500_support)/config/robot_calibration_offsets.yaml'"
+  >
+    <material name="yaskawa_blue">
+      <color rgba="0.12941 0.14902 0.74902 1" />
+    </material>
+    <xacro:unless value="${offsets_file_path == ''}">
+      <xacro:motoman_motopos_d500
+          prefix="${prefix}"
+          world_base_xyz="${world_base_xyz}"
+          world_base_rpy="${world_base_rpy}"
+          table_thickness="${table_thickness}"
+          offsets_file_path="${offsets_file_path}"
+      />
+    </xacro:unless>
+    <xacro:if value="${offsets_file_path == ''}">
+      <xacro:motoman_motopos_d500
+          prefix="${prefix}"
+          world_base_xyz="${world_base_xyz}"
+          world_base_rpy="${world_base_rpy}"
+          table_thickness="${table_thickness}"
+          offsets_file_path="'$(find motoman_motopos_d500_support)/config/robot_calibration_offsets.yaml'"
+      />
+    </xacro:if>
   </xacro:macro>
 </robot>

File: motoman_motopos_d500_support/urdf/motopos_d500_macro.xacro (robot description, xacro)
@@ -1,10 +1,13 @@
 <?xml version="1.0" ?>
 <robot xmlns:xacro="http://ros.org/wiki/xacro">
-<xacro:property name="M_PI" value="3.1415926535897931"/>
-<xacro:property name="world_base_xyz" value="0 0 0"/>
-<xacro:property name="world_base_rpy" value="0 0 0"/>
-<!-- offsets tool and positioner base/center frames to account for added tabletop -->
-<xacro:property name="table_thickness" default="0"/>
-<xacro:macro name="motoman_motopos_d500" params="prefix world_base_xyz:=^ world_base_rpy:=^ table_thickness:=^">
+<xacro:macro
+    name="motoman_motopos_d500"
+    params="prefix world_base_xyz:='0 0 0'
+    world_base_rpy:='0 0 0'
+    table_thickness:=0
+    offsets_file_path"
+>
+  <xacro:property name="M_PI" value="3.1415926535897931"/>
+  <xacro:property name="offsets" value="${load_yaml(offsets_file_path)[prefix + 'robot_calibration_offsets']}"/>
   <!-- link list -->
   <link name="${prefix}base_link">

File: motoman_motopos_mh185_vertical_support/urdf/motopos_mh185_vertical.xacro (robot description, xacro)
@@ -1,18 +1,33 @@
 <?xml version="1.0" ?>
 <robot name="motoman_motopos_mh185_vertical" xmlns:xacro="http://ros.org/wiki/xacro">
-  <!-- Properties -->
-<!--  <material name="yaskawa_blue">-->
-<!--      <color rgba="0.12941 0.14902 0.74902 1" />-->
-<!--  </material>-->
-<!--  <xacro:property name="M_PI" value="3.1415926535897931"/>-->
-<!--  <xacro:property name="world_base_xyz" value="0 0 0"/>-->
-<!--  <xacro:property name="world_base_rpy" value="0 0 0"/>-->
   <xacro:include filename="$(find motoman_motopos_mh185_vertical_support)/urdf/motopos_mh185_vertical.transmission.xacro" />
   <xacro:include filename="$(find motoman_motopos_mh185_vertical_support)/urdf/motopos_mh185_vertical_macro.xacro" />
-  <xacro:macro name="load_motoman_motopos_mh185_vertical" params="prefix:=mh185_vertical_ world_base_xyz world_base_rpy">
+  <xacro:macro
+      name="load_motoman_motopos_mh185_vertical"
+      params=
+          "prefix:=mh185_vertical_
+          world_base_xyz
+          world_base_rpy
+          offsets_file_path:='$(find motoman_motopos_mh185_vertical_support)/config/robot_calibration_offsets.yaml'"
+  >
     <material name="yaskawa_blue">
       <color rgba="0.12941 0.14902 0.74902 1" />
     </material>
-    <xacro:motoman_motopos_mh185_vertical prefix="${prefix}" world_base_xyz="${world_base_xyz}" world_base_rpy="${world_base_rpy}"/>
+    <xacro:unless value="${offsets_file_path == ''}">
+      <xacro:motoman_motopos_mh185_vertical
+          prefix="${prefix}"
+          world_base_xyz="${world_base_xyz}"
+          world_base_rpy="${world_base_rpy}"
+          offsets_file_path="${offsets_file_path}"
+      />
+    </xacro:unless>
+    <xacro:if value="${offsets_file_path == ''}">
+      <xacro:motoman_motopos_mh185_vertical
+          prefix="${prefix}"
+          world_base_xyz="${world_base_xyz}"
+          world_base_rpy="${world_base_rpy}"
+          offsets_file_path="'$(find motoman_motopos_mh185_vertical_support)/config/robot_calibration_offsets.yaml'"
+      />
+    </xacro:if>
   </xacro:macro>
 </robot>

File: motoman_motopos_mh185_vertical_support/urdf/motopos_mh185_vertical_macro.xacro (robot description, xacro)
@@ -1,12 +1,18 @@
 <?xml version="1.0" ?>
 <robot xmlns:xacro="http://ros.org/wiki/xacro">
-<xacro:property name="M_PI" value="3.1415926535897931"/>
-<xacro:property name="world_base_xyz" value="0 0 0"/>
-<xacro:property name="world_base_rpy" value="0 0 0"/>
-<!--  Should only be changed if the model for the table is changed. -->
-<xacro:property name="table_thickness" value="0.025"/>
-<!--  Height from the floor to the top of the positioner plate (not the top of the table)  -->
-<xacro:property name="positioner_height" value="0.5045"/>
-<xacro:macro name="motoman_motopos_mh185_vertical" params="prefix world_base_xyz:=^ world_base_rpy:=^">
+<xacro:macro
+    name="motoman_motopos_mh185_vertical"
+    params=
+        "prefix
+        world_base_xyz:='0 0 0'
+        world_base_rpy:='0 0 0'
+        offsets_file_path"
+>
+  <xacro:property name="M_PI" value="3.1415926535897931"/>
+  <!--  Should only be changed if the model for the table is changed. -->
+  <xacro:property name="table_thickness" value="0.025"/>
+  <!--  Height from the floor to the top of the positioner plate (not the top of the table)  -->
+  <xacro:property name="positioner_height" value="0.5045"/>
+  <xacro:property name="offsets" value="${load_yaml(offsets_file_path)[prefix + 'robot_calibration_offsets']}"/>
   <!-- link list -->
   <link name="${prefix}base_link">
@@ -35,8 +41,8 @@
   </link>
   <!-- this is here to set a base link in the URDF to link the "positioner/base" frame to for scanning -->
-  <link name="positioner/base_link"/>
+  <link name="positioner/base"/>
   <!-- this is here to set a base link in the URDF to link the "positioner/center" frame to for scanning. this is equivalent to the tool frame
   in this case, but we define this so that the naming is consistent across positioner setups -->
-  <link name="positioner/center_link"/>
+  <link name="positioner/center"/>
   <!-- end of link list -->
   <!-- joint list -->
@@ -49,6 +55,8 @@
     <parent link="${prefix}base_link"/>
     <child link="${prefix}link_1"/>
-    <origin xyz="0 0 ${positioner_height}" rpy="0 0 0" />
-<!--    <origin xyz="0 0 0.380" rpy="0 0 0" />-->
+    <origin
+        xyz="${offsets[prefix + 'joint_1']['x']} ${offsets[prefix + 'joint_1']['y']} ${positioner_height + offsets[prefix + 'joint_1']['z']}"
+        rpy="${offsets[prefix + 'joint_1']['roll']} ${offsets[prefix + 'joint_1']['pitch']} ${offsets[prefix + 'joint_1']['yaw']}"
+    />
     <axis xyz="0 0 1" />
     <limit lower="${-1*M_PI}" upper="${M_PI}" effort="1274" velocity="1.15"/>
@@ -84,10 +92,10 @@
     <origin xyz="0 0 0" rpy="0 0 0"/>
     <parent link="${prefix}table"/>
-    <child link="positioner/center_link"/>
+    <child link="positioner/center"/>
   </joint>
   <joint name="positioner/base" type="fixed">
-    <origin xyz="0 0 ${positioner_height + table_thickness}" rpy="0 0 0"/>
-    <parent link="${prefix}base_link"/>
-    <child link="positioner/base_link"/>
+    <origin xyz="0 0 ${table_thickness}" rpy="0 0 0"/>
+    <parent link="${prefix}link_1"/>
+    <child link="positioner/base"/>
   </joint>
   <!-- end of joint list -->
