Commit message: WIP - New combined ma1440-d500 moveit config set up This adds a new package that combines the ma1440 arm with the positioner, in its current state the controller_manager is not set up correctly, this is just a checkin point to revert back to as I'm trying other stuff out

File: motoman_ma1440_d500_support/urdf/ma1440_d500_gazebo.xacro (robot description, xacro)
@@ -1,7 +1,3 @@
 <?xml version="1.0" encoding="utf-8" ?>
-<!-- =================================================================================== -->
-<!-- |    This document was autogenerated by xacro from /home/path22/forge/src/motoman/motoman_ma1440_d500_support/urdf/ma1440_d500.xacro | -->
-<!-- |    EDITING THIS FILE BY HAND IS NOT RECOMMENDED                                 | -->
-<!-- =================================================================================== -->
 <!-- =================================================================================== -->
 <!-- |    This document was autogenerated by xacro from /home/path22/forge/src/motoman/motoman_ma1440_d500_support/urdf/ma1440_d500.xacro | -->
@@ -323,5 +319,5 @@
 <inertial>
             <mass value="0.1" />
-            <inertia ixx="0.03" ixy="0.0" ixz="0.0" iyy="0.03" iyz="0.0" izz="0.03" />
+            <inertia ixx="0.03" iyy="0.03" izz="0.03" ixy="0.0" ixz="0.0" iyz="0.0" />
         </inertial>
     </link>
@@ -340,5 +336,5 @@
 <inertial>
             <mass value="0.1" />
-            <inertia ixx="0.03" ixy="0.0" ixz="0.0" iyy="0.03" iyz="0.0" izz="0.03" />
+            <inertia ixx="0.03" iyy="0.03" izz="0.03" ixy="0.0" ixz="0.0" iyz="0.0" />
         </inertial>
     </link>
@@ -357,5 +353,5 @@
 <inertial>
             <mass value="0.1" />
-            <inertia ixx="0.03" ixy="0.0" ixz="0.0" iyy="0.03" iyz="0.0" izz="0.03" />
+            <inertia ixx="0.03" iyy="0.03" izz="0.03" ixy="0.0" ixz="0.0" iyz="0.0" />
         </inertial>
     </link>
@@ -368,5 +364,5 @@
         <child link="d500_base_link" />
     </joint>
-    <joint name="joint_1" type="revolute">
+    <joint name="d500_joint_1" type="revolute">
         <parent link="d500_base_link" />
         <child link="d500_link_1" />
@@ -384,5 +380,5 @@
         </joint>
     </transmission>
-    <joint name="joint_2" type="revolute">
+    <joint name="d500_joint_2" type="revolute">
         <parent link="d500_link_1" />
         <child link="d500_link_2" />
@@ -400,5 +396,5 @@
         </joint>
     </transmission>
-    <joint name="$joint_2-tool0" type="fixed">
+    <joint name="d500_joint_2-tool0" type="fixed">
         <origin rpy="0 0 0" xyz="0 0 0.150 " />
         <parent link="d500_link_2" />
@@ -477,105 +473,20 @@
         </actuator>
     </transmission>
-    <transmission name="trans_joint_1">
-        <type>transmission_interface/SimpleTransmission</type>
-        <joint name="joint_1">
-            <hardwareInterface>hardware_interface/EffortJointInterface</hardwareInterface>
-        </joint>
-        <actuator name="joint_1_motor">
-            <hardwareInterface>hardware_interface/EffortJointInterface</hardwareInterface>
-            <mechanicalReduction>1</mechanicalReduction>
-        </actuator>
-    </transmission>
-    <transmission name="trans_joint_2">
-        <type>transmission_interface/SimpleTransmission</type>
-        <joint name="joint_2">
-            <hardwareInterface>hardware_interface/EffortJointInterface</hardwareInterface>
-        </joint>
-        <actuator name="joint_2_motor">
-            <hardwareInterface>hardware_interface/EffortJointInterface</hardwareInterface>
-            <mechanicalReduction>1</mechanicalReduction>
-        </actuator>
-    </transmission>
-    <gazebo>
-        <plugin filename="libgazebo_ros_control.so" name="gazebo_ros_control">
-            <robotNamespace>/</robotNamespace>
-        </plugin>
-    </gazebo>
-    <transmission name="trans_joint_s">
-        <type>transmission_interface/SimpleTransmission</type>
-        <joint name="joint_s">
-            <hardwareInterface>hardware_interface/PositionJointInterface</hardwareInterface>
-        </joint>
-        <actuator name="joint_s_motor">
-            <hardwareInterface>hardware_interface/PositionJointInterface</hardwareInterface>
-            <mechanicalReduction>1</mechanicalReduction>
-        </actuator>
-    </transmission>
-    <transmission name="trans_joint_l">
-        <type>transmission_interface/SimpleTransmission</type>
-        <joint name="joint_l">
-            <hardwareInterface>hardware_interface/PositionJointInterface</hardwareInterface>
-        </joint>
-        <actuator name="joint_l_motor">
-            <hardwareInterface>hardware_interface/PositionJointInterface</hardwareInterface>
-            <mechanicalReduction>1</mechanicalReduction>
-        </actuator>
-    </transmission>
-    <transmission name="trans_joint_u">
-        <type>transmission_interface/SimpleTransmission</type>
-        <joint name="joint_u">
-            <hardwareInterface>hardware_interface/PositionJointInterface</hardwareInterface>
-        </joint>
-        <actuator name="joint_u_motor">
-            <hardwareInterface>hardware_interface/PositionJointInterface</hardwareInterface>
-            <mechanicalReduction>1</mechanicalReduction>
-        </actuator>
-    </transmission>
-    <transmission name="trans_joint_r">
-        <type>transmission_interface/SimpleTransmission</type>
-        <joint name="joint_r">
-            <hardwareInterface>hardware_interface/PositionJointInterface</hardwareInterface>
-        </joint>
-        <actuator name="joint_r_motor">
-            <hardwareInterface>hardware_interface/PositionJointInterface</hardwareInterface>
-            <mechanicalReduction>1</mechanicalReduction>
-        </actuator>
-    </transmission>
-    <transmission name="trans_joint_b">
-        <type>transmission_interface/SimpleTransmission</type>
-        <joint name="joint_b">
-            <hardwareInterface>hardware_interface/PositionJointInterface</hardwareInterface>
-        </joint>
-        <actuator name="joint_b_motor">
-            <hardwareInterface>hardware_interface/PositionJointInterface</hardwareInterface>
-            <mechanicalReduction>1</mechanicalReduction>
-        </actuator>
-    </transmission>
-    <transmission name="trans_joint_t">
-        <type>transmission_interface/SimpleTransmission</type>
-        <joint name="joint_t">
-            <hardwareInterface>hardware_interface/PositionJointInterface</hardwareInterface>
-        </joint>
-        <actuator name="joint_t_motor">
-            <hardwareInterface>hardware_interface/PositionJointInterface</hardwareInterface>
-            <mechanicalReduction>1</mechanicalReduction>
-        </actuator>
-    </transmission>
-    <transmission name="trans_joint_1">
-        <type>transmission_interface/SimpleTransmission</type>
-        <joint name="joint_1">
-            <hardwareInterface>hardware_interface/EffortJointInterface</hardwareInterface>
-        </joint>
-        <actuator name="joint_1_motor">
-            <hardwareInterface>hardware_interface/EffortJointInterface</hardwareInterface>
-            <mechanicalReduction>1</mechanicalReduction>
-        </actuator>
-    </transmission>
-    <transmission name="trans_joint_2">
-        <type>transmission_interface/SimpleTransmission</type>
-        <joint name="joint_2">
-            <hardwareInterface>hardware_interface/EffortJointInterface</hardwareInterface>
-        </joint>
-        <actuator name="joint_2_motor">
+    <transmission name="trans_d500_joint_1">
+        <type>transmission_interface/SimpleTransmission</type>
+        <joint name="d500_joint_1">
+            <hardwareInterface>hardware_interface/EffortJointInterface</hardwareInterface>
+        </joint>
+        <actuator name="d500_joint_1_motor">
+            <hardwareInterface>hardware_interface/EffortJointInterface</hardwareInterface>
+            <mechanicalReduction>1</mechanicalReduction>
+        </actuator>
+    </transmission>
+    <transmission name="trans_d500_joint_2">
+        <type>transmission_interface/SimpleTransmission</type>
+        <joint name="d500_joint_2">
+            <hardwareInterface>hardware_interface/EffortJointInterface</hardwareInterface>
+        </joint>
+        <actuator name="d500_joint_2_motor">
             <hardwareInterface>hardware_interface/EffortJointInterface</hardwareInterface>
             <mechanicalReduction>1</mechanicalReduction>

File: motoman_ma1440_support/urdf/ma1440/ma1440_macro.xacro (robot description, xacro)
@@ -99,5 +99,4 @@
         <link name="${prefix}link_u">
             <visual>
-<!--                <origin rpy="1.57 -3.1415 0" xyz="0 0 0"/>-->
                 <origin rpy="0 0 0" xyz="0 0 0"/>
                 <geometry>
@@ -107,5 +106,4 @@
             </visual>
             <collision>
-<!--                <origin rpy="1.57 -3.1415 0" xyz="0 0 0"/>-->
                 <origin rpy="0 0 0" xyz="0 0 0"/>
                 <geometry>
@@ -248,4 +246,5 @@
             <limit lower="-3.1415" upper="3.1415" effort="100" velocity="2.9670" />
         </joint>
+        <xacro:transmission_macro name="s"/>
         <joint name="${prefix}joint_l" type="revolute">
             <parent link="${prefix}link_s"/>
@@ -255,4 +254,5 @@
             <limit lower="-1.9198" upper="1.9198" effort="100" velocity="2.9670" />
         </joint>
+        <xacro:transmission_macro name="l"/>
         <joint name="${prefix}joint_u" type="revolute">
             <parent link="${prefix}link_l"/>
@@ -262,4 +262,5 @@
             <limit lower="-2.3561" upper="2.3561" effort="100" velocity="2.9670" />
         </joint>
+        <xacro:transmission_macro name="u"/>
         <joint name="${prefix}joint_r" type="revolute">
             <parent link="${prefix}link_u"/>
@@ -269,4 +270,5 @@
             <limit lower="-3.1415" upper="3.1415" effort="100" velocity="3.4906" />
         </joint>
+        <xacro:transmission_macro name="r"/>
         <joint name="${prefix}joint_b" type="revolute">
             <parent link="${prefix}link_r"/>
@@ -276,4 +278,5 @@
             <limit lower="-1.9198" upper="1.9198" effort="100" velocity="3.4906" />
         </joint>
+        <xacro:transmission_macro name="b"/>
         <joint name="${prefix}joint_t" type="revolute">
             <parent link="${prefix}link_b"/>
@@ -283,4 +286,5 @@
             <limit lower="-3.1415" upper="3.1415" effort="100" velocity="6.9813" />
         </joint>
+        <xacro:transmission_macro name="t"/>
         <joint name="${prefix}joint_tip" type="fixed">
             <parent link="${prefix}link_t"/>

File: motoman_motopos_d500_support/urdf/motopos_d500.xacro (robot description, xacro)
@@ -7,4 +7,4 @@
   <xacro:include filename="$(find motoman_motopos_d500_support)/urdf/motopos_d500.transmission.xacro" />
   <xacro:include filename="$(find motoman_motopos_d500_support)/urdf/motopos_d500_macro.xacro" />
-  <xacro:motoman_motopos_d500 prefix="d500"/>
+  <xacro:motoman_motopos_d500 prefix="d500_"/>
 </robot>

File: motoman_motopos_d500_support/urdf/motopos_d500_macro.xacro (robot description, xacro)
@@ -59,5 +59,5 @@
   <xacro:transmission_macro name="1"/>
   <joint name="joint_2" type="revolute">
-    <parent link="${prefix}base_link"/>
+    <parent link="${prefix}link_1"/>
     <child link="${prefix}link_2"/>
     <origin xyz="0 0 0" rpy="0 0 0" />
@@ -66,5 +66,5 @@
   </joint>
   <xacro:transmission_macro name="2"/>
-  <joint name="joint_2-tool0" type="fixed">
+  <joint name="$joint_2-tool0" type="fixed">
     <origin xyz="0 0 0.150 " rpy="0 0 0"/>
     <parent link="${prefix}link_2"/>

Commit message: added support for ma1440 with horizontally rotating positioner

File: motoman_ma1440_d500_support/urdf/ma1440_d500_gazebo.xacro (robot description, xacro)
@@ -207,40 +207,11 @@
         <material>Gazebo/White</material>
     </gazebo>
-    <link name="link_tip">
-        <visual>
-            <origin rpy="0 0 0" xyz="0 0 0" />
-            <geometry>
-                <mesh filename="package://motoman_ma1440_support/meshes/ma1440/visual/tip_link.stl" />
-            </geometry>
-            <material name="silver">
-                <color rgba="0.8 0.8 0.8 1" />
-            </material>
-        </visual>
-        <collision>
-            <origin rpy="0 0 0" xyz="0 0 0" />
-            <geometry>
-                <mesh filename="package://motoman_ma1440_support/meshes/ma1440/collision/tip_link_collision.stl" />
-            </geometry>
-            <material name="silver">
-                <color rgba="0.8 0.8 0.8 1" />
-            </material>
-        </collision>
-<inertial>
-            <mass value="4.7615" />
-            <inertia ixx="0.034062" ixy="5.0098E-05" ixz="4.7762E-05" iyy="0.020719" iyz="-0.016082" izz="0.013698" />
-            <origin rpy="0.0 0.0 0.0" xyz="0.0 0.0 0.0" />
-        </inertial>
-    </link>
-    <gazebo reference="link_t">
-        <turnGravityOff>false</turnGravityOff>
-        <selfCollide>true</selfCollide>
-        <material>Gazebo/White</material>
-    </gazebo>
     <!-- end of link list -->
     <!-- joint list -->
-    <joint name="world-base" type="fixed">
+    <joint name="ma1440_world-base" type="fixed">
         <origin rpy="0 0 0" xyz="0 0 0" />
         <parent link="world" />
         <child link="base_link" />
+        <axis xyz = "0 0 0"/>
     </joint>
     <joint name="joint_s" type="revolute">
@@ -285,10 +256,4 @@
         <axis xyz="0 0 1" />
         <limit effort="100" lower="-3.1415" upper="3.1415" velocity="6.9813" />
-    </joint>
-    <joint name="joint_tip" type="fixed">
-        <parent link="link_t" />
-        <child link="link_tip" />
-        <origin rpy="-2.35619449019 0 1.57079632679" xyz="-0.09591 0 -0.38772" />
-        <axis xyz="0 0 0" />
     </joint>
     <!-- end of joint list -->

File: motoman_ma1440_mh185_rotisserie_support/urdf/ma1440_mh185_rotisserie.xacro (robot description, xacro)
@@ -1,9 +1,9 @@
 <?xml version="1.0" ?>
  <robot name="motoman_ma1440_mh185_rotisserie" xmlns:xacro="http://ros.org/wiki/xacro">
-	<xacro:arg name="ma1440_xyz" default=""/>
-	<xacro:arg name="ma1440_rpy" default=""/>
-	<xacro:arg name="mh185_rotisserie_xyz" default=""/>
-	<xacro:arg name="mh185_rotisserie_rpy" default=""/>
-	<xacro:arg name="using_cam_mount" default=""/>
+	<xacro:arg name="ma1440_xyz" default="0 0 0"/>
+	<xacro:arg name="ma1440_rpy" default="0 0 0 "/>
+	<xacro:arg name="mh185_xyz" default="0 0 0"/>
+	<xacro:arg name="mh185_rpy" default="0 0 0"/>
+	<xacro:arg name="using_cam_mount" default="true"/>
 	<xacro:arg name="offsets_file_path" default=""/>
 	<xacro:include filename="$(find motoman_ma1440_mh185_rotisserie_support)/urdf/ma1440_mh185_rotisserie_macro.xacro" />
@@ -11,6 +11,6 @@
 			ma1440_xyz="$(arg ma1440_xyz)"
 			ma1440_rpy="$(arg ma1440_rpy)"
-			mh185_rotisserie_xyz="$(arg mh185_rotisserie_xyz)"
-			mh185_rotisserie_rpy="$(arg mh185_rotisserie_rpy)"
+			mh185_xyz="$(arg mh185_xyz)"
+			mh185_rpy="$(arg mh185_rpy)"
 			using_cam_mount="$(arg using_cam_mount)"
 			offsets_file_path="$(arg offsets_file_path)"

File: motoman_ma1440_mh185_rotisserie_support/urdf/ma1440_mh185_rotisserie_macro.xacro (robot description, xacro)
@@ -6,6 +6,6 @@
           "ma1440_xyz
           ma1440_rpy
-          mh185_rotisserie_xyz
-          mh185_rotisserie_rpy
+          mh185_xyz
+          mh185_rpy
           using_cam_mount
           offsets_file_path"
@@ -20,6 +20,6 @@
     <xacro:include filename="$(find motoman_motopos_mh185_rotisserie_support)/urdf/motopos_mh185_rotisserie.xacro" />
     <xacro:load_motoman_motopos_mh185_rotisserie
-        world_base_xyz="${mh185_rotisserie_xyz}"
-        world_base_rpy="${mh185_rotisserie_rpy}"
+        world_base_xyz="${mh185_xyz}"
+        world_base_rpy="${mh185_rpy}"
         offsets_file_path="${offsets_file_path}"
     />

File: motoman_motopos_mh185_rotisserie_support/urdf/headstock/headstock.urdf.xacro (robot description, xacro)
@@ -22,4 +22,5 @@
         izz="7.6922" />
     </inertial>
+    <xacro:arg name="visible" default="true"/>
     <xacro:if value="$(arg visible)">
       <visual>
@@ -29,5 +30,5 @@
         <geometry>
           <mesh
-              filename="package://motoman_motopos_mh185_rotisserie_support/meshes/headstock/hs_base_link.stl" />
+              filename="package://motoman_motopos_mh185_rotisserie_support/meshes/headstock/hs_base_collision_link.stl" />
         </geometry>
         <material
@@ -55,7 +56,7 @@
       rpy="0 0 0" />
     <parent
+      link="hs_base_link" />
+    <child
       link="hs_revolute_link" />
-    <child
-      link="hs_base_link" />
     <axis
       xyz="0 0 1" />
@@ -90,5 +91,5 @@
         <geometry>
           <mesh
-              filename="package://motoman_motopos_mh185_rotisserie_support/meshes/headstock/hs_revolute_link.stl" />
+              filename="package://motoman_motopos_mh185_rotisserie_support/meshes/headstock/hs_revolute_collision_link.stl" />
         </geometry>
         <material
@@ -145,5 +146,5 @@
         <geometry>
           <mesh
-              filename="package://motoman_motopos_mh185_rotisserie_support/meshes/headstock/hs_prismatic_link.stl" />
+              filename="package://motoman_motopos_mh185_rotisserie_support/meshes/headstock/hs_prismatic_collision_link.stl" />
         </geometry>
         <material

File: motoman_motopos_mh185_rotisserie_support/urdf/motopos_mh185_rotisserie.xacro (robot description, xacro)
@@ -5,5 +5,5 @@
       name="load_motoman_motopos_mh185_rotisserie"
       params=
-          "prefix:=mh185_rotisserie_
+          "prefix:=mh185_
           world_base_xyz
           world_base_rpy

File: motoman_motopos_mh185_rotisserie_support/urdf/motopos_mh185_rotisserie_macro.xacro (robot description, xacro)
@@ -10,4 +10,5 @@
 >
   <xacro:property name="M_PI" value="3.1415926535897931"/>
+  <xacro:property name="offsets" value="${load_yaml(offsets_file_path)[prefix + 'robot_calibration_offsets']}"/>
 <xacro:property name="pos2b_tf" value="${load_yaml('$(find motoman_motopos_mh185_rotisserie_support)/config/positioner_params.yaml')}"/>
   <xacro:property name="pos2b_trans" value="${pos2b_tf['positioner_params']['positioner_to_base_tf']['translation']}" />
@@ -15,4 +16,9 @@
   <xacro:property name="pos2b_xyz" value="${pos2b_trans['x']} ${pos2b_trans['y']} ${pos2b_trans['z']}"/>
   <xacro:property name="pos2b_rpy" value="${pos2b_rot['roll']} ${pos2b_rot['pitch']} ${pos2b_rot['yaw']}"/>
+<xacro:property name="world_to_pos_base_tf" value="${load_yaml('$(find motoman_motopos_mh185_rotisserie_support)/config/positioner_params.yaml')}"/>
+  <xacro:property name="world2pos_t" value="${pos2b_tf['positioner_params']['base_to_positioner_tf']['translation']}" />
+  <xacro:property name="world2pos_rot" value="${pos2b_tf['positioner_params']['base_to_positioner_tf']['rotation']}" />
+  <xacro:property name="world2pos_xyz" value="${world2pos_t['x']} ${world2pos_t['y']} ${world2pos_t['z']}"/>
+  <xacro:property name="world2pos_rpy" value="${world2pos_rot['roll']} ${world2pos_rot['pitch']} ${world2pos_rot['yaw']}"/>
   <!-- Tailstock offsets. Should be loaded from yaml file created during calibration. -->
   <xacro:property name="ts_base_offset" value="0.06985" />
@@ -30,13 +36,13 @@
   <!-- link list -->
   <!-- Add the headstock - hs_base_link, hs_revolute_link, hs_prismatic_link -->
+  <xacro:include filename="$(find motoman_motopos_mh185_rotisserie_support)/urdf/headstock/headstock.urdf.xacro" ns="hs" />
   <xacro:include filename="$(find motoman_motopos_mh185_rotisserie_support)/urdf/tailstock/tailstock.urdf.xacro" ns="ts" />
-  <xacro:include filename="$(find motoman_motopos_mh185_rotisserie_support)/urdf/headstock/headstock.urdf.xacro" ns="hs" />
   <!-- And connect positioner_link to base_link -->
   <!-- hs_base - positioner_link->base_link -->
-  <xacro:fixed_joint_macro name="hs_base"
-                           origin_xyz="${pos2b_xyz}"
-                           origin_rpy="${pos2b_rpy}"
-                           parent="hs_base_link"
-                           child="world"
+  <xacro:fixed_joint_macro name="world-hsbase"
+                           origin_xyz="${world2pos_xyz}"
+                           origin_rpy="${world2pos_rpy}"
+                           parent="world"
+                           child="hs_base_link"
                            axis_xyz="1 0 0" />
   <!-- Connect the tail stock to the headstock -->

File: motoman_motopos_mh185_rotisserie_support/urdf/tailstock/tailstock.urdf.xacro (robot description, xacro)
@@ -27,5 +27,5 @@
         <geometry>
           <mesh
-              filename="package://motoman_motopos_mh185_rotisserie_support/meshes/tailstock/ts_base_link.stl" />
+              filename="package://motoman_motopos_mh185_rotisserie_support/meshes/tailstock/ts_base_collision_link.stl" />
         </geometry>
         <material
@@ -69,5 +69,5 @@
         <geometry>
           <mesh
-              filename="package://motoman_motopos_mh185_rotisserie_support/meshes/tailstock/ts_prismatic_link.stl" />
+              filename="package://motoman_motopos_mh185_rotisserie_support/meshes/tailstock/ts_prismatic_collision_link.stl" />
         </geometry>
         <material
@@ -111,5 +111,5 @@
         <geometry>
           <mesh
-              filename="package://motoman_motopos_mh185_rotisserie_support/meshes/tailstock/ts_revolute_link.stl" />
+              filename="package://motoman_motopos_mh185_rotisserie_support/meshes/tailstock/ts_revolute_collision_link.stl" />
         </geometry>
         <material
