Commit message: Save point - get new combined package closer to working on real robot hardware Checking in code before redoing the setup assistant, here the joint state subscription is looking good and the planning is working, but getting invalid joint name errors when going to actually execute the plan

File: motoman_ma1440_d500_support/urdf/ma1440_d500.xacro (robot description, xacro)
@@ -1,7 +1,3 @@
 <?xml version="1.0" encoding="utf-8" ?>
-<!-- =================================================================================== -->
-<!-- |    This document was autogenerated by xacro from /home/path22/forge/src/motoman/motoman_ma1440_d500_support/urdf/ma1440_d500.xacro | -->
-<!-- |    EDITING THIS FILE BY HAND IS NOT RECOMMENDED                                 | -->
-<!-- =================================================================================== -->
 <!-- =================================================================================== -->
 <!-- |    This document was autogenerated by xacro from /home/path22/forge/src/motoman/motoman_ma1440_d500_support/urdf/ma1440_d500.xacro | -->
@@ -583,4 +579,89 @@
     </transmission>
     <gazebo>
+        <plugin filename="libgazebo_ros_control.so" name="gazebo_ros_control">
+            <robotNamespace>/</robotNamespace>
+        </plugin>
+    </gazebo>
+    <transmission name="trans_joint_s">
+        <type>transmission_interface/SimpleTransmission</type>
+        <joint name="joint_s">
+            <hardwareInterface>hardware_interface/EffortJointInterface</hardwareInterface>
+        </joint>
+        <actuator name="joint_s_motor">
+            <hardwareInterface>hardware_interface/EffortJointInterface</hardwareInterface>
+            <mechanicalReduction>1</mechanicalReduction>
+        </actuator>
+    </transmission>
+    <transmission name="trans_joint_l">
+        <type>transmission_interface/SimpleTransmission</type>
+        <joint name="joint_l">
+            <hardwareInterface>hardware_interface/EffortJointInterface</hardwareInterface>
+        </joint>
+        <actuator name="joint_l_motor">
+            <hardwareInterface>hardware_interface/EffortJointInterface</hardwareInterface>
+            <mechanicalReduction>1</mechanicalReduction>
+        </actuator>
+    </transmission>
+    <transmission name="trans_joint_u">
+        <type>transmission_interface/SimpleTransmission</type>
+        <joint name="joint_u">
+            <hardwareInterface>hardware_interface/EffortJointInterface</hardwareInterface>
+        </joint>
+        <actuator name="joint_u_motor">
+            <hardwareInterface>hardware_interface/EffortJointInterface</hardwareInterface>
+            <mechanicalReduction>1</mechanicalReduction>
+        </actuator>
+    </transmission>
+    <transmission name="trans_joint_r">
+        <type>transmission_interface/SimpleTransmission</type>
+        <joint name="joint_r">
+            <hardwareInterface>hardware_interface/EffortJointInterface</hardwareInterface>
+        </joint>
+        <actuator name="joint_r_motor">
+            <hardwareInterface>hardware_interface/EffortJointInterface</hardwareInterface>
+            <mechanicalReduction>1</mechanicalReduction>
+        </actuator>
+    </transmission>
+    <transmission name="trans_joint_b">
+        <type>transmission_interface/SimpleTransmission</type>
+        <joint name="joint_b">
+            <hardwareInterface>hardware_interface/EffortJointInterface</hardwareInterface>
+        </joint>
+        <actuator name="joint_b_motor">
+            <hardwareInterface>hardware_interface/EffortJointInterface</hardwareInterface>
+            <mechanicalReduction>1</mechanicalReduction>
+        </actuator>
+    </transmission>
+    <transmission name="trans_joint_t">
+        <type>transmission_interface/SimpleTransmission</type>
+        <joint name="joint_t">
+            <hardwareInterface>hardware_interface/EffortJointInterface</hardwareInterface>
+        </joint>
+        <actuator name="joint_t_motor">
+            <hardwareInterface>hardware_interface/EffortJointInterface</hardwareInterface>
+            <mechanicalReduction>1</mechanicalReduction>
+        </actuator>
+    </transmission>
+    <transmission name="trans_joint_1">
+        <type>transmission_interface/SimpleTransmission</type>
+        <joint name="joint_1">
+            <hardwareInterface>hardware_interface/EffortJointInterface</hardwareInterface>
+        </joint>
+        <actuator name="joint_1_motor">
+            <hardwareInterface>hardware_interface/EffortJointInterface</hardwareInterface>
+            <mechanicalReduction>1</mechanicalReduction>
+        </actuator>
+    </transmission>
+    <transmission name="trans_joint_2">
+        <type>transmission_interface/SimpleTransmission</type>
+        <joint name="joint_2">
+            <hardwareInterface>hardware_interface/EffortJointInterface</hardwareInterface>
+        </joint>
+        <actuator name="joint_2_motor">
+            <hardwareInterface>hardware_interface/EffortJointInterface</hardwareInterface>
+            <mechanicalReduction>1</mechanicalReduction>
+        </actuator>
+    </transmission>
+    <gazebo>
         <plugin name="gazebo_ros_control" filename="libgazebo_ros_control.so">
             <robotNamespace>/</robotNamespace>

Commit message: Minor cleanup, revert auto-generated .xacro file back to macro version

File: motoman_ma1440_d500_support/urdf/ma1440_d500.xacro (robot description, xacro)
@@ -1,670 +1,5 @@
-<?xml version="1.0" encoding="utf-8" ?>
-<!-- =================================================================================== -->
-<!-- |    This document was autogenerated by xacro from /home/path22/forge/src/motoman/motoman_ma1440_d500_support/urdf/ma1440_d500.xacro | -->
-<!-- |    EDITING THIS FILE BY HAND IS NOT RECOMMENDED                                 | -->
-<!-- =================================================================================== -->
-<robot name="motoman_ma1440_d500" xmlns:xacro="http://ros.org/wiki/xacro">
-    <!-- link list -->
-    <link name="world">
-        <origin rpy="0 0 0" xyz="0 0 0" />
-    </link>
-    <link name="base_link">
-        <visual>
-            <origin rpy="0 0 0" xyz="0 0 0" />
-            <geometry>
-                <mesh filename="package://motoman_ma1440_support/meshes/ma1440/visual/base_link.stl" />
-            </geometry>
-            <material name="blue">
-                <color rgba="0 0 1 1" />
-            </material>
-        </visual>
-        <collision>
-            <origin rpy="0 0 0" xyz="0 0 0" />
-            <geometry>
-                <mesh filename="package://motoman_ma1440_support/meshes/ma1440/collision/base_link_collision.stl" />
-            </geometry>
-            <material name="yellow">
-                <color rgba="0 1 1 1" />
-            </material>
-        </collision>
-<inertial>
-            <mass value="400" />
-            <!-- Arbitrarily large value, to simulate bolting down in case of absence of fixed joint -->
-            <inertia ixx="1.0" ixy="0.0" ixz="0.0" iyy="1.0" iyz="0.0" izz="1.0" />
-            <origin rpy="0 0 0" xyz="0 0 0" />
-        </inertial>
-    </link>
-    <gazebo reference="base_link">
-        <turnGravityOff>false</turnGravityOff>
-        <selfCollide>true</selfCollide>
-        <material>Gazebo/Blue</material>
-    </gazebo>
-    <link name="link_s">
-        <visual>
-            <!--                <origin rpy="0 0 0" xyz="0.026522 0.0082618 0.12436"/>-->
-            <origin rpy="0 0 0" xyz="0 0 0" />
-            <geometry>
-                <mesh filename="package://motoman_ma1440_support/meshes/ma1440/visual/s_link.stl" />
-            </geometry>
-            <material name="blue">
-                <color rgba="0 0 1 1" />
-            </material>
-        </visual>
-        <collision>
-            <!--                <origin rpy="0 0 0" xyz="0.026522 0.0082618 0.12436"/>-->
-            <origin rpy="0 0 0" xyz="0 0 0" />
-            <geometry>
-                <mesh filename="package://motoman_ma1440_support/meshes/ma1440/collision/s_link_collision.stl" />
-            </geometry>
-            <material name="yellow" />
-        </collision>
-<inertial>
-            <mass value="112.57" />
-            <inertia ixx="2.1336" ixy="0.197" ixz="0.8995" iyy="2.8341" iyz="0.2799" izz="2.49" />
-            <origin rpy="0 0 0" xyz="0 0 0" />
-            <!--                <origin rpy="0 0 0" xyz="0.026522 0.0082618 0.12436"/>-->
-        </inertial>
-    </link>
-    <gazebo reference="link_s">
-        <turnGravityOff>false</turnGravityOff>
-        <selfCollide>true</selfCollide>
-        <material>Gazebo/Blue</material>
-    </gazebo>
-    <link name="link_l">
-        <visual>
-            <!--                <origin rpy="1.57 3.1416 0" xyz="0 0 0"/>-->
-            <origin rpy="0 0 0" xyz="0 0 0" />
-            <geometry>
-                <mesh filename="package://motoman_ma1440_support/meshes/ma1440/visual/l_link.stl" />
-            </geometry>
-            <material name="blue" />
-        </visual>
-        <collision>
-            <!--                <origin rpy="1.57 3.1416 0" xyz="0 0 0"/>-->
-            <origin rpy="0 0 0" xyz="0 0 0" />
-            <geometry>
-                <mesh filename="package://motoman_ma1440_support/meshes/ma1440/collision/l_link_collision.stl" />
-            </geometry>
-            <material name="yellow" />
-        </collision>
-<inertial>
-            <mass value="45.143" />
-            <inertia ixx="0.1565" ixy="-0.0239" ixz="-0.0981" iyy="2.4306" iyz="0.0329" izz="2.4493" />
-            <!--                <origin xyz="0.11422130 0.0 0.018935113" rpy="0.0 0.0 0.0"/>-->
-            <origin rpy="0 0 0" xyz="0 0 0" />
-        </inertial>
-    </link>
-    <gazebo reference="link_l">
-        <turnGravityOff>false</turnGravityOff>
-        <selfCollide>true</selfCollide>
-        <material>Gazebo/Blue</material>
-    </gazebo>
-    <link name="link_u">
-        <visual>
-            <!--                <origin rpy="1.57 -3.1415 0" xyz="0 0 0"/>-->
-            <origin rpy="0 0 0" xyz="0 0 0" />
-            <geometry>
-                <mesh filename="package://motoman_ma1440_support/meshes/ma1440/visual/u_link.stl" />
-            </geometry>
-            <material name="blue" />
-        </visual>
-        <collision>
-            <!--                <origin rpy="1.57 -3.1415 0" xyz="0 0 0"/>-->
-            <origin rpy="0 0 0" xyz="0 0 0" />
-            <geometry>
-                <mesh filename="package://motoman_ma1440_support/meshes/ma1440/collision/u_link_collision.stl" />
-            </geometry>
-            <material name="yellow" />
-        </collision>
-<inertial>
-            <mass value="77.767" />
-            <inertia ixx="1.1285" ixy="-0.4562" ixz="-0.1754" iyy="0.965" iyz="0.2365" izz="1.2844" />
-            <!--                <origin xyz="0.0 -0.015659426 0.13525753" rpy="0.0 0.0 0.0"/>-->
-            <origin rpy="0 0 0" xyz="0 0 0" />
-        </inertial>
-    </link>
-    <gazebo reference="link_u">
-        <turnGravityOff>false</turnGravityOff>
-        <selfCollide>true</selfCollide>
-        <material>Gazebo/Blue</material>
-    </gazebo>
-    <link name="link_r">
-        <visual>
-            <origin rpy="0 0 0" xyz="0 0 0" />
-            <geometry>
-                <mesh filename="package://motoman_ma1440_support/meshes/ma1440/visual/r_link.stl" />
-            </geometry>
-            <material name="blue" />
-        </visual>
-        <collision>
-            <origin rpy="0 0 0" xyz="0 0 0" />
-            <geometry>
-                <mesh filename="package://motoman_ma1440_support/meshes/ma1440/collision/r_link_collision.stl" />
-            </geometry>
-            <material name="yellow" />
-        </collision>
-<inertial>
-            <mass value="31.136" />
-            <inertia ixx="0.5313" ixy="0.0027" ixz="0.0418" iyy="0.453" iyz="-0.0111" izz="0.1611" />
-            <origin rpy="0 0 0" xyz="0 0 0" />
-        </inertial>
-    </link>
-    <gazebo reference="link_r">
-        <turnGravityOff>false</turnGravityOff>
-        <selfCollide>true</selfCollide>
-        <material>Gazebo/White</material>
-    </gazebo>
-    <link name="link_b">
-        <visual>
-            <origin rpy="0 0 0" xyz="0 0 0" />
-            <geometry>
-                <mesh filename="package://motoman_ma1440_support/meshes/ma1440/visual/b_link.stl" />
-            </geometry>
-            <material name="blue" />
-        </visual>
-        <collision>
-            <origin rpy="0 0 0" xyz="0 0 0" />
-            <geometry>
-                <mesh filename="package://motoman_ma1440_support/meshes/ma1440/collision/b_link_collision.stl" />
-            </geometry>
-            <material name="yellow" />
-        </collision>
-<inertial>
-            <mass value="7.781" />
-            <inertia ixx="0.019954" ixy="6.9E-05" ixz="-0.000759" iyy="0.024524" iyz="0.000206" izz="0.019404" />
-            <origin rpy="0 0 0" xyz="0 0 0" />
-        </inertial>
-    </link>
-    <gazebo reference="link_b">
-        <turnGravityOff>false</turnGravityOff>
-        <selfCollide>true</selfCollide>
-        <material>Gazebo/Blue</material>
-    </gazebo>
-    <link name="link_t">
-        <visual>
-            <origin rpy="0 0 0" xyz="0 0 0" />
-            <geometry>
-                <mesh filename="package://motoman_ma1440_support/meshes/ma1440/visual/t_link.stl" />
-            </geometry>
-            <material name="blue" />
-        </visual>
-        <collision>
-            <origin rpy="0 0 0" xyz="0 0 0" />
-            <geometry>
-                <mesh filename="package://motoman_ma1440_support/meshes/ma1440/collision/t_link_collision.stl" />
-            </geometry>
-            <material name="yellow" />
-        </collision>
-<inertial>
-            <mass value="0.40691" />
-            <inertia ixx="0.0" ixy="0.0" ixz="0.0" iyy="0.0" iyz="0.0" izz="0.0" />
-            <origin rpy="0.0 0.0 0.0" xyz="0.0 0.0 0.0" />
-        </inertial>
-    </link>
-    <gazebo reference="link_t">
-        <turnGravityOff>false</turnGravityOff>
-        <selfCollide>true</selfCollide>
-        <material>Gazebo/White</material>
-    </gazebo>
-    <link name="link_tip">
-        <visual>
-            <origin rpy="0 0 0" xyz="0 0 0" />
-            <geometry>
-                <mesh filename="package://motoman_ma1440_support/meshes/ma1440/visual/tip_link.stl" />
-            </geometry>
-            <material name="silver">
-                <color rgba="0.8 0.8 0.8 1" />
-            </material>
-        </visual>
-        <collision>
-            <origin rpy="0 0 0" xyz="0 0 0" />
-            <geometry>
-                <mesh filename="package://motoman_ma1440_support/meshes/ma1440/collision/tip_link_collision.stl" />
-            </geometry>
-            <material name="silver">
-                <color rgba="0.8 0.8 0.8 1" />
-            </material>
-        </collision>
-<inertial>
-            <mass value="4.7615" />
-            <inertia ixx="0.034062" ixy="5.0098E-05" ixz="4.7762E-05" iyy="0.020719" iyz="-0.016082" izz="0.013698" />
-            <origin rpy="0.0 0.0 0.0" xyz="0.0 0.0 0.0" />
-        </inertial>
-    </link>
-    <gazebo reference="link_t">
-        <turnGravityOff>false</turnGravityOff>
-        <selfCollide>true</selfCollide>
-        <material>Gazebo/White</material>
-    </gazebo>
-    <!-- end of link list -->
-    <!-- joint list -->
-    <joint name="world-base" type="fixed">
-        <origin rpy="0 0 0" xyz="0 0 0" />
-        <parent link="world" />
-        <child link="base_link" />
-    </joint>
-    <joint name="joint_s" type="revolute">
-        <parent link="base_link" />
-        <child link="link_s" />
-        <origin rpy="0 0 0" xyz="0 0 0.165" />
-        <axis xyz="0 0 1" />
-        <limit effort="100" lower="-3.1415" upper="3.1415" velocity="2.9670" />
-    </joint>
-    <joint name="joint_l" type="revolute">
-        <parent link="link_s" />
-        <child link="link_l" />
-        <origin rpy="1.57079632679 -1.57079632679 3.14159265359" xyz="0.155 -0.0425 0.285" />
-        <axis xyz="0 0 1" />
-        <limit effort="100" lower="-1.9198" upper="1.9198" velocity="2.9670" />
-    </joint>
-    <joint name="joint_u" type="revolute">
-        <parent link="link_l" />
-        <child link="link_u" />
-        <origin rpy="0 0 1.57079632679" xyz="0.614 0 -0.07" />
-        <axis xyz="0 0 -1" />
-        <limit effort="100" lower="-2.3561" upper="2.3561" velocity="2.9670" />
-    </joint>
-    <joint name="joint_r" type="revolute">
-        <parent link="link_u" />
-        <child link="link_r" />
-        <origin rpy="1.57079632679 0 -1.57079632679" xyz="0.265 -0.2 0.049" />
-        <axis xyz="0 0 1" />
-        <limit effort="100" lower="-3.1415" upper="3.1415" velocity="3.4906" />
-    </joint>
-    <joint name="joint_b" type="revolute">
-        <parent link="link_r" />
-        <child link="link_b" />
-        <origin rpy="1.57079632679 1.57079632679 0" xyz="0 -0.062 -0.375" />
-        <axis xyz="0 0 1" />
-        <limit effort="100" lower="-1.9198" upper="1.9198" velocity="3.4906" />
-    </joint>
-    <joint name="joint_t" type="revolute">
-        <parent link="link_b" />
-        <child link="link_t" />
-        <origin rpy="-1.57079632679 0 1.57079632679" xyz="0.0875 0 -0.062" />
-        <axis xyz="0 0 1" />
-        <limit effort="100" lower="-3.1415" upper="3.1415" velocity="6.9813" />
-    </joint>
-    <joint name="joint_tip" type="fixed">
-        <parent link="link_t" />
-        <child link="link_tip" />
-        <origin rpy="-2.35619449019 0 1.57079632679" xyz="-0.09591 0 -0.38772" />
-        <axis xyz="0 0 0" />
-    </joint>
-    <!-- end of joint list -->
-    <!-- ROS base_link (via base_link) to Motoman Robot (not Base) Frame transform -->
-    <link name="base" />
-    <joint name="base_link-base" type="fixed">
-        <origin rpy="0 0 0" xyz="0 0 0" />
-        <parent link="base_link" />
-        <child link="base" />
-    </joint>
-    <!-- Properties -->
-    <material name="yaskawa_blue">
-        <color rgba="0.12941 0.14902 0.74902 1" />
-    </material>
-    <!-- link list -->
-    <link name="d500_base_link">
-        <visual>
-            <geometry>
-                <mesh filename="package://motoman_motopos_d500_support/meshes/motopos_d500/visual/base_link.stl" />
-            </geometry>
-            <material name="yaskawa_blue" />
-        </visual>
-        <collision>
-            <geometry>
-                <mesh filename="package://motoman_motopos_d500_support/meshes/motopos_d500/collision/base_link.stl" />
-            </geometry>
-        </collision>
-<inertial>
-            <mass value="0.1" />
-            <inertia ixx="0.03" ixy="0.0" ixz="0.0" iyy="0.03" iyz="0.0" izz="0.03" />
-        </inertial>
-    </link>
-    <link name="d500_link_1">
-        <visual>
-            <geometry>
-                <mesh filename="package://motoman_motopos_d500_support/meshes/motopos_d500/visual/link_1.stl" />
-            </geometry>
-            <material name="yaskawa_blue" />
-        </visual>
-        <collision>
-            <geometry>
-                <mesh filename="package://motoman_motopos_d500_support/meshes/motopos_d500/collision/link_1.stl" />
-            </geometry>
-        </collision>
-<inertial>
-            <mass value="0.1" />
-            <inertia ixx="0.03" ixy="0.0" ixz="0.0" iyy="0.03" iyz="0.0" izz="0.03" />
-        </inertial>
-    </link>
-    <link name="d500_link_2">
-        <visual>
-            <geometry>
-                <mesh filename="package://motoman_motopos_d500_support/meshes/motopos_d500/visual/link_2.stl" />
-            </geometry>
-            <material name="yaskawa_blue" />
-        </visual>
-        <collision>
-            <geometry>
-                <mesh filename="package://motoman_motopos_d500_support/meshes/motopos_d500/collision/link_2.stl" />
-            </geometry>
-        </collision>
-<inertial>
-            <mass value="0.1" />
-            <inertia ixx="0.03" ixy="0.0" ixz="0.0" iyy="0.03" iyz="0.0" izz="0.03" />
-        </inertial>
-    </link>
-    <link name="d500_tool0" />
-    <!-- end of link list -->
-    <!-- joint list -->
-    <joint name="d500_world-base" type="fixed">
-        <origin rpy="0 0 0" xyz="1 0 0" />
-        <parent link="world" />
-        <child link="d500_base_link" />
-    </joint>
-    <joint name="joint_1" type="revolute">
-        <parent link="d500_base_link" />
-        <child link="d500_link_1" />
-        <origin rpy="0 0 0" xyz="0 0 0.380" />
-        <axis xyz="0 -1 0" />
-        <limit effort="1274" lower="-2.3561" upper="2.3561" velocity="1.3962" />
-    </joint>
-<transmission name="1_trans">
-        <type>transmission_interface/SimpleTransmission</type>
-        <actuator name="1_motor">
-            <mechanicalReduction>1</mechanicalReduction>
-        </actuator>
-        <joint name="joint_1">
-            <hardwareInterface>hardware_interface/PositionJointInterface</hardwareInterface>
-        </joint>
-    </transmission>
-    <joint name="joint_2" type="revolute">
-        <parent link="d500_link_1" />
-        <child link="d500_link_2" />
-        <origin rpy="0 0 0" xyz="0 0 0" />
-        <axis xyz="0 0 1" />
-        <limit effort="392" lower="-3.4906" upper="3.4906" velocity="2.7925" />
-    </joint>
-    <transmission name="2_trans">
-        <type>transmission_interface/SimpleTransmission</type>
-        <actuator name="2_motor">
-            <mechanicalReduction>1</mechanicalReduction>
-        </actuator>
-        <joint name="joint_2">
-            <hardwareInterface>hardware_interface/PositionJointInterface</hardwareInterface>
-        </joint>
-    </transmission>
-    <joint name="$joint_2-tool0" type="fixed">
-        <origin rpy="0 0 0" xyz="0 0 0.150 " />
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
File: motoman_ma1440_d500_support/urdf/ma1440_d500_macro.xacro (robot description, xacro)
@@ -3,5 +3,5 @@
      <xacro:macro name="motoman_ma1440_d500" params="prefix">
         <xacro:include filename="$(find motoman_ma1440_support)/urdf/ma1440/ma1440.xacro" prefix="ma1440_"/>
-        <!-- <xacro:include filename="$(find motoman_motopos_d500_support)/urdf/motopos_d500.xacro" prefix="d500_"/> -->
+        <xacro:include filename="$(find motoman_motopos_d500_support)/urdf/motopos_d500.xacro" prefix="d500_"/>
         <!-- <xacro:motoman_ma1440 prefix="${prefix}">
         </xacro:motoman_ma1440>       -->
