Commit message: FR-277 can now specify xyz/rpy for the world pose for ma1440 and d500. Modified the combined package to support this. Updated the joint names to properly prepend the prefix in the ma1440 and d500 robot urdfs. Updated moveit package for ma1440_d500 to reflect the new joint names.

File: motoman_ma1440_d500_support/urdf/ma1440_d500.xacro (robot description, xacro)
@@ -2,4 +2,4 @@
  <robot name="motoman_ma1440_d500" xmlns:xacro="http://ros.org/wiki/xacro">
 	<xacro:include filename="$(find motoman_ma1440_d500_support)/urdf/ma1440_d500_macro.xacro" />
-	<xacro:motoman_ma1440_d500 prefix=""/>
+	<xacro:motoman_ma1440_d500/>
 </robot>

File: motoman_ma1440_d500_support/urdf/ma1440_d500_macro.xacro (robot description, xacro)
@@ -1,11 +1,16 @@
 <?xml version="1.0" ?>
 <robot name="motoman_ma1440_d500" xmlns:xacro="http://ros.org/wiki/xacro">
-     <xacro:macro name="motoman_ma1440_d500" params="prefix">
-        <xacro:include filename="$(find motoman_ma1440_support)/urdf/ma1440/ma1440.xacro" prefix="ma1440_"/>
-        <xacro:include filename="$(find motoman_motopos_d500_support)/urdf/motopos_d500.xacro" prefix="d500_"/>
-        <!-- <xacro:motoman_ma1440 prefix="${prefix}">
-        </xacro:motoman_ma1440>       -->
-        <!-- <xacro:motoman_motopos_d500 prefix="${prefix}">
-        </xacro:motoman_motopos_d500> -->
-     </xacro:macro>
+  <!--  Default values for the world positions of the robots.
+  It has to be done like this, as you can't specify initial values that contain spaces in the macro line.-->
+  <xacro:property name="_ma1440_xyz" value="1 0 0"/>
+  <xacro:property name="_ma1440_rpy" value="0 0 0"/>
+  <xacro:property name="_d500_xyz" value="1 0 0"/>
+  <xacro:property name="_d500_rpy" value="0 0 0"/>
+  <xacro:macro name="motoman_ma1440_d500"
+               params="ma1440_xyz:=${_ma1440_xyz} ma1440_rpy:=${_ma1440_rpy} d500_xyz:=${_d500_xyz} d500_rpy=${_d500_rpy}">
+    <xacro:include filename="$(find motoman_ma1440_support)/urdf/ma1440/ma1440.xacro"/>
+    <xacro:load_motoman_ma1440 world_base_xyz="${_ma1440_xyz}" world_base_rpy="${_ma1440_rpy}"/>
+    <xacro:include filename="$(find motoman_motopos_d500_support)/urdf/motopos_d500.xacro"/>
+    <xacro:load_motoman_motopos_d500 world_base_xyz="${d500_xyz}" world_base_rpy="${d500_rpy}"/>
+  </xacro:macro>
 </robot>

File: motoman_ma1440_support/urdf/ma1440/ma1440.xacro (robot description, xacro)
@@ -5,4 +5,5 @@
     <xacro:motoman_ma1440 prefix=""/>
     <!-- optionally add the cam mount to the end of the arm, this is the laserscanner enclosure used on the Corsa system -->
+<!--    <xacro:if value="$(arg cam_mount)">-->
     <xacro:if value="$(arg cam_mount)">
         <xacro:include filename="$(find motoman_ma1440_support)/urdf/cam_mount/cam_mount.xacro" />

File: motoman_ma1440_support/urdf/ma1440/ma1440_macro.xacro (robot description, xacro)
@@ -1,7 +1,9 @@
 <?xml version="1.0" ?>
 <robot xmlns:xacro="http://ros.org/wiki/xacro">
+    <xacro:property name="world_base_xyz" value="0 0 0"/>
+    <xacro:property name="world_base_rpy" value="0 0 0"/>
     <xacro:property name="M_PI" value="3.1415926535897931"/>
     <xacro:include filename="$(find motoman_ma1440_support)/urdf/ma1440/ma1440.transmission.xacro" />
-    <xacro:macro name="motoman_ma1440" params="prefix">
+    <xacro:macro name="motoman_ma1440" params="prefix world_base_xyz:=^ world_base_rpy:=^">
         <!-- link list -->
         <link name="world">
@@ -229,5 +231,5 @@
         <!-- joint list -->
         <joint name="${prefix}world-base" type="fixed">
-            <origin xyz="0 0 0" rpy="0 0 0"/>
+            <origin xyz="${world_base_xyz}" rpy="${world_base_rpy}"/>
             <parent link="world" />
             <child link="${prefix}base_link"/>

File: motoman_motopos_d500_support/urdf/motopos_d500.xacro (robot description, xacro)
@@ -7,4 +7,6 @@
   <xacro:include filename="$(find motoman_motopos_d500_support)/urdf/motopos_d500.transmission.xacro" />
   <xacro:include filename="$(find motoman_motopos_d500_support)/urdf/motopos_d500_macro.xacro" />
-  <xacro:motoman_motopos_d500 prefix="d500_"/>
+  <xacro:macro name="load_motoman_motopos_d500" params="prefix:=d500_ world_base_xyz world_base_rpy">
+    <xacro:motoman_motopos_d500 prefix="${prefix}" world_base_xyz="${world_base_xyz}" world_base_rpy="${world_base_rpy}"/>
+  </xacro:macro>
 </robot>

File: motoman_motopos_d500_support/urdf/motopos_d500_macro.xacro (robot description, xacro)
@@ -1,5 +1,7 @@
 <?xml version="1.0" ?>
 <robot xmlns:xacro="http://www.ros.org/wiki/xacro">
-<xacro:macro name="motoman_motopos_d500" params="prefix">
+<xacro:property name="world_base_xyz" value="0 0 0"/>
+<xacro:property name="world_base_rpy" value="0 0 0"/>
+<xacro:macro name="motoman_motopos_d500" params="prefix world_base_xyz:=^ world_base_rpy:=^">
   <!-- link list -->
   <link name="${prefix}base_link">
@@ -46,9 +48,9 @@
   <!-- joint list -->
   <joint name="${prefix}world-base" type="fixed">
-      <origin xyz="1 0 0" rpy="0 0 0"/>
+      <origin xyz="${world_base_xyz}" rpy="${world_base_rpy}"/>
       <parent link="world" />
       <child link="${prefix}base_link"/>
   </joint>
-  <joint name="joint_1" type="revolute">
+  <joint name="${prefix}joint_1" type="revolute">
     <parent link="${prefix}base_link"/>
     <child link="${prefix}link_1"/>
@@ -58,5 +60,5 @@
   </joint>
   <xacro:transmission_macro name="1"/>
-  <joint name="joint_2" type="revolute">
+  <joint name="${prefix}joint_2" type="revolute">
     <parent link="${prefix}link_1"/>
     <child link="${prefix}link_2"/>
@@ -66,5 +68,5 @@
   </joint>
   <xacro:transmission_macro name="2"/>
-  <joint name="joint_2-tool0" type="fixed">
+  <joint name="${prefix}joint_2-tool0" type="fixed">
     <origin xyz="0 0 0.150 " rpy="0 0 0"/>
     <parent link="${prefix}link_2"/>

Commit message: FR-277 Added functionality for cell and launch parameters.

File: motoman_ma1440_d500_support/urdf/ma1440_d500.xacro (robot description, xacro)
@@ -1,4 +1,8 @@
 <?xml version="1.0" ?>
  <robot name="motoman_ma1440_d500" xmlns:xacro="http://ros.org/wiki/xacro">
+	<xacro:property name="ma1440_xyz" value="$(arg ma1440_xyz)"/>
+	<xacro:property name="ma1440_rpy" value="$(arg ma1440_rpy)"/>
+	<xacro:property name="d500_xyz" value="$(arg d500_xyz)"/>
+	<xacro:property name="d500_rpy" value="$(arg d500_rpy)"/>
 	<xacro:include filename="$(find motoman_ma1440_d500_support)/urdf/ma1440_d500_macro.xacro" />
 	<xacro:motoman_ma1440_d500/>

File: motoman_ma1440_d500_support/urdf/ma1440_d500_macro.xacro (robot description, xacro)
@@ -1,14 +1,7 @@
 <?xml version="1.0" ?>
 <robot name="motoman_ma1440_d500" xmlns:xacro="http://ros.org/wiki/xacro">
-  <!--  Default values for the world positions of the robots.
-  It has to be done like this, as you can't specify initial values that contain spaces in the macro line.-->
-  <xacro:property name="_ma1440_xyz" value="1 0 0"/>
-  <xacro:property name="_ma1440_rpy" value="0 0 0"/>
-  <xacro:property name="_d500_xyz" value="1 0 0"/>
-  <xacro:property name="_d500_rpy" value="0 0 0"/>
-  <xacro:macro name="motoman_ma1440_d500"
-               params="ma1440_xyz:=${_ma1440_xyz} ma1440_rpy:=${_ma1440_rpy} d500_xyz:=${_d500_xyz} d500_rpy=${_d500_rpy}">
+  <xacro:macro name="motoman_ma1440_d500" params="ma1440_xyz:=^ ma1440_rpy:=^ d500_xyz:=^ d500_rpy=^">
     <xacro:include filename="$(find motoman_ma1440_support)/urdf/ma1440/ma1440.xacro"/>
-    <xacro:load_motoman_ma1440 world_base_xyz="${_ma1440_xyz}" world_base_rpy="${_ma1440_rpy}"/>
+    <xacro:load_motoman_ma1440 world_base_xyz="${ma1440_xyz}" world_base_rpy="${ma1440_rpy}"/>
     <xacro:include filename="$(find motoman_motopos_d500_support)/urdf/motopos_d500.xacro"/>
     <xacro:load_motoman_motopos_d500 world_base_xyz="${d500_xyz}" world_base_rpy="${d500_rpy}"/>

File: motoman_ma1440_support/urdf/cam_mount/cam_mount.xacro (robot description, xacro)
@@ -1,4 +1,4 @@
 <?xml version="1.0"?>
-<robot name="cam_mount" xmlns:xacro="http://www.ros.org/wiki/xacro">
+<robot name="cam_mount" xmlns:xacro="http://ros.org/wiki/xacro">
   <!-- Constants for robot dimensions -->
   <xacro:property name="M_PI" value="3.1415926535897931"/>

File: motoman_ma1440_support/urdf/ma1440/ma1440.transmission.xacro (robot description, xacro)
@@ -1,4 +1,4 @@
 <?xml version="1.0"?>
-<robot xmlns:xacro="http://www.ros.org/wiki/xacro">
+<robot xmlns:xacro="http://ros.org/wiki/xacro">
   <!-- transmission macro -->
   <xacro:macro name="transmission_macro" params="name">

File: motoman_motopos_d500_support/urdf/motopos_d500.xacro (robot description, xacro)
@@ -1,4 +1,4 @@
 <?xml version="1.0" ?>
-<robot name="motoman_motopos_d500" xmlns:xacro="http://www.ros.org/wiki/xacro">
+<robot name="motoman_motopos_d500" xmlns:xacro="http://ros.org/wiki/xacro">
   <!-- Properties -->
   <material name="yaskawa_blue">

File: motoman_motopos_d500_support/urdf/motopos_d500_macro.xacro (robot description, xacro)
@@ -1,4 +1,4 @@
 <?xml version="1.0" ?>
-<robot xmlns:xacro="http://www.ros.org/wiki/xacro">
+<robot xmlns:xacro="http://ros.org/wiki/xacro">
 <xacro:property name="world_base_xyz" value="0 0 0"/>
 <xacro:property name="world_base_rpy" value="0 0 0"/>

Commit message: Add table_thickness parameter to D500 URDF This adds a parameter to offset to the tool frame by the thickness of the welding tabletop that's attached to the rotational link

File: motoman_ma1440_d500_support/urdf/ma1440_d500.xacro (robot description, xacro)
@@ -5,4 +5,5 @@
 	<xacro:property name="d500_xyz" value="$(arg d500_xyz)"/>
 	<xacro:property name="d500_rpy" value="$(arg d500_rpy)"/>
+	<xacro:property name="table_thickness" value="$(arg table_thickness)"/>
 	<xacro:include filename="$(find motoman_ma1440_d500_support)/urdf/ma1440_d500_macro.xacro" />
 	<xacro:motoman_ma1440_d500/>

File: motoman_ma1440_d500_support/urdf/ma1440_d500_macro.xacro (robot description, xacro)
@@ -1,9 +1,9 @@
 <?xml version="1.0" ?>
 <robot name="motoman_ma1440_d500" xmlns:xacro="http://ros.org/wiki/xacro">
-  <xacro:macro name="motoman_ma1440_d500" params="ma1440_xyz:=^ ma1440_rpy:=^ d500_xyz:=^ d500_rpy=^">
+  <xacro:macro name="motoman_ma1440_d500" params="ma1440_xyz:=^ ma1440_rpy:=^ d500_xyz:=^ d500_rpy:=^ table_thickness:=^">
     <xacro:include filename="$(find motoman_ma1440_support)/urdf/ma1440/ma1440.xacro"/>
     <xacro:load_motoman_ma1440 world_base_xyz="${ma1440_xyz}" world_base_rpy="${ma1440_rpy}"/>
     <xacro:include filename="$(find motoman_motopos_d500_support)/urdf/motopos_d500.xacro"/>
-    <xacro:load_motoman_motopos_d500 world_base_xyz="${d500_xyz}" world_base_rpy="${d500_rpy}"/>
+    <xacro:load_motoman_motopos_d500 world_base_xyz="${d500_xyz}" world_base_rpy="${d500_rpy}" table_thickness="${table_thickness}"/>
   </xacro:macro>
 </robot>

File: motoman_motopos_d500_support/urdf/motopos_d500.xacro (robot description, xacro)
@@ -7,6 +7,6 @@
   <xacro:include filename="$(find motoman_motopos_d500_support)/urdf/motopos_d500.transmission.xacro" />
   <xacro:include filename="$(find motoman_motopos_d500_support)/urdf/motopos_d500_macro.xacro" />
-  <xacro:macro name="load_motoman_motopos_d500" params="prefix:=d500_ world_base_xyz world_base_rpy">
-    <xacro:motoman_motopos_d500 prefix="${prefix}" world_base_xyz="${world_base_xyz}" world_base_rpy="${world_base_rpy}"/>
+  <xacro:macro name="load_motoman_motopos_d500" params="prefix:=d500_ world_base_xyz world_base_rpy table_thickness">
+    <xacro:motoman_motopos_d500 prefix="${prefix}" world_base_xyz="${world_base_xyz}" world_base_rpy="${world_base_rpy}" table_thickness="${table_thickness}"/>
   </xacro:macro>
 </robot>

File: motoman_motopos_d500_support/urdf/motopos_d500_macro.xacro (robot description, xacro)
@@ -3,5 +3,7 @@
 <xacro:property name="world_base_xyz" value="0 0 0"/>
 <xacro:property name="world_base_rpy" value="0 0 0"/>
-<xacro:macro name="motoman_motopos_d500" params="prefix world_base_xyz:=^ world_base_rpy:=^">
+<!-- offsets tool and positioner base/center frames to account for added tabletop -->
+<xacro:property name="table_thickness" default="0"/>
+<xacro:macro name="motoman_motopos_d500" params="prefix world_base_xyz:=^ world_base_rpy:=^ table_thickness:=^">
   <!-- link list -->
   <link name="${prefix}base_link">
@@ -45,4 +47,6 @@
   </link>
   <link name="${prefix}tool0"/>
+  <!-- this is here to set a base link in the URDF to link the positioner/base frame to for scanning -->
+  <link name="positioner_base_dummy_link"/>
   <!-- end of link list -->
   <!-- joint list -->
@@ -69,7 +73,13 @@
   <xacro:transmission_macro name="2"/>
   <joint name="${prefix}joint_2-tool0" type="fixed">
-    <origin xyz="0 0 0.150 " rpy="0 0 0"/>
+    <origin xyz="0 0 ${0.150 + table_thickness}" rpy="0 0 0"/>
     <parent link="${prefix}link_2"/>
     <child link="${prefix}tool0"/>
+  </joint>
+  <xacro:transmission_macro name="2"/>
+  <joint name="positioner_base_dummy_joint" type="fixed">
+    <origin xyz="0 0 ${0.150 + table_thickness}" rpy="0 0 0"/>
+    <parent link="${prefix}link_1"/>
+    <child link="positioner_base_dummy_link"/>
   </joint>
   <!-- end of joint list -->

Commit message: FR-249 Fixed URDF/SRDF issues so cam mount works. Fixed issue with calibration camera not having the correct encoding.

File: motoman_ma1440_d500_support/urdf/ma1440_d500.xacro (robot description, xacro)
@@ -6,4 +6,5 @@
 	<xacro:property name="d500_rpy" value="$(arg d500_rpy)"/>
 	<xacro:property name="table_thickness" value="$(arg table_thickness)"/>
+	<xacro:property name="using_cam_mount" value="$(arg using_cam_mount)"/>
 	<xacro:include filename="$(find motoman_ma1440_d500_support)/urdf/ma1440_d500_macro.xacro" />
 	<xacro:motoman_ma1440_d500/>

File: motoman_ma1440_d500_support/urdf/ma1440_d500_macro.xacro (robot description, xacro)
@@ -1,7 +1,7 @@
 <?xml version="1.0" ?>
 <robot name="motoman_ma1440_d500" xmlns:xacro="http://ros.org/wiki/xacro">
-  <xacro:macro name="motoman_ma1440_d500" params="ma1440_xyz:=^ ma1440_rpy:=^ d500_xyz:=^ d500_rpy:=^ table_thickness:=^">
+  <xacro:macro name="motoman_ma1440_d500" params="ma1440_xyz:=^ ma1440_rpy:=^ d500_xyz:=^ d500_rpy:=^ table_thickness:=^ using_cam_mount:=^">
     <xacro:include filename="$(find motoman_ma1440_support)/urdf/ma1440/ma1440.xacro"/>
-    <xacro:load_motoman_ma1440 world_base_xyz="${ma1440_xyz}" world_base_rpy="${ma1440_rpy}"/>
+    <xacro:load_motoman_ma1440 world_base_xyz="${ma1440_xyz}" world_base_rpy="${ma1440_rpy}" using_cam_mount="${using_cam_mount}"/>
     <xacro:include filename="$(find motoman_motopos_d500_support)/urdf/motopos_d500.xacro"/>
     <xacro:load_motoman_motopos_d500 world_base_xyz="${d500_xyz}" world_base_rpy="${d500_rpy}" table_thickness="${table_thickness}"/>

File: motoman_ma1440_support/urdf/cam_mount/cam_mount.xacro (robot description, xacro)
@@ -3,42 +3,44 @@
   <!-- Constants for robot dimensions -->
   <xacro:property name="M_PI" value="3.1415926535897931"/>
-  <link name="cam_mount_link">
-    <visual>
-      <origin
+  <xacro:macro name="cam_mount_load" params="prefix">
+    <link name="${prefix}cam_mount_link">
+      <visual>
+        <origin
+            xyz="0 0 0"
+            rpy="0 0 0" />
+        <geometry>
+          <mesh
+              filename="package://motoman_ma1440_support/meshes/cam_mount/visual/cam_mount_link.stl" />
+        </geometry>
+        <material
+            name="">
+          <color
+              rgba="0.75294 0.75294 0.75294 1" />
+        </material>
+      </visual>
+      <collision>
+        <origin
           xyz="0 0 0"
           rpy="0 0 0" />
-      <geometry>
-        <mesh
-            filename="package://motoman_ma1440_support/meshes/cam_mount/visual/cam_mount_link.stl" />
-      </geometry>
-      <material
-          name="">
-        <color
-            rgba="0.75294 0.75294 0.75294 1" />
-      </material>
-    </visual>
-    <collision>
-      <origin
-        xyz="0 0 0"
-        rpy="0 0 0" />
-      <geometry>
-        <mesh
-          filename="package://motoman_ma1440_support/meshes/cam_mount/collision/cam_mount_link_collision.stl" />
-      </geometry>
-    </collision>
-    <inertial>
-      <origin
-              xyz="-0.006942 -0.097138 0.034574"
-              rpy="0 0 0" />
-      <mass
-              value="4.0478" />
-      <inertia
-              ixx="0.00014683"
-              ixy="0.0000294"
-              ixz="-0.00002926"
-              iyy="0.000084784"
-              iyz="0.000073415"
-              izz="0.000085483" />
-    </inertial>
-  </link>
+        <geometry>
+          <mesh
+            filename="package://motoman_ma1440_support/meshes/cam_mount/collision/cam_mount_link_collision.stl" />
+        </geometry>
+      </collision>
+      <inertial>
+        <origin
+                xyz="-0.006942 -0.097138 0.034574"
+                rpy="0 0 0" />
+        <mass
+                value="4.0478" />
+        <inertia
+                ixx="0.00014683"
+                ixy="0.0000294"
+                ixz="-0.00002926"
+                iyy="0.000084784"
+                iyz="0.000073415"
+                izz="0.000085483" />
+      </inertial>
+    </link>
+  </xacro:macro>
 </robot>

File: motoman_ma1440_support/urdf/ma1440/ma1440.xacro (robot description, xacro)
@@ -1,18 +1,19 @@
 <?xml version="1.0" ?>
 <robot name="motoman_ma1440" xmlns:xacro="http://ros.org/wiki/xacro">
-    <xacro:arg name="cam_mount" default="false"/>
+    <xacro:arg name="using_cam_mount" default="false"/>
     <xacro:include filename="$(find motoman_ma1440_support)/urdf/ma1440/ma1440_macro.xacro" />
-    <xacro:macro name="load_motoman_ma1440" params="prefix:=ma1440_ world_base_xyz world_base_rpy">
+    <xacro:macro name="load_motoman_ma1440" params="prefix:=ma1440_ world_base_xyz world_base_rpy using_cam_mount:=false">
         <xacro:motoman_ma1440 prefix="${prefix}" world_base_xyz="${world_base_xyz}" world_base_rpy="${world_base_rpy}"/>
+        <!-- optionally add the cam mount to the end of the arm, this is the laserscanner enclosure used on the Corsa system -->
+        <xacro:if value="$(arg using_cam_mount)">
+            <xacro:include filename="$(find motoman_ma1440_support)/urdf/cam_mount/cam_mount.xacro" />
+            <xacro:cam_mount_load prefix="${prefix}"/>
+            <joint name="joint_cam_mount" type="fixed">
+                <origin xyz="0 0 -0.0735" rpy="${M_PI} 0 ${M_PI/2}" />
+                <parent link="${prefix}link_t" />
+                <child link="${prefix}cam_mount_link" />
+                <axis xyz="0 0 0" />
+            </joint>
+        </xacro:if>
     </xacro:macro>
-    <!-- optionally add the cam mount to the end of the arm, this is the laserscanner enclosure used on the Corsa system -->
-    <xacro:if value="$(arg cam_mount)">
-        <xacro:include filename="$(find motoman_ma1440_support)/urdf/cam_mount/cam_mount.xacro" />
-        <joint name="joint_cam_mount" type="fixed">
-            <origin xyz="0 0 -0.0735" rpy="${M_PI} 0 ${M_PI/2}" />
-            <parent link="link_t" />
-            <child link="cam_mount_link" />
-            <axis xyz="0 0 0" />
-        </joint>
-    </xacro:if>
 </robot>
