Commit message: FR-338 Now able to specify joint offset path.

File: motoman_ma1440_d500_support/urdf/ma1440_d500.xacro (robot description, xacro)
@@ -1,11 +1,20 @@
 <?xml version="1.0" ?>
  <robot name="motoman_ma1440_d500" xmlns:xacro="http://ros.org/wiki/xacro">
-	<xacro:property name="ma1440_xyz" value="$(arg ma1440_xyz)"/>
-	<xacro:property name="ma1440_rpy" value="$(arg ma1440_rpy)"/>
-	<xacro:property name="d500_xyz" value="$(arg d500_xyz)"/>
-	<xacro:property name="d500_rpy" value="$(arg d500_rpy)"/>
-	<xacro:property name="table_thickness" value="$(arg table_thickness)"/>
-	<xacro:property name="using_cam_mount" value="$(arg using_cam_mount)"/>
-	<xacro:include filename="$(find motoman_ma1440_d500_support)/urdf/ma1440_d500_macro.xacro" />
-	<xacro:motoman_ma1440_d500/>
+	<xacro:arg name="ma1440_xyz" default=""/>
+	<xacro:arg name="ma1440_rpy" default=""/>
+	<xacro:arg name="d500_xyz" default=""/>
+	<xacro:arg name="d500_rpy" default=""/>
+	<xacro:arg name="table_thickness" default=""/>
+	<xacro:arg name="using_cam_mount" default=""/>
+	<xacro:arg name="offsets_file_path" default=""/>
+	<xacro:include filename="$(find motoman_ma1440_d500_support)/urdf/ma1440_d500_macro.xacro"/>
+	<xacro:motoman_ma1440_d500
+			ma1440_xyz="$(arg ma1440_xyz)"
+			ma1440_rpy="$(arg ma1440_rpy)"
+			d500_xyz="$(arg d500_xyz)"
+			d500_rpy="$(arg d500_rpy)"
+			table_thickness="$(arg table_thickness)"
+			using_cam_mount="$(arg using_cam_mount)"
+			offsets_file_path="$(arg offsets_file_path)"
+	/>
 </robot>

File: motoman_ma1440_d500_support/urdf/ma1440_d500_macro.xacro (robot description, xacro)
@@ -1,7 +1,21 @@
 <?xml version="1.0" ?>
 <robot name="motoman_ma1440_d500" xmlns:xacro="http://ros.org/wiki/xacro">
-  <xacro:macro name="motoman_ma1440_d500" params="ma1440_xyz:=^ ma1440_rpy:=^ d500_xyz:=^ d500_rpy:=^ table_thickness:=^ using_cam_mount:=^">
+  <xacro:macro
+      name="motoman_ma1440_d500"
+      params=
+          "ma1440_xyz
+          ma1440_rpy
+          d500_xyz
+          d500_rpy
+          table_thickness
+          using_cam_mount
+          offsets_file_path">
     <xacro:include filename="$(find motoman_ma1440_support)/urdf/ma1440/ma1440.xacro"/>
-    <xacro:load_motoman_ma1440 world_base_xyz="${ma1440_xyz}" world_base_rpy="${ma1440_rpy}" using_cam_mount="${using_cam_mount}"/>
+    <xacro:load_motoman_ma1440
+        world_base_xyz="${ma1440_xyz}"
+        world_base_rpy="${ma1440_rpy}"
+        using_cam_mount="${using_cam_mount}"
+        offsets_file_path="${offsets_file_path}"
+    />
     <xacro:include filename="$(find motoman_motopos_d500_support)/urdf/motopos_d500.xacro"/>
     <xacro:load_motoman_motopos_d500 world_base_xyz="${d500_xyz}" world_base_rpy="${d500_rpy}" table_thickness="${table_thickness}"/>

File: motoman_ma1440_support/urdf/ma1440/ma1440.xacro (robot description, xacro)
@@ -1,10 +1,32 @@
 <?xml version="1.0" ?>
 <robot name="motoman_ma1440" xmlns:xacro="http://ros.org/wiki/xacro">
-    <xacro:arg name="using_cam_mount" default="false"/>
     <xacro:include filename="$(find motoman_ma1440_support)/urdf/ma1440/ma1440_macro.xacro" />
-    <xacro:macro name="load_motoman_ma1440" params="prefix:=ma1440_ world_base_xyz world_base_rpy using_cam_mount:=false">
-        <xacro:motoman_ma1440 prefix="${prefix}" world_base_xyz="${world_base_xyz}" world_base_rpy="${world_base_rpy}"/>
+    <xacro:macro
+        name="load_motoman_ma1440"
+        params="
+            prefix:=ma1440_
+            world_base_xyz
+            world_base_rpy
+            using_cam_mount:=false
+            offsets_file_path:='$(find motoman_ma1440_support)/config/robot_calibration_offsets.yaml'"
+    >
+        <xacro:unless value="${offsets_file_path == ''}">
+            <xacro:motoman_ma1440
+                prefix="${prefix}"
+                world_base_xyz="${world_base_xyz}"
+                world_base_rpy="${world_base_rpy}"
+                offsets_file_path="${offsets_file_path}"
+            />
+        </xacro:unless>
+        <xacro:if value="${offsets_file_path == ''}">
+            <xacro:motoman_ma1440
+                prefix="${prefix}"
+                world_base_xyz="${world_base_xyz}"
+                world_base_rpy="${world_base_rpy}"
+                offsets_file_path="'$(find motoman_ma1440_support)/config/robot_calibration_offsets.yaml'"
+            />
+        </xacro:if>
         <!-- optionally add the cam mount to the end of the arm, this is the laserscanner enclosure used on the Corsa system -->
-        <xacro:if value="$(arg using_cam_mount)">
+        <xacro:if value="${using_cam_mount}">
             <xacro:include filename="$(find motoman_ma1440_support)/urdf/cam_mount/cam_mount.xacro" />
             <xacro:cam_mount_load prefix="${prefix}"/>

File: motoman_ma1440_support/urdf/ma1440/ma1440_macro.xacro (robot description, xacro)
@@ -1,12 +1,15 @@
 <?xml version="1.0" ?>
 <robot xmlns:xacro="http://ros.org/wiki/xacro">
-    <xacro:property name="world_base_xyz" value="0 0 0"/>
-    <xacro:property name="world_base_rpy" value="0 0 0"/>
-    <xacro:property name="M_PI" value="3.1415926535897931"/>
-    <xacro:property name="offsets_file_path" value="$(find motoman_ma1440_support)/config/robot_calibration_offsets.yaml"/>
     <xacro:include filename="$(find motoman_ma1440_support)/urdf/ma1440/ma1440.transmission.xacro" />
-    <xacro:macro name="motoman_ma1440" params="prefix world_base_xyz:=^ world_base_rpy:=^ offsets_file_path:=^">
-        <xacro:property name="offsets" value="${load_yaml('$(find ma1400_sim)/config/robot_calibration_offsets.yaml')['robot_calibration_offsets']}"/>
-        <!-- link list -->
+    <xacro:macro
+        name="motoman_ma1440"
+        params="
+                 prefix
+                 world_base_xyz:='0 0 0'
+                 world_base_rpy:='0 0 0'
+                 offsets_file_path"
+    >
+      <xacro:property name="M_PI" value="3.1415926535897931"/>
+      <xacro:property name="offsets" value="${load_yaml(offsets_file_path)[prefix + 'robot_calibration_offsets']}"/>
         <link name="world">
             <origin xyz="0 0 0" rpy="0 0 0"/>
@@ -248,6 +251,6 @@
             <child link="${prefix}link_s"/>
             <origin
-                xyz="${offsets['joint_s']['x']} ${offsets['joint_s']['y']} ${0.165 + offsets['joint_s']['z']}"
-                rpy="${offsets['joint_s']['roll']} ${offsets['joint_s']['pitch']} ${offsets['joint_s']['yaw']}"
+                xyz="${offsets[prefix + 'joint_s']['x']} ${offsets[prefix + 'joint_s']['y']} ${0.165 + offsets[prefix + 'joint_s']['z']}"
+                rpy="${offsets[prefix + 'joint_s']['roll']} ${offsets[prefix + 'joint_s']['pitch']} ${offsets[prefix + 'joint_s']['yaw']}"
             />
             <axis xyz="0 0 1" />
@@ -259,6 +262,6 @@
             <child link="${prefix}link_l"/>
             <origin
-                xyz="${0.155 + offsets['joint_l']['x']} ${-0.0425 + offsets['joint_l']['y']} ${0.285 + offsets['joint_l']['z']}"
-                rpy="${M_PI/2 + offsets['joint_l']['roll']} ${-M_PI/2 + offsets['joint_l']['pitch']} ${M_PI + offsets['joint_l']['yaw']}"
+                xyz="${0.155 + offsets[prefix + 'joint_l']['x']} ${-0.0425 + offsets[prefix + 'joint_l']['y']} ${0.285 + offsets[prefix + 'joint_l']['z']}"
+                rpy="${M_PI/2 + offsets[prefix + 'joint_l']['roll']} ${-M_PI/2 + offsets[prefix + 'joint_l']['pitch']} ${M_PI + offsets[prefix + 'joint_l']['yaw']}"
             />
             <axis xyz="0 0 1" />
@@ -270,6 +273,6 @@
             <child link="${prefix}link_u"/>
             <origin
-                xyz="${0.614 + offsets['joint_u']['x']} ${0.0 + offsets['joint_u']['y']} ${-0.07 + offsets['joint_u']['z']}"
-                rpy="${0 + offsets['joint_u']['roll']} ${0 + offsets['joint_u']['pitch']} ${M_PI/2 + offsets['joint_u']['yaw']}"
+                xyz="${0.614 + offsets[prefix + 'joint_u']['x']} ${0.0 + offsets[prefix + 'joint_u']['y']} ${-0.07 + offsets[prefix + 'joint_u']['z']}"
+                rpy="${0 + offsets[prefix + 'joint_u']['roll']} ${0 + offsets[prefix + 'joint_u']['pitch']} ${M_PI/2 + offsets[prefix + 'joint_u']['yaw']}"
             />
             <axis xyz="0 0 -1" />
@@ -283,6 +286,6 @@
             <child link="${prefix}link_r"/>
             <origin
-                xyz="${0.265 + offsets['joint_r']['x']} ${-0.2 + offsets['joint_r']['y']} ${0.049 + offsets['joint_r']['z']}"
-                rpy="${M_PI/2 + offsets['joint_r']['roll']} ${0 + offsets['joint_r']['pitch']} ${-M_PI/2 + offsets['joint_r']['yaw']}"
+                xyz="${0.265 + offsets[prefix + 'joint_r']['x']} ${-0.2 + offsets[prefix + 'joint_r']['y']} ${0.049 + offsets[prefix + 'joint_r']['z']}"
+                rpy="${M_PI/2 + offsets[prefix + 'joint_r']['roll']} ${0 + offsets[prefix + 'joint_r']['pitch']} ${-M_PI/2 + offsets[prefix + 'joint_r']['yaw']}"
             />
             <axis xyz="0 0 1" />
@@ -294,6 +297,6 @@
             <child link="${prefix}link_b"/>
             <origin
-                xyz="${0.0 + offsets['joint_b']['x']} ${-0.062 + offsets['joint_b']['y']} ${-0.375 + offsets['joint_b']['z']}"
-                rpy="${M_PI/2 + offsets['joint_b']['roll']} ${M_PI/2 + offsets['joint_b']['pitch']} ${0 + offsets['joint_b']['yaw']}"
+                xyz="${0.0 + offsets[prefix + 'joint_b']['x']} ${-0.062 + offsets[prefix + 'joint_b']['y']} ${-0.375 + offsets[prefix + 'joint_b']['z']}"
+                rpy="${M_PI/2 + offsets[prefix + 'joint_b']['roll']} ${M_PI/2 + offsets[prefix + 'joint_b']['pitch']} ${0 + offsets[prefix + 'joint_b']['yaw']}"
             />
             <axis xyz="0 0 1" />
@@ -307,6 +310,6 @@
             <child link="${prefix}link_t"/>
             <origin
-                xyz="${0.0875 + offsets['joint_t']['x']} ${0.0 + offsets['joint_t']['y']} ${-0.062 + offsets['joint_t']['z']}"
-                rpy="${-M_PI/2 + offsets['joint_t']['roll']} ${0 + offsets['joint_t']['pitch']} ${M_PI/2 + offsets['joint_t']['yaw']}"
+                xyz="${0.0875 + offsets[prefix + 'joint_t']['x']} ${0.0 + offsets[prefix + 'joint_t']['y']} ${-0.062 + offsets[prefix + 'joint_t']['z']}"
+                rpy="${-M_PI/2 + offsets[prefix + 'joint_t']['roll']} ${0 + offsets[prefix + 'joint_t']['pitch']} ${M_PI/2 + offsets[prefix + 'joint_t']['yaw']}"
             />
             <axis xyz="0 0 1" />

Commit message: included support for laser mount

File: motoman_ma1440_d500_support/urdf/ma1440_d500.xacro (robot description, xacro)
@@ -7,4 +7,5 @@
 	<xacro:arg name="table_thickness" default=""/>
 	<xacro:arg name="using_cam_mount" default=""/>
+	<xacro:arg name="using_laser_mount" default=""/>
 	<xacro:arg name="offsets_file_path" default=""/>
 	<xacro:include filename="$(find motoman_ma1440_d500_support)/urdf/ma1440_d500_macro.xacro"/>
@@ -16,4 +17,5 @@
 			table_thickness="$(arg table_thickness)"
 			using_cam_mount="$(arg using_cam_mount)"
+			using_laser_mount="$(arg using_laser_mount)"
 			offsets_file_path="$(arg offsets_file_path)"
 	/>

File: motoman_ma1440_d500_support/urdf/ma1440_d500_macro.xacro (robot description, xacro)
@@ -10,4 +10,5 @@
           table_thickness
           using_cam_mount
+          using_laser_mount
           offsets_file_path"
   >
@@ -17,4 +18,5 @@
         world_base_rpy="${ma1440_rpy}"
         using_cam_mount="${using_cam_mount}"
+        using_laser_mount="${using_laser_mount}"
         offsets_file_path="${offsets_file_path}"
     />

File: motoman_ma1440_mh185_rotisserie_support/urdf/ma1440_mh185_rotisserie.xacro (robot description, xacro)
@@ -6,4 +6,5 @@
 	<xacro:arg name="mh185_rpy" default=""/>
 	<xacro:arg name="using_cam_mount" default=""/>
+	<xacro:arg name="using_laser_mount" default=""/>
 	<xacro:arg name="offsets_file_path" default=""/>
 	<xacro:include filename="$(find motoman_ma1440_mh185_rotisserie_support)/urdf/ma1440_mh185_rotisserie_macro.xacro" />
@@ -14,4 +15,5 @@
 			mh185_rpy="$(arg mh185_rpy)"
 			using_cam_mount="$(arg using_cam_mount)"
+			using_laser_mount="$(arg using_laser_mount)"
 			offsets_file_path="$(arg offsets_file_path)"
 	/>

File: motoman_ma1440_mh185_rotisserie_support/urdf/ma1440_mh185_rotisserie_macro.xacro (robot description, xacro)
@@ -9,4 +9,5 @@
           mh185_rpy
           using_cam_mount
+          using_laser_mount
           offsets_file_path"
   >
@@ -16,4 +17,5 @@
         world_base_rpy="${ma1440_rpy}"
         using_cam_mount="${using_cam_mount}"
+        using_laser_mount="${using_laser_mount}"
         offsets_file_path="${offsets_file_path}"
     />

File: motoman_ma1440_support/urdf/ma1440/ma1440.xacro (robot description, xacro)
@@ -9,4 +9,5 @@
             world_base_rpy
             using_cam_mount:=false
+            using_laser_mount:=false
             offsets_file_path:='$(find motoman_ma1440_support)/config/robot_calibration_offsets.yaml'">
         <xacro:unless value="${offsets_file_path == ''}">
@@ -26,5 +27,5 @@
             />
         </xacro:if>
-        <!-- optionally add the cam mount to the end of the arm, this is the laserscanner enclosure used on the Corsa system -->
+        <!-- optionally add the cam mount to the end of the arm, this is the laser scanner enclosure used on the Corsa system -->
         <xacro:if value="${using_cam_mount}">
             <xacro:include filename="$(find motoman_ma1440_support)/urdf/cam_mount/cam_mount.xacro" />
@@ -37,4 +38,56 @@
             </joint>
         </xacro:if>
+        <xacro:if value="${using_laser_mount}">
+            <xacro:include filename="$(find motoman_ma1440_support)/urdf/laser_mount/laser_mount.xacro" />
+            <xacro:laser_mount_load prefix="${prefix}"/>
+            <joint name="joint_laser_mount" type="fixed">
+                <origin xyz="0 0 -0.0735" rpy="${M_PI} 0 ${M_PI/2}" />
+                <parent link="${prefix}link_t" />
+                <child link="${prefix}laser_mount_center_link" />
+                <axis xyz="0 0 0" />
+            </joint>
+            <joint name="joint_laser_center_to_receiver_1" type="fixed">
+                <origin xyz="0.0807 0.0777 -0.0508" rpy="0 0 0"/>
+                <parent link="${prefix}laser_mount_center_link"/>
+                <child link ="${prefix}laser_1_receiver_dummy_link"/>
+                <axis xyz="0 0 0"/>
+            </joint>
+            <joint name="joint_laser_center_to_receiver_2" type="fixed">
+                <origin xyz="-0.0807 0.0777 -0.0508" rpy="0 0 0"/>
+                <parent link="${prefix}laser_mount_center_link"/>
+                <child link ="${prefix}laser_2_receiver_dummy_link"/>
+                <axis xyz="0 0 0"/>
+            </joint>
+            <joint name="joint_laser_center_to_emitter_1" type="fixed">
+                <origin xyz="0.06788 -0.023345 -0.0508" rpy="0 0 0"/>
+                <parent link="${prefix}laser_mount_center_link"/>
+                <child link ="${prefix}laser_1_emitter_dummy_link"/>
+                <axis xyz="0 0 0"/>
+            </joint>
+            <joint name="joint_laser_center_to_emitter_2" type="fixed">
+                <origin xyz="0.03370 -0.063387 -0.0508" rpy="0 0 0"/>
+                <parent link="${prefix}laser_mount_center_link"/>
+                <child link ="${prefix}laser_2_emitter_dummy_link"/>
+                <axis xyz="0 0 0"/>
+            </joint>
+            <joint name="joint_laser_center_to_emitter_3" type="fixed">
+                <origin xyz="-0.03370 -0.063387 -0.0508" rpy="0 0 0"/>
+                <parent link="${prefix}laser_mount_center_link"/>
+                <child link ="${prefix}laser_3_emitter_dummy_link"/>
+                <axis xyz="0 0 0"/>
+            </joint>
+            <joint name="joint_laser_center_to_emitter_4" type="fixed">
+                <origin xyz="-0.06788 -0.023345 -0.0508" rpy="0 0 0"/>
+                <parent link="${prefix}laser_mount_center_link"/>
+                <child link ="${prefix}laser_4_emitter_dummy_link"/>
+                <axis xyz="0 0 0"/>
+            </joint>
+            <joint name="joint_laser_center_to_receiver_3" type="fixed">
+                <origin xyz="0.0 -0.093345 -0.0508" rpy="0 0 0"/>
+                <parent link="${prefix}laser_mount_center_link"/>
+                <child link ="${prefix}laser_3_receiver_dummy_link"/>
+                <axis xyz="0 0 0"/>
+            </joint>
+        </xacro:if>
     </xacro:macro>
 </robot>

Commit message: Add SL gantry model to URDF packages Note: right now this is in the MA1440 package for simplicity, but might be bettter suited in another package

File: motoman_ma1440_d500_support/urdf/ma1440_d500.xacro (robot description, xacro)
@@ -6,4 +6,5 @@
 	<xacro:arg name="d500_rpy" default=""/>
 	<xacro:arg name="table_thickness" default=""/>
+	<xacro:arg name="use_structured_light_gantry" default=""/>
 	<xacro:arg name="offsets_file_path" default=""/>
 	<xacro:arg name="mount_type" default=""/>
@@ -15,4 +16,5 @@
 			d500_rpy="$(arg d500_rpy)"
 			table_thickness="$(arg table_thickness)"
+			use_structured_light_gantry="$(arg use_structured_light_gantry)"
 			offsets_file_path="$(arg offsets_file_path)"
 			mount_type="$(arg mount_type)"

File: motoman_ma1440_d500_support/urdf/ma1440_d500_macro.xacro (robot description, xacro)
@@ -10,4 +10,5 @@
           table_thickness
           mount_type
+          use_structured_light_gantry
           offsets_file_path"
   >
@@ -17,4 +18,5 @@
         world_base_rpy="${ma1440_rpy}"
         offsets_file_path="${offsets_file_path}"
+        use_structured_light_gantry="${use_structured_light_gantry}"
         mount_type="${mount_type}"
     />

File: motoman_ma1440_mh185_rotisserie_support/urdf/ma1440_mh185_rotisserie.xacro (robot description, xacro)
@@ -6,4 +6,5 @@
 	<xacro:arg name="mh185_rpy" default=""/>
 	<xacro:arg name="mount_type" default=""/>
+	<xacro:arg name="use_structured_light_gantry" default=""/>
 	<xacro:arg name="offsets_file_path" default=""/>
 	<xacro:include filename="$(find motoman_ma1440_mh185_rotisserie_support)/urdf/ma1440_mh185_rotisserie_macro.xacro" />
@@ -14,4 +15,5 @@
 			mh185_rpy="$(arg mh185_rpy)"
 			mount_type="$(arg mount_type)"
+			use_structured_light_gantry="$(arg use_structured_light_gantry)"
 			offsets_file_path="$(arg offsets_file_path)"
 	/>

File: motoman_ma1440_mh185_rotisserie_support/urdf/ma1440_mh185_rotisserie_macro.xacro (robot description, xacro)
@@ -9,4 +9,5 @@
           mh185_rpy
           mount_type
+          use_structured_light_gantry
           offsets_file_path"
   >
@@ -16,4 +17,5 @@
         world_base_rpy="${ma1440_rpy}"
         mount_type="${mount_type}"
+        use_structured_light_gantry="${use_structured_light_gantry}"
         offsets_file_path="${offsets_file_path}"
     />

File: motoman_ma1440_mh185_vertical_support/urdf/ma1440_mh185_vertical.xacro (robot description, xacro)
@@ -6,4 +6,5 @@
 	<xacro:arg name="mh185_vertical_rpy" default=""/>
 	<xacro:arg name="mount_type" default=""/>
+	<xacro:arg name="use_structured_light_gantry" default=""/>
 	<xacro:arg name="offsets_file_path" default=""/>
 	<xacro:include filename="$(find motoman_ma1440_mh185_vertical_support)/urdf/ma1440_mh185_vertical_macro.xacro" />
@@ -14,4 +15,5 @@
 			mh185_vertical_rpy="$(arg mh185_vertical_rpy)"
 			mount_type="$(arg mount_type)"
+			use_structured_light_gantry="$(arg use_structured_light_gantry)"
 			offsets_file_path="$(arg offsets_file_path)"
 	/>

File: motoman_ma1440_mh185_vertical_support/urdf/ma1440_mh185_vertical_macro.xacro (robot description, xacro)
@@ -9,4 +9,5 @@
           mh185_vertical_rpy
           mount_type
+          use_structured_light_gantry
           offsets_file_path"
   >
@@ -16,4 +17,5 @@
         world_base_rpy="${ma1440_rpy}"
         mount_type="${mount_type}"
+        use_structured_light_gantry="$(arg use_structured_light_gantry)"
         offsets_file_path="${offsets_file_path}"
     />

File: motoman_ma1440_support/urdf/ma1440/ma1440.xacro (robot description, xacro)
@@ -9,4 +9,5 @@
             world_base_rpy
             mount_type
+            use_structured_light_gantry
             offsets_file_path:='$(find motoman_ma1440_support)/config/robot_calibration_offsets.yaml'">
         <xacro:unless value="${offsets_file_path == ''}">
@@ -25,4 +26,14 @@
                 offsets_file_path="'$(find motoman_ma1440_support)/config/robot_calibration_offsets.yaml'"
             />
+        </xacro:if>
+        <xacro:if value="${use_structured_light_gantry}">
+            <xacro:include filename="$(find motoman_ma1440_support)/urdf/structured_light_gantry/structured_light_gantry.xacro" />
+            <xacro:structured_light_gantry_load/>
+            <joint name="gantry_mount_joint" type="fixed">
+                <origin xyz="2.2 -1.35 0" rpy="0 0 ${M_PI/2}" />
+                <parent link="world" />
+                <child link="structured_light_gantry_link" />
+                <axis xyz="0 0 0" />
+            </joint>
         </xacro:if>
         <!-- optionally add the cam mount to the end of the arm, this is the laser scanner enclosure used on the Corsa system -->
