Commit message: FR-516 Added pedestal option to ma1440. Streamlined launch/xacro files.

File: motoman_ma1440_d500_support/urdf/ma1440_d500.xacro (robot description, xacro)
@@ -7,4 +7,5 @@
 	<xacro:arg name="table_thickness" default=""/>
 	<xacro:arg name="use_structured_light_gantry" default=""/>
+	<xacro:arg name="use_pedestal" default=""/>
 	<xacro:arg name="offsets_file_path" default=""/>
 	<xacro:arg name="mount_type" default=""/>
@@ -17,4 +18,5 @@
 			table_thickness="$(arg table_thickness)"
 			use_structured_light_gantry="$(arg use_structured_light_gantry)"
+			use_pedestal="$(arg use_pedestal)"
 			offsets_file_path="$(arg offsets_file_path)"
 			mount_type="$(arg mount_type)"

File: motoman_ma1440_d500_support/urdf/ma1440_d500_macro.xacro (robot description, xacro)
@@ -11,4 +11,5 @@
           mount_type
           use_structured_light_gantry
+          use_pedestal
           offsets_file_path"
   >
@@ -19,4 +20,5 @@
         offsets_file_path="${offsets_file_path}"
         use_structured_light_gantry="${use_structured_light_gantry}"
+        use_pedestal="${use_pedestal}"
         mount_type="${mount_type}"
     />

File: motoman_ma1440_mh185_rotisserie_support/urdf/ma1440_mh185_rotisserie.xacro (robot description, xacro)
@@ -7,4 +7,5 @@
 	<xacro:arg name="mount_type" default=""/>
 	<xacro:arg name="use_structured_light_gantry" default=""/>
+	<xacro:arg name="use_pedestal" default=""/>
 	<xacro:arg name="offsets_file_path" default=""/>
 	<xacro:include filename="$(find motoman_ma1440_mh185_rotisserie_support)/urdf/ma1440_mh185_rotisserie_macro.xacro" />
@@ -16,4 +17,5 @@
 			mount_type="$(arg mount_type)"
 			use_structured_light_gantry="$(arg use_structured_light_gantry)"
+			use_pedestal="$(arg use_pedestal)"
 			offsets_file_path="$(arg offsets_file_path)"
 	/>

File: motoman_ma1440_mh185_rotisserie_support/urdf/ma1440_mh185_rotisserie_macro.xacro (robot description, xacro)
@@ -10,4 +10,5 @@
           mount_type
           use_structured_light_gantry
+          use_pedestal
           offsets_file_path"
   >
@@ -18,4 +19,5 @@
         mount_type="${mount_type}"
         use_structured_light_gantry="${use_structured_light_gantry}"
+        use_pedestal="${use_pedestal}"
         offsets_file_path="${offsets_file_path}"
     />

File: motoman_ma1440_mh185_vertical_support/urdf/ma1440_mh185_vertical.xacro (robot description, xacro)
@@ -7,4 +7,5 @@
 	<xacro:arg name="mount_type" default=""/>
 	<xacro:arg name="use_structured_light_gantry" default=""/>
+	<xacro:arg name="use_pedestal" default=""/>
 	<xacro:arg name="offsets_file_path" default=""/>
 	<xacro:include filename="$(find motoman_ma1440_mh185_vertical_support)/urdf/ma1440_mh185_vertical_macro.xacro" />
@@ -16,4 +17,5 @@
 			mount_type="$(arg mount_type)"
 			use_structured_light_gantry="$(arg use_structured_light_gantry)"
+			use_pedestal="$(arg use_pedestal)"
 			offsets_file_path="$(arg offsets_file_path)"
 	/>

File: motoman_ma1440_mh185_vertical_support/urdf/ma1440_mh185_vertical_macro.xacro (robot description, xacro)
@@ -10,4 +10,5 @@
           mount_type
           use_structured_light_gantry
+          use_pedestal
           offsets_file_path"
   >
@@ -18,4 +19,5 @@
         mount_type="${mount_type}"
         use_structured_light_gantry="$(arg use_structured_light_gantry)"
+        use_pedestal="${use_pedestal}"
         offsets_file_path="${offsets_file_path}"
     />

File: motoman_ma1440_support/urdf/ma1440/ma1440.xacro (robot description, xacro)
@@ -2,4 +2,6 @@
 <robot name="motoman_ma1440" xmlns:xacro="http://ros.org/wiki/xacro">
     <xacro:include filename="$(find motoman_ma1440_support)/urdf/ma1440/ma1440_macro.xacro" />
+    <!-- TODO: The use_structured_light_gantry should not be taken care of in this file.
+                It is not a child of the ma1440. It should be constructed in a file that calls this one. -->
     <xacro:macro
         name="load_motoman_ma1440"
@@ -10,21 +12,16 @@
             mount_type
             use_structured_light_gantry
+            use_pedestal
             offsets_file_path:='$(find motoman_ma1440_support)/config/robot_calibration_offsets.yaml'">
-        <xacro:unless value="${offsets_file_path == ''}">
-            <xacro:motoman_ma1440
-                prefix="${prefix}"
-                world_base_xyz="${world_base_xyz}"
-                world_base_rpy="${world_base_rpy}"
-                offsets_file_path="${offsets_file_path}"
-            />
-        </xacro:unless>
-        <xacro:if value="${offsets_file_path == ''}">
-            <xacro:motoman_ma1440
-                prefix="${prefix}"
-                world_base_xyz="${world_base_xyz}"
-                world_base_rpy="${world_base_rpy}"
-                offsets_file_path="'$(find motoman_ma1440_support)/config/robot_calibration_offsets.yaml'"
-            />
-        </xacro:if>
+        <!-- This is a way to split up the xyz values. Leaving this here for future reference. -->
+        <!-- <xacro:property name="xyzList" value="${map(float, world_base_xyz.split())}"/> -->
+        <!-- world_base_xyz="${xyzList[0]} ${xyzList[1]} ${xyzList[2] + 0.7} if use_pedestal else world_base_xyz}" -->
+        <xacro:motoman_ma1440
+            prefix="${prefix}"
+            world_base_xyz="${world_base_xyz}"
+            world_base_rpy="${world_base_rpy}"
+            offsets_file_path="${offsets_file_path if offsets_file_path != '' else '$(find motoman_ma1440_support)/config/robot_calibration_offsets.yaml'}"
+            base_parent_link_name="${prefix+'pedestal_link' if use_pedestal else 'world'}"
+        />
         <xacro:if value="${use_structured_light_gantry}">
             <xacro:include filename="$(find motoman_ma1440_support)/urdf/structured_light_gantry/structured_light_gantry.xacro" />
@@ -36,4 +33,8 @@
                 <axis xyz="0 0 0" />
             </joint>
+        </xacro:if>
+        <xacro:if value="${use_pedestal}">
+            <xacro:include filename="$(find motoman_ma1440_support)/urdf/pedestal/pedestal.xacro" />
+            <xacro:pedestal_load prefix="${prefix}"/>
         </xacro:if>
         <!-- optionally add the cam mount to the end of the arm, this is the laser scanner enclosure used on the Corsa system -->

File: motoman_ma1440_support/urdf/ma1440/ma1440_macro.xacro (robot description, xacro)
@@ -8,5 +8,6 @@
                  world_base_xyz:='0 0 0'
                  world_base_rpy:='0 0 0'
-                 offsets_file_path"
+                 offsets_file_path
+                 base_parent_link_name:='world'"
     >
       <xacro:property name="M_PI" value="3.1415926535897931"/>
@@ -14,5 +15,5 @@
       <xacro:property name="M_PI_4" value="0.7853981633974483"/>
       <xacro:property name="offsets" value="${load_yaml(offsets_file_path)[prefix + 'robot_calibration_offsets']}"/>
-      <xacro:property name="vertical_offset" value="0.0"/>
+        <!-- TODO: This shouldn't be defined here. If there are two robots with world defined, things will break. Should be defined in the highest level file. -->
         <link name="world">
             <origin xyz="0 0 0" rpy="0 0 0"/>
@@ -252,6 +253,6 @@
         <!-- joint list -->
         <joint name="${prefix}world-base" type="fixed">
-            <origin xyz="0 0 ${vertical_offset}" rpy="${world_base_rpy}"/>
-            <parent link="world" />
+            <origin xyz="${world_base_xyz}" rpy="${world_base_rpy}"/>
+            <parent link="${base_parent_link_name}" />
             <child link="${prefix}base_link"/>
         </joint>
@@ -341,10 +342,10 @@
         <!-- end of joint list -->
         <!-- ROS base_link (via base_link) to Motoman Robot (not Base) Frame transform -->
-        <link name="${prefix}base" />
+        <!-- <link name="${prefix}base" />
         <joint name="${prefix}base_link-base" type="fixed">
             <origin rpy="0 0 0" xyz="0 0 0"/>
             <parent link="${prefix}base_link"/>
             <child link="${prefix}base"/>
-        </joint>
+        </joint> -->
     </xacro:macro>
 </robot>
