Commit message: hc10: use radians(..) convenience xacro function.
To specify joint position and velocity limits.

Also: fix joint B position limit.

File: motoman_hc10_support/urdf/hc10_macro.xacro (robot description, xacro)
@@ -106,5 +106,5 @@
         <origin xyz="0 0 0.275" rpy="0 0 0" />
         <axis xyz="0 0 1" />
-        <limit lower="-3.14159" upper="3.14159" effort="368.48" velocity="2.2689"/>
+        <limit lower="${radians(-180)}" upper="${radians(180)}" effort="368.48" velocity="${radians(130)}"/>
     </joint>
     <joint name="${prefix}joint_2_l" type="revolute">
@@ -113,5 +113,5 @@
         <origin xyz="0 0 0" rpy="0 0 0" />
         <axis xyz="0 1 0" />
-        <limit lower="-3.14159" upper="3.14159" effort="368.48" velocity="2.2689"/>
+        <limit lower="${radians(-180)}" upper="${radians(180)}" effort="368.48" velocity="${radians(130)}"/>
     </joint>
     <joint name="${prefix}joint_3_u" type="revolute">
@@ -120,5 +120,5 @@
         <origin xyz="0 0 0.700" rpy="0 0 0" />
         <axis xyz="0 -1 0" />
-        <limit lower="-0.08727" upper="6.19592" effort="141.12" velocity="3.1415"/>
+        <limit lower="${radians(-5)}" upper="${radians(355)}" effort="141.12" velocity="${radians(180)}"/>
     </joint>
     <joint name="${prefix}joint_4_r" type="revolute">
@@ -127,5 +127,5 @@
         <origin xyz="0 0 -0.500" rpy="0 0 0" />
         <axis xyz="0 0 1" />
-        <limit lower="-3.14159" upper="3.14159" effort="31.36" velocity="3.1415"/>
+        <limit lower="${radians(-180)}" upper="${radians(180)}" effort="31.36" velocity="${radians(180)}"/>
     </joint>
     <joint name="${prefix}joint_5_b" type="revolute">
@@ -134,5 +134,5 @@
         <origin xyz="0 0.162 0" rpy="0 0 0" />
         <axis xyz="0 -1 0" />
-        <limit lower="-2.6179" upper="2.6179" effort="31.36" velocity="4.36333"/>
+        <limit lower="${radians(-180)}" upper="${radians(180)}" effort="31.36" velocity="${radians(250)}"/>
     </joint>
     <joint name="${prefix}joint_6_t" type="revolute">
@@ -141,8 +141,8 @@
         <origin xyz="0 0 0" rpy="0 0 0" />
         <axis xyz="0 0 1" />
-        <limit lower="-3.14159" upper="3.14159" effort="31.36" velocity="4.36333"/>
+        <limit lower="${radians(-180)}" upper="${radians(180)}" effort="31.36" velocity="${radians(250)}"/>
     </joint>
     <joint name="${prefix}joint_6_t-tool0" type="fixed">
-        <origin xyz="0 0 -0.130" rpy="3.1415926 0 0"/>
+        <origin xyz="0 0 -0.130" rpy="${pi} 0 0"/>
         <parent link="${prefix}link_6_t"/>
         <child link="${prefix}tool0"/>

Commit message: hc10: correct effort limit for joint R.

File: motoman_hc10_support/urdf/hc10_macro.xacro (robot description, xacro)
@@ -127,5 +127,5 @@
         <origin xyz="0 0 -0.500" rpy="0 0 0" />
         <axis xyz="0 0 1" />
-        <limit lower="${radians(-180)}" upper="${radians(180)}" effort="31.36" velocity="${radians(180)}"/>
+        <limit lower="${radians(-180)}" upper="${radians(180)}" effort="39.20" velocity="${radians(180)}"/>
     </joint>
     <joint name="${prefix}joint_5_b" type="revolute">

Commit message: hc10: switch to Collada visual meshes.

File: motoman_hc10_support/urdf/hc10_macro.xacro (robot description, xacro)
@@ -10,5 +10,5 @@
         <visual>
             <geometry>
-                <mesh filename="package://motoman_hc10_support/meshes/hc10/visual/base_link.stl"/>
+                <mesh filename="package://motoman_hc10_support/meshes/hc10/visual/base_link.dae"/>
             </geometry>
             <material name="yaskawa_blue"/>
@@ -23,5 +23,5 @@
         <visual>
             <geometry>
-                <mesh filename="package://motoman_hc10_support/meshes/hc10/visual/link_1_s.stl"/>
+                <mesh filename="package://motoman_hc10_support/meshes/hc10/visual/link_1_s.dae"/>
             </geometry>
             <material name="yaskawa_blue"/>
@@ -36,5 +36,5 @@
         <visual>
             <geometry>
-                <mesh filename="package://motoman_hc10_support/meshes/hc10/visual/link_2_l.stl"/>
+                <mesh filename="package://motoman_hc10_support/meshes/hc10/visual/link_2_l.dae"/>
             </geometry>
             <material name="yaskawa_blue"/>
@@ -49,5 +49,5 @@
         <visual>
             <geometry>
-                <mesh filename="package://motoman_hc10_support/meshes/hc10/visual/link_3_u.stl"/>
+                <mesh filename="package://motoman_hc10_support/meshes/hc10/visual/link_3_u.dae"/>
             </geometry>
             <material name="yaskawa_blue"/>
@@ -62,5 +62,5 @@
         <visual>
             <geometry>
-                <mesh filename="package://motoman_hc10_support/meshes/hc10/visual/link_4_r.stl"/>
+                <mesh filename="package://motoman_hc10_support/meshes/hc10/visual/link_4_r.dae"/>
             </geometry>
             <material name="yaskawa_blue"/>
@@ -75,5 +75,5 @@
         <visual>
             <geometry>
-                <mesh filename="package://motoman_hc10_support/meshes/hc10/visual/link_5_b.stl"/>
+                <mesh filename="package://motoman_hc10_support/meshes/hc10/visual/link_5_b.dae"/>
             </geometry>
             <material name="yaskawa_blue"/>
@@ -88,5 +88,5 @@
         <visual>
             <geometry>
-                <mesh filename="package://motoman_hc10_support/meshes/hc10/visual/link_6_t.stl"/>
+                <mesh filename="package://motoman_hc10_support/meshes/hc10/visual/link_6_t.dae"/>
             </geometry>
             <material name="yaskawa_blue"/>

Commit message: hc10: use 2 space indent in xacro macro.

File: motoman_hc10_support/urdf/hc10_macro.xacro (robot description, xacro)
@@ -1,100 +1,100 @@
 <?xml version="1.0" ?>
 <robot xmlns:xacro="http://ros.org/wiki/xacro">
-<xacro:macro name="motoman_hc10" params="prefix">
+  <xacro:macro name="motoman_hc10" params="prefix">
     <!-- Properties -->
     <material name="yaskawa_blue">
-          <color rgba="0.12941 0.14902 0.74902 1" />
+      <color rgba="0.12941 0.14902 0.74902 1" />
     </material>
     <!-- link list -->
     <link name="${prefix}base_link">
-        <visual>
-            <geometry>
-                <mesh filename="package://motoman_hc10_support/meshes/hc10/visual/base_link.dae"/>
-            </geometry>
-            <material name="yaskawa_blue"/>
-        </visual>
-        <collision>
-            <geometry>
-                <mesh filename="package://motoman_hc10_support/meshes/hc10/collision/base_link.stl"/>
-            </geometry>
-        </collision>
+      <visual>
+        <geometry>
+          <mesh filename="package://motoman_hc10_support/meshes/hc10/visual/base_link.dae"/>
+        </geometry>
+        <material name="yaskawa_blue"/>
+      </visual>
+      <collision>
+        <geometry>
+          <mesh filename="package://motoman_hc10_support/meshes/hc10/collision/base_link.stl"/>
+        </geometry>
+      </collision>
     </link>
     <link name="${prefix}link_1_s">
-        <visual>
-            <geometry>
-                <mesh filename="package://motoman_hc10_support/meshes/hc10/visual/link_1_s.dae"/>
-            </geometry>
-            <material name="yaskawa_blue"/>
-        </visual>
-        <collision>
-            <geometry>
-                <mesh filename="package://motoman_hc10_support/meshes/hc10/collision/link_1_s.stl"/>
-            </geometry>
-        </collision>
+      <visual>
+        <geometry>
+          <mesh filename="package://motoman_hc10_support/meshes/hc10/visual/link_1_s.dae"/>
+        </geometry>
+        <material name="yaskawa_blue"/>
+      </visual>
+      <collision>
+        <geometry>
+          <mesh filename="package://motoman_hc10_support/meshes/hc10/collision/link_1_s.stl"/>
+        </geometry>
+      </collision>
     </link>
     <link name="${prefix}link_2_l">
-        <visual>
-            <geometry>
-                <mesh filename="package://motoman_hc10_support/meshes/hc10/visual/link_2_l.dae"/>
-            </geometry>
-            <material name="yaskawa_blue"/>
-        </visual>
-        <collision>
-            <geometry>
-                <mesh filename="package://motoman_hc10_support/meshes/hc10/collision/link_2_l.stl"/>
-            </geometry>
-        </collision>
+      <visual>
+        <geometry>
+          <mesh filename="package://motoman_hc10_support/meshes/hc10/visual/link_2_l.dae"/>
+        </geometry>
+        <material name="yaskawa_blue"/>
+      </visual>
+      <collision>
+        <geometry>
+          <mesh filename="package://motoman_hc10_support/meshes/hc10/collision/link_2_l.stl"/>
+        </geometry>
+      </collision>
     </link>
     <link name="${prefix}link_3_u">
-        <visual>
-            <geometry>
-                <mesh filename="package://motoman_hc10_support/meshes/hc10/visual/link_3_u.dae"/>
-            </geometry>
-            <material name="yaskawa_blue"/>
-        </visual>
-        <collision>
-            <geometry>
-                <mesh filename="package://motoman_hc10_support/meshes/hc10/collision/link_3_u.stl"/>
-            </geometry>
-        </collision>
+      <visual>
+        <geometry>
+          <mesh filename="package://motoman_hc10_support/meshes/hc10/visual/link_3_u.dae"/>
+        </geometry>
+        <material name="yaskawa_blue"/>
+      </visual>
+      <collision>
+        <geometry>
+          <mesh filename="package://motoman_hc10_support/meshes/hc10/collision/link_3_u.stl"/>
+        </geometry>
+      </collision>
     </link>
     <link name="${prefix}link_4_r">
-        <visual>
-            <geometry>
-                <mesh filename="package://motoman_hc10_support/meshes/hc10/visual/link_4_r.dae"/>
-            </geometry>
-            <material name="yaskawa_blue"/>
-        </visual>
-        <collision>
-            <geometry>
-                <mesh filename="package://motoman_hc10_support/meshes/hc10/collision/link_4_r.stl"/>
-            </geometry>
-        </collision>
+      <visual>
+        <geometry>
+          <mesh filename="package://motoman_hc10_support/meshes/hc10/visual/link_4_r.dae"/>
+        </geometry>
+        <material name="yaskawa_blue"/>
+      </visual>
+      <collision>
+        <geometry>
+          <mesh filename="package://motoman_hc10_support/meshes/hc10/collision/link_4_r.stl"/>
+        </geometry>
+      </collision>
     </link>
     <link name="${prefix}link_5_b">
-        <visual>
-            <geometry>
-                <mesh filename="package://motoman_hc10_support/meshes/hc10/visual/link_5_b.dae"/>
-            </geometry>
-            <material name="yaskawa_blue"/>
-        </visual>
-        <collision>
-            <geometry>
-                <mesh filename="package://motoman_hc10_support/meshes/hc10/collision/link_5_b.stl"/>
-            </geometry>
-        </collision>
+      <visual>
+        <geometry>
+          <mesh filename="package://motoman_hc10_support/meshes/hc10/visual/link_5_b.dae"/>
+        </geometry>
+        <material name="yaskawa_blue"/>
+      </visual>
+      <collision>
+        <geometry>
+          <mesh filename="package://motoman_hc10_support/meshes/hc10/collision/link_5_b.stl"/>
+        </geometry>
+      </collision>
     </link>
     <link name="${prefix}link_6_t">
-        <visual>
-            <geometry>
-                <mesh filename="package://motoman_hc10_support/meshes/hc10/visual/link_6_t.dae"/>
-            </geometry>
-            <material name="yaskawa_blue"/>
-        </visual>
-        <collision>
-            <geometry>
-                <mesh filename="package://motoman_hc10_support/meshes/hc10/collision/link_6_t.stl"/>
-            </geometry>
-        </collision>
+      <visual>
+        <geometry>
+          <mesh filename="package://motoman_hc10_support/meshes/hc10/visual/link_6_t.dae"/>
+        </geometry>
+        <material name="yaskawa_blue"/>
+      </visual>
+      <collision>
+        <geometry>
+          <mesh filename="package://motoman_hc10_support/meshes/hc10/collision/link_6_t.stl"/>
+        </geometry>
+      </collision>
     </link>
     <link name="${prefix}tool0"/>
@@ -102,49 +102,49 @@
     <!-- joint list -->
     <joint name="${prefix}joint_1_s" type="revolute">
-        <parent link="${prefix}base_link"/>
-        <child link="${prefix}link_1_s"/>
-        <origin xyz="0 0 0.275" rpy="0 0 0" />
-        <axis xyz="0 0 1" />
-        <limit lower="${radians(-180)}" upper="${radians(180)}" effort="368.48" velocity="${radians(130)}"/>
+      <parent link="${prefix}base_link"/>
+      <child link="${prefix}link_1_s"/>
+      <origin xyz="0 0 0.275" rpy="0 0 0" />
+      <axis xyz="0 0 1" />
+      <limit lower="${radians(-180)}" upper="${radians(180)}" effort="368.48" velocity="${radians(130)}"/>
     </joint>
     <joint name="${prefix}joint_2_l" type="revolute">
-        <parent link="${prefix}link_1_s"/>
-        <child link="${prefix}link_2_l"/>
-        <origin xyz="0 0 0" rpy="0 0 0" />
-        <axis xyz="0 1 0" />
-        <limit lower="${radians(-180)}" upper="${radians(180)}" effort="368.48" velocity="${radians(130)}"/>
+      <parent link="${prefix}link_1_s"/>
+      <child link="${prefix}link_2_l"/>
+      <origin xyz="0 0 0" rpy="0 0 0" />
+      <axis xyz="0 1 0" />
+      <limit lower="${radians(-180)}" upper="${radians(180)}" effort="368.48" velocity="${radians(130)}"/>
     </joint>
     <joint name="${prefix}joint_3_u" type="revolute">
-        <parent link="${prefix}link_2_l"/>
-        <child link="${prefix}link_3_u"/>
-        <origin xyz="0 0 0.700" rpy="0 0 0" />
-        <axis xyz="0 -1 0" />
-        <limit lower="${radians(-5)}" upper="${radians(355)}" effort="141.12" velocity="${radians(180)}"/>
+      <parent link="${prefix}link_2_l"/>
+      <child link="${prefix}link_3_u"/>
+      <origin xyz="0 0 0.700" rpy="0 0 0" />
+      <axis xyz="0 -1 0" />
+      <limit lower="${radians(-5)}" upper="${radians(355)}" effort="141.12" velocity="${radians(180)}"/>
     </joint>
     <joint name="${prefix}joint_4_r" type="revolute">
-        <parent link="${prefix}link_3_u"/>
-        <child link="${prefix}link_4_r"/>
-        <origin xyz="0 0 -0.500" rpy="0 0 0" />
-        <axis xyz="0 0 1" />
-        <limit lower="${radians(-180)}" upper="${radians(180)}" effort="39.20" velocity="${radians(180)}"/>
+      <parent link="${prefix}link_3_u"/>
+      <child link="${prefix}link_4_r"/>
+      <origin xyz="0 0 -0.500" rpy="0 0 0" />
+      <axis xyz="0 0 1" />
+      <limit lower="${radians(-180)}" upper="${radians(180)}" effort="39.20" velocity="${radians(180)}"/>
     </joint>
     <joint name="${prefix}joint_5_b" type="revolute">
-        <parent link="${prefix}link_4_r"/>
-        <child link="${prefix}link_5_b"/>
-        <origin xyz="0 0.162 0" rpy="0 0 0" />
-        <axis xyz="0 -1 0" />
-        <limit lower="${radians(-180)}" upper="${radians(180)}" effort="31.36" velocity="${radians(250)}"/>
+      <parent link="${prefix}link_4_r"/>
+      <child link="${prefix}link_5_b"/>
+      <origin xyz="0 0.162 0" rpy="0 0 0" />
+      <axis xyz="0 -1 0" />
+      <limit lower="${radians(-180)}" upper="${radians(180)}" effort="31.36" velocity="${radians(250)}"/>
     </joint>
     <joint name="${prefix}joint_6_t" type="revolute">
-        <parent link="${prefix}link_5_b"/>
-        <child link="${prefix}link_6_t"/>
-        <origin xyz="0 0 0" rpy="0 0 0" />
-        <axis xyz="0 0 1" />
-        <limit lower="${radians(-180)}" upper="${radians(180)}" effort="31.36" velocity="${radians(250)}"/>
+      <parent link="${prefix}link_5_b"/>
+      <child link="${prefix}link_6_t"/>
+      <origin xyz="0 0 0" rpy="0 0 0" />
+      <axis xyz="0 0 1" />
+      <limit lower="${radians(-180)}" upper="${radians(180)}" effort="31.36" velocity="${radians(250)}"/>
     </joint>
     <joint name="${prefix}joint_6_t-tool0" type="fixed">
-        <origin xyz="0 0 -0.130" rpy="${pi} 0 0"/>
-        <parent link="${prefix}link_6_t"/>
-        <child link="${prefix}tool0"/>
+      <origin xyz="0 0 -0.130" rpy="${pi} 0 0"/>
+      <parent link="${prefix}link_6_t"/>
+      <child link="${prefix}tool0"/>
     </joint>
     <!-- end of joint list -->
@@ -152,8 +152,8 @@
     <link name="${prefix}base" />
     <joint name="${prefix}base_link-base" type="fixed">
-        <origin xyz="0 0 0.275" rpy="0 0 0"/>
-        <parent link="${prefix}base_link"/>
-        <child link="${prefix}base"/>
+      <origin xyz="0 0 0.275" rpy="0 0 0"/>
+      <parent link="${prefix}base_link"/>
+      <child link="${prefix}base"/>
     </joint>
-    </xacro:macro>
+  </xacro:macro>
 </robot>
