Commit message: Update hc10dt_b10_macro.xacro
Added 'flange' link to model

File: motoman_hc10_support/urdf/hc10dt_b10_macro.xacro (robot description, xacro)
@@ -95,5 +95,4 @@
       </collision>
     </link>
-    <link name="${prefix}tool0"/>
     <!-- end of link list -->
     <!-- joint list -->
@@ -140,10 +139,19 @@
       <limit lower="${radians(-180)}" upper="${radians(180)}" effort="31.36" velocity="${radians(250)}"/>
     </joint>
-    <joint name="${prefix}joint_6_t-tool0" type="fixed">
+    <!-- end of joint list -->
+    <!-- ROS-Industrial 'flange' frame: attachment point for EEF models -->
+    <link name="${prefix}flange"/>
+    <joint name="${prefix}joint_6_t-flange" type="fixed">
       <origin xyz="0.170 0 0" rpy="${radians(180)} ${radians(-90)} 0"/>
       <parent link="${prefix}link_6_t"/>
+      <child link="${prefix}flange"/>
+    </joint>
+    <!-- ROS-Industrial 'tool0' frame: all-zeros tool frame -->
+    <link name="${prefix}tool0"/>
+    <joint name="${prefix}flange-tool0" type="fixed">
+      <origin xyz="0 0 0" rpy="0 0 0"/>
+      <parent link="${prefix}flange"/>
       <child link="${prefix}tool0"/>
     </joint>
-    <!-- end of joint list -->
     <!-- ROS base_link to Robot Manufacturer World Coordinates transform -->
     <link name="${prefix}base" />

Commit message: hc10: fix orientation of flange and tool0
flange == attachment point for EEF (sub)models, and as such should follow REP-103 (ie: X+ out of flange, in "forward" direction (link-local)).

tool0 == an "all-zeros toolframe", corresponding to the OEMs definition. For Yaskawa, this has Z+ forward.

File: motoman_hc10_support/urdf/hc10dt_b10_macro.xacro (robot description, xacro)
@@ -143,5 +143,5 @@
     <link name="${prefix}flange"/>
     <joint name="${prefix}joint_6_t-flange" type="fixed">
-      <origin xyz="0.170 0 0" rpy="${radians(180)} ${radians(-90)} 0"/>
+      <origin xyz="0.170 0 0" rpy="0 0 0"/>
       <parent link="${prefix}link_6_t"/>
       <child link="${prefix}flange"/>
@@ -150,5 +150,5 @@
     <link name="${prefix}tool0"/>
     <joint name="${prefix}flange-tool0" type="fixed">
-      <origin xyz="0 0 0" rpy="0 0 0"/>
+      <origin xyz="0 0 0" rpy="${radians(180)} ${radians(-90)} 0"/>
       <parent link="${prefix}flange"/>
       <child link="${prefix}tool0"/>
