Commit message: hc10: store variant meshes in separate dir.

File: motoman_hc10_support/urdf/hc10dt_macro.xacro (robot description, xacro)
@@ -104,5 +104,5 @@
       <visual>
         <geometry>
-          <mesh filename="package://motoman_hc10_support/meshes/hc10/visual/link_6_dt.stl"/>
+          <mesh filename="package://motoman_hc10_support/meshes/hc10dt/visual/link_6_dt.stl"/>
         </geometry>
         <material name="yaskawa_white"/>
@@ -110,5 +110,5 @@
       <collision>
         <geometry>
-          <mesh filename="package://motoman_hc10_support/meshes/hc10/collision/link_6_dt.stl"/>
+          <mesh filename="package://motoman_hc10_support/meshes/hc10dt/collision/link_6_dt.stl"/>
        </geometry>
       </collision>

Commit message: hc10: don't add link for DT device.
But attach it directly to link_6.

File: motoman_hc10_support/urdf/hc10dt_macro.xacro (robot description, xacro)
@@ -91,5 +91,5 @@
       <visual>
         <geometry>
-          <mesh filename="package://motoman_hc10_support/meshes/hc10/visual/link_6_t.dae"/>
+          <mesh filename="package://motoman_hc10_support/meshes/hc10dt/visual/link_6_t.stl"/>
         </geometry>
         <material name="yaskawa_blue"/>
@@ -97,18 +97,5 @@
       <collision>
         <geometry>
-          <mesh filename="package://motoman_hc10_support/meshes/hc10/collision/link_6_t.stl"/>
-       </geometry>
-      </collision>
-    </link>
-    <link name="${prefix}link_6_dt">
-      <visual>
-        <geometry>
-          <mesh filename="package://motoman_hc10_support/meshes/hc10dt/visual/link_6_dt.stl"/>
-        </geometry>
-        <material name="yaskawa_white"/>
-      </visual>
-      <collision>
-        <geometry>
-          <mesh filename="package://motoman_hc10_support/meshes/hc10dt/collision/link_6_dt.stl"/>
+          <mesh filename="package://motoman_hc10_support/meshes/hc10dt/collision/link_6_t.stl"/>
        </geometry>
       </collision>
@@ -159,9 +146,4 @@
       <limit lower="${radians(-180)}" upper="${radians(180)}" effort="31.36" velocity="${radians(250)}"/>
     </joint>
-    <joint name="${prefix}joint_6_dt" type="fixed">
-      <parent link="${prefix}link_6_t"/>
-      <child link="${prefix}link_6_dt"/>
-      <origin xyz="0 0 0" rpy="0 0 0" />
-    </joint>
     <joint name="${prefix}joint_6_t-tool0" type="fixed">
       <origin xyz="0 0 -0.170" rpy="${pi} 0 0"/>

Commit message: hc10: alternative mesh for link_6 and DT.

File: motoman_hc10_support/urdf/hc10dt_macro.xacro (robot description, xacro)
@@ -91,5 +91,5 @@
       <visual>
         <geometry>
-          <mesh filename="package://motoman_hc10_support/meshes/hc10dt/visual/link_6_t.stl"/>
+          <mesh filename="package://motoman_hc10_support/meshes/hc10dt/visual/link_6_t.dae"/>
         </geometry>
         <material name="yaskawa_blue"/>

Commit message: joint trajectory streaming demo

File: motoman_hc10_support/urdf/hc10dt_macro.xacro (robot description, xacro)
@@ -115,7 +115,7 @@
       <parent link="${prefix}link_2_l"/>
       <child link="${prefix}link_3_u"/>
-      <origin xyz="0 0 0.700" rpy="0 0 0" />
+      <origin xyz="0 0 0.700" rpy="0 ${radians(-90)}  0" />
       <axis xyz="0 -1 0" />
-      <limit lower="${radians(-5)}" upper="${radians(355)}" effort="141.12" velocity="${radians(180)}"/>
+      <limit lower="${radians(-288)}" upper="${radians(288)}" effort="141.12" velocity="${radians(180)}"/>
     </joint>
     <joint name="${prefix}joint_4_r" type="revolute">
