Commit message: fixed issues with inconsistent naming of joints

File: motoman_ma1440_mh185_rotisserie_support/urdf/ma1440_mh185_rotisserie.xacro (robot description, xacro)
@@ -1,9 +1,9 @@
 <?xml version="1.0" ?>
  <robot name="motoman_ma1440_mh185_rotisserie" xmlns:xacro="http://ros.org/wiki/xacro">
-	<xacro:arg name="ma1440_xyz" default="0 0 0"/>
-	<xacro:arg name="ma1440_rpy" default="0 0 0 "/>
-	<xacro:arg name="mh185_xyz" default="0 0 0"/>
-	<xacro:arg name="mh185_rpy" default="0 0 0"/>
-	<xacro:arg name="using_cam_mount" default="true"/>
+	<xacro:arg name="ma1440_xyz" default=""/>
+	<xacro:arg name="ma1440_rpy" default=""/>
+	<xacro:arg name="mh185_xyz" default=""/>
+	<xacro:arg name="mh185_rpy" default=""/>
+	<xacro:arg name="using_cam_mount" default=""/>
 	<xacro:arg name="offsets_file_path" default=""/>
 	<xacro:include filename="$(find motoman_ma1440_mh185_rotisserie_support)/urdf/ma1440_mh185_rotisserie_macro.xacro" />

File: motoman_ma1440_mh185_vertical_support/urdf/ma1440_mh185_vertical_macro.xacro (robot description, xacro)
@@ -14,5 +14,5 @@
     <xacro:load_motoman_ma1440
         world_base_xyz="${ma1440_xyz}"
-        world_base_rpy="${ma1440_rpy}"
+        world_base_rpy="${ma1440_rpy }"
         using_cam_mount="${using_cam_mount}"
         offsets_file_path="${offsets_file_path}"

File: motoman_motopos_mh185_rotisserie_support/urdf/headstock/headstock.urdf.xacro (robot description, xacro)
@@ -22,6 +22,4 @@
         izz="7.6922" />
     </inertial>
-    <xacro:arg name="visible" default="true"/>
-    <xacro:if value="$(arg visible)">
       <visual>
         <origin
@@ -38,5 +36,4 @@
         </material>
       </visual>
-    </xacro:if>
     <collision>
       <origin
@@ -50,5 +47,5 @@
   </link>
   <joint
-    name="joint_x"
+    name="mh185_joint_1"
     type="revolute">
     <origin
@@ -84,5 +81,4 @@
         izz="0.037392" />
     </inertial>
-    <xacro:if value="$(arg visible)">
       <visual>
         <origin
@@ -99,5 +95,4 @@
         </material>
       </visual>
-    </xacro:if>
     <collision>
       <origin
@@ -139,5 +134,4 @@
         izz="0.0066005" />
     </inertial>
-    <xacro:if value="$(arg visible)">
       <visual>
         <origin
@@ -154,5 +148,4 @@
         </material>
       </visual>
-    </xacro:if>
     <collision>
       <origin

File: motoman_motopos_mh185_rotisserie_support/urdf/motopos_mh185_rotisserie_macro.xacro (robot description, xacro)
@@ -5,24 +5,19 @@
     params=
         "prefix
-        world_base_xyz:='0 0 0'
-        world_base_rpy:='0 0 0'
+        world_base_xyz
+        world_base_rpy
         offsets_file_path"
 >
   <xacro:property name="M_PI" value="3.1415926535897931"/>
   <xacro:property name="offsets" value="${load_yaml(offsets_file_path)[prefix + 'robot_calibration_offsets']}"/>
-<xacro:property name="pos2b_tf" value="${load_yaml('$(find motoman_motopos_mh185_rotisserie_support)/config/positioner_params.yaml')}"/>
-  <xacro:property name="pos2b_trans" value="${pos2b_tf['positioner_params']['positioner_to_base_tf']['translation']}" />
-  <xacro:property name="pos2b_rot" value="${pos2b_tf['positioner_params']['positioner_to_base_tf']['rotation']}" />
-  <xacro:property name="pos2b_xyz" value="${pos2b_trans['x']} ${pos2b_trans['y']} ${pos2b_trans['z']}"/>
-  <xacro:property name="pos2b_rpy" value="${pos2b_rot['roll']} ${pos2b_rot['pitch']} ${pos2b_rot['yaw']}"/>
 <xacro:property name="world_to_pos_base_tf" value="${load_yaml('$(find motoman_motopos_mh185_rotisserie_support)/config/positioner_params.yaml')}"/>
-  <xacro:property name="world2pos_t" value="${pos2b_tf['positioner_params']['base_to_positioner_tf']['translation']}" />
-  <xacro:property name="world2pos_rot" value="${pos2b_tf['positioner_params']['base_to_positioner_tf']['rotation']}" />
+  <xacro:property name="world2pos_t" value="${world_to_pos_base_tf['positioner_params']['base_to_positioner_tf']['translation']}" />
+  <xacro:property name="world2pos_rot" value="${world_to_pos_base_tf['positioner_params']['base_to_positioner_tf']['rotation']}" />
   <xacro:property name="world2pos_xyz" value="${world2pos_t['x']} ${world2pos_t['y']} ${world2pos_t['z']}"/>
   <xacro:property name="world2pos_rpy" value="${world2pos_rot['roll']} ${world2pos_rot['pitch']} ${world2pos_rot['yaw']}"/>
   <!-- Tailstock offsets. Should be loaded from yaml file created during calibration. -->
   <xacro:property name="ts_base_offset" value="0.06985" />
-  <xacro:property name="ts_revolute_offset" value="${pos2b_tf['positioner_params']['tailstock_revolute_offset']}" />
-  <xacro:property name="hs_prismatic_offset" value="${pos2b_tf['positioner_params']['headstock_prismatic_offset']}"/>
+  <xacro:property name="ts_revolute_offset" value="${world_to_pos_base_tf['positioner_params']['tailstock_revolute_offset']}" />
+  <xacro:property name="hs_prismatic_offset" value="${world_to_pos_base_tf['positioner_params']['headstock_prismatic_offset']}"/>
   <!-- Define a fixed joint macro -->
   <xacro:macro name="fixed_joint_macro" params="name origin_xyz origin_rpy parent child axis_xyz">
@@ -39,9 +34,18 @@
   <xacro:include filename="$(find motoman_motopos_mh185_rotisserie_support)/urdf/tailstock/tailstock.urdf.xacro" ns="ts" />
   <!-- And connect positioner_link to base_link -->
+  <link name="${prefix}base_link"/>
   <!-- hs_base - positioner_link->base_link -->
-  <xacro:fixed_joint_macro name="world-hsbase"
+  <xacro:property name="world2base_xyz" value="${world_base_xyz}"/>
+  <xacro:property name="world2base_rpy" value="${world_base_rpy}"/>
+  <xacro:fixed_joint_macro name="${prefix}world-base"
+                           origin_rpy="${world2base_rpy}"
+                           origin_xyz="${world2base_xyz}"
+                           parent="world"
+                           child="${prefix}base_link"
+                           axis_xyz="0 0 0"/>
+  <xacro:fixed_joint_macro name="base-hsbase"
                            origin_xyz="${world2pos_xyz}"
                            origin_rpy="${world2pos_rpy}"
-                           parent="world"
+                           parent="${prefix}base_link"
                            child="hs_base_link"
                            axis_xyz="1 0 0" />

File: motoman_motopos_mh185_rotisserie_support/urdf/tailstock/tailstock.urdf.xacro (robot description, xacro)
@@ -3,5 +3,4 @@
   <!-- Constants for robot dimensions -->
   <xacro:property name="M_PI" value="3.1415926535897931"/>
-  <xacro:arg name="visible" default="true"/>
   <link
     name="ts_base_link">
@@ -20,5 +19,4 @@
         izz="0.19362" />
     </inertial>
-    <xacro:if value="$(arg visible)">
       <visual>
         <origin
@@ -35,5 +33,4 @@
         </material>
       </visual>
-    </xacro:if>
     <collision>
       <origin
@@ -62,5 +59,4 @@
         izz="3.7157" />
     </inertial>
-    <xacro:if value="$(arg visible)">
       <visual>
         <origin
@@ -77,5 +73,4 @@
         </material>
       </visual>
-    </xacro:if>
     <collision>
       <origin
@@ -104,5 +99,4 @@
         izz="0.017007" />
     </inertial>
-    <xacro:if value="$(arg visible)">
       <visual>
         <origin
@@ -119,5 +113,4 @@
         </material>
       </visual>
-    </xacro:if>
     <collision>
       <origin

Commit message: fixed issues with inconsistent joint names

File: motoman_ma1440_mh185_rotisserie_support/urdf/ma1440_mh185_rotisserie.xacro (robot description, xacro)
@@ -1,9 +1,9 @@
 <?xml version="1.0" ?>
  <robot name="motoman_ma1440_mh185_rotisserie" xmlns:xacro="http://ros.org/wiki/xacro">
-	<xacro:arg name="ma1440_xyz" default=""/>
-	<xacro:arg name="ma1440_rpy" default=""/>
-	<xacro:arg name="mh185_xyz" default=""/>
-	<xacro:arg name="mh185_rpy" default=""/>
-	<xacro:arg name="using_cam_mount" default=""/>
+	<xacro:arg name="ma1440_xyz" default="0 0 0"/>
+	<xacro:arg name="ma1440_rpy" default="0 0 0 "/>
+	<xacro:arg name="mh185_xyz" default="0 0 0"/>
+	<xacro:arg name="mh185_rpy" default="0 0 0"/>
+	<xacro:arg name="using_cam_mount" default="true"/>
 	<xacro:arg name="offsets_file_path" default=""/>
 	<xacro:include filename="$(find motoman_ma1440_mh185_rotisserie_support)/urdf/ma1440_mh185_rotisserie_macro.xacro" />

File: motoman_ma1440_mh185_vertical_support/urdf/ma1440_mh185_vertical_macro.xacro (robot description, xacro)
@@ -14,5 +14,5 @@
     <xacro:load_motoman_ma1440
         world_base_xyz="${ma1440_xyz}"
-        world_base_rpy="${ma1440_rpy }"
+        world_base_rpy="${ma1440_rpy}"
         using_cam_mount="${using_cam_mount}"
         offsets_file_path="${offsets_file_path}"

File: motoman_motopos_mh185_rotisserie_support/urdf/headstock/headstock.urdf.xacro (robot description, xacro)
@@ -22,4 +22,6 @@
         izz="7.6922" />
     </inertial>
+    <xacro:arg name="visible" default="true"/>
+    <xacro:if value="$(arg visible)">
       <visual>
         <origin
@@ -36,4 +38,5 @@
         </material>
       </visual>
+    </xacro:if>
     <collision>
       <origin
@@ -47,5 +50,5 @@
   </link>
   <joint
-    name="mh185_joint_1"
+    name="joint_x"
     type="revolute">
     <origin
@@ -81,4 +84,5 @@
         izz="0.037392" />
     </inertial>
+    <xacro:if value="$(arg visible)">
       <visual>
         <origin
@@ -95,4 +99,5 @@
         </material>
       </visual>
+    </xacro:if>
     <collision>
       <origin
@@ -134,4 +139,5 @@
         izz="0.0066005" />
     </inertial>
+    <xacro:if value="$(arg visible)">
       <visual>
         <origin
@@ -148,4 +154,5 @@
         </material>
       </visual>
+    </xacro:if>
     <collision>
       <origin

File: motoman_motopos_mh185_rotisserie_support/urdf/motopos_mh185_rotisserie_macro.xacro (robot description, xacro)
@@ -5,19 +5,24 @@
     params=
         "prefix
-        world_base_xyz
-        world_base_rpy
+        world_base_xyz:='0 0 0'
+        world_base_rpy:='0 0 0'
         offsets_file_path"
 >
   <xacro:property name="M_PI" value="3.1415926535897931"/>
   <xacro:property name="offsets" value="${load_yaml(offsets_file_path)[prefix + 'robot_calibration_offsets']}"/>
+<xacro:property name="pos2b_tf" value="${load_yaml('$(find motoman_motopos_mh185_rotisserie_support)/config/positioner_params.yaml')}"/>
+  <xacro:property name="pos2b_trans" value="${pos2b_tf['positioner_params']['positioner_to_base_tf']['translation']}" />
+  <xacro:property name="pos2b_rot" value="${pos2b_tf['positioner_params']['positioner_to_base_tf']['rotation']}" />
+  <xacro:property name="pos2b_xyz" value="${pos2b_trans['x']} ${pos2b_trans['y']} ${pos2b_trans['z']}"/>
+  <xacro:property name="pos2b_rpy" value="${pos2b_rot['roll']} ${pos2b_rot['pitch']} ${pos2b_rot['yaw']}"/>
 <xacro:property name="world_to_pos_base_tf" value="${load_yaml('$(find motoman_motopos_mh185_rotisserie_support)/config/positioner_params.yaml')}"/>
-  <xacro:property name="world2pos_t" value="${world_to_pos_base_tf['positioner_params']['base_to_positioner_tf']['translation']}" />
-  <xacro:property name="world2pos_rot" value="${world_to_pos_base_tf['positioner_params']['base_to_positioner_tf']['rotation']}" />
+  <xacro:property name="world2pos_t" value="${pos2b_tf['positioner_params']['base_to_positioner_tf']['translation']}" />
+  <xacro:property name="world2pos_rot" value="${pos2b_tf['positioner_params']['base_to_positioner_tf']['rotation']}" />
   <xacro:property name="world2pos_xyz" value="${world2pos_t['x']} ${world2pos_t['y']} ${world2pos_t['z']}"/>
   <xacro:property name="world2pos_rpy" value="${world2pos_rot['roll']} ${world2pos_rot['pitch']} ${world2pos_rot['yaw']}"/>
   <!-- Tailstock offsets. Should be loaded from yaml file created during calibration. -->
   <xacro:property name="ts_base_offset" value="0.06985" />
-  <xacro:property name="ts_revolute_offset" value="${world_to_pos_base_tf['positioner_params']['tailstock_revolute_offset']}" />
-  <xacro:property name="hs_prismatic_offset" value="${world_to_pos_base_tf['positioner_params']['headstock_prismatic_offset']}"/>
+  <xacro:property name="ts_revolute_offset" value="${pos2b_tf['positioner_params']['tailstock_revolute_offset']}" />
+  <xacro:property name="hs_prismatic_offset" value="${pos2b_tf['positioner_params']['headstock_prismatic_offset']}"/>
   <!-- Define a fixed joint macro -->
   <xacro:macro name="fixed_joint_macro" params="name origin_xyz origin_rpy parent child axis_xyz">
@@ -34,18 +39,9 @@
   <xacro:include filename="$(find motoman_motopos_mh185_rotisserie_support)/urdf/tailstock/tailstock.urdf.xacro" ns="ts" />
   <!-- And connect positioner_link to base_link -->
-  <link name="${prefix}base_link"/>
   <!-- hs_base - positioner_link->base_link -->
-  <xacro:property name="world2base_xyz" value="${world_base_xyz}"/>
-  <xacro:property name="world2base_rpy" value="${world_base_rpy}"/>
-  <xacro:fixed_joint_macro name="${prefix}world-base"
-                           origin_rpy="${world2base_rpy}"
-                           origin_xyz="${world2base_xyz}"
-                           parent="world"
-                           child="${prefix}base_link"
-                           axis_xyz="0 0 0"/>
-  <xacro:fixed_joint_macro name="base-hsbase"
+  <xacro:fixed_joint_macro name="world-hsbase"
                            origin_xyz="${world2pos_xyz}"
                            origin_rpy="${world2pos_rpy}"
-                           parent="${prefix}base_link"
+                           parent="world"
                            child="hs_base_link"
                            axis_xyz="1 0 0" />

File: motoman_motopos_mh185_rotisserie_support/urdf/tailstock/tailstock.urdf.xacro (robot description, xacro)
@@ -3,4 +3,5 @@
   <!-- Constants for robot dimensions -->
   <xacro:property name="M_PI" value="3.1415926535897931"/>
+  <xacro:arg name="visible" default="true"/>
   <link
     name="ts_base_link">
@@ -19,4 +20,5 @@
         izz="0.19362" />
     </inertial>
+    <xacro:if value="$(arg visible)">
       <visual>
         <origin
@@ -33,4 +35,5 @@
         </material>
       </visual>
+    </xacro:if>
     <collision>
       <origin
@@ -59,4 +62,5 @@
         izz="3.7157" />
     </inertial>
+    <xacro:if value="$(arg visible)">
       <visual>
         <origin
@@ -73,4 +77,5 @@
         </material>
       </visual>
+    </xacro:if>
     <collision>
       <origin
@@ -99,4 +104,5 @@
         izz="0.017007" />
     </inertial>
+    <xacro:if value="$(arg visible)">
       <visual>
         <origin
@@ -113,4 +119,5 @@
         </material>
       </visual>
+    </xacro:if>
     <collision>
       <origin
