Commit message: GP25 Update 1 making corrections based on reviews

File: motoman_gp25_support/urdf/gp25_macro.xacro (robot description, xacro)
@@ -10,5 +10,5 @@
         <visual>
             <geometry>
-                <mesh filename="package://motoman_gp25_support/meshes/visual/gp25_base_link.stl"/>
+                <mesh filename="package://motoman_gp25_support/meshes/visual/base_link.stl"/>
             </geometry>
             <material name="yaskawa_blue"/>
@@ -16,5 +16,5 @@
         <collision>
             <geometry>
-                <mesh filename="package://motoman_gp25_support/meshes/collision/gp25_base_link.stl"/>
+                <mesh filename="package://motoman_gp25_support/meshes/collision/base_link.stl"/>
             </geometry>
         </collision>
@@ -23,5 +23,5 @@
         <visual>
             <geometry>
-                <mesh filename="package://motoman_gp25_support/meshes/visual/gp25_link_1_s.stl"/>
+                <mesh filename="package://motoman_gp25_support/meshes/visual/link_1_s.stl"/>
             </geometry>
             <material name="yaskawa_blue"/>
@@ -29,5 +29,5 @@
         <collision>
             <geometry>
-                <mesh filename="package://motoman_gp25_support/meshes/collision/gp25_link_1_s.stl"/>
+                <mesh filename="package://motoman_gp25_support/meshes/collision/link_1_s.stl"/>
             </geometry>
         </collision>
@@ -36,5 +36,5 @@
         <visual>
             <geometry>
-                <mesh filename="package://motoman_gp25_support/meshes/visual/gp25_link_2_l.stl"/>
+                <mesh filename="package://motoman_gp25_support/meshes/visual/link_2_l.stl"/>
             </geometry>
             <material name="yaskawa_blue"/>
@@ -42,5 +42,5 @@
         <collision>
             <geometry>
-                <mesh filename="package://motoman_gp25_support/meshes/collision/gp25_link_2_l.stl"/>
+                <mesh filename="package://motoman_gp25_support/meshes/collision/link_2_l.stl"/>
             </geometry>
         </collision>
@@ -49,5 +49,5 @@
         <visual>
             <geometry>
-                <mesh filename="package://motoman_gp25_support/meshes/visual/gp25_link_3_u.stl"/>
+                <mesh filename="package://motoman_gp25_support/meshes/visual/link_3_u.stl"/>
             </geometry>
             <material name="yaskawa_blue"/>
@@ -55,5 +55,5 @@
         <collision>
             <geometry>
-                <mesh filename="package://motoman_gp25_support/meshes/collision/gp25_link_3_u.stl"/>
+                <mesh filename="package://motoman_gp25_support/meshes/collision/link_3_u.stl"/>
             </geometry>
         </collision>
@@ -62,5 +62,5 @@
         <visual>
             <geometry>
-                <mesh filename="package://motoman_gp25_support/meshes/visual/gp25_link_4_r.stl"/>
+                <mesh filename="package://motoman_gp25_support/meshes/visual/link_4_r.stl"/>
             </geometry>
             <material name="yaskawa_blue"/>
@@ -68,5 +68,5 @@
         <collision>
             <geometry>
-                <mesh filename="package://motoman_gp25_support/meshes/collision/gp25_link_4_r.stl"/>
+                <mesh filename="package://motoman_gp25_support/meshes/collision/link_4_r.stl"/>
             </geometry>
         </collision>
@@ -75,5 +75,5 @@
         <visual>
             <geometry>
-                <mesh filename="package://motoman_gp25_support/meshes/visual/gp25_link_5_b.stl"/>
+                <mesh filename="package://motoman_gp25_support/meshes/visual/link_5_b.stl"/>
             </geometry>
             <material name="yaskawa_blue"/>
@@ -81,5 +81,5 @@
         <collision>
             <geometry>
-                <mesh filename="package://motoman_gp25_support/meshes/collision/gp25_link_5_b.stl"/>
+                <mesh filename="package://motoman_gp25_support/meshes/collision/link_5_b.stl"/>
             </geometry>
         </collision>
@@ -88,5 +88,5 @@
         <visual>
             <geometry>
-                <mesh filename="package://motoman_gp25_support/meshes/visual/gp25_link_6_t.stl"/>
+                <mesh filename="package://motoman_gp25_support/meshes/visual/link_6_t.stl"/>
             </geometry>
             <material name="yaskawa_blue"/>
@@ -94,5 +94,5 @@
         <collision>
             <geometry>
-                <mesh filename="package://motoman_gp25_support/meshes/collision/gp25_link_6_t.stl"/>
+                <mesh filename="package://motoman_gp25_support/meshes/collision/link_6_t.stl"/>
             </geometry>
         </collision>
@@ -106,5 +106,5 @@
         <origin xyz="0 0 0.505" rpy="0 0 0" />
         <axis xyz="0 0 1" />
-        <limit lower="-3.1416" upper="3.1416" effort="3087" velocity="3.6651"/>
+        <limit lower="${radians(-180)}" upper="${radians(180)}" effort="3087" velocity="${radians(210)}"/>
     </joint>
     <joint name="${prefix}joint_2_l" type="revolute">
@@ -113,5 +113,5 @@
         <origin xyz="0.150 0 0" rpy="0 0 0" />
         <axis xyz="0 1 0" />
-        <limit lower="-1.8326" upper="2.7052" effort="3087" velocity="3.6651"/>
+        <limit lower="${radians(-105)}" upper="${radians(155)}" effort="3087" velocity="${radians(210)}"/>
     </joint>
     <joint name="${prefix}joint_3_u" type="revolute">
@@ -120,19 +120,19 @@
         <origin xyz="0 0 0.760" rpy="0 0 0" />
         <axis xyz="0 -1 0" />
-        <limit lower="-1.5009" upper="2.7925" effort="926.1" velocity="4.6251"/>
+        <limit lower="${radians(-86)}" upper="${radians(160)}" effort="926.1" velocity="${radians(265)}"/>
     </joint>
     <joint name="${prefix}joint_4_r" type="revolute">
         <parent link="${prefix}link_3_u"/>
         <child link="${prefix}link_4_r"/>
-        <origin xyz="0.795 0 0.200" rpy="0 0 0" />
+        <origin xyz="0 0 0.200" rpy="0 0 0" />
         <axis xyz="-1 0 0" />
-        <limit lower="-3.4906" upper="3.4906" effort="88.2" velocity="7.3303"/>
+        <limit lower="${radians(-200)}" upper="${radians(200)}" effort="88.2" velocity="${radians(420)}"/>
     </joint>
     <joint name="${prefix}joint_5_b" type="revolute">
         <parent link="${prefix}link_4_r"/>
         <child link="${prefix}link_5_b"/>
-        <origin xyz="0 0 0" rpy="0 0 0" />
+        <origin xyz="0.795 0 0" rpy="0 0 0" />
         <axis xyz="0 -1 0" />
-        <limit lower="-2.6179" upper="2.6179" effort="70.56" velocity="7.3303"/>
+        <limit lower="${radians(-155)}" upper="${radians(150)}" effort="70.56" velocity="${radians(420)}"/>
     </joint>
     <joint name="${prefix}joint_6_t" type="revolute">
@@ -141,5 +141,5 @@
         <origin xyz="0 0 0" rpy="0 0 0" />
         <axis xyz="-1 0 0" />
-        <limit lower="-7.9412" upper="7.9412" effort="50.31" velocity="15.4461"/>
+        <limit lower="${radians(-455)}" upper="${radians(455)}" effort="50.31" velocity="${radians(885)}"/>
     </joint>
     <joint name="${prefix}joint_6_t-tool0" type="fixed">
