Commit message: Update references to GP-25 resources
Replace dashes with underscores.

File: motoman_gp25_support/urdf/gp25_12.xacro (robot description, xacro)
@@ -1,5 +1,5 @@
 <?xml version="1.0" ?>
-<robot name="motoman_gp25-12" xmlns:xacro="http://ros.org/wiki/xacro">
-	<xacro:include filename="$(find motoman_gp25_support)/urdf/gp25-12_macro.xacro" />
-	<xacro:motoman_gp25-12 prefix=""/>
+<robot name="motoman_gp25_12" xmlns:xacro="http://ros.org/wiki/xacro">
+	<xacro:include filename="$(find motoman_gp25_support)/urdf/gp25_12_macro.xacro" />
+	<xacro:motoman_gp25_12 prefix=""/>
 </robot>

File: motoman_gp25_support/urdf/gp25_12_macro.xacro (robot description, xacro)
@@ -1,5 +1,5 @@
 <?xml version="1.0" ?>
 <robot xmlns:xacro="http://ros.org/wiki/xacro">
-<xacro:macro name="motoman_gp25-12" params="prefix">
+<xacro:macro name="motoman_gp25_12" params="prefix">
     <xacro:include filename="$(find motoman_resources)/urdf/common_materials.xacro"/>
     <!-- link list -->
@@ -59,5 +59,5 @@
         <visual>
             <geometry>
-                <mesh filename="package://motoman_gp25_support/meshes/gp25-12/visual/link_4_r.dae"/>
+                <mesh filename="package://motoman_gp25_support/meshes/gp25_12/visual/link_4_r.dae"/>
             </geometry>
             <xacro:material_yaskawa_blue/>
@@ -65,5 +65,5 @@
         <collision>
             <geometry>
-                <mesh filename="package://motoman_gp25_support/meshes/gp25-12/collision/link_4_r.stl"/>
+                <mesh filename="package://motoman_gp25_support/meshes/gp25_12/collision/link_4_r.stl"/>
             </geometry>
         </collision>
