Commit message: changed headstock and tailstock to be macros so that arguments can be passed to them. Prepended the positioner name to each joint and link. Reconciled velocity limits with manual. Added positioner/base dummy link. Added upper and lower joint limits to positioner.

File: motoman_motopos_mh185_rotisserie_support/urdf/headstock/headstock.urdf_macro.xacro (robot description, xacro)
@@ -1,4 +1,5 @@
 <?xml version="1.0"?>
-<robot name="headstock" xmlns:xacro="http://www.ros.org/wiki/xacro">
+<robot name="headstock" xmlns:xacro="http://www.ros.org/wiki/xacro" param="prefix">
+ <xacro:macro name ="headstock_macro" params="prefix">
   <!-- Constants for robot dimensions -->
   <xacro:property name="M_PI" value="3.1415926535897931"/>
@@ -7,5 +8,5 @@
   <xacro:property name="hs_prismatic_offset" value="${load_yaml('$(find motoman_motopos_mh185_rotisserie_support)/config/positioner_params.yaml')['positioner_params']['headstock_prismatic_offset']}"/>
   <link
-    name="hs_base_link">
+    name="${prefix}hs_base_link">
     <inertial>
       <origin
@@ -47,5 +48,5 @@
   </link>
   <joint
-    name="mh185_joint_1"
+    name="${prefix}joint_1"
     type="revolute">
     <origin
@@ -53,18 +54,18 @@
       rpy="0 0 0" />
     <parent
-      link="hs_base_link" />
+      link="${prefix}hs_base_link" />
     <child
-      link="hs_revolute_link" />
+      link="${prefix}hs_revolute_link" />
     <axis
       xyz="0 0 1" />
     <limit
-      lower="${-20*M_PI}"
-      upper="${20*M_PI}"
-      effort="10"
-      velocity="${2*M_PI}" />
+      lower="${-1.1*M_PI}"
+      upper="${1.1*M_PI}"
+      effort="100"
+      velocity="${(12.4/60)*2*M_PI}" />
   </joint>
-  <xacro:transmission_macro name="x" />
+  <xacro:transmission_macro name="${prefix}_joint_1" />
   <link
-    name="hs_revolute_link">
+    name="${prefix}hs_revolute_link">
     <inertial>
       <origin
@@ -106,5 +107,5 @@
   </link>
   <joint
-    name="joint_hs_prismatic"
+    name="${prefix}joint_hs_prismatic"
     type="fixed">
     <origin
@@ -112,12 +113,12 @@
       rpy="0 0 0" />
     <parent
-      link="hs_revolute_link" />
+      link="${prefix}hs_revolute_link" />
     <child
-      link="hs_prismatic_link" />
+      link="${prefix}hs_prismatic_link" />
     <axis
       xyz="0 0 0" />
   </joint>
   <link
-    name="hs_prismatic_link">
+    name="${prefix}hs_prismatic_link">
     <inertial>
       <origin
@@ -158,3 +159,4 @@
     </collision>
   </link>
+ </xacro:macro>
 </robot>

File: motoman_motopos_mh185_rotisserie_support/urdf/motopos_mh185_rotisserie_macro.xacro (robot description, xacro)
@@ -31,9 +31,12 @@
   <!-- link list -->
   <!-- Add the headstock - hs_base_link, hs_revolute_link, hs_prismatic_link -->
-  <xacro:include filename="$(find motoman_motopos_mh185_rotisserie_support)/urdf/headstock/headstock.urdf.xacro" ns="hs" />
-  <xacro:include filename="$(find motoman_motopos_mh185_rotisserie_support)/urdf/tailstock/tailstock.urdf.xacro" ns="ts" />
+  <xacro:include filename="$(find motoman_motopos_mh185_rotisserie_support)/urdf/headstock/headstock.urdf_macro.xacro" />
+  <xacro:headstock_macro prefix="${prefix}"/>
+  <xacro:include filename="$(find motoman_motopos_mh185_rotisserie_support)/urdf/tailstock/tailstock.urdf_macro.xacro" />
+  <xacro:tailstock_macro prefix="${prefix}"/>
   <!-- And connect positioner_link to base_link -->
   <link name="${prefix}base_link"/>
   <link name="positioner/base"/>
+  <link name="positioner/center"/>
   <!-- hs_base - positioner_link->base_link -->
   <xacro:property name="world2base_xyz" value="${world_base_xyz}"/>
@@ -49,33 +52,39 @@
                            origin_rpy="${world2pos_rpy}"
                            parent="${prefix}base_link"
-                           child="hs_base_link"
+                           child="${prefix}hs_base_link"
                            axis_xyz="1 0 0" />
   <xacro:fixed_joint_macro name="positioner/base"
                            origin_xyz="0 0 0"
                            origin_rpy="0 0 0"
-                           parent="hs_base_link"
+                           parent="${prefix}hs_base_link"
                            child="positioner/base"
-                           axis_xyz="1 0 0" />
+                           axis_xyz="0 0 0" />
   <!-- Connect the tail stock to the headstock -->
   <!-- the base and prismatic joints should be connected to a non-rotating link, i.e. the headstock base link -->
-  <xacro:fixed_joint_macro name="ts_base"
+  <xacro:fixed_joint_macro name="${prefix}ts_base"
                            origin_xyz="0 0 -${ts_base_offset}"
                            origin_rpy="0 0 0"
-                           parent="hs_base_link"
-                           child="ts_base_link"
+                           parent="${prefix}hs_base_link"
+                           child="${prefix}ts_base_link"
                            axis_xyz="1 0 0" />
-  <xacro:fixed_joint_macro name="ts_prismatic"
+  <xacro:fixed_joint_macro name="${prefix}ts_prismatic"
                            origin_xyz="0 0 -${ts_revolute_offset}"
                            origin_rpy="0 0 0"
-                           parent="hs_base_link"
-                           child="ts_prismatic_link"
+                           parent="${prefix}hs_base_link"
+                           child="${prefix}ts_prismatic_link"
                            axis_xyz="1 0 0" />
   <!-- The revolute link should be connected to a rotating link, i.e. the headstock revolute link -->
-  <xacro:fixed_joint_macro name="ts_revolute"
+  <xacro:fixed_joint_macro name="${prefix}ts_revolute"
                            origin_xyz="0 0 -${ts_revolute_offset}"
                            origin_rpy="0 0 0"
-                           parent="hs_revolute_link"
-                           child="ts_revolute_link"
+                           parent="${prefix}hs_revolute_link"
+                           child="${prefix}ts_revolute_link"
                            axis_xyz="1 0 0" />
+  <xacro:fixed_joint_macro name="${prefix}joint1-center-fixed"
+                           origin_xyz="0 0 0"
+                           origin_rpy="0 0 0"
+                           parent="${prefix}hs_revolute_link"
+                           child="positioner/center"
+                           axis_xyz="0 0 0"/>
   </xacro:macro>
 </robot>

File: motoman_motopos_mh185_rotisserie_support/urdf/tailstock/tailstock.urdf_macro.xacro (robot description, xacro)
@@ -1,8 +1,9 @@
 <?xml version="1.0"?>
 <robot name="tailstock" xmlns:xacro="http://www.ros.org/wiki/xacro">
+  <xacro:macro name="tailstock_macro" params="prefix">
   <!-- Constants for robot dimensions -->
   <xacro:property name="M_PI" value="3.1415926535897931"/>
   <link
-    name="ts_base_link">
+    name="${prefix}ts_base_link">
     <inertial>
       <origin
@@ -44,5 +45,5 @@
   </link>
   <link
-    name="ts_prismatic_link">
+    name="${prefix}ts_prismatic_link">
     <inertial>
       <origin
@@ -84,5 +85,5 @@
   </link>
   <link
-    name="ts_revolute_link">
+    name="${prefix}ts_revolute_link">
     <inertial>
       <origin
@@ -123,3 +124,4 @@
     </collision>
   </link>
+  </xacro:macro>
 </robot>

Commit message: Update min/max joint limits for MH185 packages

File: motoman_motopos_mh185_rotisserie_support/urdf/headstock/headstock.urdf_macro.xacro (robot description, xacro)
@@ -60,6 +60,6 @@
       xyz="0 0 1" />
     <limit
-      lower="${-1.1*M_PI}"
-      upper="${1.1*M_PI}"
+      lower="${-2*M_PI}"
+      upper="${2*M_PI}"
       effort="100"
       velocity="${(12.4/60)*2*M_PI}" />

File: motoman_motopos_mh185_vertical_support/urdf/motopos_mh185_vertical_macro.xacro (robot description, xacro)
@@ -66,5 +66,5 @@
     />
     <axis xyz="0 0 1" />
-    <limit lower="${-1*M_PI}" upper="${M_PI}" effort="1274" velocity="1.15"/>
+    <limit lower="${-2*M_PI}" upper="${2*M_PI}" effort="1274" velocity="1.15"/>
   </joint>
   <xacro:transmission_macro name="1"/>

Commit message: Small updates to frames/offsets for calibration

File: motoman_motopos_mh185_rotisserie_support/urdf/headstock/headstock.urdf_macro.xacro (robot description, xacro)
@@ -6,5 +6,4 @@
   <!-- Import trasnmission macro -->
   <xacro:include filename="$(find motoman_motopos_mh185_rotisserie_support)/urdf/headstock/headstock.transmission.xacro" />
-  <xacro:property name="hs_prismatic_offset" value="${load_yaml('$(find motoman_motopos_mh185_rotisserie_support)/config/positioner_params.yaml')['positioner_params']['headstock_prismatic_offset']}"/>
   <link
     name="${prefix}hs_base_link">
@@ -110,5 +109,5 @@
     type="fixed">
     <origin
-      xyz="0 ${hs_prismatic_offset} 0"
+      xyz="0 0 0"
       rpy="0 ${M_PI} 0" />
     <parent

File: motoman_motopos_mh185_rotisserie_support/urdf/motopos_mh185_rotisserie_macro.xacro (robot description, xacro)
@@ -10,14 +10,13 @@
 >
   <xacro:property name="M_PI" value="3.1415926535897931"/>
-  <xacro:property name="offsets" value="${load_yaml(offsets_file_path)[prefix + 'robot_calibration_offsets']}"/>
-<xacro:property name="world_to_pos_base_tf" value="${load_yaml('$(find motoman_motopos_mh185_rotisserie_support)/config/positioner_params.yaml')}"/>
-  <xacro:property name="world2pos_t" value="${world_to_pos_base_tf['positioner_params']['base_to_positioner_tf']['translation']}" />
-  <xacro:property name="world2pos_rot" value="${world_to_pos_base_tf['positioner_params']['base_to_positioner_tf']['rotation']}" />
+  <xacro:property name="offsets" value="${load_yaml('$(find motoman_motopos_mh185_rotisserie_support)/config/default_positioner_params.yaml')}"/>
+  <xacro:property name="world2pos_t" value="${offsets['base_to_hs_base_link_tf']['translation']}" />
+  <xacro:property name="world2pos_rot" value="${offsets['base_to_hs_base_link_tf']['rotation']}" />
   <xacro:property name="world2pos_xyz" value="${world2pos_t['x']} ${world2pos_t['y']} ${world2pos_t['z']}"/>
   <xacro:property name="world2pos_rpy" value="${world2pos_rot['roll']} ${world2pos_rot['pitch']} ${world2pos_rot['yaw']}"/>
   <!-- Tailstock offsets. Should be loaded from yaml file created during calibration. -->
   <xacro:property name="ts_base_offset" value="0.06985" />
-  <xacro:property name="ts_revolute_offset" value="${world_to_pos_base_tf['positioner_params']['tailstock_revolute_offset']}" />
-  <xacro:property name="hs_prismatic_offset" value="${world_to_pos_base_tf['positioner_params']['headstock_prismatic_offset']}"/>
+  <xacro:property name="ts_revolute_offset" value="${offsets['tailstock_revolute_offset']}" />
+  <xacro:property name="hs_prismatic_offset" value="${offsets['headstock_prismatic_offset']}"/>
   <!-- Define a fixed joint macro -->
   <xacro:macro name="fixed_joint_macro" params="name origin_xyz origin_rpy parent child axis_xyz">
@@ -40,9 +39,7 @@
   <link name="positioner/center"/>
   <!-- hs_base - positioner_link->base_link -->
-  <xacro:property name="world2base_xyz" value="${world_base_xyz}"/>
-  <xacro:property name="world2base_rpy" value="${world_base_rpy}"/>
   <xacro:fixed_joint_macro name="${prefix}world-base"
-                           origin_rpy="${world2base_rpy}"
-                           origin_xyz="${world2base_xyz}"
+                           origin_rpy="${world_base_rpy}"
+                           origin_xyz="${world_base_xyz}"
                            parent="world"
                            child="${prefix}base_link"
@@ -56,5 +53,5 @@
   <xacro:fixed_joint_macro name="positioner/base"
                            origin_xyz="0 0 0"
-                           origin_rpy="0 ${M_PI} 0"
+                           origin_rpy="0 0 0"
                            parent="${prefix}hs_base_link"
                            child="positioner/base"

Commit message: WIP - Fix frame definitons, required calibration offsets

File: motoman_motopos_mh185_rotisserie_support/urdf/headstock/headstock.urdf_macro.xacro (robot description, xacro)
@@ -158,4 +158,15 @@
     </collision>
   </link>
+   <joint name="${prefix}joint1-center-fixed" type="fixed">
+     <origin
+         xyz="0 0 0"
+         rpy="0 0 0" />
+     <parent
+         link="${prefix}hs_revolute_link" />
+     <child
+         link="positioner/center" />
+     <axis
+         xyz="0 0 0" />
+   </joint>
  </xacro:macro>
 </robot>

File: motoman_motopos_mh185_rotisserie_support/urdf/motopos_mh185_rotisserie_macro.xacro (robot description, xacro)
@@ -10,7 +10,7 @@
 >
   <xacro:property name="M_PI" value="3.1415926535897931"/>
-  <xacro:property name="offsets" value="${load_yaml('$(find motoman_motopos_mh185_rotisserie_support)/config/default_positioner_params.yaml')}"/>
-  <xacro:property name="world2pos_t" value="${offsets['base_to_hs_base_link_tf']['translation']}" />
-  <xacro:property name="world2pos_rot" value="${offsets['base_to_hs_base_link_tf']['rotation']}" />
+  <xacro:property name="offsets" value="${load_yaml('/var/local/forge/calibration/mh185_horizontal_pos_offsets.yaml')}"/>
+  <xacro:property name="world2pos_t" value="${offsets['transform']['translation']}" />
+  <xacro:property name="world2pos_rot" value="${offsets['transform']['rotation']}" />
   <xacro:property name="world2pos_xyz" value="${world2pos_t['x']} ${world2pos_t['y']} ${world2pos_t['z']}"/>
   <xacro:property name="world2pos_rpy" value="${world2pos_rot['roll']} ${world2pos_rot['pitch']} ${world2pos_rot['yaw']}"/>
@@ -18,5 +18,4 @@
   <xacro:property name="ts_base_offset" value="0.06985" />
   <xacro:property name="ts_revolute_offset" value="${offsets['tailstock_revolute_offset']}" />
-  <xacro:property name="hs_prismatic_offset" value="${offsets['headstock_prismatic_offset']}"/>
   <!-- Define a fixed joint macro -->
   <xacro:macro name="fixed_joint_macro" params="name origin_xyz origin_rpy parent child axis_xyz">
@@ -53,5 +52,5 @@
   <xacro:fixed_joint_macro name="positioner/base"
                            origin_xyz="0 0 0"
-                           origin_rpy="0 0 0"
+                           origin_rpy="0 ${M_PI} 0"
                            parent="${prefix}hs_base_link"
                            child="positioner/base"
@@ -78,10 +77,10 @@
                            child="${prefix}ts_revolute_link"
                            axis_xyz="1 0 0" />
-  <xacro:fixed_joint_macro name="${prefix}joint1-center-fixed"
-                           origin_xyz="0 0 0"
-                           origin_rpy="0 0 0"
-                           parent="positioner/base"
-                           child="positioner/center"
-                           axis_xyz="0 0 0"/>
+<!--  <xacro:fixed_joint_macro name="${prefix}joint1-center-fixed"-->
+<!--                           origin_xyz="0 0 0"-->
+<!--                           origin_rpy="0 0 0"-->
+<!--                           parent="{prefix}hs_revolute_link"-->
+<!--                           child="positioner/center"-->
+<!--                           axis_xyz="0 0 0"/>-->
   </xacro:macro>
 </robot>

Commit message: urdf changed to represent cell

File: motoman_motopos_mh185_rotisserie_support/urdf/headstock/headstock.urdf_macro.xacro (robot description, xacro)
@@ -52,5 +52,5 @@
     <origin
       xyz="0 0 0"
-      rpy="0 0 0" />
+      rpy="0 ${M_PI} 0" />
     <parent
       link="${prefix}hs_base_link" />
@@ -60,8 +60,8 @@
       xyz="0 0 1" />
     <limit
-      lower="${-1.1*M_PI}"
-      upper="${1.1*M_PI}"
+      lower="${-2*M_PI}"
+      upper="${2*M_PI}"
       effort="100"
-      velocity="${(12.4/60)*2*M_PI}" />
+      velocity="0.9" />
   </joint>
   <xacro:transmission_macro name="${prefix}_joint_1" />
@@ -110,6 +110,6 @@
     type="fixed">
     <origin
-      xyz="0 ${hs_prismatic_offset} 0"
-      rpy="0 0 0" />
+      xyz="0 0 0"
+      rpy="0 ${M_PI} 0" />
     <parent
       link="${prefix}hs_revolute_link" />
@@ -159,4 +159,15 @@
     </collision>
   </link>
+   <joint name="${prefix}joint1-center-fixed" type="fixed">
+     <origin
+         xyz="0 0 0"
+         rpy="0 0 0" />
+     <parent
+         link="${prefix}hs_revolute_link" />
+     <child
+         link="positioner/center" />
+     <axis
+         xyz="0 0 0" />
+   </joint>
  </xacro:macro>
 </robot>

File: motoman_motopos_mh185_rotisserie_support/urdf/motopos_mh185_rotisserie_macro.xacro (robot description, xacro)
@@ -56,5 +56,5 @@
   <xacro:fixed_joint_macro name="positioner/base"
                            origin_xyz="0 0 0"
-                           origin_rpy="0 0 0"
+                           origin_rpy="0 ${M_PI} 0"
                            parent="${prefix}hs_base_link"
                            child="positioner/base"
@@ -63,5 +63,5 @@
   <!-- the base and prismatic joints should be connected to a non-rotating link, i.e. the headstock base link -->
   <xacro:fixed_joint_macro name="${prefix}ts_base"
-                           origin_xyz="0 0 -${ts_base_offset}"
+                           origin_xyz="0 0 ${ts_base_offset}"
                            origin_rpy="0 0 0"
                            parent="${prefix}hs_base_link"
@@ -76,15 +76,15 @@
   <!-- The revolute link should be connected to a rotating link, i.e. the headstock revolute link -->
   <xacro:fixed_joint_macro name="${prefix}ts_revolute"
-                           origin_xyz="0 0 -${ts_revolute_offset}"
+                           origin_xyz="0 0 ${ts_revolute_offset}"
                            origin_rpy="0 0 0"
                            parent="${prefix}hs_revolute_link"
                            child="${prefix}ts_revolute_link"
                            axis_xyz="1 0 0" />
-  <xacro:fixed_joint_macro name="${prefix}joint1-center-fixed"
-                           origin_xyz="0 0 0"
-                           origin_rpy="0 0 0"
-                           parent="${prefix}hs_revolute_link"
-                           child="positioner/center"
-                           axis_xyz="0 0 0"/>
+<!--  <xacro:fixed_joint_macro name="${prefix}joint1-center-fixed"-->
+<!--                           origin_xyz="0 0 0"-->
+<!--                           origin_rpy="0 0 0"-->
+<!--                           parent="${prefix}hs_revolute_link"-->
+<!--                           child="positioner/center"-->
+<!--                           axis_xyz="0 0 0"/>-->
   </xacro:macro>
 </robot>
