Commit message: added dummy link to appease weld_planner_demo

File: motoman_motopos_mh185_rotisserie_support/urdf/motopos_mh185_rotisserie_macro.xacro (robot description, xacro)
@@ -35,4 +35,5 @@
   <!-- And connect positioner_link to base_link -->
   <link name="${prefix}base_link"/>
+  <link name="positioner/base"/>
   <!-- hs_base - positioner_link->base_link -->
   <xacro:property name="world2base_xyz" value="${world_base_xyz}"/>
@@ -49,4 +50,10 @@
                            parent="${prefix}base_link"
                            child="hs_base_link"
+                           axis_xyz="1 0 0" />
+  <xacro:fixed_joint_macro name="positioner/base"
+                           origin_xyz="0 0 0"
+                           origin_rpy="0 0 0"
+                           parent="hs_base_link"
+                           child="positioner/base"
                            axis_xyz="1 0 0" />
   <!-- Connect the tail stock to the headstock -->

Commit message: Update calibration pose and filenames

File: motoman_motopos_mh185_rotisserie_support/urdf/motopos_mh185_rotisserie_macro.xacro (robot description, xacro)
@@ -17,5 +17,6 @@
   <!-- Tailstock offsets. Should be loaded from yaml file created during calibration. -->
   <xacro:property name="ts_base_offset" value="0.06985" />
-  <xacro:property name="ts_revolute_offset" value="${offsets['tailstock_revolute_offset']}" />
+  <xacro:property name="ts_position" value="${load_yaml('/var/local/forge/calibration/mh185_horizontal_tailstock_position.yaml')}"/>
+  <xacro:property name="ts_revolute_offset" value="${ts_position['tailstock_revolute_offset']}" />
   <!-- Define a fixed joint macro -->
   <xacro:macro name="fixed_joint_macro" params="name origin_xyz origin_rpy parent child axis_xyz">
