Commit message: FR-277 Included missed ma1440 urdf update.

File: motoman_ma1440_support/urdf/ma1440/ma1440.xacro (robot description, xacro)
@@ -3,5 +3,7 @@
     <xacro:arg name="cam_mount" default="false"/>
     <xacro:include filename="$(find motoman_ma1440_support)/urdf/ma1440/ma1440_macro.xacro" />
-    <xacro:motoman_ma1440 prefix=""/>
+    <xacro:macro name="load_motoman_ma1440" params="prefix:=ma1440_ world_base_xyz world_base_rpy">
+        <xacro:motoman_ma1440 prefix="${prefix}" world_base_xyz="${world_base_xyz}" world_base_rpy="${world_base_rpy}"/>
+    </xacro:macro>
     <!-- optionally add the cam mount to the end of the arm, this is the laserscanner enclosure used on the Corsa system -->
 <!--    <xacro:if value="$(arg cam_mount)">-->

Commit message: Load default calibration values if offsets_file_path not provided

File: motoman_ma1440_support/urdf/ma1440/ma1440.xacro (robot description, xacro)
@@ -48,5 +48,5 @@
             </joint>
         </xacro:if>
-        <!-- optionally add the laser mount to the end of the armand define all of its additional frames -->
+        <!-- optionally add the laser mount to the end of the arm and define all of its additional frames -->
         <xacro:if value="${mount_type=='laser'}">
             <xacro:include filename="$(find motoman_ma1440_support)/urdf/laser_mount/laser_mount.xacro" />

File: motoman_motopos_mh185_rotisserie_support/urdf/motopos_mh185_rotisserie.xacro (robot description, xacro)
@@ -8,25 +8,16 @@
           world_base_xyz
           world_base_rpy
-          offsets_file_path:='$(find motoman_motopos_mh185_rotisserie_support)/config/robot_calibration_offsets.yaml'"
+          offsets_file_path"
   >
     <material name="yaskawa_blue">
       <color rgba="0.12941 0.14902 0.74902 1" />
     </material>
-    <xacro:unless value="${offsets_file_path == ''}">
-      <xacro:motoman_motopos_mh185_rotisserie
-          prefix="${prefix}"
-          world_base_xyz="${world_base_xyz}"
-          world_base_rpy="${world_base_rpy}"
-          offsets_file_path="${offsets_file_path}"
-      />
-    </xacro:unless>
-    <xacro:if value="${offsets_file_path == ''}">
-      <xacro:motoman_motopos_mh185_rotisserie
-          prefix="${prefix}"
-          world_base_xyz="${world_base_xyz}"
-          world_base_rpy="${world_base_rpy}"
-          offsets_file_path="'$(find motoman_motopos_mh185_rotisserie_support)/config/robot_calibration_offsets.yaml'"
-      />
-    </xacro:if>
+    <!-- Loads default calibration if offsets_file_path is blank -->
+    <xacro:motoman_motopos_mh185_rotisserie
+        prefix="${prefix}"
+        world_base_xyz="${world_base_xyz}"
+        world_base_rpy="${world_base_rpy}"
+        offsets_file_path="${offsets_file_path}"
+    />
   </xacro:macro>
 </robot>

File: motoman_motopos_mh185_rotisserie_support/urdf/motopos_mh185_rotisserie_macro.xacro (robot description, xacro)
@@ -10,12 +10,26 @@
 >
   <xacro:property name="M_PI" value="3.1415926535897931"/>
-  <xacro:property name="offsets" value="${load_yaml('/var/local/forge/calibration/mh185_horizontal_pos_offsets.yaml')}"/>
-  <xacro:property name="world2pos_t" value="${offsets['transform']['translation']}" />
-  <xacro:property name="world2pos_rot" value="${offsets['transform']['rotation']}" />
+  <!-- IMPORTANT! The filepaths for the non-default calibrations are defined in the forge-shared-definitions package as well as the API!
+                  Do not change these filenames without also changing these values in the other places! -->
+  <xacro:if value="${offsets_file_path == ''}">
+    <xacro:property name="axis_offsets_filepath" value="$(find motoman_motopos_mh185_rotisserie_support)/config/default_axis_offsets.yaml"/>
+  </xacro:if>
+  <xacro:unless value="${offsets_file_path == ''}">
+    <xacro:property name="axis_offsets_filepath" value="/var/local/forge/calibration/mh185_horizontal/axis_offsets.yaml"/>
+  </xacro:unless>
+  <xacro:if value="${offsets_file_path == ''}">
+    <xacro:property name="tailstock_offset_filepath" value="$(find motoman_motopos_mh185_rotisserie_support)/config/default_tailstock_offset.yaml"/>
+  </xacro:if>
+  <xacro:unless value="${offsets_file_path == ''}">
+    <xacro:property name="tailstock_offset_filepath" value="/var/local/forge/calibration/mh185_horizontal/tailstock_offset.yaml"/>
+  </xacro:unless>
+  <xacro:property name="axis_offsets" value="${load_yaml(axis_offsets_filepath)}"/>
+  <xacro:property name="world2pos_t" value="${axis_offsets['transform']['translation']}" />
+  <xacro:property name="world2pos_rot" value="${axis_offsets['transform']['rotation']}" />
   <xacro:property name="world2pos_xyz" value="${world2pos_t['x']} ${world2pos_t['y']} ${world2pos_t['z']}"/>
   <xacro:property name="world2pos_rpy" value="${world2pos_rot['roll']} ${world2pos_rot['pitch']} ${world2pos_rot['yaw']}"/>
   <!-- Tailstock offsets. Should be loaded from yaml file created during calibration. -->
   <xacro:property name="ts_base_offset" value="0.06985" />
-  <xacro:property name="ts_position" value="${load_yaml('/var/local/forge/calibration/mh185_horizontal_tailstock_position.yaml')}"/>
+  <xacro:property name="ts_position" value="${load_yaml(tailstock_offset_filepath)}"/>
   <xacro:property name="ts_revolute_offset" value="${ts_position['tailstock_revolute_offset']}" />
   <!-- Define a fixed joint macro -->

Commit message: add optional chessboard mount

File: motoman_ma1440_support/urdf/ma1440/ma1440.xacro (robot description, xacro)
@@ -45,4 +45,34 @@
                 <parent link="${prefix}link_t" />
                 <child link="${prefix}cam_mount_link" />
+                <axis xyz="0 0 0" />
+            </joint>
+        </xacro:if>
+        <!-- optionally add chessboard to the end of the arm, this is the laser scanner enclosure used on the Corsa system -->
+        <xacro:if value="${mount_type =='chess'}">
+            <link name="${prefix}link_chessboard">
+                <visual>
+                    <origin rpy="0 0 0" xyz="0 0 0" />
+                    <geometry>
+                        <box size="0.26 0.45 0.15" />
+                    </geometry>
+                    <material name="silver" />
+                </visual>
+                <collision>
+                    <origin rpy="0 0 0" xyz="0 0 -0.07" />
+                    <geometry>
+                        <box size="0.26 0.45 0.15" />
+                    </geometry>
+                    <material name="silver" />
+                </collision>
+                <inertial>
+                    <mass value="0.0" />
+                    <inertia ixx="0.0" ixy="0.0" ixz="0.0" iyy="0.0" iyz="0.0" izz="0.0" />
+                    <origin rpy="0.0 0.0 0.0" xyz="0.0 0.0 0.0" />
+                </inertial>
+            </link>
+            <joint name="joint_chessboard" type="fixed">
+                <origin xyz="0 0 0" rpy="0 0 0" />
+                <parent link="${prefix}link_t" />
+                <child link="${prefix}link_chessboard" />
                 <axis xyz="0 0 0" />
             </joint>

File: motoman_ma1440_support/urdf/ma1440/ma1440_macro.xacro (robot description, xacro)
@@ -312,5 +312,11 @@
             <!-- Note that the joint range here is for the A00 version,
             the A10 version is -135/+90 degrees             -->
-            <limit lower="-2.35619" upper="1.5078" effort="100" velocity="7.50492" />
+            <!--  the chessboard mount can scrape the robot if the wrist bends too far -->
+            <xacro:if value="${mount_type =='chess'}">
+                <limit lower="-1.945" upper="1.5078" effort="100" velocity="7.50492" />
+            </xacro:if>
+            <xacro:if value="${mount_type !='chess'}">
+                <limit lower="-2.35619" upper="1.5078" effort="100" velocity="7.50492" />
+            </xacro:if>
         </joint>
         <xacro:transmission_macro name="b"/>

Commit message: add top chessboard

File: motoman_ma1440_support/urdf/ma1440/ma1440.xacro (robot description, xacro)
@@ -48,9 +48,9 @@
             </joint>
         </xacro:if>
-        <!-- optionally add chessboard to the end of the arm -->
-        <xacro:if value="${mount_type =='chess'}">
+        <!-- optionally add chessboard to the end of the arm, replacing the welder tip -->
+        <xacro:if value="${mount_type =='chess_front'}">
             <link name="${prefix}link_chessboard">
                 <visual>
-                    <origin rpy="0 0 0" xyz="0 0 0" />
+                    <origin rpy="0 0 0" xyz="0 0 -0.07" />
                     <geometry>
                         <box size="0.26 0.45 0.15" />
@@ -75,4 +75,69 @@
                 <parent link="${prefix}link_t" />
                 <child link="${prefix}link_chessboard" />
+                <axis xyz="0 0 0" />
+            </joint>
+        </xacro:if>
+        <!-- optionally add chessboard on a cam mount above the welder tip -->
+        <xacro:if value="${mount_type =='chess'}">
+            <link name="${prefix}link_chessboard">
+                <visual>
+                    <origin rpy="0 0 0" xyz="0.08 0 -0.09" />
+                    <geometry>
+                        <box size="0.08 0.26 0.18" />
+                    </geometry>
+                    <material name="silver">
+                        <color rgba="0.75 0.75 0.75 0.5"/>
+                    </material>
+                </visual>
+                <collision>
+                    <origin rpy="0 0 0" xyz="0.07 0 -0.09" />
+                    <geometry>
+                        <box size="0.06 0.26 0.18" />
+                    </geometry>
+                    <material name="silver">
+                        <color rgba="0.75 0.75 0.75 0.5"/>
+                    </material>
+                </collision>
+                <inertial>
+                    <mass value="0.0" />
+                    <inertia ixx="0.0" ixy="0.0" ixz="0.0" iyy="0.0" iyz="0.0" izz="0.0" />
+                    <origin rpy="0.0 0.0 0.0" xyz="0.0 0.0 0.0" />
+                </inertial>
+            </link>
+            <joint name="joint_chessboard" type="fixed">
+                <origin xyz="0 0 0" rpy="0 0 0" />
+                <parent link="${prefix}link_t" />
+                <child link="${prefix}link_chessboard" />
+                <axis xyz="0 0 0" />
+            </joint>
+            <link name="${prefix}link_collar">
+                <visual>
+                    <origin rpy="0 0 0" xyz="0 0 -0.027" />
+                    <geometry>
+                        <cylinder length="0.054" radius="0.09"/>
+                    </geometry>
+                    <material name="black">
+                        <color rgba="0 0 0 0.5"/>
+                    </material>
+                </visual>
+                <collision>
+                    <origin rpy="0 0 0" xyz="0 0 -0.027" />
+                    <geometry>
+                        <cylinder length="0.054" radius="0.09"/>
+                    </geometry>
+                    <material name="black">
+                        <color rgba="0 0 0 1"/>
+                    </material>
+                </collision>
+                <inertial>
+                    <mass value="0.0" />
+                    <inertia ixx="0.0" ixy="0.0" ixz="0.0" iyy="0.0" iyz="0.0" izz="0.0" />
+                    <origin rpy="0.0 0.0 0.0" xyz="0.0 0.0 0.0" />
+                </inertial>
+            </link>
+            <joint name="joint_collar" type="fixed">
+                <origin xyz="0 0 0" rpy="0 0 0" />
+                <parent link="${prefix}link_t" />
+                <child link="${prefix}link_collar" />
                 <axis xyz="0 0 0" />
             </joint>

File: motoman_ma1440_support/urdf/ma1440/ma1440_macro.xacro (robot description, xacro)
@@ -313,8 +313,8 @@
             the A10 version is -135/+90 degrees             -->
             <!--  the chessboard mount can scrape the robot if the wrist bends too far -->
-            <xacro:if value="${mount_type =='chess'}">
+            <xacro:if value="${mount_type =='chess_front'}">
                 <limit lower="-1.945" upper="1.5078" effort="100" velocity="7.50492" />
             </xacro:if>
-            <xacro:unless value="${mount_type =='chess'}">
+            <xacro:unless value="${mount_type =='chess_front'}">
                 <limit lower="-2.35619" upper="1.5078" effort="100" velocity="7.50492" />
             </xacro:unless>

Commit message: match collision with visual changes

File: motoman_ma1440_support/urdf/ma1440/ma1440.xacro (robot description, xacro)
@@ -87,14 +87,14 @@
                     </geometry>
                     <material name="silver">
-                        <color rgba="0.75 0.75 0.75 0.5"/>
+                        <color rgba="0.75 0.75 0.75 1"/>
                     </material>
                 </visual>
                 <collision>
-                    <origin rpy="0 0 0" xyz="0.07 0 -0.09" />
+                    <origin rpy="0 0 0" xyz="0.08 0 -0.09" />
                     <geometry>
-                        <box size="0.06 0.26 0.18" />
+                        <box size="0.08 0.26 0.18" />
                     </geometry>
                     <material name="silver">
-                        <color rgba="0.75 0.75 0.75 0.5"/>
+                        <color rgba="0.75 0.75 0.75 1"/>
                     </material>
                 </collision>

Commit message: Update ma1440.xacro

File: motoman_ma1440_support/urdf/ma1440/ma1440.xacro (robot description, xacro)
@@ -82,5 +82,5 @@
             <link name="${prefix}link_chessboard">
                 <visual>
-                    <origin rpy="0 0 0" xyz="0.08 0 -0.09" />
+                    <origin rpy="0 0 0" xyz="0.08 0 -0.16" />
                     <geometry>
                         <box size="0.08 0.26 0.18" />
@@ -91,5 +91,5 @@
                 </visual>
                 <collision>
-                    <origin rpy="0 0 0" xyz="0.08 0 -0.09" />
+                    <origin rpy="0 0 0" xyz="0.08 0 -0.16" />
                     <geometry>
                         <box size="0.08 0.26 0.18" />
@@ -113,5 +113,5 @@
             <link name="${prefix}link_collar">
                 <visual>
-                    <origin rpy="0 0 0" xyz="0 0 -0.027" />
+                    <origin rpy="0 0 0" xyz="0 0 -0.097" />
                     <geometry>
                         <cylinder length="0.054" radius="0.09"/>
@@ -122,5 +122,5 @@
                 </visual>
                 <collision>
-                    <origin rpy="0 0 0" xyz="0 0 -0.027" />
+                    <origin rpy="0 0 0" xyz="0 0 -0.097" />
                     <geometry>
                         <cylinder length="0.054" radius="0.09"/>
