Commit message: Update joint limits/minor URDF cleanup, add datasheets

File: motoman_ma1440_support/urdf/ma1440/ma1440_macro.xacro (robot description, xacro)
@@ -40,5 +40,4 @@
         <link name="${prefix}link_s">
             <visual>
-<!--                <origin rpy="0 0 0" xyz="0.026522 0.0082618 0.12436"/>-->
                 <origin rpy="0 0 0" xyz="0 0 0"/>
                 <geometry>
@@ -50,5 +49,4 @@
             </visual>
             <collision>
-<!--                <origin rpy="0 0 0" xyz="0.026522 0.0082618 0.12436"/>-->
                 <origin rpy="0 0 0" xyz="0 0 0"/>
                 <geometry>
@@ -61,5 +59,4 @@
                 <inertia ixx="2.1336" ixy="0.197" ixz="0.8995" iyy="2.8341" iyz="0.2799" izz="2.49"/>
                 <origin rpy="0 0 0" xyz="0 0 0"/>
-<!--                <origin rpy="0 0 0" xyz="0.026522 0.0082618 0.12436"/>-->
             </inertial>
         </link>
@@ -71,5 +68,4 @@
         <link name="${prefix}link_l">
             <visual>
-<!--                <origin rpy="1.57 3.1416 0" xyz="0 0 0"/>-->
                 <origin rpy="0 0 0" xyz="0 0 0"/>
                 <geometry>
@@ -79,5 +75,4 @@
             </visual>
             <collision>
-<!--                <origin rpy="1.57 3.1416 0" xyz="0 0 0"/>-->
                 <origin rpy="0 0 0" xyz="0 0 0"/>
                 <geometry>
@@ -89,5 +84,4 @@
                 <mass value="45.143" />
                 <inertia ixx="0.1565" ixy="-0.0239" ixz="-0.0981" iyy="2.4306" iyz="0.0329" izz="2.4493"/>
-<!--                <origin xyz="0.11422130 0.0 0.018935113" rpy="0.0 0.0 0.0"/>-->
                 <origin rpy="0 0 0" xyz="0 0 0"/>
             </inertial>
@@ -116,5 +110,4 @@
                 <mass value="77.767" />
                 <inertia ixx="1.1285" ixy="-0.4562" ixz="-0.1754" iyy="0.965" iyz="0.2365" izz="1.2844"/>
-<!--                <origin xyz="0.0 -0.015659426 0.13525753" rpy="0.0 0.0 0.0"/>-->
                 <origin rpy="0 0 0" xyz="0 0 0"/>
             </inertial>
@@ -245,5 +238,5 @@
             <origin xyz="0 0 0.165" rpy="0 0 0"/>
             <axis xyz="0 0 1" />
-            <limit lower="-3.1415" upper="3.1415" effort="100" velocity="2.9670" />
+            <limit lower="-2.96706" upper="2.96706" effort="100" velocity="4.01425727959" />
         </joint>
         <xacro:transmission_macro name="s"/>
@@ -253,5 +246,5 @@
             <origin xyz="0.155 -0.0425 0.285" rpy="${M_PI/2} ${-M_PI/2} ${M_PI}"/>
             <axis xyz="0 0 1" />
-            <limit lower="-1.9198" upper="1.9198" effort="100" velocity="2.9670" />
+            <limit lower="-1.5708" upper="2.70526" effort="100" velocity="3.49066" />
         </joint>
         <xacro:transmission_macro name="l"/>
@@ -261,5 +254,5 @@
             <origin xyz="0.614 0 -0.07" rpy="0 0 ${M_PI/2}"/>
             <axis xyz="0 0 -1" />
-            <limit lower="-2.3561" upper="2.3561" effort="100" velocity="2.9670" />
+            <limit lower="-3.05433" upper="4.18879" effort="100" velocity="4.01425727959" />
         </joint>
         <xacro:transmission_macro name="u"/>
@@ -269,5 +262,5 @@
             <origin xyz="0.265 -0.2 0.049" rpy="${M_PI/2} 0 ${-M_PI/2}"/>
             <axis xyz="0 0 1" />
-            <limit lower="-3.1415" upper="3.1415" effort="100" velocity="3.4906" />
+            <limit lower="-2.61799" upper="2.61799" effort="100" velocity="7.50492" />
         </joint>
         <xacro:transmission_macro name="r"/>
@@ -277,5 +270,7 @@
             <origin xyz="0 -0.062 -0.375" rpy="${M_PI/2} ${M_PI/2} 0"/>
             <axis xyz="0 0 1" />
-            <limit lower="-1.9198" upper="1.9198" effort="100" velocity="3.4906" />
+            <!-- Note that the joint range here is for the A00 version,
+            the A10 version is -135/+90 degrees             -->
+            <limit lower="-2.35619" upper="1.5078" effort="100" velocity="7.50492" />
         </joint>
         <xacro:transmission_macro name="b"/>
@@ -285,5 +280,5 @@
             <origin xyz="0.0875 0 -0.062" rpy="${-M_PI/2} 0 ${M_PI/2}"/>
             <axis xyz="0 0 1" />
-            <limit lower="-3.1415" upper="3.1415" effort="100" velocity="6.9813" />
+            <limit lower="-3.66519" upper="3.66519" effort="100" velocity="10.9956" />
         </joint>
         <xacro:transmission_macro name="t"/>

File: motoman_motopos_d500_support/urdf/motopos_d500_macro.xacro (robot description, xacro)
@@ -66,5 +66,5 @@
   </joint>
   <xacro:transmission_macro name="2"/>
-  <joint name="$joint_2-tool0" type="fixed">
+  <joint name="joint_2-tool0" type="fixed">
     <origin xyz="0 0 0.150 " rpy="0 0 0"/>
     <parent link="${prefix}link_2"/>

Commit message: FR-249 Updated camera collision model. Added a collision box to MA1440 to account for the little bump on joint S.

File: motoman_ma1440_support/urdf/ma1440/ma1440_macro.xacro (robot description, xacro)
@@ -57,4 +57,11 @@
                 <material name="yellow"/>
             </collision>
+            <!--      TODO: Remove this once the collision model is updated to include the little bump      -->
+            <collision>
+                <origin rpy="0 0 0" xyz="0.11 -0.02 0.38"/>
+                <geometry>
+                    <box size="0.1 0.05 0.1"/>
+                </geometry>
+            </collision>
             <inertial>
                 <mass value="112.57" />

Commit message: FR-314 Changed MA1440 U joint min/max values to prevent robot collision. Updated the moveit package that uses MA1440 to reflect changes.

File: motoman_ma1440_support/urdf/ma1440/ma1440_macro.xacro (robot description, xacro)
@@ -263,5 +263,7 @@
             <origin xyz="0.614 0 -0.07" rpy="0 0 ${M_PI/2}"/>
             <axis xyz="0 0 -1" />
-            <limit lower="-3.05433" upper="4.18879" effort="100" velocity="4.01425727959" />
+<!--            The commented out line is the specification for this joint, but it allows the robot to hit itself.-->
+<!--            <limit lower="-3.05433" upper="4.18879" effort="100" velocity="4.01425727959" />-->
+            <limit lower="${-84*M_PI/180}" upper="${90*M_PI/180}" effort="100" velocity="4.01425727959" />
         </joint>
         <xacro:transmission_macro name="u"/>

Commit message: FR-338 Added joint offset loading to ma1440.

File: motoman_ma1440_support/urdf/ma1440/ma1440_macro.xacro (robot description, xacro)
@@ -4,6 +4,8 @@
     <xacro:property name="world_base_rpy" value="0 0 0"/>
     <xacro:property name="M_PI" value="3.1415926535897931"/>
+    <xacro:property name="offsets_file_path" value="$(find motoman_ma1440_support)/config/robot_calibration_offsets.yaml"/>
     <xacro:include filename="$(find motoman_ma1440_support)/urdf/ma1440/ma1440.transmission.xacro" />
-    <xacro:macro name="motoman_ma1440" params="prefix world_base_xyz:=^ world_base_rpy:=^">
+    <xacro:macro name="motoman_ma1440" params="prefix world_base_xyz:=^ world_base_rpy:=^ offsets_file_path:=^">
+        <xacro:property name="offsets" value="${load_yaml('$(find ma1400_sim)/config/robot_calibration_offsets.yaml')['robot_calibration_offsets']}"/>
         <!-- link list -->
         <link name="world">
@@ -245,5 +247,8 @@
             <parent link="${prefix}base_link"/>
             <child link="${prefix}link_s"/>
-            <origin xyz="0 0 0.165" rpy="0 0 0"/>
+            <origin
+                xyz="${offsets['joint_s']['x']} ${offsets['joint_s']['y']} ${0.165 + offsets['joint_s']['z']}"
+                rpy="${offsets['joint_s']['roll']} ${offsets['joint_s']['pitch']} ${offsets['joint_s']['yaw']}"
+            />
             <axis xyz="0 0 1" />
             <limit lower="-2.96706" upper="2.96706" effort="100" velocity="4.01425727959" />
@@ -253,5 +258,8 @@
             <parent link="${prefix}link_s"/>
             <child link="${prefix}link_l"/>
-            <origin xyz="0.155 -0.0425 0.285" rpy="${M_PI/2} ${-M_PI/2} ${M_PI}"/>
+            <origin
+                xyz="${0.155 + offsets['joint_l']['x']} ${-0.0425 + offsets['joint_l']['y']} ${0.285 + offsets['joint_l']['z']}"
+                rpy="${M_PI/2 + offsets['joint_l']['roll']} ${-M_PI/2 + offsets['joint_l']['pitch']} ${M_PI + offsets['joint_l']['yaw']}"
+            />
             <axis xyz="0 0 1" />
             <limit lower="-1.5708" upper="2.70526" effort="100" velocity="3.49066" />
@@ -261,5 +269,8 @@
             <parent link="${prefix}link_l"/>
             <child link="${prefix}link_u"/>
-            <origin xyz="0.614 0 -0.07" rpy="0 0 ${M_PI/2}"/>
+            <origin
+                xyz="${0.614 + offsets['joint_u']['x']} ${0.0 + offsets['joint_u']['y']} ${-0.07 + offsets['joint_u']['z']}"
+                rpy="${0 + offsets['joint_u']['roll']} ${0 + offsets['joint_u']['pitch']} ${M_PI/2 + offsets['joint_u']['yaw']}"
+            />
             <axis xyz="0 0 -1" />
 <!--            The commented out line is the specification for this joint, but it allows the robot to hit itself.-->
@@ -271,5 +282,8 @@
             <parent link="${prefix}link_u"/>
             <child link="${prefix}link_r"/>
-            <origin xyz="0.265 -0.2 0.049" rpy="${M_PI/2} 0 ${-M_PI/2}"/>
+            <origin
+                xyz="${0.265 + offsets['joint_r']['x']} ${-0.2 + offsets['joint_r']['y']} ${0.049 + offsets['joint_r']['z']}"
+                rpy="${M_PI/2 + offsets['joint_r']['roll']} ${0 + offsets['joint_r']['pitch']} ${-M_PI/2 + offsets['joint_r']['yaw']}"
+            />
             <axis xyz="0 0 1" />
             <limit lower="-2.61799" upper="2.61799" effort="100" velocity="7.50492" />
@@ -279,5 +293,8 @@
             <parent link="${prefix}link_r"/>
             <child link="${prefix}link_b"/>
-            <origin xyz="0 -0.062 -0.375" rpy="${M_PI/2} ${M_PI/2} 0"/>
+            <origin
+                xyz="${0.0 + offsets['joint_b']['x']} ${-0.062 + offsets['joint_b']['y']} ${-0.375 + offsets['joint_b']['z']}"
+                rpy="${M_PI/2 + offsets['joint_b']['roll']} ${M_PI/2 + offsets['joint_b']['pitch']} ${0 + offsets['joint_b']['yaw']}"
+            />
             <axis xyz="0 0 1" />
             <!-- Note that the joint range here is for the A00 version,
@@ -289,5 +306,8 @@
             <parent link="${prefix}link_b"/>
             <child link="${prefix}link_t"/>
-            <origin xyz="0.0875 0 -0.062" rpy="${-M_PI/2} 0 ${M_PI/2}"/>
+            <origin
+                xyz="${0.0875 + offsets['joint_t']['x']} ${0.0 + offsets['joint_t']['y']} ${-0.062 + offsets['joint_t']['z']}"
+                rpy="${-M_PI/2 + offsets['joint_t']['roll']} ${0 + offsets['joint_t']['pitch']} ${M_PI/2 + offsets['joint_t']['yaw']}"
+            />
             <axis xyz="0 0 1" />
             <limit lower="-3.66519" upper="3.66519" effort="100" velocity="10.9956" />

Commit message: Add welder feed box to robot collision model

File: motoman_ma1440_support/urdf/ma1440/ma1440_macro.xacro (robot description, xacro)
@@ -121,4 +121,10 @@
                 <origin rpy="0 0 0" xyz="0 0 0"/>
             </inertial>
+            <collision>
+                <origin rpy="0 0 0" xyz="-0.15 -0.10 0.10"/>
+                <geometry>
+                    <box size="0.55 0.35 0.38"/>
+                </geometry>
+            </collision>
         </link>
         <gazebo reference="${prefix}link_u">

Commit message: added vertical offset for robot base

File: motoman_ma1440_support/urdf/ma1440/ma1440_macro.xacro (robot description, xacro)
@@ -12,4 +12,5 @@
       <xacro:property name="M_PI" value="3.1415926535897931"/>
       <xacro:property name="offsets" value="${load_yaml(offsets_file_path)[prefix + 'robot_calibration_offsets']}"/>
+      <xacro:property name="vertical_offset" value="0"/>
         <link name="world">
             <origin xyz="0 0 0" rpy="0 0 0"/>
@@ -249,5 +250,5 @@
         <!-- joint list -->
         <joint name="${prefix}world-base" type="fixed">
-            <origin xyz="${world_base_xyz}" rpy="${world_base_rpy}"/>
+            <origin xyz="0 0 ${vertical_offset}" rpy="${world_base_rpy}"/>
             <parent link="world" />
             <child link="${prefix}base_link"/>

Commit message: added vertical offset

File: motoman_ma1440_support/urdf/ma1440/ma1440_macro.xacro (robot description, xacro)
@@ -12,5 +12,5 @@
       <xacro:property name="M_PI" value="3.1415926535897931"/>
       <xacro:property name="offsets" value="${load_yaml(offsets_file_path)[prefix + 'robot_calibration_offsets']}"/>
-      <xacro:property name="vertical_offset" value="0"/>
+      <xacro:property name="vertical_offset" value="0.5"/>
         <link name="world">
             <origin xyz="0 0 0" rpy="0 0 0"/>

Commit message: changed vertical offset to 0

File: motoman_ma1440_support/urdf/ma1440/ma1440_macro.xacro (robot description, xacro)
@@ -12,5 +12,5 @@
       <xacro:property name="M_PI" value="3.1415926535897931"/>
       <xacro:property name="offsets" value="${load_yaml(offsets_file_path)[prefix + 'robot_calibration_offsets']}"/>
-      <xacro:property name="vertical_offset" value="0.5"/>
+      <xacro:property name="vertical_offset" value="0.0"/>
         <link name="world">
             <origin xyz="0 0 0" rpy="0 0 0"/>

Commit message: Updated robot model to modified API model and updated meshes

File: motoman_ma1440_support/urdf/ma1440/ma1440_macro.xacro (robot description, xacro)
@@ -258,6 +258,6 @@
             <child link="${prefix}link_s"/>
             <origin
-                xyz="${offsets[prefix + 'joint_s']['x']} ${offsets[prefix + 'joint_s']['y']} ${0.165 + offsets[prefix + 'joint_s']['z']}"
-                rpy="${offsets[prefix + 'joint_s']['roll']} ${offsets[prefix + 'joint_s']['pitch']} ${offsets[prefix + 'joint_s']['yaw']}"
+                xyz="${0 + offsets[prefix + 'joint_s']['x']} ${0 + offsets[prefix + 'joint_s']['y']} ${0.45 + offsets[prefix + 'joint_s']['z']}"
+                rpy="${0 + offsets[prefix + 'joint_s']['roll']} ${0 + offsets[prefix + 'joint_s']['pitch']} ${0 + offsets[prefix + 'joint_s']['yaw']}"
             />
             <axis xyz="0 0 1" />
@@ -269,6 +269,6 @@
             <child link="${prefix}link_l"/>
             <origin
-                xyz="${0.155 + offsets[prefix + 'joint_l']['x']} ${-0.0425 + offsets[prefix + 'joint_l']['y']} ${0.285 + offsets[prefix + 'joint_l']['z']}"
-                rpy="${M_PI/2 + offsets[prefix + 'joint_l']['roll']} ${-M_PI/2 + offsets[prefix + 'joint_l']['pitch']} ${M_PI + offsets[prefix + 'joint_l']['yaw']}"
+                xyz="${0.155  + offsets[prefix + 'joint_l']['x']} ${0 + offsets[prefix + 'joint_l']['y'] + offsets[prefix + 'joint_l']['y']} ${0 + offsets[prefix + 'joint_l']['z']}"
+                rpy="${-0.7853981633974483 + offsets[prefix + 'joint_l']['roll']} ${-1.5707963267948966 + offsets[prefix + 'joint_l']['pitch']} ${-0.7853981633974483 + offsets[prefix + 'joint_l']['yaw']}"
             />
             <axis xyz="0 0 1" />
@@ -280,8 +280,8 @@
             <child link="${prefix}link_u"/>
             <origin
-                xyz="${0.614 + offsets[prefix + 'joint_u']['x']} ${0.0 + offsets[prefix + 'joint_u']['y']} ${-0.007 + offsets[prefix + 'joint_u']['z']}"
-                rpy="${0 + offsets[prefix + 'joint_u']['roll']} ${0 + offsets[prefix + 'joint_u']['pitch']} ${M_PI/2 + offsets[prefix + 'joint_u']['yaw']}"
-            />
-            <axis xyz="0 0 -1" />
+                xyz="${0.614 + offsets[prefix + 'joint_u']['x']} ${0 + offsets[prefix + 'joint_u']['y']} ${0 + offsets[prefix + 'joint_u']['z']}"
+                rpy="${3.141592653589793 + offsets[prefix + 'joint_u']['roll']} ${0+ offsets[prefix + 'joint_u']['pitch']} ${0 + offsets[prefix + 'joint_u']['yaw']}"
+            />
+            <axis xyz="0 0 1" />
 <!--            The commented out line is the specification for this joint, but it allows the robot to hit itself.-->
 <!--            <limit lower="-3.05433" upper="4.18879" effort="100" velocity="4.01425727959" />-->
@@ -293,6 +293,6 @@
             <child link="${prefix}link_r"/>
             <origin
-                xyz="${0.265 + offsets[prefix + 'joint_r']['x']} ${-0.2 + offsets[prefix + 'joint_r']['y']} ${0.049 + offsets[prefix + 'joint_r']['z']}"
-                rpy="${M_PI/2 + offsets[prefix + 'joint_r']['roll']} ${0 + offsets[prefix + 'joint_r']['pitch']} ${-M_PI/2 + offsets[prefix + 'joint_r']['yaw']}"
+                xyz="${0.2 + offsets[prefix + 'joint_r']['x']} ${-0.64 + offsets[prefix + 'joint_r']['y']} ${0 + offsets[prefix + 'joint_r']['z']}"
+                rpy="${-1.5707963267948966 + offsets[prefix + 'joint_r']['roll']} ${0 + offsets[prefix + 'joint_r']['pitch']} ${0 + offsets[prefix + 'joint_r']['yaw']}"
             />
             <axis xyz="0 0 1" />
@@ -304,6 +304,6 @@
             <child link="${prefix}link_b"/>
             <origin
-                xyz="${0.0 + offsets[prefix + 'joint_b']['x']} ${-0.062 + offsets[prefix + 'joint_b']['y']} ${-0.375 + offsets[prefix + 'joint_b']['z']}"
-                rpy="${M_PI/2 + offsets[prefix + 'joint_b']['roll']} ${M_PI/2 + offsets[prefix + 'joint_b']['pitch']} ${0 + offsets[prefix + 'joint_b']['yaw']}"
+                xyz="${0 + offsets[prefix + 'joint_b']['x']} ${0 + offsets[prefix + 'joint_b']['y']} ${0 + offsets[prefix + 'joint_b']['z']}"
+                rpy="${1.5707963267948966 + offsets[prefix + 'joint_b']['roll']} ${0 + offsets[prefix + 'joint_b']['pitch']} ${0 + offsets[prefix + 'joint_b']['yaw']}"
             />
             <axis xyz="0 0 1" />
@@ -317,6 +317,6 @@
             <child link="${prefix}link_t"/>
             <origin
-                xyz="${0.0875 + offsets[prefix + 'joint_t']['x']} ${0.0 + offsets[prefix + 'joint_t']['y']} ${-0.062 + offsets[prefix + 'joint_t']['z']}"
-                rpy="${-M_PI/2 + offsets[prefix + 'joint_t']['roll']} ${0 + offsets[prefix + 'joint_t']['pitch']} ${M_PI/2 + offsets[prefix + 'joint_t']['yaw']}"
+                xyz="${0 + offsets[prefix + 'joint_t']['x']} ${-0.1+ offsets[prefix + 'joint_t']['y']} ${0 + offsets[prefix + 'joint_t']['z']}"
+                rpy="${-1.5707963267948966 + offsets[prefix + 'joint_t']['roll']} ${0 + offsets[prefix + 'joint_t']['pitch']} ${0 + offsets[prefix + 'joint_t']['yaw']}"
             />
             <axis xyz="0 0 1" />
@@ -327,5 +327,5 @@
             <parent link="${prefix}link_t"/>
             <child link="${prefix}link_tip"/>
-            <origin xyz="-0.09591 0 -0.38772" rpy="${-135*M_PI/180} 0 ${M_PI/2}"/>
+            <origin xyz="-0.09591 0 ${-0.38772 + 0.0125}" rpy="${-135*M_PI/180} 0 ${M_PI/2}"/>
             <axis xyz="0 0 0" />
         </joint>

Commit message: fix collision models -agregg

File: motoman_ma1440_support/urdf/ma1440/ma1440_macro.xacro (robot description, xacro)
@@ -65,5 +65,5 @@
             <!--      TODO: Remove this once the collision model is updated to include the little bump      -->
             <collision>
-                <origin rpy="0 0 0" xyz="0.11 -0.02 0.38"/>
+                <origin rpy="0 0 0" xyz="0.11 -0.02 0.095"/>
                 <geometry>
                     <box size="0.1 0.05 0.1"/>
@@ -128,5 +128,5 @@
             </inertial>
             <collision>
-                <origin rpy="0 0 0" xyz="-0.15 -0.10 0.10"/>
+                <origin rpy="0 0 1.57079632679" xyz="0.10 0.15 -0.10"/>
                 <geometry>
                     <box size="0.55 0.35 0.38"/>

Commit message: Clean up offset values

File: motoman_ma1440_support/urdf/ma1440/ma1440_macro.xacro (robot description, xacro)
@@ -11,4 +11,6 @@
     >
       <xacro:property name="M_PI" value="3.1415926535897931"/>
+      <xacro:property name="M_PI_2" value="1.57079632679"/>
+      <xacro:property name="M_PI_4" value="0.7853981633974483"/>
       <xacro:property name="offsets" value="${load_yaml(offsets_file_path)[prefix + 'robot_calibration_offsets']}"/>
       <xacro:property name="vertical_offset" value="0.0"/>
@@ -128,5 +130,5 @@
             </inertial>
             <collision>
-                <origin rpy="0 0 1.57079632679" xyz="0.10 0.15 -0.10"/>
+                <origin rpy="0 0 ${M_PI_2}" xyz="0.10 0.15 -0.10"/>
                 <geometry>
                     <box size="0.55 0.35 0.38"/>
@@ -270,5 +272,5 @@
             <origin
                 xyz="${0.155  + offsets[prefix + 'joint_l']['x']} ${0 + offsets[prefix + 'joint_l']['y'] + offsets[prefix + 'joint_l']['y']} ${0 + offsets[prefix + 'joint_l']['z']}"
-                rpy="${-0.7853981633974483 + offsets[prefix + 'joint_l']['roll']} ${-1.5707963267948966 + offsets[prefix + 'joint_l']['pitch']} ${-0.7853981633974483 + offsets[prefix + 'joint_l']['yaw']}"
+                rpy="${-M_PI_4 + offsets[prefix + 'joint_l']['roll']} ${-M_PI_2 + offsets[prefix + 'joint_l']['pitch']} ${-M_PI_4 + offsets[prefix + 'joint_l']['yaw']}"
             />
             <axis xyz="0 0 1" />
@@ -281,5 +283,5 @@
             <origin
                 xyz="${0.614 + offsets[prefix + 'joint_u']['x']} ${0 + offsets[prefix + 'joint_u']['y']} ${0 + offsets[prefix + 'joint_u']['z']}"
-                rpy="${3.141592653589793 + offsets[prefix + 'joint_u']['roll']} ${0+ offsets[prefix + 'joint_u']['pitch']} ${0 + offsets[prefix + 'joint_u']['yaw']}"
+                rpy="${M_PI + offsets[prefix + 'joint_u']['roll']} ${0+ offsets[prefix + 'joint_u']['pitch']} ${0 + offsets[prefix + 'joint_u']['yaw']}"
             />
             <axis xyz="0 0 1" />
@@ -294,5 +296,5 @@
             <origin
                 xyz="${0.2 + offsets[prefix + 'joint_r']['x']} ${-0.64 + offsets[prefix + 'joint_r']['y']} ${0 + offsets[prefix + 'joint_r']['z']}"
-                rpy="${-1.5707963267948966 + offsets[prefix + 'joint_r']['roll']} ${0 + offsets[prefix + 'joint_r']['pitch']} ${0 + offsets[prefix + 'joint_r']['yaw']}"
+                rpy="${-M_PI_2 + offsets[prefix + 'joint_r']['roll']} ${0 + offsets[prefix + 'joint_r']['pitch']} ${0 + offsets[prefix + 'joint_r']['yaw']}"
             />
             <axis xyz="0 0 1" />
@@ -305,5 +307,5 @@
             <origin
                 xyz="${0 + offsets[prefix + 'joint_b']['x']} ${0 + offsets[prefix + 'joint_b']['y']} ${0 + offsets[prefix + 'joint_b']['z']}"
-                rpy="${1.5707963267948966 + offsets[prefix + 'joint_b']['roll']} ${0 + offsets[prefix + 'joint_b']['pitch']} ${0 + offsets[prefix + 'joint_b']['yaw']}"
+                rpy="${M_PI_2 + offsets[prefix + 'joint_b']['roll']} ${0 + offsets[prefix + 'joint_b']['pitch']} ${0 + offsets[prefix + 'joint_b']['yaw']}"
             />
             <axis xyz="0 0 1" />
@@ -318,5 +320,5 @@
             <origin
                 xyz="${0 + offsets[prefix + 'joint_t']['x']} ${-0.1+ offsets[prefix + 'joint_t']['y']} ${0 + offsets[prefix + 'joint_t']['z']}"
-                rpy="${-1.5707963267948966 + offsets[prefix + 'joint_t']['roll']} ${0 + offsets[prefix + 'joint_t']['pitch']} ${0 + offsets[prefix + 'joint_t']['yaw']}"
+                rpy="${-M_PI_2 + offsets[prefix + 'joint_t']['roll']} ${0 + offsets[prefix + 'joint_t']['pitch']} ${0 + offsets[prefix + 'joint_t']['yaw']}"
             />
             <axis xyz="0 0 1" />
