Commit message: Fix U link collision model orientation

File: motoman_ma1440_support/urdf/ma1440/ma1440_macro.xacro (robot description, xacro)
@@ -118,5 +118,5 @@
             </visual>
             <collision>
-                <origin rpy="0 0 0" xyz="0 0 0"/>
+                <origin rpy="0 ${M_PI} ${M_PI_2}" xyz="0 0 0"/>
                 <geometry>
                     <mesh filename="package://motoman_ma1440_support/meshes/ma1440/collision/u_link_collision.stl" />

Commit message: modifications to support loading tip calib offsets from urdf

File: motoman_ma1440_support/urdf/ma1440/ma1440_macro.xacro (robot description, xacro)
@@ -1,343 +1,649 @@
 <?xml version="1.0" ?>
-<robot xmlns:xacro="http://ros.org/wiki/xacro">
-    <xacro:include filename="$(find motoman_ma1440_support)/urdf/ma1440/ma1440.transmission.xacro" />
-    <xacro:macro
-        name="motoman_ma1440"
-        params="
+<robot
+    xmlns:xacro="http://ros.org/wiki/xacro">
+  <xacro:include
+      filename="$(find motoman_ma1440_support)/urdf/ma1440/ma1440.transmission.xacro"/>
+  <xacro:macro
+      name="motoman_ma1440"
+      params="
                  prefix
                  world_base_xyz:='0 0 0'
                  world_base_rpy:='0 0 0'
                  offsets_file_path"
-    >
-      <xacro:property name="M_PI" value="3.1415926535897931"/>
-      <xacro:property name="M_PI_2" value="1.57079632679"/>
-      <xacro:property name="M_PI_4" value="0.7853981633974483"/>
-      <xacro:property name="offsets" value="${load_yaml(offsets_file_path)[prefix + 'robot_calibration_offsets']}"/>
-      <xacro:property name="vertical_offset" value="0.0"/>
-        <link name="world">
-            <origin xyz="0 0 0" rpy="0 0 0"/>
-        </link>
-        <link name="${prefix}base_link">
-            <visual>
-                <origin rpy="0 0 0" xyz="0 0 0"/>
-                <geometry>
-                    <mesh filename="package://motoman_ma1440_support/meshes/ma1440/visual/base_link.stl" />
-                </geometry>
-                <material name="blue">
-                    <color rgba="0 0 1 1"/>
-                </material>
-            </visual>
-            <collision>
-                <origin rpy="0 0 0" xyz="0 0 0"/>
-                <geometry>
-                    <mesh filename="package://motoman_ma1440_support/meshes/ma1440/collision/base_link_collision.stl" />
-                </geometry>
-                <material name="yellow">
-                    <color rgba="0 1 1 1"/>
-                </material>
-            </collision>
-            <inertial>
-                <mass value="400" /> 	<!-- Arbitrarily large value, to simulate bolting down in case of absence of fixed joint -->
-                <inertia ixx="1.0" ixy="0.0" ixz="0.0" iyy="1.0" iyz="0.0" izz="1.0"/>
-                <origin rpy="0 0 0" xyz="0 0 0"/>
-            </inertial>
-        </link>
-        <gazebo reference="${prefix}base_link">
-            <turnGravityOff>false</turnGravityOff>
-            <selfCollide>true</selfCollide>
-            <material>Gazebo/Blue</material>
-        </gazebo>
-        <link name="${prefix}link_s">
-            <visual>
-                <origin rpy="0 0 0" xyz="0 0 0"/>
-                <geometry>
-                    <mesh filename="package://motoman_ma1440_support/meshes/ma1440/visual/s_link.stl"/>
-                </geometry>
-                <material name="blue">
-                    <color rgba="0 0 1 1"/>
-                </material>
-            </visual>
-            <collision>
-                <origin rpy="0 0 0" xyz="0 0 0"/>
-                <geometry>
-                    <mesh filename="package://motoman_ma1440_support/meshes/ma1440/collision/s_link_collision.stl" />
-                </geometry>
-                <material name="yellow"/>
-            </collision>
-            <!--      TODO: Remove this once the collision model is updated to include the little bump      -->
-            <collision>
-                <origin rpy="0 0 0" xyz="0.11 -0.02 0.095"/>
-                <geometry>
-                    <box size="0.1 0.05 0.1"/>
-                </geometry>
-            </collision>
-            <inertial>
-                <mass value="112.57" />
-                <inertia ixx="2.1336" ixy="0.197" ixz="0.8995" iyy="2.8341" iyz="0.2799" izz="2.49"/>
-                <origin rpy="0 0 0" xyz="0 0 0"/>
-            </inertial>
-        </link>
-        <gazebo reference="${prefix}link_s">
-            <turnGravityOff>false</turnGravityOff>
-            <selfCollide>true</selfCollide>
-            <material>Gazebo/Blue</material>
-        </gazebo>
-        <link name="${prefix}link_l">
-            <visual>
-                <origin rpy="0 0 0" xyz="0 0 0"/>
-                <geometry>
-                    <mesh filename="package://motoman_ma1440_support/meshes/ma1440/visual/l_link.stl"/>
-                </geometry>
-                <material name="blue"/>
-            </visual>
-            <collision>
-                <origin rpy="0 0 0" xyz="0 0 0"/>
-                <geometry>
-                    <mesh filename="package://motoman_ma1440_support/meshes/ma1440/collision/l_link_collision.stl" />
-                </geometry>
-                <material name="yellow"/>
-            </collision>
-            <inertial>
-                <mass value="45.143" />
-                <inertia ixx="0.1565" ixy="-0.0239" ixz="-0.0981" iyy="2.4306" iyz="0.0329" izz="2.4493"/>
-                <origin rpy="0 0 0" xyz="0 0 0"/>
-            </inertial>
-        </link>
-        <gazebo reference="${prefix}link_l">
-            <turnGravityOff>false</turnGravityOff>
-            <selfCollide>true</selfCollide>
-            <material>Gazebo/Blue</material>
-        </gazebo>
-        <link name="${prefix}link_u">
-            <visual>
-                <origin rpy="0 0 0" xyz="0 0 0"/>
-                <geometry>
-                    <mesh filename="package://motoman_ma1440_support/meshes/ma1440/visual/u_link.stl"/>
-                </geometry>
-                <material name="blue"/>
-            </visual>
-            <collision>
-                <origin rpy="0 ${M_PI} ${M_PI_2}" xyz="0 0 0"/>
-                <geometry>
-                    <mesh filename="package://motoman_ma1440_support/meshes/ma1440/collision/u_link_collision.stl" />
-                </geometry>
-                <material name="yellow"/>
-            </collision>
-            <inertial>
-                <mass value="77.767" />
-                <inertia ixx="1.1285" ixy="-0.4562" ixz="-0.1754" iyy="0.965" iyz="0.2365" izz="1.2844"/>
-                <origin rpy="0 0 0" xyz="0 0 0"/>
-            </inertial>
-            <collision>
-                <origin rpy="0 0 ${M_PI_2}" xyz="0.10 0.15 -0.10"/>
-                <geometry>
-                    <box size="0.55 0.35 0.38"/>
-                </geometry>
-            </collision>
-        </link>
-        <gazebo reference="${prefix}link_u">
-            <turnGravityOff>false</turnGravityOff>
-            <selfCollide>true</selfCollide>
-            <material>Gazebo/Blue</material>
-        </gazebo>
-        <link name="${prefix}link_r">
-            <visual>
-                <origin rpy="0 0 0" xyz="0 0 0"/>
-                <geometry>
-                    <mesh filename="package://motoman_ma1440_support/meshes/ma1440/visual/r_link.stl"/>
-                </geometry>
-                <material name="blue"/>
-            </visual>
-            <collision>
-                <origin rpy="0 0 0" xyz="0 0 0"/>
-                <geometry>
-                    <mesh filename="package://motoman_ma1440_support/meshes/ma1440/collision/r_link_collision.stl" />
-                </geometry>
-                <material name="yellow"/>
-            </collision>
-            <inertial>
-                <mass value="31.136" />
-                <inertia ixx="0.5313" ixy="0.0027" ixz="0.0418" iyy="0.453" iyz="-0.0111" izz="0.1611"/>
-                <origin rpy="0 0 0" xyz="0 0 0"/>
-            </inertial>
-        </link>
-        <gazebo reference="${prefix}link_r">
-            <turnGravityOff>false</turnGravityOff>
-            <selfCollide>true</selfCollide>
-            <material>Gazebo/White</material>
-        </gazebo>
-        <link name="${prefix}link_b">
-            <visual>
-                <origin rpy="0 0 0" xyz="0 0 0"/>
-                <geometry>
-                    <mesh filename="package://motoman_ma1440_support/meshes/ma1440/visual/b_link.stl" />
-                </geometry>
-                <material name="blue"/>
-            </visual>
-            <collision>
-                <origin rpy="0 0 0" xyz="0 0 0"/>
-                <geometry>
-                    <mesh filename="package://motoman_ma1440_support/meshes/ma1440/collision/b_link_collision.stl" />
-                </geometry>
-                <material name="yellow"/>
-            </collision>
-            <inertial>
-                <mass value="7.781" />
-                <inertia ixx="0.019954" ixy="6.9E-05" ixz="-0.000759" iyy="0.024524" iyz="0.000206" izz="0.019404"/>
-                <origin rpy="0 0 0" xyz="0 0 0"/>
-            </inertial>
-        </link>
-        <gazebo reference="${prefix}link_b">
-            <turnGravityOff>false</turnGravityOff>
-            <selfCollide>true</selfCollide>
-            <material>Gazebo/Blue</material>
-        </gazebo>
-        <link name="${prefix}link_t">
-            <visual>
-                <origin rpy="0 0 0" xyz="0 0 0"/>
-                <geometry>
-                    <mesh filename="package://motoman_ma1440_support/meshes/ma1440/visual/t_link.stl" />
-                </geometry>
-                <material name="blue"/>
-            </visual>
-            <collision>
-                <origin rpy="0 0 0" xyz="0 0 0"/>
-                <geometry>
-                    <mesh filename="package://motoman_ma1440_support/meshes/ma1440/collision/t_link_collision.stl" />
-                </geometry>
-                <material name="yellow"/>
-            </collision>
-            <inertial>
-                <mass value="0.40691" />
-                <inertia ixx="0.0" ixy="0.0" ixz="0.0" iyy="0.0" iyz="0.0" izz="0.0"/>
-                <origin xyz="0.0 0.0 0.0" rpy="0.0 0.0 0.0"/>
-            </inertial>
-        </link>
-        <gazebo reference="${prefix}link_t">
-            <turnGravityOff>false</turnGravityOff>
-            <selfCollide>true</selfCollide>
-            <material>Gazebo/White</material>
-        </gazebo>
-        <link name="${prefix}link_tip">
-            <visual>
-                <origin rpy="0 0 0" xyz="0 0 0"/>
-                <geometry>
-                    <mesh filename="package://motoman_ma1440_support/meshes/ma1440/visual/tip_link.stl" />
-                </geometry>
-                <material name="silver">
-                    <color rgba="0.8 0.8 0.8 1"/>
-                </material>
-            </visual>
-            <collision>
-                <origin rpy="0 0 0" xyz="0 0 0"/>
-                <geometry>
-                    <mesh filename="package://motoman_ma1440_support/meshes/ma1440/collision/tip_link_collision.stl" />
-                </geometry>
-                <material name="silver">
-                    <color rgba="0.8 0.8 0.8 1"/>
-                </material>
-            </collision>
-            <inertial>
-                <mass value="4.7615" />
-                <inertia ixx="0.034062" ixy="5.0098E-05" ixz="4.7762E-05" iyy="0.020719" iyz="-0.016082" izz="0.013698"/>
-                <origin xyz="0.0 0.0 0.0" rpy="0.0 0.0 0.0"/>
-            </inertial>
-        </link>
-        <gazebo reference="${prefix}link_t">
-            <turnGravityOff>false</turnGravityOff>
-            <selfCollide>true</selfCollide>
-            <material>Gazebo/White</material>
-        </gazebo>
-        <!-- end of link list -->
-        <!-- joint list -->
-        <joint name="${prefix}world-base" type="fixed">
-            <origin xyz="0 0 ${vertical_offset}" rpy="${world_base_rpy}"/>
-            <parent link="world" />
-            <child link="${prefix}base_link"/>
-        </joint>
-        <joint name="${prefix}joint_s" type="revolute">
-            <parent link="${prefix}base_link"/>
-            <child link="${prefix}link_s"/>
-            <origin
-                xyz="${0 + offsets[prefix + 'joint_s']['x']} ${0 + offsets[prefix + 'joint_s']['y']} ${0.45 + offsets[prefix + 'joint_s']['z']}"
-                rpy="${0 + offsets[prefix + 'joint_s']['roll']} ${0 + offsets[prefix + 'joint_s']['pitch']} ${0 + offsets[prefix + 'joint_s']['yaw']}"
-            />
-            <axis xyz="0 0 1" />
-            <limit lower="-2.96706" upper="2.96706" effort="100" velocity="4.01425727959" />
-        </joint>
-        <xacro:transmission_macro name="s"/>
-        <joint name="${prefix}joint_l" type="revolute">
-            <parent link="${prefix}link_s"/>
-            <child link="${prefix}link_l"/>
-            <origin
-                xyz="${0.155  + offsets[prefix + 'joint_l']['x']} ${0 + offsets[prefix + 'joint_l']['y'] + offsets[prefix + 'joint_l']['y']} ${0 + offsets[prefix + 'joint_l']['z']}"
-                rpy="${-M_PI_4 + offsets[prefix + 'joint_l']['roll']} ${-M_PI_2 + offsets[prefix + 'joint_l']['pitch']} ${-M_PI_4 + offsets[prefix + 'joint_l']['yaw']}"
-            />
-            <axis xyz="0 0 1" />
-            <limit lower="-1.5708" upper="2.70526" effort="100" velocity="3.49066" />
-        </joint>
-        <xacro:transmission_macro name="l"/>
-        <joint name="${prefix}joint_u" type="revolute">
-            <parent link="${prefix}link_l"/>
-            <child link="${prefix}link_u"/>
-            <origin
-                xyz="${0.614 + offsets[prefix + 'joint_u']['x']} ${0 + offsets[prefix + 'joint_u']['y']} ${0 + offsets[prefix + 'joint_u']['z']}"
-                rpy="${M_PI + offsets[prefix + 'joint_u']['roll']} ${0+ offsets[prefix + 'joint_u']['pitch']} ${0 + offsets[prefix + 'joint_u']['yaw']}"
-            />
-            <axis xyz="0 0 1" />
-<!--            The commented out line is the specification for this joint, but it allows the robot to hit itself.-->
-<!--            <limit lower="-3.05433" upper="4.18879" effort="100" velocity="4.01425727959" />-->
-            <limit lower="${-84*M_PI/180}" upper="${90*M_PI/180}" effort="100" velocity="4.01425727959" />
-        </joint>
-        <xacro:transmission_macro name="u"/>
-        <joint name="${prefix}joint_r" type="revolute">
-            <parent link="${prefix}link_u"/>
-            <child link="${prefix}link_r"/>
-            <origin
-                xyz="${0.2 + offsets[prefix + 'joint_r']['x']} ${-0.64 + offsets[prefix + 'joint_r']['y']} ${0 + offsets[prefix + 'joint_r']['z']}"
-                rpy="${-M_PI_2 + offsets[prefix + 'joint_r']['roll']} ${0 + offsets[prefix + 'joint_r']['pitch']} ${0 + offsets[prefix + 'joint_r']['yaw']}"
-            />
-            <axis xyz="0 0 1" />
-            <limit lower="-2.61799" upper="2.61799" effort="100" velocity="7.50492" />
-        </joint>
-        <xacro:transmission_macro name="r"/>
-        <joint name="${prefix}joint_b" type="revolute">
-            <parent link="${prefix}link_r"/>
-            <child link="${prefix}link_b"/>
-            <origin
-                xyz="${0 + offsets[prefix + 'joint_b']['x']} ${0 + offsets[prefix + 'joint_b']['y']} ${0 + offsets[prefix + 'joint_b']['z']}"
-                rpy="${M_PI_2 + offsets[prefix + 'joint_b']['roll']} ${0 + offsets[prefix + 'joint_b']['pitch']} ${0 + offsets[prefix + 'joint_b']['yaw']}"
-            />
-            <axis xyz="0 0 1" />
-            <!-- Note that the joint range here is for the A00 version,
-            the A10 version is -135/+90 degrees             -->
-            <limit lower="-2.35619" upper="1.5078" effort="100" velocity="7.50492" />
-        </joint>
-        <xacro:transmission_macro name="b"/>
-        <joint name="${prefix}joint_t" type="revolute">
-            <parent link="${prefix}link_b"/>
-            <child link="${prefix}link_t"/>
-            <origin
-                xyz="${0 + offsets[prefix + 'joint_t']['x']} ${-0.1+ offsets[prefix + 'joint_t']['y']} ${0 + offsets[prefix + 'joint_t']['z']}"
-                rpy="${-M_PI_2 + offsets[prefix + 'joint_t']['roll']} ${0 + offsets[prefix + 'joint_t']['pitch']} ${0 + offsets[prefix + 'joint_t']['yaw']}"
-            />
-            <axis xyz="0 0 1" />
-            <limit lower="-3.66519" upper="3.66519" effort="100" velocity="10.9956" />
-        </joint>
-        <xacro:transmission_macro name="t"/>
-        <joint name="${prefix}joint_tip" type="fixed">
-            <parent link="${prefix}link_t"/>
-            <child link="${prefix}link_tip"/>
-            <origin xyz="-0.09591 0 ${-0.38772 + 0.0125}" rpy="${-135*M_PI/180} 0 ${M_PI/2}"/>
-            <axis xyz="0 0 0" />
-        </joint>
-        <!-- end of joint list -->
-        <!-- ROS base_link (via base_link) to Motoman Robot (not Base) Frame transform -->
-        <link name="${prefix}base" />
-        <joint name="${prefix}base_link-base" type="fixed">
-            <origin rpy="0 0 0" xyz="0 0 0"/>
-            <parent link="${prefix}base_link"/>
-            <child link="${prefix}base"/>
-        </joint>
-    </xacro:macro>
+  >
+    <xacro:property
+        name="M_PI"
+        value="3.1415926535897931"/>
+    <xacro:property
+        name="M_PI_2"
+        value="1.57079632679"/>
+    <xacro:property
+        name="M_PI_4"
+        value="0.7853981633974483"/>
+    <xacro:property
+        name="offsets"
+        value="${load_yaml(offsets_file_path)[prefix + 'robot_calibration_offsets']}"/>
+    <xacro:property
+        name="vertical_offset"
+        value="0.5"/>
+    <link
+        name="world">
+      <origin
+          xyz="0 0 0"
+          rpy="0 0 0"/>
+    </link>
+    <link
+        name="${prefix}base_link">
+      <visual>
+        <origin
+            rpy="0 0 0"
+            xyz="0 0 0"/>
+        <geometry>
+          <mesh
+              filename="package://motoman_ma1440_support/meshes/ma1440/visual/base_link.stl"/>
+        </geometry>
+        <material
+            name="blue">
+          <color
+              rgba="0 0 1 1"/>
+        </material>
+      </visual>
+      <collision>
+        <origin
+            rpy="0 0 0"
+            xyz="0 0 0"/>
+        <geometry>
+          <mesh
+              filename="package://motoman_ma1440_support/meshes/ma1440/collision/base_link_collision.stl"/>
+        </geometry>
+        <material
+            name="yellow">
+          <color
+              rgba="0 1 1 1"/>
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