Commit message: Revert "modifications to support loading tip calib offsets from urdf"
This reverts commit edf6723b80a3ee4244bf3047dccc9ffba6bde09a.

File: motoman_ma1440_support/urdf/ma1440/ma1440_macro.xacro (robot description, xacro)
@@ -1,649 +1,343 @@
 <?xml version="1.0" ?>
-<robot
-    xmlns:xacro="http://ros.org/wiki/xacro">
-  <xacro:include
-      filename="$(find motoman_ma1440_support)/urdf/ma1440/ma1440.transmission.xacro"/>
-  <xacro:macro
-      name="motoman_ma1440"
-      params="
+<robot xmlns:xacro="http://ros.org/wiki/xacro">
+    <xacro:include filename="$(find motoman_ma1440_support)/urdf/ma1440/ma1440.transmission.xacro" />
+    <xacro:macro
+        name="motoman_ma1440"
+        params="
                  prefix
                  world_base_xyz:='0 0 0'
                  world_base_rpy:='0 0 0'
                  offsets_file_path"
-  >
-    <xacro:property
-        name="M_PI"
-        value="3.1415926535897931"/>
-    <xacro:property
-        name="M_PI_2"
-        value="1.57079632679"/>
-    <xacro:property
-        name="M_PI_4"
-        value="0.7853981633974483"/>
-    <xacro:property
-        name="offsets"
-        value="${load_yaml(offsets_file_path)[prefix + 'robot_calibration_offsets']}"/>
-    <xacro:property
-        name="vertical_offset"
-        value="0.5"/>
-    <link
-        name="world">
-      <origin
-          xyz="0 0 0"
-          rpy="0 0 0"/>
-    </link>
-    <link
-        name="${prefix}base_link">
-      <visual>
-        <origin
-            rpy="0 0 0"
-            xyz="0 0 0"/>
-        <geometry>
-          <mesh
-              filename="package://motoman_ma1440_support/meshes/ma1440/visual/base_link.stl"/>
-        </geometry>
-        <material
-            name="blue">
-          <color
-              rgba="0 0 1 1"/>
-        </material>
-      </visual>
-      <collision>
-        <origin
-            rpy="0 0 0"
-            xyz="0 0 0"/>
-        <geometry>
-          <mesh
-              filename="package://motoman_ma1440_support/meshes/ma1440/collision/base_link_collision.stl"/>
-        </geometry>
-        <material
-            name="yellow">
-          <color
-              rgba="0 1 1 1"/>
-        </material>
-      </collision>
-      <inertial>
-        <mass
-            value="400"/>  <!-- Arbitrarily large value, to simulate bolting down in case of absence of fixed joint -->
-        <inertia
-            ixx="1.0"
-            ixy="0.0"
-            ixz="0.0"
-            iyy="1.0"
-            iyz="0.0"
-            izz="1.0"/>
-        <origin
-            rpy="0 0 0"
-            xyz="0 0 0"/>
-      </inertial>
-    </link>
-    <gazebo
-        reference="${prefix}base_link">
-      <turnGravityOff>
-        false
-      </turnGravityOff>
-      <selfCollide>
-        true
-      </selfCollide>
-      <material>
-        Gazebo/Blue
-      </material>
-    </gazebo>
-    <link
-        name="${prefix}link_s">
-      <visual>
-        <origin
-            rpy="0 0 0"
-            xyz="0 0 0"/>
-        <geometry>
-          <mesh
-              filename="package://motoman_ma1440_support/meshes/ma1440/visual/s_link.stl"/>
-        </geometry>
-        <material
-            name="blue">
-          <color
-              rgba="0 0 1 1"/>
-        </material>
-      </visual>
-      <collision>
-        <origin
-            rpy="0 0 0"
-            xyz="0 0 0"/>
-        <geometry>
-          <mesh
-              filename="package://motoman_ma1440_support/meshes/ma1440/collision/s_link_collision.stl"/>
-        </geometry>
-        <material
-            name="yellow"/>
-      </collision>
-      <!--      TODO: Remove this once the collision model is updated to include the little bump      -->
-      <collision>
-        <origin
-            rpy="0 0 0"
-            xyz="0.11 -0.02 0.095"/>
-        <geometry>
-          <box
-              size="0.1 0.05 0.1"/>
-        </geometry>
-      </collision>
-      <inertial>
-        <mass
-            value="112.57"/>
-        <inertia
-            ixx="2.1336"
-            ixy="0.197"
-            ixz="0.8995"
-            iyy="2.8341"
-            iyz="0.2799"
-            izz="2.49"/>
-        <origin
-            rpy="0 0 0"
-            xyz="0 0 0"/>
-      </inertial>
-    </link>
-    <gazebo
-        reference="${prefix}link_s">
-      <turnGravityOff>
-        false
-      </turnGravityOff>
-      <selfCollide>
-        true
-      </selfCollide>
-      <material>
-        Gazebo/Blue
-      </material>
-    </gazebo>
-    <link
-        name="${prefix}link_l">
-      <visual>
-        <origin
-            rpy="0 0 0"
-            xyz="0 0 0"/>
-        <geometry>
-          <mesh
-              filename="package://motoman_ma1440_support/meshes/ma1440/visual/l_link.stl"/>
-        </geometry>
-        <material
-            name="blue"/>
-      </visual>
-      <collision>
-        <origin
-            rpy="0 0 0"
-            xyz="0 0 0"/>
-        <geometry>
-          <mesh
-              filename="package://motoman_ma1440_support/meshes/ma1440/collision/l_link_collision.stl"/>
-        </geometry>
-        <material
-            name="yellow"/>
-      </collision>
-      <inertial>
-        <mass
-            value="45.143"/>
-        <inertia
-            ixx="0.1565"
-            ixy="-0.0239"
-            ixz="-0.0981"
-            iyy="2.4306"
-            iyz="0.0329"
-            izz="2.4493"/>
-        <origin
-            rpy="0 0 0"
-            xyz="0 0 0"/>
-      </inertial>
-    </link>
-    <gazebo
-        reference="${prefix}link_l">
-      <turnGravityOff>
-        false
-      </turnGravityOff>
-      <selfCollide>
-        true
-      </selfCollide>
-      <material>
-        Gazebo/Blue
-      </material>
-    </gazebo>
-    <link
-        name="${prefix}link_u">
-      <visual>
-        <origin
-            rpy="0 0 0"
-            xyz="0 0 0"/>
-        <geometry>
-          <mesh
-              filename="package://motoman_ma1440_support/meshes/ma1440/visual/u_link.stl"/>
-        </geometry>
-        <material
-            name="blue"/>
-      </visual>
-      <collision>
-        <origin
-            rpy="0 ${M_PI} ${M_PI_2}"
-            xyz="0 0 0"/>
-        <geometry>
-          <mesh
-              filename="package://motoman_ma1440_support/meshes/ma1440/collision/u_link_collision.stl"/>
-        </geometry>
-        <material
-            name="yellow"/>
-      </collision>
-      <inertial>
-        <mass
-            value="77.767"/>
-        <inertia
-            ixx="1.1285"
-            ixy="-0.4562"
-            ixz="-0.1754"
-            iyy="0.965"
-            iyz="0.2365"
-            izz="1.2844"/>
-        <origin
-            rpy="0 0 0"
-            xyz="0 0 0"/>
-      </inertial>
-      <collision>
-        <origin
-            rpy="0 0 ${M_PI_2}"
-            xyz="0.10 0.15 -0.10"/>
-        <geometry>
-          <box
-              size="0.55 0.35 0.38"/>
-        </geometry>
-      </collision>
-    </link>
-    <gazebo
-        reference="${prefix}link_u">
-      <turnGravityOff>
-        false
-      </turnGravityOff>
-      <selfCollide>
-        true
-      </selfCollide>
-      <material>
-        Gazebo/Blue
-      </material>
-    </gazebo>
-    <link
-        name="${prefix}link_r">
-      <visual>
-        <origin
-            rpy="0 0 0"
-            xyz="0 0 0"/>
-        <geometry>
-          <mesh
-              filename="package://motoman_ma1440_support/meshes/ma1440/visual/r_link.stl"/>
-        </geometry>
-        <material
-            name="blue"/>
-      </visual>
-      <collision>
-        <origin
-            rpy="0 0 0"
-            xyz="0 0 0"/>
-        <geometry>
-          <mesh
-              filename="package://motoman_ma1440_support/meshes/ma1440/collision/r_link_collision.stl"/>
-        </geometry>
-        <material
-            name="yellow"/>
-      </collision>
-      <inertial>
-        <mass
-            value="31.136"/>
-        <inertia
-            ixx="0.5313"
-            ixy="0.0027"
-            ixz="0.0418"
-            iyy="0.453"
-            iyz="-0.0111"
-            izz="0.1611"/>
-        <origin
-            rpy="0 0 0"
-            xyz="0 0 0"/>
-      </inertial>
-    </link>
-    <gazebo
-        reference="${prefix}link_r">
-      <turnGravityOff>
-        false
-      </turnGravityOff>
-      <selfCollide>
-        true
-      </selfCollide>
-      <material>
-        Gazebo/White
-      </material>
-    </gazebo>
-    <link
-        name="${prefix}link_b">
-      <visual>
-        <origin
-            rpy="0 0 0"
-            xyz="0 0 0"/>
-        <geometry>
-          <mesh
-              filename="package://motoman_ma1440_support/meshes/ma1440/visual/b_link.stl"/>
-        </geometry>
-        <material
-            name="blue"/>
-      </visual>
-      <collision>
-        <origin
-            rpy="0 0 0"
-            xyz="0 0 0"/>
-        <geometry>
-          <mesh
-              filename="package://motoman_ma1440_support/meshes/ma1440/collision/b_link_collision.stl"/>
-        </geometry>
-        <material
-            name="yellow"/>
-      </collision>
-      <inertial>
-        <mass
-            value="7.781"/>
-        <inertia
-            ixx="0.019954"
-            ixy="6.9E-05"
-            ixz="-0.000759"
-            iyy="0.024524"
-            iyz="0.000206"
-            izz="0.019404"/>
-        <origin
-            rpy="0 0 0"
-            xyz="0 0 0"/>
-      </inertial>
-    </link>
-    <gazebo
-        reference="${prefix}link_b">
-      <turnGravityOff>
-        false
-      </turnGravityOff>
-      <selfCollide>
-        true
-      </selfCollide>
-      <material>
-        Gazebo/Blue
-      </material>
-    </gazebo>
-    <link
-        name="${prefix}link_t">
-      <visual>
-        <origin
-            rpy="0 0 0"
-            xyz="0 0 0"/>
-        <geometry>
-          <mesh
-              filename="package://motoman_ma1440_support/meshes/ma1440/visual/t_link.stl"/>
-        </geometry>
-        <material
-            name="blue"/>
-      </visual>
-      <collision>
-        <origin
-            rpy="0 0 0"
-            xyz="0 0 0"/>
-        <geometry>
-          <mesh
-              filename="package://motoman_ma1440_support/meshes/ma1440/collision/t_link_collision.stl"/>
-        </geometry>
-        <material
-            name="yellow"/>
-      </collision>
-      <inertial>
-        <mass
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
Commit message: support for tip calib in urdf without reformatting

File: motoman_ma1440_support/urdf/ma1440/ma1440_macro.xacro (robot description, xacro)
@@ -329,5 +329,6 @@
             <parent link="${prefix}link_t"/>
             <child link="${prefix}link_tip"/>
-            <origin xyz="-0.09591 0 ${-0.38772 + 0.0125}" rpy="${-135*M_PI/180} 0 ${M_PI/2}"/>
+            <origin xyz="${-0.09591+ + offsets[prefix + 'joint_tip']['x']} ${0+ + offsets[prefix + 'joint_tip']['y']} ${-0.38772 + 0.0125 + offsets[prefix + 'joint_tip']['z']}"
+                    rpy="${-135*M_PI/180 + offsets[prefix + 'joint_tip']['roll']} ${0 + offsets[prefix + 'joint_tip']['pitch']} ${M_PI/2 + offsets[prefix + 'joint_tip']['yaw']}"/>
             <axis xyz="0 0 0" />
         </joint>
