Commit message: gp88: use 'offset tool0 from link_6_t' convention in the urdf
Does not move the pose of tool0 relative to base_link

File: motoman_gp88_support/urdf/gp88_macro.xacro (robot description, xacro)
@@ -139,10 +139,10 @@
         <parent link="${prefix}link_5_b"/>
         <child link="${prefix}link_6_t"/>
-        <origin xyz="0.175 0 0" rpy="0 0 0" />
+        <origin xyz="0 0 0" rpy="0 0 0" />
         <axis xyz="-1 0 0" />
         <limit lower="${radians(-360)}" upper="${radians(360)}" effort="375.1" velocity="${radians(350)}"/>
     </joint>
     <joint name="${prefix}joint_6_t-tool0" type="fixed">
-        <origin xyz="0 0 0" rpy="${radians(180)} ${radians(-90)} 0"/>
+        <origin xyz="0.175 0 0" rpy="${radians(180)} ${radians(-90)} 0"/>
         <parent link="${prefix}link_6_t"/>
         <child link="${prefix}tool0"/>

Commit message: gp88: group convenience frames together.

File: motoman_gp88_support/urdf/gp88_macro.xacro (robot description, xacro)
@@ -98,5 +98,4 @@
         </collision>
     </link>
-    <link name="${prefix}tool0"/>
     <!-- end of link list -->
     <!-- joint list -->
@@ -143,9 +142,4 @@
         <limit lower="${radians(-360)}" upper="${radians(360)}" effort="375.1" velocity="${radians(350)}"/>
     </joint>
-    <joint name="${prefix}joint_6_t-tool0" type="fixed">
-        <origin xyz="0.175 0 0" rpy="${radians(180)} ${radians(-90)} 0"/>
-        <parent link="${prefix}link_6_t"/>
-        <child link="${prefix}tool0"/>
-    </joint>
     <!-- end of joint list -->
     <!-- ROS base_link to Robot Manufacturer World Coordinates transform -->
@@ -156,4 +150,11 @@
         <child link="${prefix}base"/>
     </joint>
+    <!-- ROS-Industrial 'tool0' frame: all-zeros tool frame -->
+    <link name="${prefix}tool0"/>
+    <joint name="${prefix}joint_6_t-tool0" type="fixed">
+        <origin xyz="0.175 0 0" rpy="${radians(180)} ${radians(-90)} 0"/>
+        <parent link="${prefix}link_6_t"/>
+        <child link="${prefix}tool0"/>
+    </joint>
 </xacro:macro>
 </robot>
