Commit message: sia50_support: Rename package to drop "d" suffix

File: motoman_sia50_support/urdf/sia50d.xacro (robot description, xacro)
@@ -1,5 +1,5 @@
 <?xml version="1.0" ?>
 <robot name="motoman_sia50d" xmlns:xacro="http://ros.org/wiki/xacro">
-  <xacro:include filename="$(find motoman_sia50d_support)/urdf/sia50d_macro.xacro" />
+  <xacro:include filename="$(find motoman_sia50_support)/urdf/sia50d_macro.xacro" />
   <xacro:motoman_sia50d prefix=""/>
 </robot>

File: motoman_sia50_support/urdf/sia50d_macro.xacro (robot description, xacro)
@@ -6,5 +6,5 @@
             <visual>
                 <geometry>
-                    <mesh filename="package://motoman_sia50d_support/meshes/sia50d/visual/base_link.stl" />
+                    <mesh filename="package://motoman_sia50_support/meshes/sia50d/visual/base_link.stl" />
                 </geometry>
                 <material name="blue">
@@ -14,5 +14,5 @@
             <collision>
                 <geometry>
-                    <mesh filename="package://motoman_sia50d_support/meshes/sia50d/collision/base_link.stl" />
+                    <mesh filename="package://motoman_sia50_support/meshes/sia50d/collision/base_link.stl" />
                 </geometry>
                 <material name="yellow">
@@ -25,5 +25,5 @@
                 <origin rpy="0 0 0" xyz="0 0 0"/>
                 <geometry>
-                    <mesh filename="package://motoman_sia50d_support/meshes/sia50d/visual/link_1_s.stl"/>
+                    <mesh filename="package://motoman_sia50_support/meshes/sia50d/visual/link_1_s.stl"/>
                 </geometry>
                 <material name="silver">
@@ -34,5 +34,5 @@
                 <origin rpy="0 0 0" xyz="0 0 0"/>
                 <geometry>
-                    <mesh filename="package://motoman_sia50d_support/meshes/sia50d/collision/link_1_s.stl" />
+                    <mesh filename="package://motoman_sia50_support/meshes/sia50d/collision/link_1_s.stl" />
                 </geometry>
                 <material name="yellow"/>
@@ -43,5 +43,5 @@
                 <origin rpy="0 0 0" xyz="0 0 0"/>
                 <geometry>
-                    <mesh filename="package://motoman_sia50d_support/meshes/sia50d/visual/link_2_l.stl"/>
+                    <mesh filename="package://motoman_sia50_support/meshes/sia50d/visual/link_2_l.stl"/>
                 </geometry>
                 <material name="blue"/>
@@ -50,5 +50,5 @@
                 <origin rpy="0 0 0" xyz="0 0 0"/>
                 <geometry>
-                    <mesh filename="package://motoman_sia50d_support/meshes/sia50d/collision/link_2_l.stl"/>
+                    <mesh filename="package://motoman_sia50_support/meshes/sia50d/collision/link_2_l.stl"/>
                 </geometry>
                 <material name="yellow"/>
@@ -59,5 +59,5 @@
                 <origin rpy="0 0 0" xyz="0 0 0"/>
                 <geometry>
-                    <mesh filename="package://motoman_sia50d_support/meshes/sia50d/visual/link_3_e.stl"/>
+                    <mesh filename="package://motoman_sia50_support/meshes/sia50d/visual/link_3_e.stl"/>
                 </geometry>
                 <material name="silver"/>
@@ -66,5 +66,5 @@
                 <origin rpy="0 0 0" xyz="0 0 0"/>
                 <geometry>
-                    <mesh filename="package://motoman_sia50d_support/meshes/sia50d/collision/link_3_e.stl"/>
+                    <mesh filename="package://motoman_sia50_support/meshes/sia50d/collision/link_3_e.stl"/>
                 </geometry>
                 <material name="yellow"/>
@@ -75,5 +75,5 @@
                 <origin rpy="0 0 0" xyz="0 0 0"/>
                 <geometry>
-                    <mesh filename="package://motoman_sia50d_support/meshes/sia50d/visual/link_4_u.stl"/>
+                    <mesh filename="package://motoman_sia50_support/meshes/sia50d/visual/link_4_u.stl"/>
                 </geometry>
                 <material name="blue"/>
@@ -82,5 +82,5 @@
                 <origin rpy="0 0 0" xyz="0 0 0"/>
                 <geometry>
-                    <mesh filename="package://motoman_sia50d_support/meshes/sia50d/collision/link_4_u.stl"/>
+                    <mesh filename="package://motoman_sia50_support/meshes/sia50d/collision/link_4_u.stl"/>
                 </geometry>
                 <material name="yellow"/>
@@ -91,5 +91,5 @@
                 <origin rpy="0 0 0" xyz="0 0 0"/>
                 <geometry>
-                    <mesh filename="package://motoman_sia50d_support/meshes/sia50d/visual/link_5_r.stl"/>
+                    <mesh filename="package://motoman_sia50_support/meshes/sia50d/visual/link_5_r.stl"/>
                 </geometry>
                 <material name="silver"/>
@@ -98,5 +98,5 @@
                 <origin rpy="0 0 0" xyz="0 0 0"/>
                 <geometry>
-                    <mesh filename="package://motoman_sia50d_support/meshes/sia50d/collision/link_5_r.stl"/>
+                    <mesh filename="package://motoman_sia50_support/meshes/sia50d/collision/link_5_r.stl"/>
                 </geometry>
                 <material name="yellow"/>
@@ -107,5 +107,5 @@
                 <origin rpy="0 0 0" xyz="0 0 0"/>
                 <geometry>
-                    <mesh filename="package://motoman_sia50d_support/meshes/sia50d/visual/link_6_b.stl"/>
+                    <mesh filename="package://motoman_sia50_support/meshes/sia50d/visual/link_6_b.stl"/>
                 </geometry>
                 <material name="blue"/>
@@ -114,5 +114,5 @@
                 <origin rpy="0 0 0" xyz="0 0 0"/>
                 <geometry>
-                    <mesh filename="package://motoman_sia50d_support/meshes/sia50d/collision/link_6_b.stl"/>
+                    <mesh filename="package://motoman_sia50_support/meshes/sia50d/collision/link_6_b.stl"/>
                 </geometry>
                 <material name="yellow"/>
@@ -122,5 +122,5 @@
             <visual>
                 <geometry>
-                    <mesh filename="package://motoman_sia50d_support/meshes/sia50d/visual/link_7_t.stl" />
+                    <mesh filename="package://motoman_sia50_support/meshes/sia50d/visual/link_7_t.stl" />
                 </geometry>
                 <material name="silver"/>
@@ -128,5 +128,5 @@
             <collision>
                 <geometry>
-                    <mesh filename="package://motoman_sia50d_support/meshes/sia50d/collision/link_7_t.stl" />
+                    <mesh filename="package://motoman_sia50_support/meshes/sia50d/collision/link_7_t.stl" />
                 </geometry>
                 <material name="yellow"/>
@@ -149,5 +149,6 @@
             <origin xyz="0.145 0 0.228" rpy="0 0 0"/>
             <axis xyz="0 1 0" />
-            <limit lower="-1.047198" upper="2.181662" effort="28.4" velocity="2.268928" /><!-- 5883.99 -->
+            <limit lower="-1.047198" upper="2.181662" effort="28.4" velocity="2.268928" />
+            <!-- 5883.99 -->
         </joint>
         <joint name="${prefix}joint_e" type="revolute">
@@ -156,5 +157,6 @@
             <origin xyz="0 0 0.875" rpy="0 0 0"/>
             <axis xyz="0 0 1" />
-            <limit lower="-2.967064" upper="2.967064" effort="22" velocity="2.26893" /><!-- 2549.73 -->
+            <limit lower="-2.967064" upper="2.967064" effort="22" velocity="2.26893" />
+            <!-- 2549.73 -->
         </joint>
         <joint name="${prefix}joint_u" type="revolute">
@@ -163,5 +165,6 @@
             <origin xyz="0 0 0" rpy="0 0 0"/>
             <axis xyz="0 -1 0" />
-            <limit lower="-0.610869" upper="3.752462" effort="22" velocity="2.26893" /><!-- 2549.73 -->
+            <limit lower="-0.610869" upper="3.752462" effort="22" velocity="2.26893" />
+            <!-- 2549.73 -->
         </joint>
         <joint name="${prefix}joint_r" type="revolute">
@@ -170,5 +173,6 @@
             <origin xyz="0.61 0 0" rpy="0 0 0"/>
             <axis xyz="-1 0 0" />
-            <limit lower="-2.96706" upper="2.96706" effort="6" velocity="2.268928" /><!-- 720.2 -->
+            <limit lower="-2.96706" upper="2.96706" effort="6" velocity="2.268928" />
+            <!-- 720.2 -->
         </joint>
         <joint name="${prefix}joint_b" type="revolute">
@@ -177,5 +181,6 @@
             <origin xyz="0 0 0" rpy="0 0 0"/>
             <axis xyz="0 -1 0" />
-            <limit lower="-2.181662" upper="2.181662" effort="6" velocity="2.268928" /><!-- 720.2 -->
+            <limit lower="-2.181662" upper="2.181662" effort="6" velocity="2.268928" />
+            <!-- 720.2 -->
         </joint>
         <joint name="${prefix}joint_t" type="revolute">
@@ -184,5 +189,6 @@
             <origin xyz="0.35 0 0" rpy="0 0 0"/>
             <axis xyz="-1 0 0" />
-            <limit lower="-3.141593" upper="3.141593" effort="2.5" velocity="3.490659" /><!-- 255.76 -->
+            <limit lower="-3.141593" upper="3.141593" effort="2.5" velocity="3.490659" />
+            <!-- 255.76 -->
         </joint>
         <joint name="${prefix}link_t-tool0" type="fixed">
