Commit message: sia50_support: Fix xml indentation using 2 spaces

File: motoman_sia50_support/urdf/sia50.xacro (robot description, xacro)
@@ -1,4 +1,5 @@
 <?xml version="1.0" ?>
-<robot name="motoman_sia50" xmlns:xacro="http://ros.org/wiki/xacro">
+<robot name="motoman_sia50"
+  xmlns:xacro="http://ros.org/wiki/xacro">
   <xacro:include filename="$(find motoman_sia50_support)/urdf/sia50_macro.xacro" />
   <xacro:motoman_sia50 prefix=""/>

File: motoman_sia50_support/urdf/sia50_macro.xacro (robot description, xacro)
@@ -1,201 +1,201 @@
 <?xml version="1.0" ?>
 <robot xmlns:xacro="http://ros.org/wiki/xacro">
-    <xacro:macro name="motoman_sia50" params="prefix">
-        <!-- link list -->
-        <link name="${prefix}base_link">
-            <visual>
-                <geometry>
-                    <mesh filename="package://motoman_sia50_support/meshes/sia50/visual/base_link.stl" />
-                </geometry>
-                <material name="blue">
-                    <color rgba="0 0 1 1"/>
-                </material>
-            </visual>
-            <collision>
-                <geometry>
-                    <mesh filename="package://motoman_sia50_support/meshes/sia50/collision/base_link.stl" />
-                </geometry>
-                <material name="yellow">
-                    <color rgba="0 1 1 1"/>
-                </material>
-            </collision>
-        </link>
-        <link name="${prefix}link_s">
-            <visual>
-                <origin rpy="0 0 0" xyz="0 0 0"/>
-                <geometry>
-                    <mesh filename="package://motoman_sia50_support/meshes/sia50/visual/link_1_s.stl"/>
-                </geometry>
-                <material name="silver">
-                    <color rgba="0.8 0.8 0.8 1"/>
-                </material>
-            </visual>
-            <collision>
-                <origin rpy="0 0 0" xyz="0 0 0"/>
-                <geometry>
-                    <mesh filename="package://motoman_sia50_support/meshes/sia50/collision/link_1_s.stl" />
-                </geometry>
-                <material name="yellow"/>
-            </collision>
-        </link>
-        <link name="${prefix}link_l">
-            <visual>
-                <origin rpy="0 0 0" xyz="0 0 0"/>
-                <geometry>
-                    <mesh filename="package://motoman_sia50_support/meshes/sia50/visual/link_2_l.stl"/>
-                </geometry>
-                <material name="blue"/>
-            </visual>
-            <collision>
-                <origin rpy="0 0 0" xyz="0 0 0"/>
-                <geometry>
-                    <mesh filename="package://motoman_sia50_support/meshes/sia50/collision/link_2_l.stl"/>
-                </geometry>
-                <material name="yellow"/>
-            </collision>
-        </link>
-        <link name="${prefix}link_e">
-            <visual>
-                <origin rpy="0 0 0" xyz="0 0 0"/>
-                <geometry>
-                    <mesh filename="package://motoman_sia50_support/meshes/sia50/visual/link_3_e.stl"/>
-                </geometry>
-                <material name="silver"/>
-            </visual>
-            <collision>
-                <origin rpy="0 0 0" xyz="0 0 0"/>
-                <geometry>
-                    <mesh filename="package://motoman_sia50_support/meshes/sia50/collision/link_3_e.stl"/>
-                </geometry>
-                <material name="yellow"/>
-            </collision>
-        </link>
-        <link name="${prefix}link_u">
-            <visual>
-                <origin rpy="0 0 0" xyz="0 0 0"/>
-                <geometry>
-                    <mesh filename="package://motoman_sia50_support/meshes/sia50/visual/link_4_u.stl"/>
-                </geometry>
-                <material name="blue"/>
-            </visual>
-            <collision>
-                <origin rpy="0 0 0" xyz="0 0 0"/>
-                <geometry>
-                    <mesh filename="package://motoman_sia50_support/meshes/sia50/collision/link_4_u.stl"/>
-                </geometry>
-                <material name="yellow"/>
-            </collision>
-        </link>
-        <link name="${prefix}link_r">
-            <visual>
-                <origin rpy="0 0 0" xyz="0 0 0"/>
-                <geometry>
-                    <mesh filename="package://motoman_sia50_support/meshes/sia50/visual/link_5_r.stl"/>
-                </geometry>
-                <material name="silver"/>
-            </visual>
-            <collision>
-                <origin rpy="0 0 0" xyz="0 0 0"/>
-                <geometry>
-                    <mesh filename="package://motoman_sia50_support/meshes/sia50/collision/link_5_r.stl"/>
-                </geometry>
-                <material name="yellow"/>
-            </collision>
-        </link>
-        <link name="${prefix}link_b">
-            <visual>
-                <origin rpy="0 0 0" xyz="0 0 0"/>
-                <geometry>
-                    <mesh filename="package://motoman_sia50_support/meshes/sia50/visual/link_6_b.stl"/>
-                </geometry>
-                <material name="blue"/>
-            </visual>
-            <collision>
-                <origin rpy="0 0 0" xyz="0 0 0"/>
-                <geometry>
-                    <mesh filename="package://motoman_sia50_support/meshes/sia50/collision/link_6_b.stl"/>
-                </geometry>
-                <material name="yellow"/>
-            </collision>
-        </link>
-        <link name="${prefix}link_t">
-            <visual>
-                <geometry>
-                    <mesh filename="package://motoman_sia50_support/meshes/sia50/visual/link_7_t.stl" />
-                </geometry>
-                <material name="silver"/>
-            </visual>
-            <collision>
-                <geometry>
-                    <mesh filename="package://motoman_sia50_support/meshes/sia50/collision/link_7_t.stl" />
-                </geometry>
-                <material name="yellow"/>
-            </collision>
-        </link>
-        <link name="${prefix}tool0" />
-        <!-- end of link list -->
-        <!-- joint list -->
-        <joint name="${prefix}joint_s" type="revolute">
-            <parent link="${prefix}base_link"/>
-            <child link="${prefix}link_s"/>
-            <origin xyz="0 0 0.312" rpy="0 0 0"/>
-            <axis xyz="0 0 1" />
-            <limit lower="${radians(-180)}" upper="${radians(180)}" effort="4903.32" velocity="${radians(170)}" />
-        </joint>
-        <joint name="${prefix}joint_l" type="revolute">
-            <parent link="${prefix}link_s"/>
-            <child link="${prefix}link_l"/>
-            <origin xyz="0.145 0 0.228" rpy="0 0 0"/>
-            <axis xyz="0 1 0" />
-            <limit lower="${radians(-60)}" upper="${radians(125)}" effort="5883.99" velocity="${radians(130)}" />
-        </joint>
-        <joint name="${prefix}joint_e" type="revolute">
-            <parent link="${prefix}link_l"/>
-            <child link="${prefix}link_e"/>
-            <origin xyz="0 0 0.875" rpy="0 0 0"/>
-            <axis xyz="0 0 1" />
-            <limit lower="${radians(-170)}" upper="${radians(170)}" effort="2549.73" velocity="${radians(130)}" />
-        </joint>
-        <joint name="${prefix}joint_u" type="revolute">
-            <parent link="${prefix}link_e"/>
-            <child link="${prefix}link_u"/>
-            <origin xyz="0 0 0" rpy="0 0 0"/>
-            <axis xyz="0 -1 0" />
-            <limit lower="${radians(-35)}" upper="${radians(215)}" effort="2549.73" velocity="${radians(130)}" />
-        </joint>
-        <joint name="${prefix}joint_r" type="revolute">
-            <parent link="${prefix}link_u"/>
-            <child link="${prefix}link_r"/>
-            <origin xyz="0.61 0 0" rpy="0 0 0"/>
-            <axis xyz="-1 0 0" />
-            <limit lower="${radians(-170)}" upper="${radians(170)}" effort="720.2" velocity="${radians(130)}" />
-        </joint>
-        <joint name="${prefix}joint_b" type="revolute">
-            <parent link="${prefix}link_r"/>
-            <child link="${prefix}link_b"/>
-            <origin xyz="0 0 0" rpy="0 0 0"/>
-            <axis xyz="0 -1 0" />
-            <limit lower="${radians(-125)}" upper="${radians(125)}" effort="720.2" velocity="${radians(130)}" />
-        </joint>
-        <joint name="${prefix}joint_t" type="revolute">
-            <parent link="${prefix}link_b"/>
-            <child link="${prefix}link_t"/>
-            <origin xyz="0.35 0 0" rpy="0 0 0"/>
-            <axis xyz="-1 0 0" />
-            <limit lower="${radians(-180)}" upper="${radians(180)}" effort="255.76" velocity="${radians(200)}" />
-        </joint>
-        <joint name="${prefix}link_t-tool0" type="fixed">
-            <origin xyz="0 0 0.0" rpy="0 0 ${radians(-180)}"/>
-            <parent link="${prefix}link_t" />
-            <child link="${prefix}tool0" />
-        </joint>
-        <!-- end of joint list -->
-        <!-- ROS base_link (via base_link) to Motoman Robot (not Base) Frame transform -->
-        <link name="${prefix}base" />
-        <joint name="${prefix}base_link-base" type="fixed">
-            <origin xyz="0 0 0.540" rpy="0 0 0"/>
-            <parent link="${prefix}base_link"/>
-            <child link="${prefix}base"/>
-        </joint>
-    </xacro:macro>
+  <xacro:macro name="motoman_sia50" params="prefix">
+    <!-- link list -->
+    <link name="${prefix}base_link">
+      <visual>
+        <geometry>
+          <mesh filename="package://motoman_sia50_support/meshes/sia50/visual/base_link.stl" />
+        </geometry>
+        <material name="blue">
+          <color rgba="0 0 1 1"/>
+        </material>
+      </visual>
+      <collision>
+        <geometry>
+          <mesh filename="package://motoman_sia50_support/meshes/sia50/collision/base_link.stl" />
+        </geometry>
+        <material name="yellow">
+          <color rgba="0 1 1 1"/>
+        </material>
+      </collision>
+    </link>
+    <link name="${prefix}link_s">
+      <visual>
+        <origin rpy="0 0 0" xyz="0 0 0"/>
+        <geometry>
+          <mesh filename="package://motoman_sia50_support/meshes/sia50/visual/link_1_s.stl"/>
+        </geometry>
+        <material name="silver">
+          <color rgba="0.8 0.8 0.8 1"/>
+        </material>
+      </visual>
+      <collision>
+        <origin rpy="0 0 0" xyz="0 0 0"/>
+        <geometry>
+          <mesh filename="package://motoman_sia50_support/meshes/sia50/collision/link_1_s.stl" />
+        </geometry>
+        <material name="yellow"/>
+      </collision>
+    </link>
+    <link name="${prefix}link_l">
+      <visual>
+        <origin rpy="0 0 0" xyz="0 0 0"/>
+        <geometry>
+          <mesh filename="package://motoman_sia50_support/meshes/sia50/visual/link_2_l.stl"/>
+        </geometry>
+        <material name="blue"/>
+      </visual>
+      <collision>
+        <origin rpy="0 0 0" xyz="0 0 0"/>
+        <geometry>
+          <mesh filename="package://motoman_sia50_support/meshes/sia50/collision/link_2_l.stl"/>
+        </geometry>
+        <material name="yellow"/>
+      </collision>
+    </link>
+    <link name="${prefix}link_e">
+      <visual>
+        <origin rpy="0 0 0" xyz="0 0 0"/>
+        <geometry>
+          <mesh filename="package://motoman_sia50_support/meshes/sia50/visual/link_3_e.stl"/>
+        </geometry>
+        <material name="silver"/>
+      </visual>
+      <collision>
+        <origin rpy="0 0 0" xyz="0 0 0"/>
+        <geometry>
+          <mesh filename="package://motoman_sia50_support/meshes/sia50/collision/link_3_e.stl"/>
+        </geometry>
+        <material name="yellow"/>
+      </collision>
+    </link>
+    <link name="${prefix}link_u">
+      <visual>
+        <origin rpy="0 0 0" xyz="0 0 0"/>
+        <geometry>
+          <mesh filename="package://motoman_sia50_support/meshes/sia50/visual/link_4_u.stl"/>
+        </geometry>
+        <material name="blue"/>
+      </visual>
+      <collision>
+        <origin rpy="0 0 0" xyz="0 0 0"/>
+        <geometry>
+          <mesh filename="package://motoman_sia50_support/meshes/sia50/collision/link_4_u.stl"/>
+        </geometry>
+        <material name="yellow"/>
+      </collision>
+    </link>
+    <link name="${prefix}link_r">
+      <visual>
+        <origin rpy="0 0 0" xyz="0 0 0"/>
+        <geometry>
+          <mesh filename="package://motoman_sia50_support/meshes/sia50/visual/link_5_r.stl"/>
+        </geometry>
+        <material name="silver"/>
+      </visual>
+      <collision>
+        <origin rpy="0 0 0" xyz="0 0 0"/>
+        <geometry>
+          <mesh filename="package://motoman_sia50_support/meshes/sia50/collision/link_5_r.stl"/>
+        </geometry>
+        <material name="yellow"/>
+      </collision>
+    </link>
+    <link name="${prefix}link_b">
+      <visual>
+        <origin rpy="0 0 0" xyz="0 0 0"/>
+        <geometry>
+          <mesh filename="package://motoman_sia50_support/meshes/sia50/visual/link_6_b.stl"/>
+        </geometry>
+        <material name="blue"/>
+      </visual>
+      <collision>
+        <origin rpy="0 0 0" xyz="0 0 0"/>
+        <geometry>
+          <mesh filename="package://motoman_sia50_support/meshes/sia50/collision/link_6_b.stl"/>
+        </geometry>
+        <material name="yellow"/>
+      </collision>
+    </link>
+    <link name="${prefix}link_t">
+      <visual>
+        <geometry>
+          <mesh filename="package://motoman_sia50_support/meshes/sia50/visual/link_7_t.stl" />
+        </geometry>
+        <material name="silver"/>
+      </visual>
+      <collision>
+        <geometry>
+          <mesh filename="package://motoman_sia50_support/meshes/sia50/collision/link_7_t.stl" />
+        </geometry>
+        <material name="yellow"/>
+      </collision>
+    </link>
+    <link name="${prefix}tool0" />
+    <!-- end of link list -->
+    <!-- joint list -->
+    <joint name="${prefix}joint_s" type="revolute">
+      <parent link="${prefix}base_link"/>
+      <child link="${prefix}link_s"/>
+      <origin xyz="0 0 0.312" rpy="0 0 0"/>
+      <axis xyz="0 0 1" />
+      <limit lower="${radians(-180)}" upper="${radians(180)}" effort="4903.32" velocity="${radians(170)}" />
+    </joint>
+    <joint name="${prefix}joint_l" type="revolute">
+      <parent link="${prefix}link_s"/>
+      <child link="${prefix}link_l"/>
+      <origin xyz="0.145 0 0.228" rpy="0 0 0"/>
+      <axis xyz="0 1 0" />
+      <limit lower="${radians(-60)}" upper="${radians(125)}" effort="5883.99" velocity="${radians(130)}" />
+    </joint>
+    <joint name="${prefix}joint_e" type="revolute">
+      <parent link="${prefix}link_l"/>
+      <child link="${prefix}link_e"/>
+      <origin xyz="0 0 0.875" rpy="0 0 0"/>
+      <axis xyz="0 0 1" />
+      <limit lower="${radians(-170)}" upper="${radians(170)}" effort="2549.73" velocity="${radians(130)}" />
+    </joint>
+    <joint name="${prefix}joint_u" type="revolute">
+      <parent link="${prefix}link_e"/>
+      <child link="${prefix}link_u"/>
+      <origin xyz="0 0 0" rpy="0 0 0"/>
+      <axis xyz="0 -1 0" />
+      <limit lower="${radians(-35)}" upper="${radians(215)}" effort="2549.73" velocity="${radians(130)}" />
+    </joint>
+    <joint name="${prefix}joint_r" type="revolute">
+      <parent link="${prefix}link_u"/>
+      <child link="${prefix}link_r"/>
+      <origin xyz="0.61 0 0" rpy="0 0 0"/>
+      <axis xyz="-1 0 0" />
+      <limit lower="${radians(-170)}" upper="${radians(170)}" effort="720.2" velocity="${radians(130)}" />
+    </joint>
+    <joint name="${prefix}joint_b" type="revolute">
+      <parent link="${prefix}link_r"/>
+      <child link="${prefix}link_b"/>
+      <origin xyz="0 0 0" rpy="0 0 0"/>
+      <axis xyz="0 -1 0" />
+      <limit lower="${radians(-125)}" upper="${radians(125)}" effort="720.2" velocity="${radians(130)}" />
+    </joint>
+    <joint name="${prefix}joint_t" type="revolute">
+      <parent link="${prefix}link_b"/>
+      <child link="${prefix}link_t"/>
+      <origin xyz="0.35 0 0" rpy="0 0 0"/>
+      <axis xyz="-1 0 0" />
+      <limit lower="${radians(-180)}" upper="${radians(180)}" effort="255.76" velocity="${radians(200)}" />
+    </joint>
+    <joint name="${prefix}link_t-tool0" type="fixed">
+      <origin xyz="0 0 0.0" rpy="0 0 ${radians(-180)}"/>
+      <parent link="${prefix}link_t" />
+      <child link="${prefix}tool0" />
+    </joint>
+    <!-- end of joint list -->
+    <!-- ROS base_link (via base_link) to Motoman Robot (not Base) Frame transform -->
+    <link name="${prefix}base" />
+    <joint name="${prefix}base_link-base" type="fixed">
+      <origin xyz="0 0 0.540" rpy="0 0 0"/>
+      <parent link="${prefix}base_link"/>
+      <child link="${prefix}base"/>
+    </joint>
+  </xacro:macro>
 </robot>
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