Commit message: sia50_support: Address PR review comments

File: motoman_sia50_support/urdf/sia50_macro.xacro (robot description, xacro)
@@ -1,10 +1,10 @@
 <?xml version="1.0" ?>
 <robot xmlns:xacro="http://ros.org/wiki/xacro">
-    <xacro:macro name="motoman_sia50d" params="prefix">
+    <xacro:macro name="motoman_sia50" params="prefix">
         <!-- link list -->
         <link name="${prefix}base_link">
             <visual>
                 <geometry>
-                    <mesh filename="package://motoman_sia50_support/meshes/sia50d/visual/base_link.stl" />
+                    <mesh filename="package://motoman_sia50_support/meshes/sia50/visual/base_link.stl" />
                 </geometry>
                 <material name="blue">
@@ -14,5 +14,5 @@
             <collision>
                 <geometry>
-                    <mesh filename="package://motoman_sia50_support/meshes/sia50d/collision/base_link.stl" />
+                    <mesh filename="package://motoman_sia50_support/meshes/sia50/collision/base_link.stl" />
                 </geometry>
                 <material name="yellow">
@@ -25,5 +25,5 @@
                 <origin rpy="0 0 0" xyz="0 0 0"/>
                 <geometry>
-                    <mesh filename="package://motoman_sia50_support/meshes/sia50d/visual/link_1_s.stl"/>
+                    <mesh filename="package://motoman_sia50_support/meshes/sia50/visual/link_1_s.stl"/>
                 </geometry>
                 <material name="silver">
@@ -34,5 +34,5 @@
                 <origin rpy="0 0 0" xyz="0 0 0"/>
                 <geometry>
-                    <mesh filename="package://motoman_sia50_support/meshes/sia50d/collision/link_1_s.stl" />
+                    <mesh filename="package://motoman_sia50_support/meshes/sia50/collision/link_1_s.stl" />
                 </geometry>
                 <material name="yellow"/>
@@ -43,5 +43,5 @@
                 <origin rpy="0 0 0" xyz="0 0 0"/>
                 <geometry>
-                    <mesh filename="package://motoman_sia50_support/meshes/sia50d/visual/link_2_l.stl"/>
+                    <mesh filename="package://motoman_sia50_support/meshes/sia50/visual/link_2_l.stl"/>
                 </geometry>
                 <material name="blue"/>
@@ -50,5 +50,5 @@
                 <origin rpy="0 0 0" xyz="0 0 0"/>
                 <geometry>
-                    <mesh filename="package://motoman_sia50_support/meshes/sia50d/collision/link_2_l.stl"/>
+                    <mesh filename="package://motoman_sia50_support/meshes/sia50/collision/link_2_l.stl"/>
                 </geometry>
                 <material name="yellow"/>
@@ -59,5 +59,5 @@
                 <origin rpy="0 0 0" xyz="0 0 0"/>
                 <geometry>
-                    <mesh filename="package://motoman_sia50_support/meshes/sia50d/visual/link_3_e.stl"/>
+                    <mesh filename="package://motoman_sia50_support/meshes/sia50/visual/link_3_e.stl"/>
                 </geometry>
                 <material name="silver"/>
@@ -66,5 +66,5 @@
                 <origin rpy="0 0 0" xyz="0 0 0"/>
                 <geometry>
-                    <mesh filename="package://motoman_sia50_support/meshes/sia50d/collision/link_3_e.stl"/>
+                    <mesh filename="package://motoman_sia50_support/meshes/sia50/collision/link_3_e.stl"/>
                 </geometry>
                 <material name="yellow"/>
@@ -75,5 +75,5 @@
                 <origin rpy="0 0 0" xyz="0 0 0"/>
                 <geometry>
-                    <mesh filename="package://motoman_sia50_support/meshes/sia50d/visual/link_4_u.stl"/>
+                    <mesh filename="package://motoman_sia50_support/meshes/sia50/visual/link_4_u.stl"/>
                 </geometry>
                 <material name="blue"/>
@@ -82,5 +82,5 @@
                 <origin rpy="0 0 0" xyz="0 0 0"/>
                 <geometry>
-                    <mesh filename="package://motoman_sia50_support/meshes/sia50d/collision/link_4_u.stl"/>
+                    <mesh filename="package://motoman_sia50_support/meshes/sia50/collision/link_4_u.stl"/>
                 </geometry>
                 <material name="yellow"/>
@@ -91,5 +91,5 @@
                 <origin rpy="0 0 0" xyz="0 0 0"/>
                 <geometry>
-                    <mesh filename="package://motoman_sia50_support/meshes/sia50d/visual/link_5_r.stl"/>
+                    <mesh filename="package://motoman_sia50_support/meshes/sia50/visual/link_5_r.stl"/>
                 </geometry>
                 <material name="silver"/>
@@ -98,5 +98,5 @@
                 <origin rpy="0 0 0" xyz="0 0 0"/>
                 <geometry>
-                    <mesh filename="package://motoman_sia50_support/meshes/sia50d/collision/link_5_r.stl"/>
+                    <mesh filename="package://motoman_sia50_support/meshes/sia50/collision/link_5_r.stl"/>
                 </geometry>
                 <material name="yellow"/>
@@ -107,5 +107,5 @@
                 <origin rpy="0 0 0" xyz="0 0 0"/>
                 <geometry>
-                    <mesh filename="package://motoman_sia50_support/meshes/sia50d/visual/link_6_b.stl"/>
+                    <mesh filename="package://motoman_sia50_support/meshes/sia50/visual/link_6_b.stl"/>
                 </geometry>
                 <material name="blue"/>
@@ -114,5 +114,5 @@
                 <origin rpy="0 0 0" xyz="0 0 0"/>
                 <geometry>
-                    <mesh filename="package://motoman_sia50_support/meshes/sia50d/collision/link_6_b.stl"/>
+                    <mesh filename="package://motoman_sia50_support/meshes/sia50/collision/link_6_b.stl"/>
                 </geometry>
                 <material name="yellow"/>
@@ -122,5 +122,5 @@
             <visual>
                 <geometry>
-                    <mesh filename="package://motoman_sia50_support/meshes/sia50d/visual/link_7_t.stl" />
+                    <mesh filename="package://motoman_sia50_support/meshes/sia50/visual/link_7_t.stl" />
                 </geometry>
                 <material name="silver"/>
@@ -128,5 +128,5 @@
             <collision>
                 <geometry>
-                    <mesh filename="package://motoman_sia50_support/meshes/sia50d/collision/link_7_t.stl" />
+                    <mesh filename="package://motoman_sia50_support/meshes/sia50/collision/link_7_t.stl" />
                 </geometry>
                 <material name="yellow"/>
@@ -139,8 +139,7 @@
             <parent link="${prefix}base_link"/>
             <child link="${prefix}link_s"/>
-            <origin xyz="0 0 0.312000" rpy="0 0 0"/>
+            <origin xyz="0 0 0.312" rpy="0 0 0"/>
             <axis xyz="0 0 1" />
-            <!-- Max Acc/Dec Torque: 4903.32, Rated Motor Torque: 18.5 -->
-            <limit lower="-3.1415" upper="3.1415" effort="18.5" velocity="2.967051" />
+            <limit lower="${radians(-180)}" upper="${radians(180)}" effort="4903.32" velocity="${radians(170)}" />
         </joint>
         <joint name="${prefix}joint_l" type="revolute">
@@ -149,6 +148,5 @@
             <origin xyz="0.145 0 0.228" rpy="0 0 0"/>
             <axis xyz="0 1 0" />
-            <limit lower="-1.047198" upper="2.181662" effort="28.4" velocity="2.268928" />
-            <!-- 5883.99 -->
+            <limit lower="${radians(-60)}" upper="${radians(125)}" effort="5883.99" velocity="${radians(130)}" />
         </joint>
         <joint name="${prefix}joint_e" type="revolute">
@@ -157,6 +155,5 @@
             <origin xyz="0 0 0.875" rpy="0 0 0"/>
             <axis xyz="0 0 1" />
-            <limit lower="-2.967064" upper="2.967064" effort="22" velocity="2.26893" />
-            <!-- 2549.73 -->
+            <limit lower="${radians(-170)}" upper="${radians(170)}" effort="2549.73" velocity="${radians(130)}" />
         </joint>
         <joint name="${prefix}joint_u" type="revolute">
@@ -165,6 +162,5 @@
             <origin xyz="0 0 0" rpy="0 0 0"/>
             <axis xyz="0 -1 0" />
-            <limit lower="-0.610869" upper="3.752462" effort="22" velocity="2.26893" />
-            <!-- 2549.73 -->
+            <limit lower="${radians(-35)}" upper="${radians(215)}" effort="2549.73" velocity="${radians(130)}" />
         </joint>
         <joint name="${prefix}joint_r" type="revolute">
@@ -173,6 +169,5 @@
             <origin xyz="0.61 0 0" rpy="0 0 0"/>
             <axis xyz="-1 0 0" />
-            <limit lower="-2.96706" upper="2.96706" effort="6" velocity="2.268928" />
-            <!-- 720.2 -->
+            <limit lower="${radians(-170)}" upper="${radians(170)}" effort="720.2" velocity="${radians(130)}" />
         </joint>
         <joint name="${prefix}joint_b" type="revolute">
@@ -181,6 +176,5 @@
             <origin xyz="0 0 0" rpy="0 0 0"/>
             <axis xyz="0 -1 0" />
-            <limit lower="-2.181662" upper="2.181662" effort="6" velocity="2.268928" />
-            <!-- 720.2 -->
+            <limit lower="${radians(-125)}" upper="${radians(125)}" effort="720.2" velocity="${radians(130)}" />
         </joint>
         <joint name="${prefix}joint_t" type="revolute">
@@ -189,9 +183,8 @@
             <origin xyz="0.35 0 0" rpy="0 0 0"/>
             <axis xyz="-1 0 0" />
-            <limit lower="-3.141593" upper="3.141593" effort="2.5" velocity="3.490659" />
-            <!-- 255.76 -->
+            <limit lower="${radians(-180)}" upper="${radians(180)}" effort="255.76" velocity="${radians(200)}" />
         </joint>
         <joint name="${prefix}link_t-tool0" type="fixed">
-            <origin xyz="0 0 0.0" rpy="0 0 -3.1415926535"/>
+            <origin xyz="0 0 0.0" rpy="0 0 ${radians(-180)}"/>
             <parent link="${prefix}link_t" />
             <child link="${prefix}tool0" />
@@ -199,10 +192,10 @@
         <!-- end of joint list -->
         <!-- ROS base_link (via base_link) to Motoman Robot (not Base) Frame transform -->
-        <!-- <link name="${prefix}base" />
+        <link name="${prefix}base" />
         <joint name="${prefix}base_link-base" type="fixed">
-            <origin xyz="0 0 0.410" rpy="0 0 0"/>
+            <origin xyz="0 0 0.540" rpy="0 0 0"/>
             <parent link="${prefix}base_link"/>
             <child link="${prefix}base"/>
-        </joint> -->
+        </joint>
     </xacro:macro>
 </robot>

Commit message: sia50: translate only in one dimension (xacro).
Update meshes as well.

File: motoman_sia50_support/urdf/sia50_macro.xacro (robot description, xacro)
@@ -139,5 +139,5 @@
       <parent link="${prefix}base_link"/>
       <child link="${prefix}link_s"/>
-      <origin xyz="0 0 0.312" rpy="0 0 0"/>
+      <origin xyz="0 0 0.540" rpy="0 0 0"/>
       <axis xyz="0 0 1" />
       <limit lower="${radians(-180)}" upper="${radians(180)}" effort="4903.32" velocity="${radians(170)}" />
@@ -146,5 +146,5 @@
       <parent link="${prefix}link_s"/>
       <child link="${prefix}link_l"/>
-      <origin xyz="0.145 0 0.228" rpy="0 0 0"/>
+      <origin xyz="0.145 0 0" rpy="0 0 0"/>
       <axis xyz="0 1 0" />
       <limit lower="${radians(-60)}" upper="${radians(125)}" effort="5883.99" velocity="${radians(130)}" />
