Commit message: gp50: indent fix xacro macro.

File: motoman_gp50_support/urdf/gp50.xacro (robot description, xacro)
@@ -1,5 +1,5 @@
 <?xml version="1.0" ?>
 <robot name="motoman_gp50" xmlns:xacro="http://ros.org/wiki/xacro">
-	<xacro:include filename="$(find motoman_gp50_support)/urdf/gp50_macro.xacro" />
-	<xacro:motoman_gp50 prefix=""/>
+  <xacro:include filename="$(find motoman_gp50_support)/urdf/gp50_macro.xacro" />
+  <xacro:motoman_gp50 prefix=""/>
 </robot>

File: motoman_gp50_support/urdf/gp50_macro.xacro (robot description, xacro)
@@ -1,5 +1,5 @@
 <?xml version="1.0" ?>
 <robot xmlns:xacro="http://ros.org/wiki/xacro">
-<xacro:macro name="motoman_gp50" params="prefix">
+  <xacro:macro name="motoman_gp50" params="prefix">
     <!-- Properties -->
     <material name="yaskawa_blue">
@@ -156,4 +156,4 @@
         <child link="${prefix}base"/>
     </joint>
-    </xacro:macro>
+  </xacro:macro>
 </robot>
