Commit message: Added "gp50" subfolder under the "meshes" folder
Added "gp50" subfolder under the "meshes" folder and made corresponding changes to the gp50_macro.xacro file.

File: motoman_gp50_support/urdf/gp50_macro.xacro (robot description, xacro)
@@ -10,5 +10,5 @@
         <visual>
             <geometry>
-                <mesh filename="package://motoman_gp50_support/meshes/visual/base_link.stl"/>
+                <mesh filename="package://motoman_gp50_support/meshes/gp50/visual/base_link.stl"/>
             </geometry>
             <material name="yaskawa_blue"/>
@@ -16,5 +16,5 @@
         <collision>
             <geometry>
-                <mesh filename="package://motoman_gp50_support/meshes/collision/base_link.stl"/>
+                <mesh filename="package://motoman_gp50_support/meshes/gp50/collision/base_link.stl"/>
             </geometry>
         </collision>
@@ -23,5 +23,5 @@
         <visual>
             <geometry>
-                <mesh filename="package://motoman_gp50_support/meshes/visual/link_1_s.stl"/>
+                <mesh filename="package://motoman_gp50_support/meshes/gp50/visual/link_1_s.stl"/>
             </geometry>
             <material name="yaskawa_blue"/>
@@ -29,5 +29,5 @@
         <collision>
             <geometry>
-                <mesh filename="package://motoman_gp50_support/meshes/collision/link_1_s.stl"/>
+                <mesh filename="package://motoman_gp50_support/meshes/gp50/collision/link_1_s.stl"/>
             </geometry>
         </collision>
@@ -36,5 +36,5 @@
         <visual>
             <geometry>
-                <mesh filename="package://motoman_gp50_support/meshes/visual/link_2_l.stl"/>
+                <mesh filename="package://motoman_gp50_support/meshes/gp50/visual/link_2_l.stl"/>
             </geometry>
             <material name="yaskawa_blue"/>
@@ -42,5 +42,5 @@
         <collision>
             <geometry>
-                <mesh filename="package://motoman_gp50_support/meshes/collision/link_2_l.stl"/>
+                <mesh filename="package://motoman_gp50_support/meshes/gp50/collision/link_2_l.stl"/>
             </geometry>
         </collision>
@@ -49,5 +49,5 @@
         <visual>
             <geometry>
-                <mesh filename="package://motoman_gp50_support/meshes/visual/link_3_u.stl"/>
+                <mesh filename="package://motoman_gp50_support/meshes/gp50/visual/link_3_u.stl"/>
             </geometry>
             <material name="yaskawa_blue"/>
@@ -55,5 +55,5 @@
         <collision>
             <geometry>
-                <mesh filename="package://motoman_gp50_support/meshes/collision/link_3_u.stl"/>
+                <mesh filename="package://motoman_gp50_support/meshes/gp50/collision/link_3_u.stl"/>
             </geometry>
         </collision>
@@ -62,5 +62,5 @@
         <visual>
             <geometry>
-                <mesh filename="package://motoman_gp50_support/meshes/visual/link_4_r.stl"/>
+                <mesh filename="package://motoman_gp50_support/meshes/gp50/visual/link_4_r.stl"/>
             </geometry>
             <material name="yaskawa_blue"/>
@@ -68,5 +68,5 @@
         <collision>
             <geometry>
-                <mesh filename="package://motoman_gp50_support/meshes/collision/link_4_r.stl"/>
+                <mesh filename="package://motoman_gp50_support/meshes/gp50/collision/link_4_r.stl"/>
             </geometry>
         </collision>
@@ -75,5 +75,5 @@
         <visual>
             <geometry>
-                <mesh filename="package://motoman_gp50_support/meshes/visual/link_5_b.stl"/>
+                <mesh filename="package://motoman_gp50_support/meshes/gp50/visual/link_5_b.stl"/>
             </geometry>
             <material name="yaskawa_blue"/>
@@ -81,5 +81,5 @@
         <collision>
             <geometry>
-                <mesh filename="package://motoman_gp50_support/meshes/collision/link_5_b.stl"/>
+                <mesh filename="package://motoman_gp50_support/meshes/gp50/collision/link_5_b.stl"/>
             </geometry>
         </collision>
@@ -88,5 +88,5 @@
         <visual>
             <geometry>
-                <mesh filename="package://motoman_gp50_support/meshes/visual/link_6_t.stl"/>
+                <mesh filename="package://motoman_gp50_support/meshes/gp50/visual/link_6_t.stl"/>
             </geometry>
             <material name="yaskawa_blue"/>
@@ -94,5 +94,5 @@
         <collision>
             <geometry>
-                <mesh filename="package://motoman_gp50_support/meshes/collision/link_6_t.stl"/>
+                <mesh filename="package://motoman_gp50_support/meshes/gp50/collision/link_6_t.stl"/>
             </geometry>
         </collision>

Commit message: gp50: translate in one dimension only.
So move X translation to link_5 (and update meshes accordingly).

File: motoman_gp50_support/urdf/gp50_macro.xacro (robot description, xacro)
@@ -125,5 +125,5 @@
         <parent link="${prefix}link_3_u"/>
         <child link="${prefix}link_4_r"/>
-        <origin xyz="1.025 0 0.210" rpy="0 0 0" />
+        <origin xyz="0 0 0.210" rpy="0 0 0" />
         <axis xyz="-1 0 0" />
         <limit lower="${radians(-360)}" upper="${radians(360)}" effort="926" velocity="${radians(250)}"/>
@@ -132,5 +132,5 @@
         <parent link="${prefix}link_4_r"/>
         <child link="${prefix}link_5_b"/>
-        <origin xyz="0 0 0" rpy="0 0 0" />
+        <origin xyz="1.025 0 0" rpy="0 0 0" />
         <axis xyz="0 -1 0" />
         <limit lower="${radians(-125)}" upper="${radians(125)}" effort="794" velocity="${radians(250)}"/>
