Commit message: hc20: remove stray 'pi'.
Probably copy-pasted by accident.

File: motoman_hc20_support/urdf/hc20_macro.xacro (robot description, xacro)
@@ -86,5 +86,5 @@
     </link>
     <link name="${prefix}link_6_t">
-      <visual>pi
+      <visual>
         <geometry>
           <mesh filename="package://motoman_hc20_support/meshes/hc20/visual/link_6_t.stl"/>

Commit message: Updated model color
Updated model color

File: motoman_hc20_support/urdf/hc20_macro.xacro (robot description, xacro)
@@ -3,6 +3,6 @@
   <xacro:macro name="motoman_hc20" params="prefix">
     <!-- Properties -->
-    <material name="yaskawa_blue">
-      <color rgba="0.12941 0.14902 0.74902 1" />
+    <material name="yaskawa_white">
+      <color rgba="0.99 0.99 0.99 1" />
     </material>
     <!-- link list -->
@@ -12,5 +12,5 @@
           <mesh filename="package://motoman_hc20_support/meshes/hc20/visual/base_link.stl"/>
         </geometry>
-        <material name="yaskawa_blue"/>
+        <material name="yaskawa_white"/>
       </visual>
       <collision>
@@ -25,5 +25,5 @@
           <mesh filename="package://motoman_hc20_support/meshes/hc20/visual/link_1_s.stl"/>
         </geometry>
-        <material name="yaskawa_blue"/>
+        <material name="yaskawa_white"/>
       </visual>
       <collision>
@@ -38,5 +38,5 @@
           <mesh filename="package://motoman_hc20_support/meshes/hc20/visual/link_2_l.stl"/>
         </geometry>
-        <material name="yaskawa_blue"/>
+        <material name="yaskawa_white"/>
       </visual>
       <collision>
@@ -51,5 +51,5 @@
           <mesh filename="package://motoman_hc20_support/meshes/hc20/visual/link_3_u.stl"/>
         </geometry>
-        <material name="yaskawa_blue"/>
+        <material name="yaskawa_white"/>
       </visual>
       <collision>
@@ -64,5 +64,5 @@
           <mesh filename="package://motoman_hc20_support/meshes/hc20/visual/link_4_r.stl"/>
         </geometry>
-        <material name="yaskawa_blue"/>
+        <material name="yaskawa_white"/>
       </visual>
       <collision>
@@ -77,5 +77,5 @@
           <mesh filename="package://motoman_hc20_support/meshes/hc20/visual/link_5_b.stl"/>
         </geometry>
-        <material name="yaskawa_blue"/>
+        <material name="yaskawa_white"/>
       </visual>
       <collision>
@@ -90,5 +90,5 @@
           <mesh filename="package://motoman_hc20_support/meshes/hc20/visual/link_6_t.stl"/>
         </geometry>
-        <material name="yaskawa_blue"/>
+        <material name="yaskawa_white"/>
       </visual>
       <collision>
