Commit message: HC20DTP and HC30PL Update
The HC20 package was updated with the HC20DTP and HC30PL variant. HC20 visual meshes were changed from .stl to .dae format to improve rendering.

File: motoman_hc20_support/urdf/hc20dtp_macro.xacro (robot description, xacro)
@@ -1,5 +1,5 @@
 <?xml version="1.0" ?>
 <robot xmlns:xacro="http://ros.org/wiki/xacro">
-  <xacro:macro name="motoman_hc20" params="prefix">
+  <xacro:macro name="motoman_hc20dtp" params="prefix">
     <xacro:include filename="$(find motoman_resources)/urdf/common_materials.xacro"/>
     <!-- link list -->
@@ -72,5 +72,5 @@
       <visual>
         <geometry>
-          <mesh filename="package://motoman_hc20_support/meshes/hc20/visual/link_5_b.dae"/>
+          <mesh filename="package://motoman_hc20_support/meshes/hc20dtp/visual/link_5_b.dae"/>
         </geometry>
         <xacro:material_yaskawa_white/>
@@ -78,5 +78,5 @@
       <collision>
         <geometry>
-          <mesh filename="package://motoman_hc20_support/meshes/hc20/collision/link_5_b.stl"/>
+          <mesh filename="package://motoman_hc20_support/meshes/hc20dtp/collision/link_5_b.stl"/>
         </geometry>
       </collision>
@@ -85,5 +85,5 @@
       <visual>
         <geometry>
-          <mesh filename="package://motoman_hc20_support/meshes/hc20/visual/link_6_t.dae"/>
+          <mesh filename="package://motoman_hc20_support/meshes/hc20dtp/visual/link_6_t.dae"/>
         </geometry>
         <xacro:material_yaskawa_white/>
@@ -91,5 +91,5 @@
       <collision>
         <geometry>
-          <mesh filename="package://motoman_hc20_support/meshes/hc20/collision/link_6_t.stl"/>
+          <mesh filename="package://motoman_hc20_support/meshes/hc20dtp/collision/link_6_t.stl"/>
         </geometry>
       </collision>
@@ -103,5 +103,5 @@
       <origin xyz="0 0 0.380" rpy="0 0 0" />
       <axis xyz="0 0 1" />
-      <limit lower="${radians(-180)}" upper="${radians(180)}" effort="917.28" velocity="${radians(80)}"/>
+      <limit lower="${radians(-210)}" upper="${radians(210)}" effort="917.28" velocity="${radians(80)}"/>
     </joint>
     <joint name="${prefix}joint_2_l" type="revolute">

File: motoman_hc20_support/urdf/hc30pl_macro.xacro (robot description, xacro)
@@ -1,5 +1,5 @@
 <?xml version="1.0" ?>
 <robot xmlns:xacro="http://ros.org/wiki/xacro">
-  <xacro:macro name="motoman_hc20" params="prefix">
+  <xacro:macro name="motoman_hc30pl" params="prefix">
     <xacro:include filename="$(find motoman_resources)/urdf/common_materials.xacro"/>
     <!-- link list -->
@@ -72,12 +72,14 @@
       <visual>
         <geometry>
-          <mesh filename="package://motoman_hc20_support/meshes/hc20/visual/link_5_b.dae"/>
+          <mesh filename="package://motoman_hc20_support/meshes/hc20dtp/visual/link_5_b.dae"/>
         </geometry>
+		<origin rpy="0 1.57075 0"/>
         <xacro:material_yaskawa_white/>
       </visual>
       <collision>
         <geometry>
-          <mesh filename="package://motoman_hc20_support/meshes/hc20/collision/link_5_b.stl"/>
+          <mesh filename="package://motoman_hc20_support/meshes/hc20dtp/collision/link_5_b.stl"/>
         </geometry>
+		<origin rpy="0 1.57075 0"/>
       </collision>
     </link>
@@ -85,12 +87,14 @@
       <visual>
         <geometry>
-          <mesh filename="package://motoman_hc20_support/meshes/hc20/visual/link_6_t.dae"/>
+          <mesh filename="package://motoman_hc20_support/meshes/hc20dtp/visual/link_6_t.dae"/>
         </geometry>
+		<origin rpy="0 1.57075 0"/>
         <xacro:material_yaskawa_white/>
       </visual>
       <collision>
         <geometry>
-          <mesh filename="package://motoman_hc20_support/meshes/hc20/collision/link_6_t.stl"/>
+          <mesh filename="package://motoman_hc20_support/meshes/hc20dtp/collision/link_6_t.stl"/>
         </geometry>
+		<origin rpy="0 1.57075 0"/>
       </collision>
     </link>
@@ -103,5 +107,5 @@
       <origin xyz="0 0 0.380" rpy="0 0 0" />
       <axis xyz="0 0 1" />
-      <limit lower="${radians(-180)}" upper="${radians(180)}" effort="917.28" velocity="${radians(80)}"/>
+      <limit lower="${radians(-210)}" upper="${radians(210)}" effort="917.28" velocity="${radians(80)}"/>
     </joint>
     <joint name="${prefix}joint_2_l" type="revolute">
@@ -110,5 +114,5 @@
       <origin xyz="0 0 0" rpy="0 0 0" />
       <axis xyz="0 1 0" />
-      <limit lower="${radians(-180)}" upper="${radians(180)}" effort="1223.04" velocity="${radians(80)}"/>
+      <limit lower="${radians(-154)}" upper="${radians(180)}" effort="1223.04" velocity="${radians(80)}"/>
     </joint>
     <joint name="${prefix}joint_3_u" type="revolute">
@@ -124,5 +128,5 @@
       <origin xyz="0.880 0 0" rpy="0 0 0" />
       <axis xyz="-1 0 0" />
-      <limit lower="${radians(-210)}" upper="${radians(210)}" effort="368.48" velocity="${radians(130)}"/>
+      <limit lower="${radians(-15)}" upper="${radians(15)}" effort="368.48" velocity="${radians(112)}"/>
     </joint>
     <joint name="${prefix}joint_5_b" type="revolute">
@@ -131,5 +135,5 @@
       <origin xyz="0 0 0" rpy="0 0 0" />
       <axis xyz="0 -1 0" />
-      <limit lower="${radians(-180)}" upper="${radians(180)}" effort="141.12" velocity="${radians(180)}"/>
+      <limit lower="${radians(-15)}" upper="${radians(15)}" effort="141.12" velocity="${radians(132)}"/>
     </joint>
     <joint name="${prefix}joint_6_t" type="revolute">
@@ -137,9 +141,9 @@
       <child link="${prefix}link_6_t"/>
       <origin xyz="0 0 0" rpy="0 0 0" />
-      <axis xyz="-1 0 0" />
+      <axis xyz="0 0 1" />
       <limit lower="${radians(-210)}" upper="${radians(210)}" effort="141.12" velocity="${radians(180)}"/>
     </joint>
     <joint name="${prefix}joint_6_t-tool0" type="fixed">
-      <origin xyz="0.200 0 0" rpy="${radians(180)} ${radians(-90)} 0"/>
+      <origin xyz="0 0 -0.200" rpy="0 ${radians(180)} ${radians(180)}"/>
       <parent link="${prefix}link_6_t"/>
       <child link="${prefix}tool0"/>
