Commit message: Updated URDF to pull controller-specific joint velocities

File: motoman_es_support/urdf/es165rdii.xacro (robot description, xacro)
@@ -2,4 +2,5 @@
 <robot name="motoman_es165rdii" xmlns:xacro="http://ros.org/wiki/xacro">
   <xacro:include filename="$(find motoman_es_support)/urdf/es165rdii_macro.xacro"/>
-  <xacro:motoman_es165rdii prefix=""/>
+  <xacro:arg name="joint_velocities_file" default=""/>
+  <xacro:motoman_es165rdii prefix="" joint_velocities_file="$(arg joint_velocities_file)"/>
 </robot>

File: motoman_es_support/urdf/es165rdii_macro.xacro (robot description, xacro)
@@ -1,5 +1,5 @@
 <?xml version="1.0"?>
 <robot xmlns:xacro="http://ros.org/wiki/xacro">
-  <xacro:macro name="motoman_es165rdii" params="prefix">
+  <xacro:macro name="motoman_es165rdii" params="prefix joint_velocities_file">
     <!-- link list -->
     <link name="${prefix}base_link">
@@ -163,4 +163,5 @@
     <!-- end of link list -->
     <!-- joint list -->
+    <xacro:property name="velocities" value="${load_yaml(joint_velocities_file)}" />
     <joint name="${prefix}joint_1_s" type="revolute">
       <origin xyz="0 0 0.450" rpy="0 0 0"/>
@@ -168,5 +169,5 @@
       <child link="${prefix}link_s"/>
       <axis xyz="0 0 1"/>
-      <limit lower="${radians(-180)}" upper="${radians(180)}" effort="0" velocity="${radians(105)}"/>
+      <limit lower="${radians(-180)}" upper="${radians(180)}" effort="0" velocity="${radians(velocities['joint_1_s'])}"/>
     </joint>
     <joint name="${prefix}joint_2_l" type="revolute">
@@ -175,5 +176,5 @@
       <child link="${prefix}link_l"/>
       <axis xyz="0 1 0"/>
-      <limit lower="${radians(-130)}" upper="${radians(80)}" effort="0" velocity="${radians(105)}"/>
+      <limit lower="${radians(-130)}" upper="${radians(80)}" effort="0" velocity="${radians(velocities['joint_2_l'])}"/>
     </joint>
     <joint name="${prefix}joint_3_u" type="revolute">
@@ -182,5 +183,5 @@
       <child link="${prefix}link_u"/>
       <axis xyz="0 -1 0"/>
-      <limit lower="${radians(-112)}" upper="${radians(208)}" effort="0" velocity="${radians(105)}"/>
+      <limit lower="${radians(-112)}" upper="${radians(208)}" effort="0" velocity="${radians(velocities['joint_3_u'])}"/>
     </joint>
     <joint name="${prefix}joint_4_r" type="revolute">
@@ -189,5 +190,5 @@
       <child link="${prefix}link_r"/>
       <axis xyz="0 0 1"/>
-      <limit lower="${radians(-360)}" upper="${radians(360)}" effort="0" velocity="${radians(175)}"/>
+      <limit lower="${radians(-360)}" upper="${radians(360)}" effort="0" velocity="${radians(velocities['joint_4_r'])}"/>
     </joint>
     <joint name="${prefix}joint_5_b" type="revolute">
@@ -196,5 +197,5 @@
       <child link="${prefix}link_b"/>
       <axis xyz="0 -1 0"/>
-      <limit lower="${radians(-130)}" upper="${radians(130)}" effort="0" velocity="${radians(150)}"/>
+      <limit lower="${radians(-130)}" upper="${radians(130)}" effort="0" velocity="${radians(velocities['joint_5_b'])}"/>
     </joint>
     <joint name="${prefix}joint_6_t" type="revolute">
@@ -203,5 +204,5 @@
       <child link="${prefix}link_t"/>
       <axis xyz="0 0 1"/>
-      <limit lower="${radians(-360)}" upper="${radians(360)}" effort="0" velocity="${radians(240)}"/>
+      <limit lower="${radians(-360)}" upper="${radians(360)}" effort="0" velocity="${radians(velocities['joint_6_t'])}"/>
     </joint>
     <joint name="${prefix}joint_t-tool0" type="fixed">
