Commit message: Renamed from es200rn_120 to es200_120

File: motoman_es_support/urdf/es200_120_macro.xacro (robot description, xacro)
@@ -1,5 +1,5 @@
 <?xml version="1.0"?>
 <robot xmlns:xacro="http://ros.org/wiki/xacro">
-  <xacro:macro name="motoman_es200rn_120" params="prefix">
+  <xacro:macro name="motoman_es200_120" params="prefix">
     <!-- link list -->
     <link name="${prefix}base_link">
@@ -58,12 +58,12 @@
         <origin xyz="0 0 0" rpy="0 0 0"/>
         <geometry>
-          <mesh filename="package://motoman_es_support/meshes/es200rn_120/visual/link_u.stl"/>
-        </geometry>
-        <material name="blue"/>
-      </visual>
-      <collision>
-        <origin xyz="0 0 0" rpy="0 0 0"/>
-        <geometry>
-          <mesh filename="package://motoman_es_support/meshes/es200rn_120/collision/link_u.stl"/>
+          <mesh filename="package://motoman_es_support/meshes/es200_120/visual/link_u.stl"/>
+        </geometry>
+        <material name="blue"/>
+      </visual>
+      <collision>
+        <origin xyz="0 0 0" rpy="0 0 0"/>
+        <geometry>
+          <mesh filename="package://motoman_es_support/meshes/es200_120/collision/link_u.stl"/>
         </geometry>
         <material name="yellow"/>
@@ -74,12 +74,12 @@
         <origin xyz="0 0 0" rpy="0 0 0"/>
         <geometry>
-          <mesh filename="package://motoman_es_support/meshes/es200rn_120/visual/link_r.stl"/>
-        </geometry>
-        <material name="blue"/>
-      </visual>
-      <collision>
-        <origin xyz="0 0 0" rpy="0 0 0"/>
-        <geometry>
-          <mesh filename="package://motoman_es_support/meshes/es200rn_120/collision/link_r.stl"/>
+          <mesh filename="package://motoman_es_support/meshes/es200_120/visual/link_r.stl"/>
+        </geometry>
+        <material name="blue"/>
+      </visual>
+      <collision>
+        <origin xyz="0 0 0" rpy="0 0 0"/>
+        <geometry>
+          <mesh filename="package://motoman_es_support/meshes/es200_120/collision/link_r.stl"/>
         </geometry>
         <material name="yellow"/>
