Commit message: Update MS210 Support Package
Changes
- Add Joint Effort Limits
- Update STL mesh origins for S,R,T links
- Update joint origins limit changes in orientation to 1-DOF per joint.

File: motoman_ms210_support/urdf/ms210_macro.xacro (robot description, xacro)
@@ -142,10 +142,10 @@
     <parent link="${prefix}base_link" />
     <child  link="${prefix}link_s" />
-    <origin xyz="0 0 0.342" rpy="0 0 0" />
+    <origin xyz="0 0 0.650" rpy="0 0 0" />
     <axis   xyz="0 0 1" />
     <limit
       lower="-3.1416"
       upper="3.1416"
-      effort="0"
+      effort="6276.26"
       velocity="2.09440" />
   </joint>
@@ -153,10 +153,10 @@
     <parent link="${prefix}link_s" />
     <child link="${prefix}link_l" />
-    <origin xyz="0.325 0 0.333" rpy="0 0 0" />
+    <origin xyz="0.325 0 0" rpy="0 0 0" />
     <axis xyz="0 1 0" />
     <limit
       lower="-1.0472"
       upper="1.3265"
-      effort="0"
+      effort="9806.65"
       velocity="1.69297" />
   </joint>
@@ -164,10 +164,10 @@
     <parent link="${prefix}link_l" />
     <child link="${prefix}link_u" />
-    <origin xyz="0 0 1.15" rpy="0 0 0" />
+    <origin xyz="0 0 1.150" rpy="0 0 0" />
     <axis xyz="0 1 0" />
     <limit
       lower="-2.5656"
       upper="1.5708"
-      effort="0"
+      effort="9806.65"
       velocity="2.00713" />
   </joint>
@@ -175,25 +175,25 @@
     <parent link="${prefix}link_u" />
     <child link="${prefix}link_r" />
-    <origin xyz="0.9735 0 0.3" rpy="0 0 0" />
+    <origin xyz="0 0 0.300" rpy="0 0 0" />
     <axis xyz="1 0 0" />
     <limit
       lower="-3.6652"
       upper="3.6652"
-      effort="0"
+      effort="2451.66"
       velocity="2.53073" />
   </joint>
   <joint name="${prefix}joint_b" type="revolute">
-    <origin xyz="0.2515 0 0" rpy="0 0 0" />
     <parent link="${prefix}link_r" />
     <child link="${prefix}link_b" />
+    <origin xyz="1.225 0 0" rpy="0 0 0" />
     <axis xyz="0 1 0" />
     <limit
       lower="-2.1816"
       upper="2.1816"
-      effort="0"
+      effort="2745.86"
       velocity="2.53073" />
   </joint>
   <joint name="${prefix}joint_t" type="revolute">
-    <origin xyz="0.21695 0 0" rpy="0 0 0" />
+    <origin xyz="0.250 0 0" rpy="0 0 0" />
     <parent link="${prefix}link_b" />
     <child link="${prefix}link_t" />
@@ -202,13 +202,20 @@
       lower="-3.6652"
       upper="3.6652"
-      effort="0"
+      effort="1800.5"
       velocity="3.83972" />
   </joint>
   <joint name="${prefix}joint_t-tool0" type="fixed">
-    <origin xyz="0.035 0 0 " rpy="0 0 0 "/><!-- ATTN USERS! MODIFY THIS LINE TO MATCH YOUR MOUNTED TOOLING -->
+    <origin xyz="0 0 0 " rpy="3.1415926 -1.570796 0"/>
     <parent link="${prefix}link_t"/>
     <child link="${prefix}tool0"/>
   </joint>
   <!-- end of joint list -->
+  <!-- ROS base_link to Robot Manufacturer World Coordinates transform -->
+  <link name="${prefix}base" />
+  <joint name="${prefix}base_link-base" type="fixed">
+    <origin xyz="0 0 0.650" rpy="0 0 0"/>
+    <parent link="${prefix}base_link"/>
+    <child link="${prefix}base"/>
+  </joint>
   </xacro:macro>
 </robot>

Commit message: Reorient URBT axis in MS210 Support
Following physical robot testing (state_visualize only), identified that
URBT axis' were inverted. Correcting this here by setting live axis to
`-1`

File: motoman_ms210_support/urdf/ms210_macro.xacro (robot description, xacro)
@@ -133,5 +133,5 @@
     <child link="${prefix}link_u" />
     <origin xyz="0 0 1.150" rpy="0 0 0" />
-    <axis xyz="0 1 0" />
+    <axis xyz="0 -1 0" />
     <limit lower="${radians(-147)}" upper="${radians(90)}" effort="9806.65" velocity="${radians(115)}" />
   </joint>
@@ -140,5 +140,5 @@
     <child link="${prefix}link_r" />
     <origin xyz="0 0 0.300" rpy="0 0 0" />
-    <axis xyz="1 0 0" />
+    <axis xyz="-1 0 0" />
     <limit lower="${radians(-210)}" upper="${radians(210)}" effort="2451.66" velocity="${radians(145)}" />
   </joint>
@@ -147,5 +147,5 @@
     <child link="${prefix}link_b" />
     <origin xyz="1.225 0 0" rpy="0 0 0" />
-    <axis xyz="0 1 0" />
+    <axis xyz="0 -1 0" />
     <limit lower="${radians(-125)}" upper="${radians(125)}" effort="2745.86" velocity="${radians(145)}" />
   </joint>
@@ -154,5 +154,5 @@
     <parent link="${prefix}link_b" />
     <child link="${prefix}link_t" />
-    <axis xyz="1 0 0" />
+    <axis xyz="-1 0 0" />
     <limit lower="${radians(-210)}" upper="${radians(210)}" effort="1800.5" velocity="${radians(220)}" />
   </joint>

Commit message: Standardize Joint & Link Names

File: motoman_ms210_support/urdf/ms210_macro.xacro (robot description, xacro)
@@ -22,5 +22,5 @@
     </collision>
   </link>
-  <link  name="${prefix}link_s">
+  <link  name="${prefix}link_1_s">
     <visual>
       <origin xyz="0 0 0" rpy="0 0 0" />
@@ -37,5 +37,5 @@
     </collision>
   </link>
-  <link  name="${prefix}link_l">
+  <link  name="${prefix}link_2_l">
     <visual>
       <origin xyz="0 0 0" rpy="0 0 0" />
@@ -52,5 +52,5 @@
     </collision>
   </link>
-  <link  name="${prefix}link_u">
+  <link  name="${prefix}link_3_u">
     <visual>
       <origin xyz="0 0 0" rpy="0 0 0" />
@@ -67,5 +67,5 @@
     </collision>
   </link>
-  <link  name="${prefix}link_r">
+  <link  name="${prefix}link_4_r">
     <visual>
       <origin xyz="0 0 0" rpy="0 0 0" />
@@ -82,5 +82,5 @@
     </collision>
   </link>
-  <link  name="${prefix}link_b">
+  <link  name="${prefix}link_5_b">
     <visual>
       <origin xyz="0 0 0" rpy="0 0 0" />
@@ -97,5 +97,5 @@
     </collision>
   </link>
-  <link  name="${prefix}link_t">
+  <link  name="${prefix}link_6_t">
     <visual>
       <origin xyz="0 0 0" rpy="0 0 0" />
@@ -115,50 +115,50 @@
   <!-- end of link list -->
   <!-- joint list -->
-  <joint name="${prefix}joint_s" type="revolute">
+  <joint name="${prefix}joint_1_s" type="revolute">
     <parent link="${prefix}base_link" />
-    <child  link="${prefix}link_s" />
+    <child  link="${prefix}link_1_s" />
     <origin xyz="0 0 0.650" rpy="0 0 0" />
     <axis   xyz="0 0 1" />
     <limit lower="${radians(-180)}" upper="${radians(180)}" effort="6276.26" velocity="${radians(120)}" />
   </joint>
-  <joint name="${prefix}joint_l" type="revolute">
-    <parent link="${prefix}link_s" />
-    <child link="${prefix}link_l" />
+  <joint name="${prefix}joint_2_l" type="revolute">
+    <parent link="${prefix}link_1_s" />
+    <child link="${prefix}link_2_l" />
     <origin xyz="0.325 0 0" rpy="0 0 0" />
     <axis xyz="0 1 0" />
     <limit lower="${radians(-60)}" upper="${radians(76)}" effort="9806.65" velocity="${radians(97)}" />
   </joint>
-  <joint name="${prefix}joint_u" type="revolute">
-    <parent link="${prefix}link_l" />
-    <child link="${prefix}link_u" />
+  <joint name="${prefix}joint_3_u" type="revolute">
+    <parent link="${prefix}link_2_l" />
+    <child link="${prefix}link_3_u" />
     <origin xyz="0 0 1.150" rpy="0 0 0" />
     <axis xyz="0 -1 0" />
     <limit lower="${radians(-147)}" upper="${radians(90)}" effort="9806.65" velocity="${radians(115)}" />
   </joint>
-  <joint name="${prefix}joint_r" type="revolute">
-    <parent link="${prefix}link_u" />
-    <child link="${prefix}link_r" />
+  <joint name="${prefix}joint_4_r" type="revolute">
+    <parent link="${prefix}link_3_u" />
+    <child link="${prefix}link_4_r" />
     <origin xyz="0 0 0.300" rpy="0 0 0" />
     <axis xyz="-1 0 0" />
     <limit lower="${radians(-210)}" upper="${radians(210)}" effort="2451.66" velocity="${radians(145)}" />
   </joint>
-  <joint name="${prefix}joint_b" type="revolute">
-    <parent link="${prefix}link_r" />
-    <child link="${prefix}link_b" />
+  <joint name="${prefix}joint_5_b" type="revolute">
+    <parent link="${prefix}link_4_r" />
+    <child link="${prefix}link_5_b" />
     <origin xyz="1.225 0 0" rpy="0 0 0" />
     <axis xyz="0 -1 0" />
     <limit lower="${radians(-125)}" upper="${radians(125)}" effort="2745.86" velocity="${radians(145)}" />
   </joint>
-  <joint name="${prefix}joint_t" type="revolute">
+  <joint name="${prefix}joint_6_t" type="revolute">
+    <parent link="${prefix}link_5_b" />
+    <child link="${prefix}link_6_t" />
     <origin xyz="0.250 0 0" rpy="0 0 0" />
-    <parent link="${prefix}link_b" />
-    <child link="${prefix}link_t" />
     <axis xyz="-1 0 0" />
     <limit lower="${radians(-210)}" upper="${radians(210)}" effort="1800.5" velocity="${radians(220)}" />
   </joint>
-  <joint name="${prefix}joint_t-tool0" type="fixed">
+  <joint name="${prefix}joint_6_t-tool0" type="fixed">
+    <parent link="${prefix}link_6_t"/>
+    <child link="${prefix}tool0"/>
     <origin xyz="0 0 0 " rpy="${radians(180)} ${radians(-90)} 0"/>
-    <parent link="${prefix}link_t"/>
-    <child link="${prefix}tool0"/>
   </joint>
   <!-- end of joint list -->

Commit message: ms210: whitespace and formatting.

File: motoman_ms210_support/urdf/ms210_macro.xacro (robot description, xacro)
@@ -117,7 +117,7 @@
   <joint name="${prefix}joint_1_s" type="revolute">
     <parent link="${prefix}base_link" />
-    <child  link="${prefix}link_1_s" />
+    <child link="${prefix}link_1_s" />
     <origin xyz="0 0 0.650" rpy="0 0 0" />
-    <axis   xyz="0 0 1" />
+    <axis xyz="0 0 1" />
     <limit lower="${radians(-180)}" upper="${radians(180)}" effort="6276.26" velocity="${radians(120)}" />
   </joint>

Commit message: ms210: 'special' links go at the end of the file.
So move 'tool0' to the end.

File: motoman_ms210_support/urdf/ms210_macro.xacro (robot description, xacro)
@@ -112,5 +112,4 @@
     </collision>
   </link>
-  <link name="${prefix}tool0"/>
   <!-- end of link list -->
   <!-- joint list -->
@@ -157,9 +156,4 @@
     <limit lower="${radians(-210)}" upper="${radians(210)}" effort="1800.5" velocity="${radians(220)}" />
   </joint>
-  <joint name="${prefix}joint_6_t-tool0" type="fixed">
-    <parent link="${prefix}link_6_t"/>
-    <child link="${prefix}tool0"/>
-    <origin xyz="0 0 0 " rpy="${radians(180)} ${radians(-90)} 0"/>
-  </joint>
   <!-- end of joint list -->
   <!-- ROS base_link to Robot Manufacturer World Coordinates transform -->
@@ -170,4 +164,11 @@
     <child link="${prefix}base"/>
   </joint>
-  </xacro:macro>
+    <!-- ROS-Industrial 'tool0' frame: all-zeros tool frame -->
+  <link name="${prefix}tool0"/>
+  <joint name="${prefix}joint_6_t-tool0" type="fixed">
+    <parent link="${prefix}link_6_t"/>
+    <child link="${prefix}tool0"/>
+    <origin xyz="0 0 0 " rpy="${radians(180)} ${radians(-90)} 0"/>
+  </joint>
+</xacro:macro>
 </robot>
