Commit message: Updated URDFs to have proper flange and tool0.
Did not update any of the S series (sda, sia)

File: motoman_gp12_support/urdf/gp12_macro.xacro (robot description, xacro)
@@ -98,5 +98,4 @@
         </collision>
     </link>
-    <link name="${prefix}tool0"/>
     <!-- end of link list -->
     <!-- joint list -->
@@ -143,9 +142,4 @@
         <limit lower="-7.9412" upper="7.9412" effort="33.30" velocity="12.2143"/>
     </joint>
-    <joint name="${prefix}joint_6_t-tool0" type="fixed">
-        <origin xyz="0.100 0 0" rpy="3.1415926 -1.570796 0"/>
-        <parent link="${prefix}link_6_t"/>
-        <child link="${prefix}tool0"/>
-    </joint>
     <!-- end of joint list -->
     <!-- ROS base_link to Robot Manufacturer World Coordinates transform -->
@@ -156,4 +150,18 @@
         <child link="${prefix}base"/>
     </joint>
+    <!-- ROS-Industrial 'flange' frame: attachment point for EEF models -->
+    <link name="${prefix}flange" />
+    <joint name="${prefix}joint_6_t-flange" type="fixed">
+        <origin xyz="0.100 0 0" rpy="0 0 0" />
+        <parent link="${prefix}link_6_t" />
+        <child link="${prefix}flange" />
+    </joint>
+    <!-- ROS-Industrial 'tool0' frame: all-zeros tool frame -->
+    <link name="${prefix}tool0" />
+    <joint name="${prefix}flange-tool0" type="fixed">
+        <origin xyz="0 0 0" rpy="${pi} ${-pi/2.0} 0" />
+        <parent link="${prefix}flange" />
+        <child link="${prefix}tool0" />
+    </joint>
     </xacro:macro>
 </robot>

File: motoman_gp180_support/urdf/gp180_120_macro.xacro (robot description, xacro)
@@ -98,5 +98,4 @@
         </collision>
     </link>
-    <link name="${prefix}tool0"/>
     <!-- end of link list -->
     <!-- joint list -->
@@ -143,9 +142,4 @@
         <limit lower="${radians(-360)}" upper="${radians(360)}" effort="926.73" velocity="${radians(265)}"/>
     </joint>
-    <joint name="${prefix}joint_6_t-tool0" type="fixed">
-        <origin xyz="0 0 0" rpy="${radians(180)} ${radians(-90)} 0"/>
-        <parent link="${prefix}link_6_t"/>
-        <child link="${prefix}tool0"/>
-    </joint>
     <!-- end of joint list -->
     <!-- ROS base_link to Robot Manufacturer World Coordinates transform -->
@@ -156,4 +150,18 @@
         <child link="${prefix}base"/>
     </joint>
+    <!-- ROS-Industrial 'flange' frame: attachment point for EEF models -->
+    <link name="${prefix}flange" />
+    <joint name="${prefix}joint_6_t-flange" type="fixed">
+        <origin xyz="0.0 0 0" rpy="0 0 0" />
+        <parent link="${prefix}link_6_t" />
+        <child link="${prefix}flange" />
+    </joint>
+    <!-- ROS-Industrial 'tool0' frame: all-zeros tool frame -->
+    <link name="${prefix}tool0" />
+    <joint name="${prefix}flange-tool0" type="fixed">
+        <origin xyz="0 0 0" rpy="${pi} ${-pi/2.0} 0" />
+        <parent link="${prefix}flange" />
+        <child link="${prefix}tool0" />
+    </joint>
 </xacro:macro>
 </robot>

File: motoman_gp25_support/urdf/gp25_macro.xacro (robot description, xacro)
@@ -98,5 +98,4 @@
         </collision>
     </link>
-    <link name="${prefix}tool0"/>
     <!-- end of link list -->
     <!-- joint list -->
@@ -143,9 +142,4 @@
         <limit lower="${radians(-455)}" upper="${radians(455)}" effort="50.31" velocity="${radians(885)}"/>
     </joint>
-    <joint name="${prefix}joint_6_t-tool0" type="fixed">
-        <origin xyz="0.100 0 0" rpy="3.1415926 -1.570796 0"/>
-        <parent link="${prefix}link_6_t"/>
-        <child link="${prefix}tool0"/>
-    </joint>
     <!-- end of joint list -->
     <!-- ROS base_link to Robot Manufacturer World Coordinates transform -->
@@ -156,4 +150,18 @@
         <child link="${prefix}base"/>
     </joint>
+    <!-- ROS-Industrial 'flange' frame: attachment point for EEF models -->
+    <link name="${prefix}flange" />
+    <joint name="${prefix}joint_6_t-flange" type="fixed">
+        <origin xyz="0.10 0 0" rpy="0 0 0" />
+        <parent link="${prefix}link_6_t" />
+        <child link="${prefix}flange" />
+    </joint>
+    <!-- ROS-Industrial 'tool0' frame: all-zeros tool frame -->
+    <link name="${prefix}tool0" />
+    <joint name="${prefix}flange-tool0" type="fixed">
+        <origin xyz="0 0 0" rpy="${pi} ${-pi/2.0} 0" />
+        <parent link="${prefix}flange" />
+        <child link="${prefix}tool0" />
+    </joint>
     </xacro:macro>
 </robot>

File: motoman_gp50_support/urdf/gp50_macro.xacro (robot description, xacro)
@@ -98,5 +98,4 @@
         </collision>
     </link>
-    <link name="${prefix}tool0"/>
     <!-- end of link list -->
     <!-- joint list -->
@@ -143,9 +142,4 @@
         <limit lower="${radians(-360)}" upper="${radians(360)}" effort="375" velocity="${radians(360)}"/>
     </joint>
-    <joint name="${prefix}joint_6_t-tool0" type="fixed">
-        <origin xyz="0.175 0 0" rpy="3.1415926 -1.570796 0"/>
-        <parent link="${prefix}link_6_t"/>
-        <child link="${prefix}tool0"/>
-    </joint>
     <!-- end of joint list -->
     <!-- ROS base_link to Robot Manufacturer World Coordinates transform -->
@@ -156,4 +150,18 @@
         <child link="${prefix}base"/>
     </joint>
+    <!-- ROS-Industrial 'flange' frame: attachment point for EEF models -->
+    <link name="${prefix}flange" />
+    <joint name="${prefix}joint_6_t-flange" type="fixed">
+      <origin xyz="0.175 0 0" rpy="0 0 0" />
+      <parent link="${prefix}link_6_t" />
+      <child link="${prefix}flange" />
+    </joint>
+    <!-- ROS-Industrial 'tool0' frame: all-zeros tool frame -->
+    <link name="${prefix}tool0" />
+    <joint name="${prefix}flange-tool0" type="fixed">
+      <origin xyz="0 0 0" rpy="${pi} ${-pi/2.0} 0" />
+      <parent link="${prefix}flange" />
+      <child link="${prefix}tool0" />
+    </joint>
   </xacro:macro>
 </robot>

File: motoman_gp7_support/urdf/gp7_macro.xacro (robot description, xacro)
@@ -98,5 +98,4 @@
         </collision>
     </link>
-    <link name="${prefix}tool0"/>
     <!-- end of link list -->
     <!-- joint list -->
@@ -143,9 +142,4 @@
         <limit lower="-6.2944" upper="6.2944" effort="22.54" velocity="17.4845"/>
     </joint>
-    <joint name="${prefix}joint_6_t-tool0" type="fixed">
-        <origin xyz="0.080 0 0" rpy="3.1415926 -1.570796 0"/>
-        <parent link="${prefix}link_6_t"/>
-        <child link="${prefix}tool0"/>
-    </joint>
     <!-- end of joint list -->
     <!-- ROS base_link to Robot Manufacturer World Coordinates transform -->
@@ -156,4 +150,18 @@
         <child link="${prefix}base"/>
     </joint>
+    <!-- ROS-Industrial 'flange' frame: attachment point for EEF models -->
+    <link name="${prefix}flange" />
+    <joint name="${prefix}joint_6_t-flange" type="fixed">
+        <origin xyz="0.080 0 0" rpy="0 0 0" />
+        <parent link="${prefix}link_6_t" />
+        <child link="${prefix}flange" />
+    </joint>
+    <!-- ROS-Industrial 'tool0' frame: all-zeros tool frame -->
+    <link name="${prefix}tool0" />
+    <joint name="${prefix}flange-tool0" type="fixed">
+        <origin xyz="0 0 0" rpy="${pi} ${-pi/2.0} 0" />
+        <parent link="${prefix}flange" />
+        <child link="${prefix}tool0" />
+    </joint>
     </xacro:macro>
 </robot>

File: motoman_gp88_support/urdf/gp88_macro.xacro (robot description, xacro)
@@ -150,10 +150,17 @@
       <child link="${prefix}base"/>
     </joint>
+    <!-- ROS-Industrial 'flange' frame: attachment point for EEF models -->
+    <link name="${prefix}flange" />
+    <joint name="${prefix}joint_6_t-flange" type="fixed">
+      <origin xyz="0.175 0 0" rpy="0 0 0" />
+      <parent link="${prefix}link_6_t" />
+      <child link="${prefix}flange" />
+    </joint>
     <!-- ROS-Industrial 'tool0' frame: all-zeros tool frame -->
-    <link name="${prefix}tool0"/>
-    <joint name="${prefix}joint_6_t-tool0" type="fixed">
-      <origin xyz="0.175 0 0" rpy="${radians(180)} ${radians(-90)} 0"/>
-      <parent link="${prefix}link_6_t"/>
-      <child link="${prefix}tool0"/>
+    <link name="${prefix}tool0" />
+    <joint name="${prefix}flange-tool0" type="fixed">
+      <origin xyz="0 0 0" rpy="${pi} ${-pi/2.0} 0" />
+      <parent link="${prefix}flange" />
+      <child link="${prefix}tool0" />
     </joint>
   </xacro:macro>

File: motoman_gp8_support/urdf/gp8_macro.xacro (robot description, xacro)
@@ -98,5 +98,4 @@
         </collision>
     </link>
-    <link name="${prefix}tool0"/>
     <!-- end of link list -->
     <!-- joint list -->
@@ -143,9 +142,4 @@
         <limit lower="-6.2944" upper="6.2944" effort="22.54" velocity="17.4845"/>
     </joint>
-    <joint name="${prefix}joint_6_t-tool0" type="fixed">
-        <origin xyz="0.080 0 0" rpy="3.1415926 -1.570796 0"/>
-        <parent link="${prefix}link_6_t"/>
-        <child link="${prefix}tool0"/>
-    </joint>
     <!-- end of joint list -->
     <!-- ROS base_link to Robot Manufacturer World Coordinates transform -->
@@ -156,4 +150,18 @@
         <child link="${prefix}base"/>
     </joint>
+    <!-- ROS-Industrial 'flange' frame: attachment point for EEF models -->
+    <link name="${prefix}flange" />
+    <joint name="${prefix}joint_6_t-flange" type="fixed">
+        <origin xyz="0.080 0 0" rpy="0 0 0" />
+        <parent link="${prefix}link_6_t" />
+        <child link="${prefix}flange" />
+    </joint>
+    <!-- ROS-Industrial 'tool0' frame: all-zeros tool frame -->
+    <link name="${prefix}tool0" />
+    <joint name="${prefix}flange-tool0" type="fixed">
+        <origin xyz="0 0 0" rpy="${pi} ${-pi/2.0} 0" />
+        <parent link="${prefix}flange" />
+        <child link="${prefix}tool0" />
+    </joint>
     </xacro:macro>
 </robot>

File: motoman_hc10_support/urdf/hc10_macro.xacro (robot description, xacro)
@@ -98,5 +98,4 @@
       </collision>
     </link>
-    <link name="${prefix}tool0"/>
     <!-- end of link list -->
     <!-- joint list -->
@@ -143,9 +142,4 @@
       <limit lower="${radians(-180)}" upper="${radians(180)}" effort="31.36" velocity="${radians(250)}"/>
     </joint>
-    <joint name="${prefix}joint_6_t-tool0" type="fixed">
-      <origin xyz="0 0 -0.130" rpy="${pi} 0 0"/>
-      <parent link="${prefix}link_6_t"/>
-      <child link="${prefix}tool0"/>
-    </joint>
     <!-- end of joint list -->
     <!-- ROS base_link to Robot Manufacturer World Coordinates transform -->
@@ -156,4 +150,18 @@
       <child link="${prefix}base"/>
     </joint>
+    <!-- ROS-Industrial 'flange' frame: attachment point for EEF models -->
+    <link name="${prefix}flange" />
+    <joint name="${prefix}joint_6_t-flange" type="fixed">
+      <origin xyz="0 0 -0.130" rpy="0 ${pi/2} 0" />
+      <parent link="${prefix}link_6_t" />
+      <child link="${prefix}flange" />
+    </joint>
+    <!-- ROS-Industrial 'tool0' frame: all-zeros tool frame -->
+    <link name="${prefix}tool0" />
+    <joint name="${prefix}flange-tool0" type="fixed">
+      <origin xyz="0 0 0" rpy="${pi} ${-pi/2.0} 0" />
+      <parent link="${prefix}flange" />
+      <child link="${prefix}tool0" />
+    </joint>
   </xacro:macro>
 </robot>

File: motoman_hc10_support/urdf/hc10dt_macro.xacro (robot description, xacro)
@@ -101,5 +101,4 @@
       </collision>
     </link>
-    <link name="${prefix}tool0"/>
     <!-- end of link list -->
     <!-- joint list -->
@@ -146,9 +145,4 @@
       <limit lower="${radians(-180)}" upper="${radians(180)}" effort="31.36" velocity="${radians(250)}"/>
     </joint>
-    <joint name="${prefix}joint_6_t-tool0" type="fixed">
-      <origin xyz="0 0 -0.170" rpy="${pi} 0 0"/>
-      <parent link="${prefix}link_6_t"/>
-      <child link="${prefix}tool0"/>
-    </joint>
     <!-- end of joint list -->
     <!-- ROS base_link to Robot Manufacturer World Coordinates transform -->
@@ -159,4 +153,18 @@
       <child link="${prefix}base"/>
     </joint>
+    <!-- ROS-Industrial 'flange' frame: attachment point for EEF models -->
+    <link name="${prefix}flange" />
+    <joint name="${prefix}joint_6_t-flange" type="fixed">
+      <origin xyz="0 0 -0.170" rpy="0 ${pi/2} 0" />
+      <parent link="${prefix}link_6_t" />
+      <child link="${prefix}flange" />
+    </joint>
+    <!-- ROS-Industrial 'tool0' frame: all-zeros tool frame -->
+    <link name="${prefix}tool0" />
+    <joint name="${prefix}flange-tool0" type="fixed">
+      <origin xyz="0 0 0" rpy="${pi} ${-pi/2.0} 0" />
+      <parent link="${prefix}flange" />
+      <child link="${prefix}tool0" />
+    </joint>
   </xacro:macro>
 </robot>

File: motoman_hc20_support/urdf/hc20_macro.xacro (robot description, xacro)
@@ -98,5 +98,4 @@
       </collision>
     </link>
-    <link name="${prefix}tool0"/>
     <!-- end of link list -->
     <!-- joint list -->
@@ -143,9 +142,4 @@
       <limit lower="${radians(-210)}" upper="${radians(210)}" effort="141.12" velocity="${radians(180)}"/>
     </joint>
-    <joint name="${prefix}joint_6_t-tool0" type="fixed">
-      <origin xyz="0.200 0 0" rpy="${radians(180)} ${radians(-90)} 0"/>
-      <parent link="${prefix}link_6_t"/>
-      <child link="${prefix}tool0"/>
-    </joint>
     <!-- end of joint list -->
     <!-- ROS base_link to Robot Manufacturer World Coordinates transform -->
@@ -156,4 +150,18 @@
       <child link="${prefix}base"/>
     </joint>
+    <!-- ROS-Industrial 'flange' frame: attachment point for EEF models -->
+    <link name="${prefix}flange" />
+    <joint name="${prefix}joint_6_t-flange" type="fixed">
+      <origin xyz="0.200 0 -0" rpy="0 0 0" />
+      <parent link="${prefix}link_6_t" />
+      <child link="${prefix}flange" />
+    </joint>
+    <!-- ROS-Industrial 'tool0' frame: all-zeros tool frame -->
+    <link name="${prefix}tool0" />
+    <joint name="${prefix}flange-tool0" type="fixed">
+      <origin xyz="0 0 0" rpy="${pi} ${-pi/2.0} 0" />
+      <parent link="${prefix}flange" />
+      <child link="${prefix}tool0" />
+    </joint>
   </xacro:macro>
 </robot>

File: motoman_mh12_support/urdf/mh12_macro.xacro (robot description, xacro)
@@ -98,5 +98,4 @@
         </collision>
     </link>
-    <link name="${prefix}tool0"/>
     <!-- end of link list -->
     <!-- joint list -->
@@ -143,9 +142,4 @@
         <limit lower="-6.2832" upper="6.2832" effort="14.80" velocity="10.6465"/>
     </joint>
-    <joint name="${prefix}joint_6_t-tool0" type="fixed">
-        <origin xyz="0.100 0 0" rpy="3.1415926 -1.570796 0"/>
-        <parent link="${prefix}link_6_t"/>
-        <child link="${prefix}tool0"/>
-    </joint>
     <!-- end of joint list -->
     <!-- ROS base_link to Robot Manufacturer World Coordinates transform -->
@@ -156,4 +150,18 @@
         <child link="${prefix}base"/>
     </joint>
+    <!-- ROS-Industrial 'flange' frame: attachment point for EEF models -->
+    <link name="${prefix}flange" />
+    <joint name="${prefix}joint_6_t-flange" type="fixed">
+        <origin xyz="0.100 0 0" rpy="0 0 0" />
+        <parent link="${prefix}link_6_t" />
+        <child link="${prefix}flange" />
+    </joint>
+    <!-- ROS-Industrial 'tool0' frame: all-zeros tool frame -->
+    <link name="${prefix}tool0" />
+    <joint name="${prefix}flange-tool0" type="fixed">
+        <origin xyz="0 0 0" rpy="${pi} ${-pi/2.0} 0" />
+        <parent link="${prefix}flange" />
+        <child link="${prefix}tool0" />
+    </joint>
     </xacro:macro>
 </robot>

File: motoman_mh50_support/urdf/mh50_macro.xacro (robot description, xacro)
@@ -98,5 +98,4 @@
         </collision>
     </link>
-    <link name="${prefix}tool0"/>
     <!-- end of link list -->
     <!-- joint list -->
@@ -143,9 +142,4 @@
         <limit lower="-6.2831" upper="6.2831" effort="333.43" velocity="6.283"/>
     </joint>
-    <joint name="${prefix}joint_6_t-tool0" type="fixed">
-        <origin xyz="0.175 0 0" rpy="3.1415926 -1.570796 0"/>
-        <parent link="${prefix}link_6_t"/>
-        <child link="${prefix}tool0"/>
-    </joint>
     <!-- end of joint list -->
     <!-- ROS base_link to Robot Manufacturer World Coordinates transform -->
@@ -156,4 +150,18 @@
         <child link="${prefix}base"/>
     </joint>
+    <!-- ROS-Industrial 'flange' frame: attachment point for EEF models -->
+    <link name="${prefix}flange" />
+    <joint name="${prefix}link_6_t-flange" type="fixed">
+        <origin xyz="0.175 0 0" rpy="0 0 0" />
+        <parent link="${prefix}link_6_t" />
+        <child link="${prefix}flange" />
+    </joint>
+    <!-- ROS-Industrial 'tool0' frame: all-zeros tool frame -->
+    <link name="${prefix}tool0" />
+    <joint name="${prefix}flange-tool0" type="fixed">
+        <origin xyz="0 0 0" rpy="${pi} ${-pi/2.0} 0" />
+        <parent link="${prefix}flange" />
+        <child link="${prefix}tool0" />
+    </joint>
     </xacro:macro>
 </robot>

File: motoman_mh5_support/urdf/mh5_macro.xacro (robot description, xacro)
@@ -167,4 +167,18 @@
 		</joint>
 		<!-- end of joint list -->
+		<!-- ROS-Industrial 'flange' frame: attachment point for EEF models -->
+		<link name="${prefix}flange" />
+		<joint name="${prefix}link_t-flange" type="fixed">
+			<origin xyz="0 0 0" rpy="0 0 0" />
+			<parent link="${prefix}link_t" />
+			<child link="${prefix}flange" />
+		</joint>
+		<!-- ROS-Industrial 'tool0' frame: all-zeros tool frame -->
+		<link name="${prefix}tool0" />
+		<joint name="${prefix}flange-tool0" type="fixed">
+			<origin xyz="0 0 0" rpy="${pi} ${-pi/2.0} 0" />
+			<parent link="${prefix}flange" />
+			<child link="${prefix}tool0" />
+		</joint>
 	</xacro:macro>
 </robot>

File: motoman_motomini_support/urdf/motomini_macro.xacro (robot description, xacro)
@@ -98,5 +98,4 @@
     </collision>
   </link>
-  <link name="${prefix}tool0"/>
   <!-- end of link list -->
   <!-- joint list -->
@@ -143,9 +142,4 @@
     <limit lower="-6.2831" upper="6.2831" effort="0.07" velocity="10.4719"/>
   </joint>
-  <joint name="${prefix}joint_6_t-tool0" type="fixed">
-    <origin xyz="0 0 -0.040 " rpy="${pi} 0 0"/>
-    <parent link="${prefix}link_6_t"/>
-    <child link="${prefix}tool0"/>
-  </joint>
   <!-- end of joint list -->
   <!-- ROS base_link to Robot Manufacturer World Coordinates transform -->
@@ -156,4 +150,18 @@
     <child link="${prefix}base"/>
   </joint>
+  <!-- ROS-Industrial 'flange' frame: attachment point for EEF models -->
+  <link name="${prefix}flange" />
+  <joint name="${prefix}joint_6_t-flange" type="fixed">
+    <origin xyz="0 0 -0.040" rpy="0 ${pi/2.0} 0" />
+    <parent link="${prefix}link_6_t" />
+    <child link="${prefix}flange" />
+  </joint>
+  <!-- ROS-Industrial 'tool0' frame: all-zeros tool frame -->
+  <link name="${prefix}tool0" />
+  <joint name="${prefix}flange-tool0" type="fixed">
+    <origin xyz="0 0 0" rpy="${pi} ${-pi/2.0} 0" />
+    <parent link="${prefix}flange" />
+    <child link="${prefix}tool0" />
+  </joint>
   </xacro:macro>
 </robot>
