Commit message: Use new resources package.
And remove macro-local definitions of colors and materials from .xacro files.

File: motoman_gp12_support/urdf/gp12_macro.xacro (robot description, xacro)
@@ -2,8 +2,5 @@
 <robot xmlns:xacro="http://ros.org/wiki/xacro">
 <xacro:macro name="motoman_gp12" params="prefix">
-    <!-- Properties -->
-    <material name="yaskawa_blue">
-          <color rgba="0.12941 0.14902 0.74902 1" />
-    </material>
+    <xacro:include filename="$(find motoman_resources)/urdf/common_materials.xacro"/>
     <!-- link list -->
     <link name="${prefix}base_link">
@@ -12,5 +9,5 @@
                 <mesh filename="package://motoman_gp12_support/meshes/visual/gp12_base_link.stl"/>
             </geometry>
-            <material name="yaskawa_blue"/>
+            <xacro:material_yaskawa_blue/>
         </visual>
         <collision>
@@ -25,5 +22,5 @@
                 <mesh filename="package://motoman_gp12_support/meshes/visual/gp12_link_1_s.stl"/>
             </geometry>
-            <material name="yaskawa_blue"/>
+            <xacro:material_yaskawa_blue/>
         </visual>
         <collision>
@@ -38,5 +35,5 @@
                 <mesh filename="package://motoman_gp12_support/meshes/visual/gp12_link_2_l.stl"/>
             </geometry>
-            <material name="yaskawa_blue"/>
+            <xacro:material_yaskawa_blue/>
         </visual>
         <collision>
@@ -51,5 +48,5 @@
                 <mesh filename="package://motoman_gp12_support/meshes/visual/gp12_link_3_u.stl"/>
             </geometry>
-            <material name="yaskawa_blue"/>
+            <xacro:material_yaskawa_blue/>
         </visual>
         <collision>
@@ -64,5 +61,5 @@
                 <mesh filename="package://motoman_gp12_support/meshes/visual/gp12_link_4_r.stl"/>
             </geometry>
-            <material name="yaskawa_blue"/>
+            <xacro:material_yaskawa_blue/>
         </visual>
         <collision>
@@ -77,5 +74,5 @@
                 <mesh filename="package://motoman_gp12_support/meshes/visual/gp12_link_5_b.stl"/>
             </geometry>
-            <material name="yaskawa_blue"/>
+            <xacro:material_yaskawa_blue/>
         </visual>
         <collision>
@@ -90,5 +87,5 @@
                 <mesh filename="package://motoman_gp12_support/meshes/visual/gp12_link_6_t.stl"/>
             </geometry>
-            <material name="yaskawa_blue"/>
+            <xacro:material_yaskawa_blue/>
         </visual>
         <collision>

File: motoman_gp180_support/urdf/gp180_120_macro.xacro (robot description, xacro)
@@ -2,8 +2,5 @@
 <robot xmlns:xacro="http://ros.org/wiki/xacro">
 <xacro:macro name="motoman_gp180_120" params="prefix">
-    <!-- Properties -->
-    <material name="yaskawa_blue">
-        <color rgba="0 0.35546875 0.671875 1" />
-    </material>
+    <xacro:include filename="$(find motoman_resources)/urdf/common_materials.xacro"/>
     <!-- link list -->
     <link name="${prefix}base_link">
@@ -12,5 +9,5 @@
                 <mesh filename="package://motoman_gp180_support/meshes/gp180_120/visual/base_link.stl"/>
             </geometry>
-            <material name="yaskawa_blue"/>
+            <xacro:material_yaskawa_blue/>
         </visual>
         <collision>
@@ -25,5 +22,5 @@
                 <mesh filename="package://motoman_gp180_support/meshes/gp180_120/visual/link_1_s.stl"/>
             </geometry>
-            <material name="yaskawa_blue"/>
+            <xacro:material_yaskawa_blue/>
         </visual>
         <collision>
@@ -38,5 +35,5 @@
                 <mesh filename="package://motoman_gp180_support/meshes/gp180_120/visual/link_2_l.stl"/>
             </geometry>
-            <material name="yaskawa_blue"/>
+            <xacro:material_yaskawa_blue/>
         </visual>
         <collision>
@@ -51,5 +48,5 @@
                 <mesh filename="package://motoman_gp180_support/meshes/gp180_120/visual/link_3_u.stl"/>
             </geometry>
-            <material name="yaskawa_blue"/>
+            <xacro:material_yaskawa_blue/>
         </visual>
         <collision>
@@ -64,5 +61,5 @@
                 <mesh filename="package://motoman_gp180_support/meshes/gp180_120/visual/link_4_r.stl"/>
             </geometry>
-            <material name="yaskawa_blue"/>
+            <xacro:material_yaskawa_blue/>
         </visual>
         <collision>
@@ -77,5 +74,5 @@
                 <mesh filename="package://motoman_gp180_support/meshes/gp180_120/visual/link_5_b.stl"/>
             </geometry>
-            <material name="yaskawa_blue"/>
+            <xacro:material_yaskawa_blue/>
         </visual>
         <collision>
@@ -90,5 +87,5 @@
                 <mesh filename="package://motoman_gp180_support/meshes/gp180_120/visual/link_6_t.stl"/>
             </geometry>
-            <material name="yaskawa_blue"/>
+            <xacro:material_yaskawa_blue/>
         </visual>
         <collision>

File: motoman_gp25_support/urdf/gp25_macro.xacro (robot description, xacro)
@@ -2,8 +2,5 @@
 <robot xmlns:xacro="http://ros.org/wiki/xacro">
 <xacro:macro name="motoman_gp25" params="prefix">
-    <!-- Properties -->
-    <material name="yaskawa_blue">
-          <color rgba="0.12941 0.14902 0.74902 1" />
-    </material>
+    <xacro:include filename="$(find motoman_resources)/urdf/common_materials.xacro"/>
     <!-- link list -->
     <link name="${prefix}base_link">
@@ -12,5 +9,5 @@
                 <mesh filename="package://motoman_gp25_support/meshes/visual/base_link.stl"/>
             </geometry>
-            <material name="yaskawa_blue"/>
+            <xacro:material_yaskawa_blue/>
         </visual>
         <collision>
@@ -25,5 +22,5 @@
                 <mesh filename="package://motoman_gp25_support/meshes/visual/link_1_s.stl"/>
             </geometry>
-            <material name="yaskawa_blue"/>
+            <xacro:material_yaskawa_blue/>
         </visual>
         <collision>
@@ -38,5 +35,5 @@
                 <mesh filename="package://motoman_gp25_support/meshes/visual/link_2_l.stl"/>
             </geometry>
-            <material name="yaskawa_blue"/>
+            <xacro:material_yaskawa_blue/>
         </visual>
         <collision>
@@ -51,5 +48,5 @@
                 <mesh filename="package://motoman_gp25_support/meshes/visual/link_3_u.stl"/>
             </geometry>
-            <material name="yaskawa_blue"/>
+            <xacro:material_yaskawa_blue/>
         </visual>
         <collision>
@@ -64,5 +61,5 @@
                 <mesh filename="package://motoman_gp25_support/meshes/visual/link_4_r.stl"/>
             </geometry>
-            <material name="yaskawa_blue"/>
+            <xacro:material_yaskawa_blue/>
         </visual>
         <collision>
@@ -77,5 +74,5 @@
                 <mesh filename="package://motoman_gp25_support/meshes/visual/link_5_b.stl"/>
             </geometry>
-            <material name="yaskawa_blue"/>
+            <xacro:material_yaskawa_blue/>
         </visual>
         <collision>
@@ -90,5 +87,5 @@
                 <mesh filename="package://motoman_gp25_support/meshes/visual/link_6_t.stl"/>
             </geometry>
-            <material name="yaskawa_blue"/>
+            <xacro:material_yaskawa_blue/>
         </visual>
         <collision>

File: motoman_gp50_support/urdf/gp50_macro.xacro (robot description, xacro)
@@ -2,8 +2,5 @@
 <robot xmlns:xacro="http://ros.org/wiki/xacro">
   <xacro:macro name="motoman_gp50" params="prefix">
-    <!-- Properties -->
-    <material name="yaskawa_blue">
-          <color rgba="0.12941 0.14902 0.74902 1" />
-    </material>
+    <xacro:include filename="$(find motoman_resources)/urdf/common_materials.xacro"/>
     <!-- link list -->
     <link name="${prefix}base_link">
@@ -12,5 +9,5 @@
                 <mesh filename="package://motoman_gp50_support/meshes/gp50/visual/base_link.stl"/>
             </geometry>
-            <material name="yaskawa_blue"/>
+            <xacro:material_yaskawa_blue/>
         </visual>
         <collision>
@@ -25,5 +22,5 @@
                 <mesh filename="package://motoman_gp50_support/meshes/gp50/visual/link_1_s.stl"/>
             </geometry>
-            <material name="yaskawa_blue"/>
+            <xacro:material_yaskawa_blue/>
         </visual>
         <collision>
@@ -38,5 +35,5 @@
                 <mesh filename="package://motoman_gp50_support/meshes/gp50/visual/link_2_l.stl"/>
             </geometry>
-            <material name="yaskawa_blue"/>
+            <xacro:material_yaskawa_blue/>
         </visual>
         <collision>
@@ -51,5 +48,5 @@
                 <mesh filename="package://motoman_gp50_support/meshes/gp50/visual/link_3_u.stl"/>
             </geometry>
-            <material name="yaskawa_blue"/>
+            <xacro:material_yaskawa_blue/>
         </visual>
         <collision>
@@ -64,5 +61,5 @@
                 <mesh filename="package://motoman_gp50_support/meshes/gp50/visual/link_4_r.stl"/>
             </geometry>
-            <material name="yaskawa_blue"/>
+            <xacro:material_yaskawa_blue/>
         </visual>
         <collision>
@@ -77,5 +74,5 @@
                 <mesh filename="package://motoman_gp50_support/meshes/gp50/visual/link_5_b.stl"/>
             </geometry>
-            <material name="yaskawa_blue"/>
+            <xacro:material_yaskawa_blue/>
         </visual>
         <collision>
@@ -90,5 +87,5 @@
                 <mesh filename="package://motoman_gp50_support/meshes/gp50/visual/link_6_t.stl"/>
             </geometry>
-            <material name="yaskawa_blue"/>
+            <xacro:material_yaskawa_blue/>
         </visual>
         <collision>

File: motoman_gp7_support/urdf/gp7_macro.xacro (robot description, xacro)
@@ -2,8 +2,5 @@
 <robot xmlns:xacro="http://ros.org/wiki/xacro">
 <xacro:macro name="motoman_gp7" params="prefix">
-    <!-- Properties -->
-    <material name="yaskawa_blue">
-          <color rgba="0.12941 0.14902 0.74902 1" />
-    </material>
+    <xacro:include filename="$(find motoman_resources)/urdf/common_materials.xacro"/>
     <!-- link list -->
     <link name="${prefix}base_link">
@@ -12,5 +9,5 @@
                 <mesh filename="package://motoman_gp7_support/meshes/visual/gp7_base_link.stl"/>
             </geometry>
-            <material name="yaskawa_blue"/>
+            <xacro:material_yaskawa_blue/>
         </visual>
         <collision>
@@ -25,5 +22,5 @@
                 <mesh filename="package://motoman_gp7_support/meshes/visual/gp7_link_1_s.stl"/>
             </geometry>
-            <material name="yaskawa_blue"/>
+            <xacro:material_yaskawa_blue/>
         </visual>
         <collision>
@@ -38,5 +35,5 @@
                 <mesh filename="package://motoman_gp7_support/meshes/visual/gp7_link_2_l.stl"/>
             </geometry>
-            <material name="yaskawa_blue"/>
+            <xacro:material_yaskawa_blue/>
         </visual>
         <collision>
@@ -51,5 +48,5 @@
                 <mesh filename="package://motoman_gp7_support/meshes/visual/gp7_link_3_u.stl"/>
             </geometry>
-            <material name="yaskawa_blue"/>
+            <xacro:material_yaskawa_blue/>
         </visual>
         <collision>
@@ -64,5 +61,5 @@
                 <mesh filename="package://motoman_gp7_support/meshes/visual/gp7_link_4_r.stl"/>
             </geometry>
-            <material name="yaskawa_blue"/>
+            <xacro:material_yaskawa_blue/>
         </visual>
         <collision>
@@ -77,5 +74,5 @@
                 <mesh filename="package://motoman_gp7_support/meshes/visual/gp7_link_5_b.stl"/>
             </geometry>
-            <material name="yaskawa_blue"/>
+            <xacro:material_yaskawa_blue/>
         </visual>
         <collision>
@@ -90,5 +87,5 @@
                 <mesh filename="package://motoman_gp7_support/meshes/visual/gp7_link_6_t.stl"/>
             </geometry>
-            <material name="yaskawa_blue"/>
+            <xacro:material_yaskawa_blue/>
         </visual>
         <collision>

File: motoman_gp88_support/urdf/gp88_macro.xacro (robot description, xacro)
@@ -2,8 +2,5 @@
 <robot xmlns:xacro="http://ros.org/wiki/xacro">
   <xacro:macro name="motoman_gp88" params="prefix">
-    <!-- Properties -->
-    <material name="yaskawa_blue">
-      <color rgba="0 0.35546875 0.671875 1" />
-    </material>
+    <xacro:include filename="$(find motoman_resources)/urdf/common_materials.xacro"/>
     <!-- link list -->
     <link name="${prefix}base_link">
@@ -12,5 +9,5 @@
           <mesh filename="package://motoman_gp88_support/meshes/gp88/visual/base_link.stl"/>
         </geometry>
-        <material name="yaskawa_blue"/>
+        <xacro:material_yaskawa_blue/>
       </visual>
       <collision>
@@ -25,5 +22,5 @@
           <mesh filename="package://motoman_gp88_support/meshes/gp88/visual/link_1_s.stl"/>
         </geometry>
-        <material name="yaskawa_blue"/>
+        <xacro:material_yaskawa_blue/>
       </visual>
       <collision>
@@ -38,5 +35,5 @@
           <mesh filename="package://motoman_gp88_support/meshes/gp88/visual/link_2_l.stl"/>
         </geometry>
-        <material name="yaskawa_blue"/>
+        <xacro:material_yaskawa_blue/>
       </visual>
       <collision>
@@ -51,5 +48,5 @@
           <mesh filename="package://motoman_gp88_support/meshes/gp88/visual/link_3_u.stl"/>
         </geometry>
-        <material name="yaskawa_blue"/>
+        <xacro:material_yaskawa_blue/>
       </visual>
       <collision>
@@ -64,5 +61,5 @@
           <mesh filename="package://motoman_gp88_support/meshes/gp88/visual/link_4_r.stl"/>
         </geometry>
-        <material name="yaskawa_blue"/>
+        <xacro:material_yaskawa_blue/>
       </visual>
       <collision>
@@ -77,5 +74,5 @@
           <mesh filename="package://motoman_gp88_support/meshes/gp88/visual/link_5_b.stl"/>
         </geometry>
-        <material name="yaskawa_blue"/>
+        <xacro:material_yaskawa_blue/>
       </visual>
       <collision>
@@ -90,5 +87,5 @@
           <mesh filename="package://motoman_gp88_support/meshes/gp88/visual/link_6_t.stl"/>
         </geometry>
-        <material name="yaskawa_blue"/>
+        <xacro:material_yaskawa_blue/>
       </visual>
       <collision>

File: motoman_gp8_support/urdf/gp8_macro.xacro (robot description, xacro)
@@ -2,8 +2,5 @@
 <robot xmlns:xacro="http://ros.org/wiki/xacro">
 <xacro:macro name="motoman_gp8" params="prefix">
-    <!-- Properties -->
-    <material name="yaskawa_blue">
-          <color rgba="0.12941 0.14902 0.74902 1" />
-    </material>
+    <xacro:include filename="$(find motoman_resources)/urdf/common_materials.xacro"/>
     <!-- link list -->
     <link name="${prefix}base_link">
@@ -12,5 +9,5 @@
                 <mesh filename="package://motoman_gp8_support/meshes/visual/gp8_base_link.stl"/>
             </geometry>
-            <material name="yaskawa_blue"/>
+            <xacro:material_yaskawa_blue/>
         </visual>
         <collision>
@@ -25,5 +22,5 @@
                 <mesh filename="package://motoman_gp8_support/meshes/visual/gp8_link_1_s.stl"/>
             </geometry>
-            <material name="yaskawa_blue"/>
+            <xacro:material_yaskawa_blue/>
         </visual>
         <collision>
@@ -38,5 +35,5 @@
                 <mesh filename="package://motoman_gp8_support/meshes/visual/gp8_link_2_l.stl"/>
             </geometry>
-            <material name="yaskawa_blue"/>
+            <xacro:material_yaskawa_blue/>
         </visual>
         <collision>
@@ -51,5 +48,5 @@
                 <mesh filename="package://motoman_gp8_support/meshes/visual/gp8_link_3_u.stl"/>
             </geometry>
-            <material name="yaskawa_blue"/>
+            <xacro:material_yaskawa_blue/>
         </visual>
         <collision>
@@ -64,5 +61,5 @@
                 <mesh filename="package://motoman_gp8_support/meshes/visual/gp8_link_4_r.stl"/>
             </geometry>
-            <material name="yaskawa_blue"/>
+            <xacro:material_yaskawa_blue/>
         </visual>
         <collision>
@@ -77,5 +74,5 @@
                 <mesh filename="package://motoman_gp8_support/meshes/visual/gp8_link_5_b.stl"/>
             </geometry>
-            <material name="yaskawa_blue"/>
+            <xacro:material_yaskawa_blue/>
         </visual>
         <collision>
@@ -90,5 +87,5 @@
                 <mesh filename="package://motoman_gp8_support/meshes/visual/gp8_link_6_t.stl"/>
             </geometry>
-            <material name="yaskawa_blue"/>
+            <xacro:material_yaskawa_blue/>
         </visual>
         <collision>

File: motoman_hc10_support/urdf/hc10_macro.xacro (robot description, xacro)
@@ -2,8 +2,5 @@
 <robot xmlns:xacro="http://ros.org/wiki/xacro">
   <xacro:macro name="motoman_hc10" params="prefix">
-    <!-- Properties -->
-    <material name="yaskawa_blue">
-      <color rgba="0.12941 0.14902 0.74902 1" />
-    </material>
+    <xacro:include filename="$(find motoman_resources)/urdf/common_materials.xacro"/>
     <!-- link list -->
     <link name="${prefix}base_link">
@@ -12,5 +9,5 @@
           <mesh filename="package://motoman_hc10_support/meshes/hc10/visual/base_link.dae"/>
         </geometry>
-        <material name="yaskawa_blue"/>
+        <xacro:material_yaskawa_blue/>
       </visual>
       <collision>
@@ -25,5 +22,5 @@
           <mesh filename="package://motoman_hc10_support/meshes/hc10/visual/link_1_s.dae"/>
         </geometry>
-        <material name="yaskawa_blue"/>
+        <xacro:material_yaskawa_blue/>
       </visual>
       <collision>
@@ -38,5 +35,5 @@
           <mesh filename="package://motoman_hc10_support/meshes/hc10/visual/link_2_l.dae"/>
         </geometry>
-        <material name="yaskawa_blue"/>
+        <xacro:material_yaskawa_blue/>
       </visual>
       <collision>
@@ -51,5 +48,5 @@
           <mesh filename="package://motoman_hc10_support/meshes/hc10/visual/link_3_u.dae"/>
         </geometry>
-        <material name="yaskawa_blue"/>
+        <xacro:material_yaskawa_blue/>
       </visual>
       <collision>
@@ -64,5 +61,5 @@
           <mesh filename="package://motoman_hc10_support/meshes/hc10/visual/link_4_r.dae"/>
         </geometry>
-        <material name="yaskawa_blue"/>
+        <xacro:material_yaskawa_blue/>
       </visual>
       <collision>
@@ -77,5 +74,5 @@
           <mesh filename="package://motoman_hc10_support/meshes/hc10/visual/link_5_b.dae"/>
         </geometry>
-        <material name="yaskawa_blue"/>
+        <xacro:material_yaskawa_blue/>
       </visual>
       <collision>
@@ -90,5 +87,5 @@
           <mesh filename="package://motoman_hc10_support/meshes/hc10/visual/link_6_t.dae"/>
         </geometry>
-        <material name="yaskawa_blue"/>
+        <xacro:material_yaskawa_blue/>
       </visual>
       <collision>

File: motoman_hc10_support/urdf/hc10dt_macro.xacro (robot description, xacro)
@@ -2,11 +2,5 @@
 <robot xmlns:xacro="http://ros.org/wiki/xacro">
   <xacro:macro name="motoman_hc10dt" params="prefix">
-    <!-- Properties -->
-    <material name="yaskawa_blue">
-      <color rgba="0.12941 0.14902 0.74902 1" />
-    </material>
-    <material name="yaskawa_white">
-      <color rgba="0.95294 0.95294 0.95294 1" />
-    </material>
+    <xacro:include filename="$(find motoman_resources)/urdf/common_materials.xacro"/>
     <!-- link list -->
     <link name="${prefix}base_link">
@@ -15,5 +9,5 @@
           <mesh filename="package://motoman_hc10_support/meshes/hc10/visual/base_link.dae"/>
         </geometry>
-        <material name="yaskawa_blue"/>
+        <xacro:material_yaskawa_blue/>
       </visual>
       <collision>
@@ -28,5 +22,5 @@
           <mesh filename="package://motoman_hc10_support/meshes/hc10/visual/link_1_s.dae"/>
         </geometry>
-        <material name="yaskawa_blue"/>
+        <xacro:material_yaskawa_blue/>
       </visual>
       <collision>
@@ -41,5 +35,5 @@
           <mesh filename="package://motoman_hc10_support/meshes/hc10/visual/link_2_l.dae"/>
         </geometry>
-        <material name="yaskawa_blue"/>
+        <xacro:material_yaskawa_blue/>
       </visual>
       <collision>
@@ -54,5 +48,5 @@
           <mesh filename="package://motoman_hc10_support/meshes/hc10/visual/link_3_u.dae"/>
         </geometry>
-        <material name="yaskawa_blue"/>
+        <xacro:material_yaskawa_blue/>
       </visual>
       <collision>
@@ -67,5 +61,5 @@
           <mesh filename="package://motoman_hc10_support/meshes/hc10/visual/link_4_r.dae"/>
         </geometry>
-        <material name="yaskawa_blue"/>
+        <xacro:material_yaskawa_blue/>
       </visual>
       <collision>
@@ -80,5 +74,5 @@
           <mesh filename="package://motoman_hc10_support/meshes/hc10/visual/link_5_b.dae"/>
         </geometry>
-        <material name="yaskawa_blue"/>
+        <xacro:material_yaskawa_blue/>
       </visual>
       <collision>
@@ -93,5 +87,5 @@
           <mesh filename="package://motoman_hc10_support/meshes/hc10dt/visual/link_6_t.dae"/>
         </geometry>
-        <material name="yaskawa_blue"/>
+        <xacro:material_yaskawa_blue/>
       </visual>
       <collision>
