Commit message: Use new resources package.
And remove macro-local definitions of colors and materials from .xacro files.

File: motoman_hc20_support/urdf/hc20_macro.xacro (robot description, xacro)
@@ -2,8 +2,5 @@
 <robot xmlns:xacro="http://ros.org/wiki/xacro">
   <xacro:macro name="motoman_hc20" params="prefix">
-    <!-- Properties -->
-    <material name="yaskawa_white">
-      <color rgba="0.99 0.99 0.99 1" />
-    </material>
+    <xacro:include filename="$(find motoman_resources)/urdf/common_materials.xacro"/>
     <!-- link list -->
     <link name="${prefix}base_link">
@@ -12,5 +9,5 @@
           <mesh filename="package://motoman_hc20_support/meshes/hc20/visual/base_link.stl"/>
         </geometry>
-        <material name="yaskawa_white"/>
+        <xacro:material_yaskawa_white/>
       </visual>
       <collision>
@@ -25,5 +22,5 @@
           <mesh filename="package://motoman_hc20_support/meshes/hc20/visual/link_1_s.stl"/>
         </geometry>
-        <material name="yaskawa_white"/>
+        <xacro:material_yaskawa_white/>
       </visual>
       <collision>
@@ -38,5 +35,5 @@
           <mesh filename="package://motoman_hc20_support/meshes/hc20/visual/link_2_l.stl"/>
         </geometry>
-        <material name="yaskawa_white"/>
+        <xacro:material_yaskawa_white/>
       </visual>
       <collision>
@@ -51,5 +48,5 @@
           <mesh filename="package://motoman_hc20_support/meshes/hc20/visual/link_3_u.stl"/>
         </geometry>
-        <material name="yaskawa_white"/>
+        <xacro:material_yaskawa_white/>
       </visual>
       <collision>
@@ -64,5 +61,5 @@
           <mesh filename="package://motoman_hc20_support/meshes/hc20/visual/link_4_r.stl"/>
         </geometry>
-        <material name="yaskawa_white"/>
+        <xacro:material_yaskawa_white/>
       </visual>
       <collision>
@@ -77,5 +74,5 @@
           <mesh filename="package://motoman_hc20_support/meshes/hc20/visual/link_5_b.stl"/>
         </geometry>
-        <material name="yaskawa_white"/>
+        <xacro:material_yaskawa_white/>
       </visual>
       <collision>
@@ -90,5 +87,5 @@
           <mesh filename="package://motoman_hc20_support/meshes/hc20/visual/link_6_t.stl"/>
         </geometry>
-        <material name="yaskawa_white"/>
+        <xacro:material_yaskawa_white/>
       </visual>
       <collision>

File: motoman_mh12_support/urdf/mh12_macro.xacro (robot description, xacro)
@@ -2,8 +2,5 @@
 <robot xmlns:xacro="http://ros.org/wiki/xacro">
 <xacro:macro name="motoman_mh12" params="prefix">
-    <!-- Properties -->
-    <material name="yaskawa_blue">
-          <color rgba="0.12941 0.14902 0.74902 1" />
-    </material>
+    <xacro:include filename="$(find motoman_resources)/urdf/common_materials.xacro"/>
     <!-- link list -->
     <link name="${prefix}base_link">
@@ -12,5 +9,5 @@
                 <mesh filename="package://motoman_mh12_support/meshes/visual/mh12_base_link.stl"/>
             </geometry>
-            <material name="yaskawa_blue"/>
+            <xacro:material_yaskawa_blue/>
         </visual>
         <collision>
@@ -25,5 +22,5 @@
                 <mesh filename="package://motoman_mh12_support/meshes/visual/mh12_link_1_s.stl"/>
             </geometry>
-            <material name="yaskawa_blue"/>
+            <xacro:material_yaskawa_blue/>
         </visual>
         <collision>
@@ -38,5 +35,5 @@
                 <mesh filename="package://motoman_mh12_support/meshes/visual/mh12_link_2_l.stl"/>
             </geometry>
-            <material name="yaskawa_blue"/>
+            <xacro:material_yaskawa_blue/>
         </visual>
         <collision>
@@ -51,5 +48,5 @@
                 <mesh filename="package://motoman_mh12_support/meshes/visual/mh12_link_3_u.stl"/>
             </geometry>
-            <material name="yaskawa_blue"/>
+            <xacro:material_yaskawa_blue/>
         </visual>
         <collision>
@@ -64,5 +61,5 @@
                 <mesh filename="package://motoman_mh12_support/meshes/visual/mh12_link_4_r.stl"/>
             </geometry>
-            <material name="yaskawa_blue"/>
+            <xacro:material_yaskawa_blue/>
         </visual>
         <collision>
@@ -77,5 +74,5 @@
                 <mesh filename="package://motoman_mh12_support/meshes/visual/mh12_link_5_b.stl"/>
             </geometry>
-            <material name="yaskawa_blue"/>
+            <xacro:material_yaskawa_blue/>
         </visual>
         <collision>
@@ -90,5 +87,5 @@
                 <mesh filename="package://motoman_mh12_support/meshes/visual/mh12_link_6_t.stl"/>
             </geometry>
-            <material name="yaskawa_blue"/>
+            <xacro:material_yaskawa_blue/>
         </visual>
         <collision>

File: motoman_mh50_support/urdf/mh50_macro.xacro (robot description, xacro)
@@ -2,8 +2,5 @@
 <robot xmlns:xacro="http://ros.org/wiki/xacro">
 <xacro:macro name="motoman_mh50" params="prefix">
-    <!-- Properties -->
-    <material name="yaskawa_blue">
-          <color rgba="0.12941 0.14902 0.74902 1" />
-    </material>
+    <xacro:include filename="$(find motoman_resources)/urdf/common_materials.xacro"/>
     <!-- link list -->
     <link name="${prefix}base_link">
@@ -12,5 +9,5 @@
                 <mesh filename="package://motoman_mh50_support/meshes/visual/mh50_base_link.stl"/>
             </geometry>
-            <material name="yaskawa_blue"/>
+            <xacro:material_yaskawa_blue/>
         </visual>
         <collision>
@@ -25,5 +22,5 @@
                 <mesh filename="package://motoman_mh50_support/meshes/visual/mh50_link_1_s.stl"/>
             </geometry>
-            <material name="yaskawa_blue"/>
+            <xacro:material_yaskawa_blue/>
         </visual>
         <collision>
@@ -38,5 +35,5 @@
                 <mesh filename="package://motoman_mh50_support/meshes/visual/mh50_link_2_l.stl"/>
             </geometry>
-            <material name="yaskawa_blue"/>
+            <xacro:material_yaskawa_blue/>
         </visual>
         <collision>
@@ -51,5 +48,5 @@
                 <mesh filename="package://motoman_mh50_support/meshes/visual/mh50_link_3_u.stl"/>
             </geometry>
-            <material name="yaskawa_blue"/>
+            <xacro:material_yaskawa_blue/>
         </visual>
         <collision>
@@ -64,5 +61,5 @@
                 <mesh filename="package://motoman_mh50_support/meshes/visual/mh50_link_4_r.stl"/>
             </geometry>
-            <material name="yaskawa_blue"/>
+            <xacro:material_yaskawa_blue/>
         </visual>
         <collision>
@@ -77,5 +74,5 @@
                 <mesh filename="package://motoman_mh50_support/meshes/visual/mh50_link_5_b.stl"/>
             </geometry>
-            <material name="yaskawa_blue"/>
+            <xacro:material_yaskawa_blue/>
         </visual>
         <collision>
@@ -90,5 +87,5 @@
                 <mesh filename="package://motoman_mh50_support/meshes/visual/mh50_link_6_t.stl"/>
             </geometry>
-            <material name="yaskawa_blue"/>
+            <xacro:material_yaskawa_blue/>
         </visual>
         <collision>

File: motoman_motomini_support/urdf/motomini_macro.xacro (robot description, xacro)
@@ -2,8 +2,5 @@
 <robot xmlns:xacro="http://ros.org/wiki/xacro">
 <xacro:macro name="motoman_motomini" params="prefix">
-  <!-- Properties -->
-  <material name="yaskawa_blue">
-      <color rgba="0.12941 0.14902 0.74902 1" />
-  </material>
+  <xacro:include filename="$(find motoman_resources)/urdf/common_materials.xacro"/>
   <!-- link list -->
   <link name="${prefix}base_link">
@@ -12,5 +9,5 @@
         <mesh filename="package://motoman_motomini_support/meshes/motomini/visual/base_link.stl"/>
       </geometry>
-      <material name="yaskawa_blue"/>
+      <xacro:material_yaskawa_blue/>
     </visual>
     <collision>
@@ -25,5 +22,5 @@
         <mesh filename="package://motoman_motomini_support/meshes/motomini/visual/link_1_s.stl"/>
       </geometry>
-      <material name="yaskawa_blue"/>
+      <xacro:material_yaskawa_blue/>
     </visual>
     <collision>
@@ -38,5 +35,5 @@
         <mesh filename="package://motoman_motomini_support/meshes/motomini/visual/link_2_l.stl"/>
       </geometry>
-      <material name="yaskawa_blue"/>
+      <xacro:material_yaskawa_blue/>
     </visual>
     <collision>
@@ -51,5 +48,5 @@
         <mesh filename="package://motoman_motomini_support/meshes/motomini/visual/link_3_u.stl"/>
       </geometry>
-      <material name="yaskawa_blue"/>
+      <xacro:material_yaskawa_blue/>
     </visual>
     <collision>
@@ -64,5 +61,5 @@
         <mesh filename="package://motoman_motomini_support/meshes/motomini/visual/link_4_r.stl"/>
       </geometry>
-      <material name="yaskawa_blue"/>
+      <xacro:material_yaskawa_blue/>
     </visual>
     <collision>
@@ -77,5 +74,5 @@
         <mesh filename="package://motoman_motomini_support/meshes/motomini/visual/link_5_b.stl"/>
       </geometry>
-      <material name="yaskawa_blue"/>
+      <xacro:material_yaskawa_blue/>
     </visual>
     <collision>
@@ -90,5 +87,5 @@
         <mesh filename="package://motoman_motomini_support/meshes/motomini/visual/link_6_t.stl"/>
       </geometry>
-      <material name="yaskawa_blue"/>
+      <xacro:material_yaskawa_blue/>
     </visual>
     <collision>
