Commit message: resources: add two commonly used colours and materials
Both not necessarily 'official' in any way, but used in (old) xacro:macros.

File: motoman_resources/urdf/common_colors.xacro (robot description, xacro)
@@ -3,3 +3,7 @@
   <xacro:property name="color_yaskawa_blue" value="${33/255} ${38/255} ${191/255} 1.0"/>
   <xacro:property name="color_yaskawa_white" value="0.99 0.99 0.99 1"/>
+  <!-- not an official colour, but used in some old xacro:macros -->
+  <xacro:property name="color_yaskawa_yellow" value="0 1 1 1"/>
+  <!-- not an official colour, but used in some old xacro:macros -->
+  <xacro:property name="color_yaskawa_silver" value="0.8 0.8 0.8 1"/>
 </robot>

File: motoman_resources/urdf/common_materials.xacro (robot description, xacro)
@@ -12,3 +12,15 @@
     </material>
   </xacro:macro>
+  <!-- not an official colour, but used in some old xacro:macros -->
+  <xacro:macro name="material_yaskawa_yellow">
+    <material name="">
+      <color rgba="${color_yaskawa_yellow}"/>
+    </material>
+  </xacro:macro>
+  <!-- not an official colour, but used in some old xacro:macros -->
+  <xacro:macro name="material_yaskawa_silver">
+    <material name="">
+      <color rgba="${color_yaskawa_silver}"/>
+    </material>
+  </xacro:macro>
 </robot>
