Commit message: Use resources package in the rest of the support pkgs

File: motoman_ma2010_support/urdf/ma2010.xacro (robot description, xacro)
@@ -1,8 +1,4 @@
 <?xml version="1.0" ?>
 <robot name="motoman_ma2010" xmlns:xacro="http://ros.org/wiki/xacro">
-  <!-- Properties -->
-  <material name="yaskawa_blue">
-      <color rgba="0.12941 0.14902 0.74902 1" />
-  </material>
   <xacro:include filename="$(find motoman_ma2010_support)/urdf/ma2010_macro.xacro" />
   <xacro:motoman_ma2010 prefix=""/>

File: motoman_ma2010_support/urdf/ma2010_macro.xacro (robot description, xacro)
@@ -2,4 +2,5 @@
 <robot xmlns:xacro="http://ros.org/wiki/xacro">
   <xacro:macro name="motoman_ma2010" params="prefix">
+    <xacro:include filename="$(find motoman_resources)/urdf/common_materials.xacro"/>
     <!-- link list -->
     <link name="${prefix}base_link">
@@ -8,5 +9,5 @@
           <mesh filename="package://motoman_ma2010_support/meshes/ma2010/visual/base_link.stl"/>
         </geometry>
-        <material name="yaskawa_blue"/>
+        <xacro:material_yaskawa_blue/>
       </visual>
       <collision>
@@ -21,5 +22,5 @@
           <mesh filename="package://motoman_ma2010_support/meshes/ma2010/visual/link_1_s.stl"/>
         </geometry>
-        <material name="yaskawa_blue"/>
+        <xacro:material_yaskawa_blue/>
       </visual>
       <collision>
@@ -34,5 +35,5 @@
           <mesh filename="package://motoman_ma2010_support/meshes/ma2010/visual/link_2_l.stl"/>
         </geometry>
-        <material name="yaskawa_blue"/>
+        <xacro:material_yaskawa_blue/>
       </visual>
       <collision>
@@ -47,5 +48,5 @@
           <mesh filename="package://motoman_ma2010_support/meshes/ma2010/visual/link_3_u.stl"/>
         </geometry>
-        <material name="yaskawa_blue"/>
+        <xacro:material_yaskawa_blue/>
       </visual>
       <collision>
@@ -60,5 +61,5 @@
           <mesh filename="package://motoman_ma2010_support/meshes/ma2010/visual/link_4_r.stl"/>
         </geometry>
-        <material name="yaskawa_blue"/>
+        <xacro:material_yaskawa_blue/>
       </visual>
       <collision>
@@ -73,5 +74,5 @@
           <mesh filename="package://motoman_ma2010_support/meshes/ma2010/visual/link_5_b.stl"/>
         </geometry>
-        <material name="yaskawa_blue"/>
+        <xacro:material_yaskawa_blue/>
       </visual>
       <collision>
@@ -86,5 +87,5 @@
           <mesh filename="package://motoman_ma2010_support/meshes/ma2010/visual/link_6_t.stl"/>
         </geometry>
-        <material name="yaskawa_blue"/>
+        <xacro:material_yaskawa_blue/>
       </visual>
       <collision>

File: motoman_motopos_d500_support/urdf/motopos_d500_macro.xacro (robot description, xacro)
@@ -2,4 +2,5 @@
 <robot xmlns:xacro="http://ros.org/wiki/xacro">
   <xacro:macro name="motoman_motopos_d500" params="prefix">
+    <xacro:include filename="$(find motoman_resources)/urdf/common_materials.xacro"/>
     <!-- link list -->
     <link name="${prefix}base_link">
@@ -8,5 +9,5 @@
           <mesh filename="package://motoman_motopos_d500_support/meshes/motopos_d500/visual/base_link.stl"/>
         </geometry>
-        <material name="yaskawa_blue"/>
+        <xacro:material_yaskawa_blue/>
       </visual>
       <collision>
@@ -21,5 +22,5 @@
           <mesh filename="package://motoman_motopos_d500_support/meshes/motopos_d500/visual/link_1.stl"/>
         </geometry>
-        <material name="yaskawa_blue"/>
+        <xacro:material_yaskawa_blue/>
       </visual>
       <collision>
@@ -34,5 +35,5 @@
           <mesh filename="package://motoman_motopos_d500_support/meshes/motopos_d500/visual/link_2.stl"/>
         </geometry>
-        <material name="yaskawa_blue"/>
+        <xacro:material_yaskawa_blue/>
       </visual>
       <collision>

File: motoman_ms210_support/urdf/ms210_macro.xacro (robot description, xacro)
@@ -2,8 +2,5 @@
 <robot xmlns:xacro="http://ros.org/wiki/xacro">
 <xacro:macro name="motoman_ms210" params="prefix">
-  <!-- Properties -->
-  <material name="yaskawa_blue">
-    <color rgba="0 0.35546875 0.671875 1" />
-  </material>
+  <xacro:include filename="$(find motoman_resources)/urdf/common_materials.xacro"/>
   <!-- link list -->
   <link  name="${prefix}base_link">
@@ -13,5 +10,5 @@
         <mesh filename="package://motoman_ms210_support/meshes/ms210/visual/base_link.stl" />
       </geometry>
-      <material name="yaskawa_blue"/>
+      <xacro:material_yaskawa_blue/>
     </visual>
     <collision>
@@ -28,5 +25,5 @@
         <mesh filename="package://motoman_ms210_support/meshes/ms210/visual/link_1_s.stl" />
       </geometry>
-      <material name="yaskawa_blue"/>
+      <xacro:material_yaskawa_blue/>
     </visual>
     <collision>
@@ -43,5 +40,5 @@
         <mesh filename="package://motoman_ms210_support/meshes/ms210/visual/link_2_l.stl" />
       </geometry>
-      <material name="yaskawa_blue"/>
+      <xacro:material_yaskawa_blue/>
     </visual>
     <collision>
@@ -58,5 +55,5 @@
         <mesh filename="package://motoman_ms210_support/meshes/ms210/visual/link_3_u.stl" />
       </geometry>
-      <material name="yaskawa_blue"/>
+      <xacro:material_yaskawa_blue/>
     </visual>
     <collision>
@@ -73,5 +70,5 @@
         <mesh filename="package://motoman_ms210_support/meshes/ms210/visual/link_4_r.stl" />
       </geometry>
-      <material name="yaskawa_blue"/>
+      <xacro:material_yaskawa_blue/>
     </visual>
     <collision>
@@ -88,5 +85,5 @@
         <mesh filename="package://motoman_ms210_support/meshes/ms210/visual/link_5_b.stl" />
       </geometry>
-      <material name="yaskawa_blue"/>
+      <xacro:material_yaskawa_blue/>
     </visual>
     <collision>
@@ -103,5 +100,5 @@
         <mesh filename="package://motoman_ms210_support/meshes/ms210/visual/link_6_t.stl" />
       </geometry>
-      <material name="yaskawa_blue"/>
+      <xacro:material_yaskawa_blue/>
     </visual>
     <collision>
