Commit message: add support for d500 kinematic offsets from file

File: motoman_motopos_d500_support/urdf/motopos_d500.xacro (robot description, xacro)
@@ -6,4 +6,5 @@
   </material>
   <xacro:include filename="$(find motoman_motopos_d500_support)/urdf/motopos_d500_macro.xacro" />
+  <xacro:property name="kinematics_offsets" value="${load_yaml('$(find motoman_ar2010_support)' + '/config/default_kinematic_offsets.yaml')}"/>
   <xacro:motoman_motopos_d500 prefix=""/>
 </robot>

File: motoman_motopos_d500_support/urdf/motopos_d500_macro.xacro (robot description, xacro)
@@ -1,5 +1,5 @@
 <?xml version="1.0" ?>
 <robot xmlns:xacro="http://ros.org/wiki/xacro">
-<xacro:macro name="motoman_motopos_d500" params="prefix">
+<xacro:macro name="motoman_motopos_d500" params="prefix kinematic_offsets">
   <xacro:include filename="$(find motoman_resources)/urdf/common_materials.xacro"/>
   <!-- link list -->
@@ -50,5 +50,6 @@
     <parent link="${prefix}base_link"/>
     <child link="${prefix}link_1"/>
-    <origin xyz="0 0 0.380" rpy="0 0 0" />
+    <origin xyz="${0 + kinematic_offsets['link_1']['x']} ${0 + kinematic_offsets['link_1']['y']} ${0.380 + kinematic_offsets['link_1']['z']}"
+            rpy="${0 + kinematic_offsets['link_1']['roll']} ${0 + kinematic_offsets['link_1']['pitch']} ${0.380 + kinematic_offsets['link_1']['yaw']}" />
     <axis xyz="0 -1 0" />
     <limit lower="-2.3561" upper="2.3561" effort="1274" velocity="1.3962"/>
@@ -57,5 +58,6 @@
     <parent link="${prefix}link_1"/>
     <child link="${prefix}link_2"/>
-    <origin xyz="0 0 0" rpy="0 0 0" />
+    <origin xyz="${0 + kinematic_offsets['link_2']['x']} ${0 + kinematic_offsets['link_2']['y']} ${0 + kinematic_offsets['link_2']['z']}"
+            rpy="${0 + kinematic_offsets['link_2']['roll']} ${0 + kinematic_offsets['link_2']['pitch']} ${0.380 + kinematic_offsets['link_2']['yaw']}" />
     <axis xyz="0 0 -1" />
     <limit lower="-3.4906" upper="3.4906" effort="392" velocity="2.7925"/>

Commit message: find d500 support not ar2010

File: motoman_motopos_d500_support/urdf/motopos_d500.xacro (robot description, xacro)
@@ -6,5 +6,5 @@
   </material>
   <xacro:include filename="$(find motoman_motopos_d500_support)/urdf/motopos_d500_macro.xacro" />
-  <xacro:property name="kinematics_offsets" value="${load_yaml('$(find motoman_ar2010_support)' + '/config/default_kinematic_offsets.yaml')}"/>
+  <xacro:property name="kinematics_offsets" value="${load_yaml('$(find motoman_motopos_d500_support)' + '/config/default_kinematic_offsets.yaml')}"/>
   <xacro:motoman_motopos_d500 prefix=""/>
 </robot>
