Commit message: Add static broadcasters to link positioner frames to planning tree

File: motoman_motopos_d500_support/urdf/motopos_d500_macro.xacro (robot description, xacro)
@@ -47,6 +47,9 @@
   </link>
   <link name="${prefix}tool0"/>
-  <!-- this is here to set a base link in the URDF to link the positioner/base frame to for scanning -->
+  <!-- this is here to set a base link in the URDF to link the "positioner/base" frame to for scanning -->
   <link name="positioner_base_dummy_link"/>
+  <!-- this is here to set a base link in the URDF to link the "positioner/center" frame to for scanning. this is equivalent to the tool frame
+  in this case, but we define this so that the naming is consistent across positioner setups -->
+  <link name="positioner_center_dummy_link"/>
   <!-- end of link list -->
   <!-- joint list -->
@@ -83,4 +86,9 @@
     <child link="positioner_base_dummy_link"/>
   </joint>
+  <joint name="positioner_center_dummy_joint" type="fixed">
+    <origin xyz="0 0 0" rpy="0 0 0"/>
+    <parent link="${prefix}tool0"/>
+    <child link="positioner_center_dummy_link"/>
+  </joint>
   <!-- end of joint list -->
   <!-- ROS base_link to Robot Manufacturer World Coordinates transform -->

Commit message: Fix rotation axis direction on D500 positioner

File: motoman_motopos_d500_support/urdf/motopos_d500_macro.xacro (robot description, xacro)
@@ -71,5 +71,5 @@
     <child link="${prefix}link_2"/>
     <origin xyz="0 0 0" rpy="0 0 0" />
-    <axis xyz="0 0 1" />
+    <axis xyz="0 0 -1" />
     <limit lower="-3.4906" upper="3.4906" effort="392" velocity="2.7925"/>
   </joint>

Commit message: Add table to D500 positioner model

File: motoman_motopos_d500_support/urdf/motopos_d500_macro.xacro (robot description, xacro)
@@ -46,5 +46,20 @@
     </collision>
   </link>
-  <link name="${prefix}tool0"/>
+  <link name="${prefix}tool0">
+    <visual>
+      <geometry>
+          <cylinder length="${table_thickness}" radius="0.5" />
+      </geometry>
+      <origin xyz="0 0 0" rpy="0 0 0 " />
+      <material name="Cast Carbon Steel">
+        <color rgba="0.52941 0.54902 0.54902 1" />
+      </material>
+    </visual>
+    <collision>
+      <geometry>
+        <cylinder length="${table_thickness}" radius="0.5" />
+      </geometry>
+    </collision>
+  </link>
   <!-- this is here to set a base link in the URDF to link the "positioner/base" frame to for scanning -->
   <link name="positioner_base_dummy_link"/>
@@ -76,5 +91,5 @@
   <xacro:transmission_macro name="2"/>
   <joint name="${prefix}joint_2-tool0" type="fixed">
-    <origin xyz="0 0 ${0.150 + table_thickness}" rpy="0 0 0"/>
+    <origin xyz="0 0 ${0.165}" rpy="0 0 0"/>
     <parent link="${prefix}link_2"/>
     <child link="${prefix}tool0"/>
@@ -82,5 +97,5 @@
   <xacro:transmission_macro name="2"/>
   <joint name="positioner_base_dummy_joint" type="fixed">
-    <origin xyz="0 0 ${0.150 + table_thickness}" rpy="0 0 0"/>
+    <origin xyz="0 0 ${0.165 + table_thickness}" rpy="0 0 0"/>
     <parent link="${prefix}link_1"/>
     <child link="positioner_base_dummy_link"/>

Commit message: Fix height offset for D500 positioner center frame

File: motoman_motopos_d500_support/urdf/motopos_d500_macro.xacro (robot description, xacro)
@@ -1,4 +1,5 @@
 <?xml version="1.0" ?>
 <robot xmlns:xacro="http://ros.org/wiki/xacro">
+<xacro:property name="M_PI" value="3.1415926535897931"/>
 <xacro:property name="world_base_xyz" value="0 0 0"/>
 <xacro:property name="world_base_rpy" value="0 0 0"/>
@@ -102,5 +103,5 @@
   </joint>
   <joint name="positioner_center_dummy_joint" type="fixed">
-    <origin xyz="0 0 0" rpy="0 0 0"/>
+    <origin xyz="0 0 ${table_thickness}" rpy="0 0 0"/>
     <parent link="${prefix}tool0"/>
     <child link="positioner_center_dummy_link"/>

Commit message: FR-338 Removed d500 dummy links.

File: motoman_motopos_d500_support/urdf/motopos_d500_macro.xacro (robot description, xacro)
@@ -67,8 +67,8 @@
   </link>
   <!-- this is here to set a base link in the URDF to link the "positioner/base" frame to for scanning -->
-  <link name="positioner_base_dummy_link"/>
+  <link name="positioner/base"/>
   <!-- this is here to set a base link in the URDF to link the "positioner/center" frame to for scanning. this is equivalent to the tool frame
   in this case, but we define this so that the naming is consistent across positioner setups -->
-  <link name="positioner_center_dummy_link"/>
+  <link name="positioner/center"/>
   <!-- end of link list -->
   <!-- joint list -->
@@ -100,13 +100,13 @@
   </joint>
   <xacro:transmission_macro name="2"/>
-  <joint name="positioner_base_dummy_joint" type="fixed">
+  <joint name="positioner/base" type="fixed">
     <origin xyz="0 0 ${0.165 + table_thickness}" rpy="0 0 0"/>
     <parent link="${prefix}link_1"/>
-    <child link="positioner_base_dummy_link"/>
+    <child link="positioner/base"/>
   </joint>
-  <joint name="positioner_center_dummy_joint" type="fixed">
+  <joint name="positioner/center" type="fixed">
     <origin xyz="0 0 ${table_thickness}" rpy="0 0 0"/>
     <parent link="${prefix}tool0"/>
-    <child link="positioner_center_dummy_link"/>
+    <child link="positioner/center"/>
   </joint>
   <!-- end of joint list -->

Commit message: FR-338 d500 and mh185_vertical now use offsets. More modification will likely be required based on how the offset format is being saved.

File: motoman_motopos_d500_support/urdf/motopos_d500_macro.xacro (robot description, xacro)
@@ -89,5 +89,13 @@
     <parent link="${prefix}link_1"/>
     <child link="${prefix}link_2"/>
-    <origin xyz="0 0 0" rpy="0 0 0" />
+    <origin
+        xyz=
+            "${offsets[prefix + 'joint_2']['x']}
+             ${offsets[prefix + 'joint_2']['y']}
+             ${offsets[prefix + 'joint_2']['z']}"
+        rpy=
+            "${offsets[prefix + 'joint_2']['roll']}
+             ${offsets[prefix + 'joint_2']['pitch']}
+             ${offsets[prefix + 'joint_2']['yaw']}"/>
     <axis xyz="0 0 -1" />
     <limit lower="-3.4906" upper="3.4906" effort="392" velocity="2.7925"/>
@@ -101,5 +109,13 @@
   <xacro:transmission_macro name="2"/>
   <joint name="positioner/base" type="fixed">
-    <origin xyz="0 0 ${0.165 + table_thickness}" rpy="0 0 0"/>
+    <origin
+        xyz=
+            "${offsets[prefix + 'joint_2']['x']}
+             ${offsets[prefix + 'joint_2']['y']}
+             ${offsets[prefix + 'joint_2']['z'] + 0.165 + table_thickness}"
+        rpy=
+            "${offsets[prefix + 'joint_2']['roll']}
+             ${offsets[prefix + 'joint_2']['pitch']}
+             ${offsets[prefix + 'joint_2']['yaw']}"/>
     <parent link="${prefix}link_1"/>
     <child link="positioner/base"/>

File: motoman_motopos_mh185_vertical_support/urdf/motopos_mh185_vertical_macro.xacro (robot description, xacro)
@@ -56,6 +56,12 @@
     <child link="${prefix}link_1"/>
     <origin
-        xyz="${offsets[prefix + 'joint_1']['x']} ${offsets[prefix + 'joint_1']['y']} ${positioner_height + offsets[prefix + 'joint_1']['z']}"
-        rpy="${offsets[prefix + 'joint_1']['roll']} ${offsets[prefix + 'joint_1']['pitch']} ${offsets[prefix + 'joint_1']['yaw']}"
+        xyz=
+            "${offsets[prefix + 'joint_1']['x']}
+             ${offsets[prefix + 'joint_1']['y']}
+             ${offsets[prefix + 'joint_1']['z'] + positioner_height}"
+        rpy=
+            "${offsets[prefix + 'joint_1']['roll']}
+             ${offsets[prefix + 'joint_1']['pitch']}
+             ${offsets[prefix + 'joint_1']['yaw']}"
     />
     <axis xyz="0 0 1" />
@@ -95,6 +101,15 @@
   </joint>
   <joint name="positioner/base" type="fixed">
-    <origin xyz="0 0 ${table_thickness}" rpy="0 0 0"/>
-    <parent link="${prefix}link_1"/>
+    <origin
+        xyz=
+            "${offsets[prefix + 'joint_1']['x']}
+             ${offsets[prefix + 'joint_1']['y']}
+             ${offsets[prefix + 'joint_1']['z'] + positioner_height + table_thickness}"
+        rpy=
+            "${offsets[prefix + 'joint_1']['roll']}
+             ${offsets[prefix + 'joint_1']['pitch']}
+             ${offsets[prefix + 'joint_1']['yaw']}"
+    />
+    <parent link="${prefix}base_link"/>
     <child link="positioner/base"/>
   </joint>

Commit message: ENG-104 Updated D500 to have standard frames

File: motoman_motopos_d500_support/urdf/motopos_d500_macro.xacro (robot description, xacro)
@@ -42,4 +42,5 @@
     </collision>
   </link>
+  <link name="${prefix}flange"/>
   <link name="${prefix}tool0"/>
   <!-- end of link list -->
@@ -59,7 +60,12 @@
     <limit lower="-3.4906" upper="3.4906" effort="392" velocity="2.7925"/>
   </joint>
-  <joint name="${prefix}joint_2-tool0" type="fixed">
-    <origin xyz="0 0 0.150 " rpy="0 0 0"/>
-    <parent link="${prefix}link_2"/>
+  <joint name="${prefix}joint_2-flange" type="fixed">
+    <origin xyz="0 0 0.150" rpy="0 0 0"/>
+    <parent link="${prefix}link_1"/>
+    <child link="${prefix}flange"/>
+  </joint>
+  <joint name="${prefix}flange-tool0" type="fixed">
+    <origin xyz="0 0 0" rpy="${pi} ${-pi/2} 0"/>
+    <parent link="${prefix}flange"/>
     <child link="${prefix}tool0"/>
   </joint>

Commit message: ENG-104 Fixed issues with d500 macro.

File: motoman_motopos_d500_support/urdf/motopos_d500_macro.xacro (robot description, xacro)
@@ -2,4 +2,5 @@
 <robot xmlns:xacro="http://ros.org/wiki/xacro">
 <xacro:macro name="motoman_motopos_d500" params="prefix">
+  <xacro:include filename="$(find motoman_resources)/urdf/common_materials.xacro"/>
   <!-- link list -->
   <link name="${prefix}base_link">
@@ -8,5 +9,5 @@
         <mesh filename="package://motoman_motopos_d500_support/meshes/motopos_d500/visual/base_link.stl"/>
       </geometry>
-      <material name="yaskawa_blue"/>
+      <xacro:material_yaskawa_blue/>
     </visual>
     <collision>
@@ -21,5 +22,5 @@
         <mesh filename="package://motoman_motopos_d500_support/meshes/motopos_d500/visual/link_1.stl"/>
       </geometry>
-      <material name="yaskawa_blue"/>
+      <xacro:material_yaskawa_blue/>
     </visual>
     <collision>
@@ -34,5 +35,5 @@
         <mesh filename="package://motoman_motopos_d500_support/meshes/motopos_d500/visual/link_2.stl"/>
       </geometry>
-      <material name="yaskawa_blue"/>
+      <xacro:material_yaskawa_blue/>
     </visual>
     <collision>
@@ -61,10 +62,10 @@
   </joint>
   <joint name="${prefix}joint_2-flange" type="fixed">
-    <origin xyz="0 0 0.150" rpy="0 0 0"/>
-    <parent link="${prefix}link_1"/>
+    <origin xyz="0 0 0.150" rpy="0 ${-pi/2} 0"/>
+    <parent link="${prefix}link_2"/>
     <child link="${prefix}flange"/>
   </joint>
   <joint name="${prefix}flange-tool0" type="fixed">
-    <origin xyz="0 0 0" rpy="${pi} ${-pi/2} 0"/>
+    <origin xyz="0 0 0" rpy="0 ${pi/2} 0"/>
     <parent link="${prefix}flange"/>
     <child link="${prefix}tool0"/>

Commit message: update d500 joint limits

File: motoman_motopos_d500_support/urdf/motopos_d500_macro.xacro (robot description, xacro)
@@ -53,5 +53,5 @@
             rpy="${0 + kinematic_offsets['link_1']['roll']} ${0 + kinematic_offsets['link_1']['pitch']} ${0 + kinematic_offsets['link_1']['yaw']}" />
     <axis xyz="0 -1 0" />
-    <limit lower="-2.3561" upper="2.3561" effort="1274" velocity="1.3962"/>
+    <limit lower="-1.51" upper="1.51" effort="1274" velocity="1.3962"/>
   </joint>
   <joint name="${prefix}joint_2" type="revolute">

Commit message: change by 0.01

File: motoman_motopos_d500_support/urdf/motopos_d500_macro.xacro (robot description, xacro)
@@ -53,5 +53,5 @@
             rpy="${0 + kinematic_offsets['link_1']['roll']} ${0 + kinematic_offsets['link_1']['pitch']} ${0 + kinematic_offsets['link_1']['yaw']}" />
     <axis xyz="0 -1 0" />
-    <limit lower="-1.51" upper="1.51" effort="1274" velocity="1.3962"/>
+    <limit lower="-1.50" upper="1.50" effort="1274" velocity="1.3962"/>
   </joint>
   <joint name="${prefix}joint_2" type="revolute">

Commit message: updated formatting

File: motoman_motopos_d500_support/urdf/motopos_d500_macro.xacro (robot description, xacro)
@@ -1,84 +1,84 @@
 <?xml version="1.0" ?>
 <robot xmlns:xacro="http://ros.org/wiki/xacro">
-<xacro:macro name="motoman_motopos_d500" params="prefix kinematic_offsets">
-  <xacro:include filename="$(find motoman_resources)/urdf/common_materials.xacro"/>
-  <!-- link list -->
-  <link name="${prefix}base_link">
-    <visual>
-      <geometry>
-        <mesh filename="package://motoman_motopos_d500_support/meshes/motopos_d500/visual/base_link.stl"/>
-      </geometry>
-      <xacro:material_yaskawa_blue/>
-    </visual>
-    <collision>
-      <geometry>
-        <mesh filename="package://motoman_motopos_d500_support/meshes/motopos_d500/collision/base_link.stl"/>
-      </geometry>
-    </collision>
-  </link>
-  <link name="${prefix}link_1">
-    <visual>
-      <geometry>
-        <mesh filename="package://motoman_motopos_d500_support/meshes/motopos_d500/visual/link_1.stl"/>
-      </geometry>
-      <xacro:material_yaskawa_blue/>
-    </visual>
-    <collision>
-      <geometry>
-        <mesh filename="package://motoman_motopos_d500_support/meshes/motopos_d500/collision/link_1.stl"/>
-      </geometry>
-    </collision>
-  </link>
-  <link name="${prefix}link_2">
-    <visual>
-      <geometry>
-        <mesh filename="package://motoman_motopos_d500_support/meshes/motopos_d500/visual/link_2.stl"/>
-      </geometry>
-      <xacro:material_yaskawa_blue/>
-    </visual>
-    <collision>
-      <geometry>
-        <mesh filename="package://motoman_motopos_d500_support/meshes/motopos_d500/collision/link_2.stl"/>
-      </geometry>
-    </collision>
-  </link>
-  <link name="${prefix}flange"/>
-  <link name="${prefix}tool0"/>
-  <!-- end of link list -->
-  <!-- joint list -->
-  <joint name="${prefix}joint_1" type="revolute">
-    <parent link="${prefix}base_link"/>
-    <child link="${prefix}link_1"/>
-    <origin xyz="${0 + kinematic_offsets['link_1']['x']} ${0 + kinematic_offsets['link_1']['y']} ${0.380 + kinematic_offsets['link_1']['z']}"
-            rpy="${0 + kinematic_offsets['link_1']['roll']} ${0 + kinematic_offsets['link_1']['pitch']} ${0 + kinematic_offsets['link_1']['yaw']}" />
-    <axis xyz="0 -1 0" />
-    <limit lower="-1.50" upper="1.50" effort="1274" velocity="1.3962"/>
-  </joint>
-  <joint name="${prefix}joint_2" type="revolute">
-    <parent link="${prefix}link_1"/>
-    <child link="${prefix}link_2"/>
-    <origin xyz="${0 + kinematic_offsets['link_2']['x']} ${0 + kinematic_offsets['link_2']['y']} ${0 + kinematic_offsets['link_2']['z']}"
-            rpy="${0 + kinematic_offsets['link_2']['roll']} ${0 + kinematic_offsets['link_2']['pitch']} ${0 + kinematic_offsets['link_2']['yaw']}" />
-    <axis xyz="0 0 -1" />
-    <limit lower="-10" upper="10" effort="392" velocity="2.7925"/>
-  </joint>
-  <joint name="${prefix}joint_2-flange" type="fixed">
-    <origin xyz="0 0 0.150" rpy="0 ${-pi/2} 0"/>
-    <parent link="${prefix}link_2"/>
-    <child link="${prefix}flange"/>
-  </joint>
-  <joint name="${prefix}flange-tool0" type="fixed">
-    <origin xyz="0 0 0" rpy="0 ${pi/2} 0"/>
-    <parent link="${prefix}flange"/>
-    <child link="${prefix}tool0"/>
-  </joint>
-  <!-- end of joint list -->
-  <!-- ROS base_link to Robot Manufacturer World Coordinates transform -->
-  <link name="${prefix}base" />
-  <joint name="${prefix}base_link-base" type="fixed">
-    <origin xyz="0 0 0.380" rpy="0 0 0"/>
-    <parent link="${prefix}base_link"/>
-    <child link="${prefix}base"/>
-  </joint>
+  <xacro:macro name="motoman_motopos_d500" params="prefix kinematic_offsets">
+    <xacro:include filename="$(find motoman_resources)/urdf/common_materials.xacro"/>
+    <!-- link list -->
+    <link name="${prefix}base_link">
+      <visual>
+        <geometry>
+          <mesh filename="package://motoman_motopos_d500_support/meshes/motopos_d500/visual/base_link.stl"/>
+        </geometry>
+        <xacro:material_yaskawa_blue/>
+      </visual>
+      <collision>
+        <geometry>
+          <mesh filename="package://motoman_motopos_d500_support/meshes/motopos_d500/collision/base_link.stl"/>
+        </geometry>
+      </collision>
+    </link>
+    <link name="${prefix}link_1">
+      <visual>
+        <geometry>
+          <mesh filename="package://motoman_motopos_d500_support/meshes/motopos_d500/visual/link_1.stl"/>
+        </geometry>
+        <xacro:material_yaskawa_blue/>
+      </visual>
+      <collision>
+        <geometry>
+          <mesh filename="package://motoman_motopos_d500_support/meshes/motopos_d500/collision/link_1.stl"/>
+        </geometry>
+      </collision>
+    </link>
+    <link name="${prefix}link_2">
+      <visual>
+        <geometry>
+          <mesh filename="package://motoman_motopos_d500_support/meshes/motopos_d500/visual/link_2.stl"/>
+        </geometry>
+        <xacro:material_yaskawa_blue/>
+      </visual>
+      <collision>
+        <geometry>
+          <mesh filename="package://motoman_motopos_d500_support/meshes/motopos_d500/collision/link_2.stl"/>
+        </geometry>
+      </collision>
+    </link>
+    <link name="${prefix}flange"/>
+    <link name="${prefix}tool0"/>
+    <!-- end of link list -->
+    <!-- joint list -->
+    <joint name="${prefix}joint_1" type="revolute">
+      <parent link="${prefix}base_link"/>
+      <child link="${prefix}link_1"/>
+      <origin xyz="${0 + kinematic_offsets['link_1']['x']} ${0 + kinematic_offsets['link_1']['y']} ${0.380 + kinematic_offsets['link_1']['z']}"
+              rpy="${0 + kinematic_offsets['link_1']['roll']} ${0 + kinematic_offsets['link_1']['pitch']} ${0 + kinematic_offsets['link_1']['yaw']}"/>
+      <axis xyz="0 -1 0"/>
+      <limit lower="-1.50" upper="1.50" effort="1274" velocity="1.3962"/>
+    </joint>
+    <joint name="${prefix}joint_2" type="revolute">
+      <parent link="${prefix}link_1"/>
+      <child link="${prefix}link_2"/>
+      <origin xyz="${0 + kinematic_offsets['link_2']['x']} ${0 + kinematic_offsets['link_2']['y']} ${0 + kinematic_offsets['link_2']['z']}"
+              rpy="${0 + kinematic_offsets['link_2']['roll']} ${0 + kinematic_offsets['link_2']['pitch']} ${0 + kinematic_offsets['link_2']['yaw']}"/>
+      <axis xyz="0 0 -1"/>
+      <limit lower="-10" upper="10" effort="392" velocity="2.7925"/>
+    </joint>
+    <joint name="${prefix}joint_2-flange" type="fixed">
+      <origin xyz="0 0 0.150" rpy="0 ${-pi/2} 0"/>
+      <parent link="${prefix}link_2"/>
+      <child link="${prefix}flange"/>
+    </joint>
+    <joint name="${prefix}flange-tool0" type="fixed">
+      <origin xyz="0 0 0" rpy="0 ${pi/2} 0"/>
+      <parent link="${prefix}flange"/>
+      <child link="${prefix}tool0"/>
+    </joint>
+    <!-- end of joint list -->
+    <!-- ROS base_link to Robot Manufacturer World Coordinates transform -->
+    <link name="${prefix}base"/>
+    <joint name="${prefix}base_link-base" type="fixed">
+      <origin xyz="0 0 0.380" rpy="0 0 0"/>
+      <parent link="${prefix}base_link"/>
+      <child link="${prefix}base"/>
+    </joint>
   </xacro:macro>
 </robot>
