Commit message: updated mh1655 to include kinematic offsets and material color

File: motoman_motopos_mh1655_support/urdf/motopos_mh1655.xacro (robot description, xacro)
@@ -1,5 +1,11 @@
 <?xml version="1.0" ?>
 <robot name="motoman_motopos_mh1655" xmlns:xacro="http://ros.org/wiki/xacro">
+  <!-- Properties -->
+  <material name="yaskawa_blue">
+    <color rgba="0.12941 0.14902 0.74902 1" />
+  </material>
   <xacro:include filename="$(find motoman_motopos_mh1655_support)/urdf/motopos_mh1655_macro.xacro" />
+  <xacro:property name="kinematics_offsets" value="${load_yaml('$(find motoman_motopos_mh1655_support)' + '/config/default_kinematic_offsets.yaml')}"/>
+  <xacro:motoman_motopos_d500 prefix="" kinematic_offsets="${kinematics_offsets['kinematic_offsets']}"/>
   <xacro:motoman_motopos_mh1655 prefix="" use_pedestal="false"/>
 </robot>

File: motoman_motopos_mh1655_support/urdf/motopos_mh1655_macro.xacro (robot description, xacro)
@@ -1,5 +1,5 @@
 <?xml version="1.0" ?>
 <robot xmlns:xacro="http://ros.org/wiki/xacro">
-  <xacro:macro name="motoman_motopos_mh1655" params="prefix use_pedestal:=false">
+  <xacro:macro name="motoman_motopos_mh1655" params="prefix use_pedestal:=false kinematic_offsets">
     <xacro:include filename="$(find motoman_resources)/urdf/common_materials.xacro"/>
     <!-- link list -->
@@ -51,5 +51,6 @@
       <parent link="${prefix}base_link"/>
       <child link="${prefix}link_1"/>
-      <origin xyz="0 0 0.305" rpy="0 0 0"/>
+      <origin xyz="${0 + kinematic_offsets['link_1']['x']} ${0 + kinematic_offsets['link_1']['y']} ${0.305 + kinematic_offsets['link_1']['z']}"
+              rpy="${0 + kinematic_offsets['link_1']['roll']} ${0 + kinematic_offsets['link_1']['pitch']} ${0 + kinematic_offsets['link_1']['yaw']}"/>
       <axis xyz="1 0 0"/>
       <limit lower="${-2*pi}" upper="${2*pi}" effort="1274" velocity="1.3962"/>
