Commit message: fixed joint axis

File: motoman_motopos_mh1655_support/urdf/motopos_mh1655_macro.xacro (robot description, xacro)
@@ -52,6 +52,6 @@
       <child link="${prefix}link_1"/>
       <origin xyz="${0 + kinematic_offsets['link_1']['x']} ${0 + kinematic_offsets['link_1']['y']} ${0.305 + kinematic_offsets['link_1']['z']}"
-              rpy="${0 + kinematic_offsets['link_1']['roll']} ${0 + kinematic_offsets['link_1']['pitch']} ${0 + kinematic_offsets['link_1']['yaw']}"/>
-      <axis xyz="1 0 0"/>
+              rpy="${pi + kinematic_offsets['link_1']['roll']} ${-pi/2 + kinematic_offsets['link_1']['pitch']} ${0 + kinematic_offsets['link_1']['yaw']}"/>
+      <axis xyz="0 0 1"/>
       <limit lower="${-2*pi}" upper="${2*pi}" effort="1274" velocity="1.3962"/>
     </joint>
@@ -67,5 +67,5 @@
     <link name="${prefix}flange"/>
     <joint name="${prefix}joint_1-flange" type="fixed">
-      <origin xyz="0.2768 0 0" rpy="0 0 0"/>
+      <origin xyz="0 0 0.2768" rpy="0 0 0"/>
       <parent link="${prefix}link_1"/>
       <child link="${prefix}flange"/>
@@ -74,5 +74,5 @@
     <link name="${prefix}tool0"/>
     <joint name="${prefix}flange-tool0" type="fixed">
-      <origin xyz="0 0 0" rpy="${pi} ${-pi/2} 0"/>
+      <origin xyz="0 0 0" rpy="0 0 0"/>
       <parent link="${prefix}flange"/>
       <child link="${prefix}tool0"/>

Commit message: improved conditional pedestal

File: motoman_motopos_mh1655_support/urdf/motopos_mh1655_macro.xacro (robot description, xacro)
@@ -3,4 +3,5 @@
   <xacro:macro name="motoman_motopos_mh1655" params="prefix use_pedestal:=false kinematic_offsets">
     <xacro:include filename="$(find motoman_resources)/urdf/common_materials.xacro"/>
+    <xacro:property name="pedestal_offset" value="0.695" />
     <!-- link list -->
     <link name="${prefix}base_link">
@@ -9,4 +10,7 @@
           <mesh filename="package://motoman_motopos_mh1655_support/meshes/motopos_mh1655/visual/base_link.stl"/>
         </geometry>
+        <xacro:if value="${use_pedestal}">
+          <origin xyz="0 0 ${pedestal_offset}" rpy="0 0 0"/>
+        </xacro:if>
         <xacro:material_yaskawa_blue/>
       </visual>
@@ -15,4 +19,7 @@
           <mesh filename="package://motoman_motopos_mh1655_support/meshes/motopos_mh1655/collision/base_link.stl"/>
         </geometry>
+        <xacro:if value="${use_pedestal}">
+          <origin xyz="0 0 ${pedestal_offset}" rpy="0 0 0"/>
+        </xacro:if>
       </collision>
       <xacro:if value="${use_pedestal}">
@@ -22,4 +29,5 @@
             <mesh filename="package://motoman_motopos_mh1655_support/meshes/motopos_mh1655/visual/pedestal.stl"/>
           </geometry>
+          <origin xyz="0 0 ${pedestal_offset}" rpy="0 0 0"/>
           <xacro:material_yaskawa_blue/>
         </visual>
@@ -28,4 +36,5 @@
             <mesh filename="package://motoman_motopos_mh1655_support/meshes/motopos_mh1655/collision/pedestal.stl"/>
           </geometry>
+          <origin xyz="0 0 ${pedestal_offset}" rpy="0 0 0"/>
         </collision>
       </xacro:if>
@@ -51,5 +60,5 @@
       <parent link="${prefix}base_link"/>
       <child link="${prefix}link_1"/>
-      <origin xyz="${0 + kinematic_offsets['link_1']['x']} ${0 + kinematic_offsets['link_1']['y']} ${0.305 + kinematic_offsets['link_1']['z']}"
+      <origin xyz="${0 + kinematic_offsets['link_1']['x']} ${0 + kinematic_offsets['link_1']['y']} ${pedestal_offset + 0.305 + kinematic_offsets['link_1']['z']}"
               rpy="${pi + kinematic_offsets['link_1']['roll']} ${-pi/2 + kinematic_offsets['link_1']['pitch']} ${0 + kinematic_offsets['link_1']['yaw']}"/>
       <axis xyz="0 0 1"/>
