Commit message: Fix gp20hl_macro.xacro for link_4_r

File: motoman_gp20hl_support/urdf/gp20hl_macro.xacro (robot description, xacro)
@@ -125,5 +125,5 @@
       <parent link="${prefix}link_3_u"/>
       <child link="${prefix}link_4_r"/>
-      <origin xyz="${0.250 + kinematic_offsets['4_r']['x']} ${0 + kinematic_offsets['4_r']['y']} ${0 + kinematic_offsets['4_r']['z']}"
+      <origin xyz="${0.250 + kinematic_offsets['4_r']['x']} ${-1.812 + kinematic_offsets['4_r']['y']} ${0 + kinematic_offsets['4_r']['z']}"
               rpy="${radians(-90) + kinematic_offsets['4_r']['roll']} ${0 + kinematic_offsets['4_r']['pitch']} ${0 + kinematic_offsets['4_r']['yaw']}"/>
       <axis xyz="0 0 1"/>
@@ -133,5 +133,5 @@
       <parent link="${prefix}link_4_r"/>
       <child link="${prefix}link_5_b"/>
-      <origin xyz="${0 + kinematic_offsets['5_b']['x']} ${0 + kinematic_offsets['5_b']['y']} ${-1.812 + kinematic_offsets['5_b']['z']}"
+      <origin xyz="${0 + kinematic_offsets['5_b']['x']} ${0 + kinematic_offsets['5_b']['y']} ${0 + kinematic_offsets['5_b']['z']}"
               rpy="${radians(90) + kinematic_offsets['5_b']['roll']} ${0 + kinematic_offsets['5_b']['pitch']} ${0 + kinematic_offsets['5_b']['yaw']}"/>
       <axis xyz="0 0 1"/>

Commit message: update meshes and kinematic parameters to reflect DH param frame origins

File: motoman_gp20hl_support/urdf/gp20hl_macro.xacro (robot description, xacro)
@@ -110,5 +110,5 @@
       <child link="${prefix}link_2_l"/>
       <origin xyz="${0.145 + kinematic_offsets['2_l']['x']} ${0 + kinematic_offsets['2_l']['y']} ${0 + kinematic_offsets['2_l']['z']}"
-              rpy="${radians(90) + kinematic_offsets['2_l']['roll']} ${radians(-90) + kinematic_offsets['2_l']['pitch']} ${radians(-180) + kinematic_offsets['2_l']['yaw']}"/>
+              rpy="${0 + kinematic_offsets['2_l']['roll']} ${radians(-90) + kinematic_offsets['2_l']['pitch']} ${radians(-90) + kinematic_offsets['2_l']['yaw']}"/>
       <axis xyz="0 0 1"/>
       <limit lower="${radians(-90)}" upper="${radians(135)}" effort="3087" velocity="${radians(180)}"/>
@@ -125,5 +125,5 @@
       <parent link="${prefix}link_3_u"/>
       <child link="${prefix}link_4_r"/>
-      <origin xyz="${0.250 + kinematic_offsets['4_r']['x']} ${0 + kinematic_offsets['4_r']['y']} ${0 + kinematic_offsets['4_r']['z']}"
+      <origin xyz="${0.250 + kinematic_offsets['4_r']['x']} ${-1.812 + kinematic_offsets['4_r']['y']} ${0 + kinematic_offsets['4_r']['z']}"
               rpy="${radians(-90) + kinematic_offsets['4_r']['roll']} ${0 + kinematic_offsets['4_r']['pitch']} ${0 + kinematic_offsets['4_r']['yaw']}"/>
       <axis xyz="0 0 1"/>
@@ -133,5 +133,5 @@
       <parent link="${prefix}link_4_r"/>
       <child link="${prefix}link_5_b"/>
-      <origin xyz="${0 + kinematic_offsets['5_b']['x']} ${0 + kinematic_offsets['5_b']['y']} ${-1.812 + kinematic_offsets['5_b']['z']}"
+      <origin xyz="${0 + kinematic_offsets['5_b']['x']} ${0 + kinematic_offsets['5_b']['y']} ${0 + kinematic_offsets['5_b']['z']}"
               rpy="${radians(90) + kinematic_offsets['5_b']['roll']} ${0 + kinematic_offsets['5_b']['pitch']} ${0 + kinematic_offsets['5_b']['yaw']}"/>
       <axis xyz="0 0 1"/>
@@ -144,5 +144,5 @@
               rpy="${radians(-90) + kinematic_offsets['6_t']['roll']} ${0 + kinematic_offsets['6_t']['pitch']} ${0 + kinematic_offsets['6_t']['yaw']}"/>
       <axis xyz="0 0 1"/>
-      <limit lower="${radians(-455)}" upper="${radians(455)}" effort="19.6" velocity="${radians(700)}"/>
+      <limit lower="${radians(-210)}" upper="${radians(210)}" effort="19.6" velocity="${radians(700)}"/>
     </joint>
     <!-- end of joint list -->
