Commit message: Added calibration offsets to AR2010

File: motoman_ar2010_support/urdf/ar2010.xacro (robot description, xacro)
@@ -2,4 +2,5 @@
 <robot name="motoman_ar2010" xmlns:xacro="http://ros.org/wiki/xacro">
 	<xacro:include filename="$(find motoman_ar2010_support)/urdf/ar2010_macro.xacro" />
-	<xacro:motoman_ar2010 prefix=""/>
+	<xacro:property name="kinematics_offsets" value="${load_yaml('$(find motoman_ar2010_support)' + '/config/default_kinematic_offsets.yaml')}"/>
+	<xacro:motoman_ar2010 prefix="" kinematic_offsets="${kinematics_offsets['kinematic_offsets']}"/>
 </robot>

File: motoman_ar2010_support/urdf/ar2010_macro.xacro (robot description, xacro)
@@ -1,5 +1,5 @@
 <?xml version="1.0" ?>
 <robot xmlns:xacro="http://ros.org/wiki/xacro">
-  <xacro:macro name="motoman_ar2010" params="prefix">
+  <xacro:macro name="motoman_ar2010" params="prefix kinematic_offsets">
     <xacro:include filename="$(find motoman_resources)/urdf/common_materials.xacro"/>
     <!-- link list -->
@@ -101,5 +101,6 @@
       <parent link="${prefix}base_link"/>
       <child link="${prefix}link_1_s"/>
-      <origin xyz="0 0 0.505" rpy="0 0 0"/>
+      <origin xyz="${0 + kinematic_offsets['1_s']['x']} ${0 + kinematic_offsets['1_s']['y']} ${0.505 + kinematic_offsets['1_s']['z']}"
+              rpy="${0 + kinematic_offsets['1_s']['roll']} ${0 + kinematic_offsets['1_s']['pitch']} ${0 + kinematic_offsets['1_s']['yaw']}"/>
       <axis xyz="0 0 1"/>
       <limit lower="${radians(-180)}" upper="${radians(180)}" effort="3087" velocity="${radians(210)}"/>
@@ -108,5 +109,6 @@
       <parent link="${prefix}link_1_s"/>
       <child link="${prefix}link_2_l"/>
-      <origin xyz="0.150 0 0" rpy="${pi/2} ${-pi/2} ${-pi}"/>
+      <origin xyz="${0.150 + kinematic_offsets['2_l']['x']} ${0 + kinematic_offsets['2_l']['y']} ${0 + kinematic_offsets['2_l']['z']}"
+              rpy="${radians(90) + kinematic_offsets['2_l']['roll']} ${radians(-90) + kinematic_offsets['2_l']['pitch']} ${radians(-180) + kinematic_offsets['2_l']['yaw']}"/>
       <axis xyz="0 0 1"/>
       <limit lower="${radians(-105)}" upper="${radians(155)}" effort="3087" velocity="${radians(210)}"/>
@@ -115,5 +117,6 @@
       <parent link="${prefix}link_2_l"/>
       <child link="${prefix}link_3_u"/>
-      <origin xyz="0.760 0 0" rpy="${pi} 0 0"/>
+      <origin xyz="${0.760 + kinematic_offsets['3_u']['x']} ${0 + kinematic_offsets['3_u']['y']} ${0 + kinematic_offsets['3_u']['z']}"
+              rpy="${radians(180) + kinematic_offsets['3_u']['roll']} ${0 + kinematic_offsets['3_u']['pitch']} ${0 + kinematic_offsets['3_u']['yaw']}"/>
       <axis xyz="0 0 1"/>
       <limit lower="${radians(-86)}" upper="${radians(160)}" effort="926.1" velocity="${radians(220)}"/>
@@ -122,5 +125,6 @@
       <parent link="${prefix}link_3_u"/>
       <child link="${prefix}link_4_r"/>
-      <origin xyz="0.200 0 0" rpy="${-pi/2} 0 0"/>
+      <origin xyz="${0.200 + kinematic_offsets['4_r']['x']} ${0 + kinematic_offsets['4_r']['y']} ${0 + kinematic_offsets['4_r']['z']}"
+              rpy="${radians(-90) + kinematic_offsets['4_r']['roll']} ${0 + kinematic_offsets['4_r']['pitch']} ${0 + kinematic_offsets['4_r']['yaw']}"/>
       <axis xyz="0 0 1"/>
       <limit lower="${radians(-150)}" upper="${radians(150)}" effort="78.4" velocity="${radians(435)}"/>
@@ -129,5 +133,6 @@
       <parent link="${prefix}link_4_r"/>
       <child link="${prefix}link_5_b"/>
-      <origin xyz="0 0 -1.082" rpy="${pi/2} 0 0"/>
+      <origin xyz="${0 + kinematic_offsets['5_b']['x']} ${0 + kinematic_offsets['5_b']['y']} ${-1.082 + kinematic_offsets['5_b']['z']}"
+              rpy="${radians(90) + kinematic_offsets['5_b']['roll']} ${0 + kinematic_offsets['5_b']['pitch']} ${0 + kinematic_offsets['5_b']['yaw']}"/>
       <axis xyz="0 0 1"/>
       <limit lower="${radians(-135)}" upper="${radians(90)}" effort="67.03" velocity="${radians(435)}"/>
@@ -136,5 +141,6 @@
       <parent link="${prefix}link_5_b"/>
       <child link="${prefix}link_6_t"/>
-      <origin xyz="0 0 0" rpy="${-pi/2} 0 0"/>
+      <origin xyz="${0 + kinematic_offsets['6_t']['x']} ${0 + kinematic_offsets['6_t']['y']} ${0 + kinematic_offsets['6_t']['z']}"
+              rpy="${radians(-90) + kinematic_offsets['6_t']['roll']} ${0 + kinematic_offsets['6_t']['pitch']} ${0 + kinematic_offsets['6_t']['yaw']}"/>
       <axis xyz="0 0 1"/>
       <limit lower="${radians(-210)}" upper="${radians(210)}" effort="33.3" velocity="${radians(700)}"/>

Commit message: fix load_yaml() warning

File: motoman_ar2010_support/urdf/ar2010.xacro (robot description, xacro)
@@ -2,5 +2,5 @@
 <robot name="motoman_ar2010" xmlns:xacro="http://ros.org/wiki/xacro">
 	<xacro:include filename="$(find motoman_ar2010_support)/urdf/ar2010_macro.xacro" />
-	<xacro:property name="kinematics_offsets" value="${load_yaml('$(find motoman_ar2010_support)' + '/config/default_kinematic_offsets.yaml')}"/>
+	<xacro:property name="kinematics_offsets" value="${xacro.load_yaml('$(find motoman_ar2010_support)' + '/config/default_kinematic_offsets.yaml')}"/>
 	<xacro:motoman_ar2010 prefix="" kinematic_offsets="${kinematics_offsets['kinematic_offsets']}"/>
 </robot>

File: motoman_gp180_support/urdf/gp180.xacro (robot description, xacro)
@@ -2,5 +2,5 @@
 <robot name="motoman_gp180" xmlns:xacro="http://ros.org/wiki/xacro">
     <xacro:include filename="$(find motoman_gp180_support)/urdf/gp180_macro.xacro" />
-    <xacro:property name="kinematics_offsets" value="${load_yaml('$(find motoman_gp180_support)' + '/config/default_kinematic_offsets.yaml')}"/>
+    <xacro:property name="kinematics_offsets" value="${xacro.load_yaml('$(find motoman_gp180_support)' + '/config/default_kinematic_offsets.yaml')}"/>
     <xacro:motoman_gp180 prefix="" kinematic_offsets="${kinematics_offsets['kinematic_offsets']}"/>
 </robot>

File: motoman_gp20hl_support/urdf/gp20hl.xacro (robot description, xacro)
@@ -2,5 +2,5 @@
 <robot name="motoman_gp20hl" xmlns:xacro="http://ros.org/wiki/xacro">
 	<xacro:include filename="$(find motoman_gp20hl_support)/urdf/gp20hl_macro.xacro" />
-	<xacro:property name="kinematics_offsets" value="${load_yaml('$(find motoman_gp20hl_support)' + '/config/default_kinematic_offsets.yaml')}"/>
+	<xacro:property name="kinematics_offsets" value="${xacro.load_yaml('$(find motoman_gp20hl_support)' + '/config/default_kinematic_offsets.yaml')}"/>
 	<xacro:motoman_gp20hl prefix="" kinematic_offsets="${kinematics_offsets['kinematic_offsets']}"/>
 </robot>

File: motoman_motopos_d500_support/urdf/motopos_d500.xacro (robot description, xacro)
@@ -6,5 +6,5 @@
   </material>
   <xacro:include filename="$(find motoman_motopos_d500_support)/urdf/motopos_d500_macro.xacro" />
-  <xacro:property name="kinematics_offsets" value="${load_yaml('$(find motoman_motopos_d500_support)' + '/config/default_kinematic_offsets.yaml')}"/>
+  <xacro:property name="kinematics_offsets" value="${xacro.load_yaml('$(find motoman_motopos_d500_support)' + '/config/default_kinematic_offsets.yaml')}"/>
   <xacro:motoman_motopos_d500 prefix="" kinematic_offsets="${kinematics_offsets['kinematic_offsets']}"/>
 </robot>

File: motoman_motopos_mh1655_support/urdf/motopos_mh1655.xacro (robot description, xacro)
@@ -6,5 +6,5 @@
   </material>
   <xacro:include filename="$(find motoman_motopos_mh1655_support)/urdf/motopos_mh1655_macro.xacro" />
-  <xacro:property name="kinematics_offsets" value="${load_yaml('$(find motoman_motopos_mh1655_support)' + '/config/default_kinematic_offsets.yaml')}"/>
+  <xacro:property name="kinematics_offsets" value="${xacro.load_yaml('$(find motoman_motopos_mh1655_support)' + '/config/default_kinematic_offsets.yaml')}"/>
   <xacro:motoman_motopos_mh1655 prefix="" use_pedestal="false" kinematic_offsets="${kinematics_offsets['kinematic_offsets']}"/>
 </robot>
