Commit message: Offset t-link orientation by 0.1 to match old urdf

File: motoman_ar2010_support/urdf/ar2010_macro.xacro (robot description, xacro)
@@ -141,5 +141,5 @@
       <parent link="${prefix}link_5_b"/>
       <child link="${prefix}link_6_t"/>
-      <origin xyz="${0 + kinematic_offsets['6_t']['x']} ${0 + kinematic_offsets['6_t']['y']} ${0 + kinematic_offsets['6_t']['z']}"
+      <origin xyz="${0 + kinematic_offsets['6_t']['x']} ${-0.1 + kinematic_offsets['6_t']['y']} ${0 + kinematic_offsets['6_t']['z']}"
               rpy="${radians(-90) + kinematic_offsets['6_t']['roll']} ${0 + kinematic_offsets['6_t']['pitch']} ${0 + kinematic_offsets['6_t']['yaw']}"/>
       <axis xyz="0 0 1"/>
@@ -157,5 +157,5 @@
     <link name="${prefix}flange"/>
     <joint name="${prefix}joint_6_t-flange" type="fixed">
-      <origin xyz="0 0 -0.100" rpy="0 ${pi/2} 0"/>
+      <origin xyz="0 0 0" rpy="0 ${pi/2} 0"/>
       <parent link="${prefix}link_6_t"/>
       <child link="${prefix}flange"/>

Commit message: fixed discrepancy in nominal urdf's xyzrpy coordinates

File: motoman_ar2010_support/urdf/ar2010_macro.xacro (robot description, xacro)
@@ -110,5 +110,5 @@
       <child link="${prefix}link_2_l"/>
       <origin xyz="${0.150 + kinematic_offsets['2_l']['x']} ${0 + kinematic_offsets['2_l']['y']} ${0 + kinematic_offsets['2_l']['z']}"
-              rpy="${radians(90) + kinematic_offsets['2_l']['roll']} ${radians(-90) + kinematic_offsets['2_l']['pitch']} ${radians(-180) + kinematic_offsets['2_l']['yaw']}"/>
+              rpy="${0 + kinematic_offsets['2_l']['roll']} ${radians(-90) + kinematic_offsets['2_l']['pitch']} ${radians(-90) + kinematic_offsets['2_l']['yaw']}"/>
       <axis xyz="0 0 1"/>
       <limit lower="${radians(-105)}" upper="${radians(155)}" effort="3087" velocity="${radians(210)}"/>
@@ -125,5 +125,5 @@
       <parent link="${prefix}link_3_u"/>
       <child link="${prefix}link_4_r"/>
-      <origin xyz="${0.200 + kinematic_offsets['4_r']['x']} ${0 + kinematic_offsets['4_r']['y']} ${0 + kinematic_offsets['4_r']['z']}"
+      <origin xyz="${0.200 + kinematic_offsets['4_r']['x']} ${-1.082 + kinematic_offsets['4_r']['y']} ${0 + kinematic_offsets['4_r']['z']}"
               rpy="${radians(-90) + kinematic_offsets['4_r']['roll']} ${0 + kinematic_offsets['4_r']['pitch']} ${0 + kinematic_offsets['4_r']['yaw']}"/>
       <axis xyz="0 0 1"/>
@@ -133,5 +133,5 @@
       <parent link="${prefix}link_4_r"/>
       <child link="${prefix}link_5_b"/>
-      <origin xyz="${0 + kinematic_offsets['5_b']['x']} ${0 + kinematic_offsets['5_b']['y']} ${-1.082 + kinematic_offsets['5_b']['z']}"
+      <origin xyz="${0 + kinematic_offsets['5_b']['x']} ${0 + kinematic_offsets['5_b']['y']} ${0 + kinematic_offsets['5_b']['z']}"
               rpy="${radians(90) + kinematic_offsets['5_b']['roll']} ${0 + kinematic_offsets['5_b']['pitch']} ${0 + kinematic_offsets['5_b']['yaw']}"/>
       <axis xyz="0 0 1"/>

Commit message: ar2010: remove Gazebo-isms

File: motoman_ar2010_support/urdf/ar2010_macro.xacro (robot description, xacro)
@@ -162,40 +162,4 @@
       <child link="${prefix}tool0"/>
     </joint>
-    <!-- Gazebo -->
-    <gazebo reference="${prefix}base_link">
-      <turnGravityOff>false</turnGravityOff>
-      <selfCollide>true</selfCollide>
-      <material>Gazebo/Blue</material>
-    </gazebo>
-    <gazebo reference="${prefix}link_s">
-      <turnGravityOff>false</turnGravityOff>
-      <selfCollide>true</selfCollide>
-      <material>Gazebo/Blue</material>
-    </gazebo>
-    <gazebo reference="${prefix}link_l">
-      <turnGravityOff>false</turnGravityOff>
-      <selfCollide>true</selfCollide>
-      <material>Gazebo/Blue</material>
-    </gazebo>
-    <gazebo reference="${prefix}link_u">
-      <turnGravityOff>false</turnGravityOff>
-      <selfCollide>true</selfCollide>
-      <material>Gazebo/Blue</material>
-    </gazebo>
-    <gazebo reference="${prefix}link_r">
-      <turnGravityOff>false</turnGravityOff>
-      <selfCollide>true</selfCollide>
-      <material>Gazebo/White</material>
-    </gazebo>
-    <gazebo reference="${prefix}link_b">
-      <turnGravityOff>false</turnGravityOff>
-      <selfCollide>true</selfCollide>
-      <material>Gazebo/Blue</material>
-    </gazebo>
-    <gazebo reference="${prefix}link_t">
-      <turnGravityOff>false</turnGravityOff>
-      <selfCollide>true</selfCollide>
-      <material>Gazebo/White</material>
-    </gazebo>
   </xacro:macro>
 </robot>
