Commit message: Indent with spaces, not tabs

File: motoman_sia30d_support/urdf/sia30d.xacro (robot description, xacro)
@@ -1,5 +1,5 @@
 <?xml version="1.0" ?>
 <robot name="motoman_sia30d" xmlns:xacro="http://ros.org/wiki/xacro">
-	<xacro:include filename="$(find motoman_sia30d_support)/urdf/sia30d_macro.xacro" />
-	<xacro:motoman_sia30d prefix=""/>
+  <xacro:include filename="$(find motoman_sia30d_support)/urdf/sia30d_macro.xacro" />
+  <xacro:motoman_sia30d prefix=""/>
 </robot>

File: motoman_sia30d_support/urdf/sia30d_macro.xacro (robot description, xacro)
@@ -1,182 +1,182 @@
 <?xml version="1.0" ?>
 <robot xmlns:xacro="http://ros.org/wiki/xacro">
-	<xacro:macro name="motoman_sia30d" params="prefix">
-		<!-- Properties -->
-		<material name="yaskawa_blue">
-			<color rgba="0.12941 0.14902 0.74902 1" />
-		</material>
-	    <material name="silver">
-			<color rgba="0.8 0.8 0.8 1"/>
-		</material>
-		<!-- link list -->
-		<link name="${prefix}base_link">
-			<visual>
-				<geometry>
-					<mesh filename="package://motoman_sia30d_support/meshes/visual/base_link.stl"/>
-				</geometry>
-				<material name="yaskawa_blue"/>
-			</visual>
-			<collision>
-				<geometry>
-					<mesh filename="package://motoman_sia30d_support/meshes/collision/base_link.stl"/>
-				</geometry>
-			</collision>
-		</link>
-		<link name="${prefix}link_1_s">
-			<visual>
-				<geometry>
-					<mesh filename="package://motoman_sia30d_support/meshes/visual/link_1_s.stl"/>
-				</geometry>
-				<material name="silver"/>
-			</visual>
-			<collision>
-				<geometry>
-					<mesh filename="package://motoman_sia30d_support/meshes/collision/link_1_s.stl"/>
-				</geometry>
-			</collision>
-		</link>
-		<link name="${prefix}link_2_l">
-			<visual>
-				<geometry>
-					<mesh filename="package://motoman_sia30d_support/meshes/visual/link_2_l.stl"/>
-				</geometry>
-				<material name="yaskawa_blue"/>
-			</visual>
-			<collision>
-				<geometry>
-					<mesh filename="package://motoman_sia30d_support/meshes/collision/link_2_l.stl"/>
-				</geometry>
-			</collision>
-		</link>
-		<link name="${prefix}link_3_e">
-			<visual>
-				<geometry>
-					<mesh filename="package://motoman_sia30d_support/meshes/visual/link_3_e.stl"/>
-				</geometry>
-				<material name="silver"/>
-			</visual>
-			<collision>
-				<geometry>
-					<mesh filename="package://motoman_sia30d_support/meshes/collision/link_3_e.stl"/>
-				</geometry>
-			</collision>
-		</link>
-		<link name="${prefix}link_4_u">
-			<visual>
-				<geometry>
-					<mesh filename="package://motoman_sia30d_support/meshes/visual/link_4_u.stl"/>
-				</geometry>
-				<material name="yaskawa_blue"/>
-			</visual>
-			<collision>
-				<geometry>
-					<mesh filename="package://motoman_sia30d_support/meshes/collision/link_4_u.stl"/>
-				</geometry>
-			</collision>
-		</link>
-		<link name="${prefix}link_5_r">
-			<visual>
-				<geometry>
-					<mesh filename="package://motoman_sia30d_support/meshes/visual/link_5_r.stl"/>
-				</geometry>
-				<material name="silver"/>
-			</visual>
-			<collision>
-				<geometry>
-					<mesh filename="package://motoman_sia30d_support/meshes/collision/link_5_r.stl"/>
-				</geometry>
-			</collision>
-		</link>
-		<link name="${prefix}link_6_b">
-			<visual>
-				<geometry>
-					<mesh filename="package://motoman_sia30d_support/meshes/visual/link_6_b.stl"/>
-				</geometry>
-				<material name="yaskawa_blue"/>
-			</visual>
-			<collision>
-				<geometry>
-					<mesh filename="package://motoman_sia30d_support/meshes/collision/link_6_b.stl"/>
-				</geometry>
-			</collision>
-		</link>
-		<link name="${prefix}link_7_t">
-			<visual>
-				<geometry>
-					<mesh filename="package://motoman_sia30d_support/meshes/visual/link_7_t.stl"/>
-				</geometry>
-				<material name="silver"/>
-			</visual>
-			<collision>
-				<geometry>
-					<mesh filename="package://motoman_sia30d_support/meshes/collision/link_7_t.stl"/>
-				</geometry>
-			</collision>
-		</link>
-		<link name="${prefix}tool0" />
-		<!-- end of link list -->
-		<!-- joint list -->
-		<joint name="${prefix}joint_1_s" type="revolute">
-			<parent link="${prefix}base_link"/>
-			<child link="${prefix}link_1_s"/>
-			<origin xyz="0 0 0.598" rpy="0 0 0" />
-			<axis xyz="0 0 1" />
-			<limit lower="${radians(-180)}" upper="${radians(180)}" effort="1911" velocity="${radians(130)}"/>
-		</joint>
-		<joint name="${prefix}joint_2_l" type="revolute">
-			<parent link="${prefix}link_1_s"/>
-			<child link="${prefix}link_2_l"/>
-			<origin xyz="0 0 0" rpy="0 0 0" />
-			<axis xyz="0 1 0" />
-			<limit lower="${radians(-125)}" upper="${radians(125)}" effort="2388" velocity="${radians(130)}"/>
-		</joint>
-		<joint name="${prefix}joint_3_e" type="revolute">
-			<parent link="${prefix}link_2_l"/>
-			<child link="${prefix}link_3_e"/>
-			<origin xyz="0 0 0.875" rpy="0 0 0" />
-			<axis xyz="0 0 1" />
-			<limit lower="${radians(-170)}" upper="${radians(170)}" effort="674" velocity="${radians(130)}"/>
-		</joint>
-		<joint name="${prefix}joint_4_u" type="revolute">
-			<parent link="${prefix}link_3_e"/>
-			<child link="${prefix}link_4_u"/>
-			<origin xyz="0 0 0" rpy="0 0 0" />
-			<axis xyz="0 -1 0" />
-			<limit lower="${radians(-110)}" upper="${radians(110)}" effort="674" velocity="${radians(130)}"/>
-		</joint>
-		<joint name="${prefix}joint_5_r" type="revolute">
-			<parent link="${prefix}link_4_u"/>
-			<child link="${prefix}link_5_r"/>
-			<origin xyz="0 0 0.610" rpy="0 0 0" />
-			<axis xyz="0 0 -1" />
-			<limit lower="${radians(-170)}" upper="${radians(170)}" effort="191" velocity="${radians(170)}"/>
-		</joint>
-		<joint name="${prefix}joint_6_b" type="revolute">
-			<parent link="${prefix}link_5_r"/>
-			<child link="${prefix}link_6_b"/>
-			<origin xyz="0 0 0" rpy="0 0 0" />
-			<axis xyz="0 -1 0" />
-			<limit lower="${radians(-110)}" upper="${radians(110)}" effort="191" velocity="${radians(170)}"/>
-		</joint>
-		<joint name="${prefix}joint_7_t" type="revolute">
-			<parent link="${prefix}link_6_b"/>
-			<child link="${prefix}link_7_t"/>
-			<origin xyz="0 0 0" rpy="0 0 0" />
-			<axis xyz="0 0 -1" />
-			<limit lower="${radians(-180)}" upper="${radians(180)}" effort="77" velocity="${radians(200)}"/>
-		</joint>
-		<joint name="${prefix}link_7_t-tool0" type="fixed" >
-		  <origin xyz="0 0 0.217" rpy="0 0 ${pi}"/>
-		  <parent link="${prefix}link_7_t" />
-		  <child link="${prefix}tool0" />
-		</joint>
-		<!-- end of joint list -->
-		<!-- ROS base_link to Robot Manufacturer World Coordinates transform -->
-		<link name="${prefix}base" />
-		<joint name="${prefix}base_link-base" type="fixed">
-			<origin xyz="0 0 0.598" rpy="0 0 0"/>
-			<parent link="${prefix}base_link"/>
-			<child link="${prefix}base"/>
-		</joint>
-	</xacro:macro>
+  <xacro:macro name="motoman_sia30d" params="prefix">
+    <!-- Properties -->
+    <material name="yaskawa_blue">
+      <color rgba="0.12941 0.14902 0.74902 1" />
+    </material>
+      <material name="silver">
+      <color rgba="0.8 0.8 0.8 1"/>
+    </material>
+    <!-- link list -->
+    <link name="${prefix}base_link">
+      <visual>
+        <geometry>
+          <mesh filename="package://motoman_sia30d_support/meshes/visual/base_link.stl"/>
+        </geometry>
+        <material name="yaskawa_blue"/>
+      </visual>
+      <collision>
+        <geometry>
+          <mesh filename="package://motoman_sia30d_support/meshes/collision/base_link.stl"/>
+        </geometry>
+      </collision>
+    </link>
+    <link name="${prefix}link_1_s">
+      <visual>
+        <geometry>
+          <mesh filename="package://motoman_sia30d_support/meshes/visual/link_1_s.stl"/>
+        </geometry>
+        <material name="silver"/>
+      </visual>
+      <collision>
+        <geometry>
+          <mesh filename="package://motoman_sia30d_support/meshes/collision/link_1_s.stl"/>
+        </geometry>
+      </collision>
+    </link>
+    <link name="${prefix}link_2_l">
+      <visual>
+        <geometry>
+          <mesh filename="package://motoman_sia30d_support/meshes/visual/link_2_l.stl"/>
+        </geometry>
+        <material name="yaskawa_blue"/>
+      </visual>
+      <collision>
+        <geometry>
+          <mesh filename="package://motoman_sia30d_support/meshes/collision/link_2_l.stl"/>
+        </geometry>
+      </collision>
+    </link>
+    <link name="${prefix}link_3_e">
+      <visual>
+        <geometry>
+          <mesh filename="package://motoman_sia30d_support/meshes/visual/link_3_e.stl"/>
+        </geometry>
+        <material name="silver"/>
+      </visual>
+      <collision>
+        <geometry>
+          <mesh filename="package://motoman_sia30d_support/meshes/collision/link_3_e.stl"/>
+        </geometry>
+      </collision>
+    </link>
+    <link name="${prefix}link_4_u">
+      <visual>
+        <geometry>
+          <mesh filename="package://motoman_sia30d_support/meshes/visual/link_4_u.stl"/>
+        </geometry>
+        <material name="yaskawa_blue"/>
+      </visual>
+      <collision>
+        <geometry>
+          <mesh filename="package://motoman_sia30d_support/meshes/collision/link_4_u.stl"/>
+        </geometry>
+      </collision>
+    </link>
+    <link name="${prefix}link_5_r">
+      <visual>
+        <geometry>
+          <mesh filename="package://motoman_sia30d_support/meshes/visual/link_5_r.stl"/>
+        </geometry>
+        <material name="silver"/>
+      </visual>
+      <collision>
+        <geometry>
+          <mesh filename="package://motoman_sia30d_support/meshes/collision/link_5_r.stl"/>
+        </geometry>
+      </collision>
+    </link>
+    <link name="${prefix}link_6_b">
+      <visual>
+        <geometry>
+          <mesh filename="package://motoman_sia30d_support/meshes/visual/link_6_b.stl"/>
+        </geometry>
+        <material name="yaskawa_blue"/>
+      </visual>
+      <collision>
+        <geometry>
+          <mesh filename="package://motoman_sia30d_support/meshes/collision/link_6_b.stl"/>
+        </geometry>
+      </collision>
+    </link>
+    <link name="${prefix}link_7_t">
+      <visual>
+        <geometry>
+          <mesh filename="package://motoman_sia30d_support/meshes/visual/link_7_t.stl"/>
+        </geometry>
+        <material name="silver"/>
+      </visual>
+      <collision>
+        <geometry>
+          <mesh filename="package://motoman_sia30d_support/meshes/collision/link_7_t.stl"/>
+        </geometry>
+      </collision>
+    </link>
+    <link name="${prefix}tool0" />
+    <!-- end of link list -->
+    <!-- joint list -->
+    <joint name="${prefix}joint_1_s" type="revolute">
+      <parent link="${prefix}base_link"/>
+      <child link="${prefix}link_1_s"/>
+      <origin xyz="0 0 0.598" rpy="0 0 0" />
+      <axis xyz="0 0 1" />
+      <limit lower="${radians(-180)}" upper="${radians(180)}" effort="1911" velocity="${radians(130)}"/>
+    </joint>
+    <joint name="${prefix}joint_2_l" type="revolute">
+      <parent link="${prefix}link_1_s"/>
+      <child link="${prefix}link_2_l"/>
+      <origin xyz="0 0 0" rpy="0 0 0" />
+      <axis xyz="0 1 0" />
+      <limit lower="${radians(-125)}" upper="${radians(125)}" effort="2388" velocity="${radians(130)}"/>
+    </joint>
+    <joint name="${prefix}joint_3_e" type="revolute">
+      <parent link="${prefix}link_2_l"/>
+      <child link="${prefix}link_3_e"/>
+      <origin xyz="0 0 0.875" rpy="0 0 0" />
+      <axis xyz="0 0 1" />
+      <limit lower="${radians(-170)}" upper="${radians(170)}" effort="674" velocity="${radians(130)}"/>
+    </joint>
+    <joint name="${prefix}joint_4_u" type="revolute">
+      <parent link="${prefix}link_3_e"/>
+      <child link="${prefix}link_4_u"/>
+      <origin xyz="0 0 0" rpy="0 0 0" />
+      <axis xyz="0 -1 0" />
+      <limit lower="${radians(-110)}" upper="${radians(110)}" effort="674" velocity="${radians(130)}"/>
+    </joint>
+    <joint name="${prefix}joint_5_r" type="revolute">
+      <parent link="${prefix}link_4_u"/>
+      <child link="${prefix}link_5_r"/>
+      <origin xyz="0 0 0.610" rpy="0 0 0" />
+      <axis xyz="0 0 -1" />
+      <limit lower="${radians(-170)}" upper="${radians(170)}" effort="191" velocity="${radians(170)}"/>
+    </joint>
+    <joint name="${prefix}joint_6_b" type="revolute">
+      <parent link="${prefix}link_5_r"/>
+      <child link="${prefix}link_6_b"/>
+      <origin xyz="0 0 0" rpy="0 0 0" />
+      <axis xyz="0 -1 0" />
+      <limit lower="${radians(-110)}" upper="${radians(110)}" effort="191" velocity="${radians(170)}"/>
+    </joint>
+    <joint name="${prefix}joint_7_t" type="revolute">
+      <parent link="${prefix}link_6_b"/>
+      <child link="${prefix}link_7_t"/>
+      <origin xyz="0 0 0" rpy="0 0 0" />
+      <axis xyz="0 0 -1" />
+      <limit lower="${radians(-180)}" upper="${radians(180)}" effort="77" velocity="${radians(200)}"/>
+    </joint>
+    <joint name="${prefix}link_7_t-tool0" type="fixed" >
+      <origin xyz="0 0 0.217" rpy="0 0 ${pi}"/>
+      <parent link="${prefix}link_7_t" />
+      <child link="${prefix}tool0" />
+    </joint>
+    <!-- end of joint list -->
+    <!-- ROS base_link to Robot Manufacturer World Coordinates transform -->
+    <link name="${prefix}base" />
+    <joint name="${prefix}base_link-base" type="fixed">
+      <origin xyz="0 0 0.598" rpy="0 0 0"/>
+      <parent link="${prefix}base_link"/>
+      <child link="${prefix}base"/>
+    </joint>
+  </xacro:macro>
 </robot>
