Commit message: Move tool0 link & joint to end of file

File: motoman_sia30d_support/urdf/sia30d_macro.xacro (robot description, xacro)
@@ -114,5 +114,4 @@
       </collision>
     </link>
-    <link name="${prefix}tool0" />
     <!-- end of link list -->
     <!-- joint list -->
@@ -166,9 +165,4 @@
       <limit lower="${radians(-180)}" upper="${radians(180)}" effort="77" velocity="${radians(200)}"/>
     </joint>
-    <joint name="${prefix}link_7_t-tool0" type="fixed" >
-      <origin xyz="0 0 0.217" rpy="0 0 ${pi}"/>
-      <parent link="${prefix}link_7_t" />
-      <child link="${prefix}tool0" />
-    </joint>
     <!-- end of joint list -->
     <!-- ROS base_link to Robot Manufacturer World Coordinates transform -->
@@ -179,4 +173,11 @@
       <child link="${prefix}base"/>
     </joint>
+    <!-- ROS-Industrial 'tool0' frame: all-zeros tool frame -->
+    <link name="${prefix}tool0" />
+    <joint name="${prefix}link_7_t-tool0" type="fixed">
+      <origin xyz="0 0 0.217" rpy="0 0 ${pi}"/>
+      <parent link="${prefix}link_7_t" />
+      <child link="${prefix}tool0" />
+    </joint>
   </xacro:macro>
 </robot>

Commit message: sia30: use materials from resources package
Instead of package-local material defs.

File: motoman_sia30d_support/urdf/sia30d_macro.xacro (robot description, xacro)
@@ -2,11 +2,5 @@
 <robot xmlns:xacro="http://ros.org/wiki/xacro">
   <xacro:macro name="motoman_sia30d" params="prefix">
-    <!-- Properties -->
-    <material name="yaskawa_blue">
-      <color rgba="0.12941 0.14902 0.74902 1" />
-    </material>
-      <material name="silver">
-      <color rgba="0.8 0.8 0.8 1"/>
-    </material>
+    <xacro:include filename="$(find motoman_resources)/urdf/common_materials.xacro"/>
     <!-- link list -->
     <link name="${prefix}base_link">
@@ -15,5 +9,5 @@
           <mesh filename="package://motoman_sia30d_support/meshes/visual/base_link.stl"/>
         </geometry>
-        <material name="yaskawa_blue"/>
+        <xacro:material_yaskawa_blue/>
       </visual>
       <collision>
@@ -28,5 +22,5 @@
           <mesh filename="package://motoman_sia30d_support/meshes/visual/link_1_s.stl"/>
         </geometry>
-        <material name="silver"/>
+        <xacro:material_yaskawa_silver/>
       </visual>
       <collision>
@@ -41,5 +35,5 @@
           <mesh filename="package://motoman_sia30d_support/meshes/visual/link_2_l.stl"/>
         </geometry>
-        <material name="yaskawa_blue"/>
+        <xacro:material_yaskawa_blue/>
       </visual>
       <collision>
@@ -54,5 +48,5 @@
           <mesh filename="package://motoman_sia30d_support/meshes/visual/link_3_e.stl"/>
         </geometry>
-        <material name="silver"/>
+        <xacro:material_yaskawa_silver/>
       </visual>
       <collision>
@@ -67,5 +61,5 @@
           <mesh filename="package://motoman_sia30d_support/meshes/visual/link_4_u.stl"/>
         </geometry>
-        <material name="yaskawa_blue"/>
+        <xacro:material_yaskawa_blue/>
       </visual>
       <collision>
@@ -80,5 +74,5 @@
           <mesh filename="package://motoman_sia30d_support/meshes/visual/link_5_r.stl"/>
         </geometry>
-        <material name="silver"/>
+        <xacro:material_yaskawa_silver/>
       </visual>
       <collision>
@@ -93,5 +87,5 @@
           <mesh filename="package://motoman_sia30d_support/meshes/visual/link_6_b.stl"/>
         </geometry>
-        <material name="yaskawa_blue"/>
+        <xacro:material_yaskawa_blue/>
       </visual>
       <collision>
@@ -106,5 +100,5 @@
           <mesh filename="package://motoman_sia30d_support/meshes/visual/link_7_t.stl"/>
         </geometry>
-        <material name="silver"/>
+        <xacro:material_yaskawa_silver/>
       </visual>
       <collision>
