Commit message: fixed joint limits

File: motoman_gp200r_support/urdf/gp200r_macro.xacro (robot description, xacro)
@@ -106,5 +106,5 @@
         <origin xyz="0 0 0.450" rpy="0 0 0" />
         <axis xyz="0 0 1" />
-        <limit lower="${radians(-179)}" upper="${radians(179)}" effort="9414.38" velocity="${radians(125)}"/>
+        <limit lower="${radians(-180)}" upper="${radians(180)}" effort="9414.38" velocity="${radians(125)}"/>
     </joint>
     <joint name="${prefix}joint_2_l" type="revolute">
@@ -113,5 +113,5 @@
         <origin xyz="0.740 0 0" rpy="0 ${radians(90)} 0" />
         <axis xyz="0 1 0" />
-        <limit lower="${radians(-39)}" upper="${radians(169)}" effort="11645.4" velocity="${radians(115)}"/>
+        <limit lower="${radians(-130)}" upper="${radians(80)}" effort="11645.4" velocity="${radians(115)}"/>
     </joint>
     <joint name="${prefix}joint_3_u" type="revolute">
@@ -120,5 +120,5 @@
         <origin xyz="0 0 1.150" rpy="0 0 0" />
         <axis xyz="0 -1 0" />
-        <limit lower="${radians(-78.3)}" upper="${radians(77)}" effort="7060.79" velocity="${radians(125)}"/>
+        <limit lower="${radians(-78.4)}" upper="${radians(78)}" effort="7060.79" velocity="${radians(125)}"/>
     </joint>
     <joint name="${prefix}joint_4_r" type="revolute">
@@ -127,5 +127,5 @@
         <origin xyz="0 0 0.250" rpy="0 0 0" />
         <axis xyz="-1 0 0" />
-        <limit lower="${-3.13}" upper="${3.13}" effort="1392.54" velocity="${radians(182)}"/>
+        <limit lower="${-3.14}" upper="${3.14}" effort="1392.54" velocity="${radians(182)}"/>
     </joint>
     <joint name="${prefix}joint_5_b" type="revolute">
@@ -134,5 +134,5 @@
         <origin xyz="1.225 0 0" rpy="0 0 0" />
         <axis xyz="0 -1 0" />
-        <limit lower="${radians(-124)}" upper="${radians(124)}" effort="1863.26" velocity="${radians(175)}"/>
+        <limit lower="${radians(-125)}" upper="${radians(125)}" effort="1863.26" velocity="${radians(175)}"/>
     </joint>
     <joint name="${prefix}joint_6_t" type="revolute">
@@ -141,5 +141,5 @@
         <origin xyz="0.250 0 0" rpy="0 0 0" />
         <axis xyz="1 0 0" />
-        <limit lower="${-3.13}" upper="${3.13}" effort="926.73" velocity="${radians(265)}"/>
+        <limit lower="${-3.14}" upper="${3.14}" effort="926.73" velocity="${radians(265)}"/>
     </joint>
     <joint name="${prefix}joint_6_t-tool0" type="fixed">

Commit message: added base_link to robot transform back into urdf

File: motoman_gp200r_support/urdf/gp200r_macro.xacro (robot description, xacro)
@@ -150,10 +150,10 @@
     <!-- end of joint list -->
     <!-- ROS base_link to Robot Manufacturer World Coordinates transform -->
-    <!-- <link name="${prefix}base" />
+    <link name="${prefix}base" />
     <joint name="${prefix}base_link-base" type="fixed">
         <origin xyz="0 0 0.650" rpy="0 0 0"/>
         <parent link="${prefix}base_link"/>
         <child link="${prefix}base"/>
-    </joint> -->
+    </joint>
 </xacro:macro>
 </robot>

Commit message: fixed pr comments from ros-industrial

File: motoman_gp200r_support/urdf/gp200r_macro.xacro (robot description, xacro)
@@ -3,18 +3,16 @@
 <xacro:macro name="motoman_gp200r" params="prefix">
     <!-- Properties -->
-    <material name="yaskawa_blue">
-        <color rgba="0 0.35546875 0.671875 1" />
-    </material>
+    <xacro:include filename="$(find motoman_resources)/urdf/common_materials.xacro"/>
     <!-- link list -->
     <link name="${prefix}base_link">
         <visual>
             <geometry>
-                <mesh filename="package://motoman_gp200r_support/meshes/gp200r/visual/base_link.STL" scale="0.001 0.001 0.001"/>
+                <mesh filename="package://motoman_gp200r_support/meshes/gp200r/visual/base_link.stl"/>
             </geometry>
-            <material name="yaskawa_blue"/>
+            <xacro:material_yaskawa_blue/>
         </visual>
         <collision>
             <geometry>
-                <mesh filename="package://motoman_gp200r_support/meshes/gp200r/visual/base_link.STL" scale="0.001 0.001 0.001"/>
+                <mesh filename="package://motoman_gp200r_support/meshes/gp200r/collision/base_link.stl"/>
             </geometry>
         </collision>
@@ -23,11 +21,11 @@
         <visual>
             <geometry>
-                <mesh filename="package://motoman_gp200r_support/meshes/gp200r/visual/link_1_s.STL" scale="0.001 0.001 0.001"/>
+                <mesh filename="package://motoman_gp200r_support/meshes/gp200r/visual/link_1_s.stl"/>
             </geometry>
-            <material name="yaskawa_blue"/>
+            <xacro:material_yaskawa_blue/>
         </visual>
         <collision>
             <geometry>
-                <mesh filename="package://motoman_gp200r_support/meshes/gp200r/visual/link_1_s.STL" scale="0.001 0.001 0.001"/>
+                <mesh filename="package://motoman_gp200r_support/meshes/gp200r/collision/link_1_s.stl"/>
             </geometry>
         </collision>
@@ -36,11 +34,11 @@
         <visual>
             <geometry>
-                <mesh filename="package://motoman_gp200r_support/meshes/gp200r/visual/link_2_l.STL" scale="0.001 0.001 0.001"/>
+                <mesh filename="package://motoman_gp200r_support/meshes/gp200r/visual/link_2_l.stl"/>
             </geometry>
-            <material name="yaskawa_blue"/>
+            <xacro:material_yaskawa_blue/>
         </visual>
         <collision>
             <geometry>
-                <mesh filename="package://motoman_gp200r_support/meshes/gp200r/visual/link_2_l.STL" scale="0.001 0.001 0.001"/>
+                <mesh filename="package://motoman_gp200r_support/meshes/gp200r/collision/link_2_l.stl"/>
             </geometry>
         </collision>
@@ -49,11 +47,11 @@
         <visual>
             <geometry>
-                <mesh filename="package://motoman_gp200r_support/meshes/gp200r/visual/link_3_u.STL" scale="0.001 0.001 0.001"/>
+                <mesh filename="package://motoman_gp200r_support/meshes/gp200r/visual/link_3_u.stl"/>
             </geometry>
-            <material name="yaskawa_blue"/>
+            <xacro:material_yaskawa_blue/>
         </visual>
         <collision>
             <geometry>
-                <mesh filename="package://motoman_gp200r_support/meshes/gp200r/visual/link_3_u.STL" scale="0.001 0.001 0.001"/>
+                <mesh filename="package://motoman_gp200r_support/meshes/gp200r/collision/link_3_u.stl"/>
             </geometry>
         </collision>
@@ -62,11 +60,11 @@
         <visual>
             <geometry>
-                <mesh filename="package://motoman_gp200r_support/meshes/gp200r/visual/link_4_r.STL" scale="0.001 0.001 0.001"/>
+                <mesh filename="package://motoman_gp200r_support/meshes/gp200r/visual/link_4_r.stl"/>
             </geometry>
-            <material name="yaskawa_blue"/>
+            <xacro:material_yaskawa_blue/>
         </visual>
         <collision>
             <geometry>
-                <mesh filename="package://motoman_gp200r_support/meshes/gp200r/visual/link_4_r.STL" scale="0.001 0.001 0.001"/>
+                <mesh filename="package://motoman_gp200r_support/meshes/gp200r/collision/link_4_r.stl"/>
             </geometry>
         </collision>
@@ -75,11 +73,11 @@
         <visual>
             <geometry>
-                <mesh filename="package://motoman_gp200r_support/meshes/gp200r/visual/link_5_b.STL" scale="0.001 0.001 0.001"/>
+                <mesh filename="package://motoman_gp200r_support/meshes/gp200r/visual/link_5_b.stl"/>
             </geometry>
-            <material name="yaskawa_blue"/>
+            <xacro:material_yaskawa_blue/>
         </visual>
         <collision>
             <geometry>
-                <mesh filename="package://motoman_gp200r_support/meshes/gp200r/visual/link_5_b.STL" scale="0.001 0.001 0.001"/>
+                <mesh filename="package://motoman_gp200r_support/meshes/gp200r/collision/link_5_b.stl"/>
             </geometry>
         </collision>
@@ -88,15 +86,14 @@
         <visual>
             <geometry>
-                <mesh filename="package://motoman_gp200r_support/meshes/gp200r/visual/link_6_t.STL" scale="0.001 0.001 0.001"/>
+                <mesh filename="package://motoman_gp200r_support/meshes/gp200r/visual/link_6_t.stl"/>
             </geometry>
-            <material name="yaskawa_blue"/>
+            <xacro:material_yaskawa_blue/>
         </visual>
         <collision>
             <geometry>
-                <mesh filename="package://motoman_gp200r_support/meshes/gp200r/visual/link_6_t.STL" scale="0.001 0.001 0.001"/>
+                <mesh filename="package://motoman_gp200r_support/meshes/gp200r/collision/link_6_t.stl"/>
             </geometry>
         </collision>
     </link>
-    <link name="${prefix}tool0"/>
     <!-- end of link list -->
     <!-- joint list -->
@@ -106,26 +103,26 @@
         <origin xyz="0 0 0.450" rpy="0 0 0" />
         <axis xyz="0 0 1" />
-        <limit lower="${radians(-180)}" upper="${radians(180)}" effort="9414.38" velocity="${radians(125)}"/>
+        <limit lower="${radians(-180)}" upper="${radians(180)}" effort="7060.79" velocity="${radians(90)}"/>
     </joint>
     <joint name="${prefix}joint_2_l" type="revolute">
         <parent link="${prefix}link_1_s"/>
         <child link="${prefix}link_2_l"/>
-        <origin xyz="0.740 0 0" rpy="0 ${radians(90)} 0" />
+        <origin xyz="0.740 0 0" rpy="0 0 0" />
         <axis xyz="0 1 0" />
-        <limit lower="${radians(-130)}" upper="${radians(80)}" effort="11645.4" velocity="${radians(115)}"/>
+        <limit lower="${radians(-130)}" upper="${radians(80)}" effort="11032.48" velocity="${radians(85)}"/>
     </joint>
     <joint name="${prefix}joint_3_u" type="revolute">
         <parent link="${prefix}link_2_l"/>
         <child link="${prefix}link_3_u"/>
-        <origin xyz="0 0 1.150" rpy="0 0 0" />
+        <origin xyz="1.150 0 0" rpy="0 0 0" />
         <axis xyz="0 -1 0" />
-        <limit lower="${radians(-78.4)}" upper="${radians(78)}" effort="7060.79" velocity="${radians(125)}"/>
+        <limit lower="${radians(-78.4)}" upper="${radians(78)}" effort="9929.23" velocity="${radians(85)}"/>
     </joint>
     <joint name="${prefix}joint_4_r" type="revolute">
         <parent link="${prefix}link_3_u"/>
         <child link="${prefix}link_4_r"/>
-        <origin xyz="0 0 0.250" rpy="0 0 0" />
+        <origin xyz="0.250 0 0" rpy="0 ${radians(90)} 0" />
         <axis xyz="-1 0 0" />
-        <limit lower="${-3.14}" upper="${3.14}" effort="1392.54" velocity="${radians(182)}"/>
+        <limit lower="${radians(-180)}" upper="${radians(180)}" effort="2621.3" velocity="${radians(120)}"/>
     </joint>
     <joint name="${prefix}joint_5_b" type="revolute">
@@ -134,5 +131,5 @@
         <origin xyz="1.225 0 0" rpy="0 0 0" />
         <axis xyz="0 -1 0" />
-        <limit lower="${radians(-125)}" upper="${radians(125)}" effort="1863.26" velocity="${radians(175)}"/>
+        <limit lower="${radians(-125)}" upper="${radians(180)}" effort="3530.38" velocity="${radians(120)}"/>
     </joint>
     <joint name="${prefix}joint_6_t" type="revolute">
@@ -141,10 +138,10 @@
         <origin xyz="0.250 0 0" rpy="0 0 0" />
         <axis xyz="1 0 0" />
-        <limit lower="${-3.14}" upper="${3.14}" effort="926.73" velocity="${radians(265)}"/>
+        <limit lower="${radians(-180)}" upper="${radians(180)}" effort="1765.19" velocity="${radians(190)}"/>
     </joint>
     <joint name="${prefix}joint_6_t-tool0" type="fixed">
         <origin xyz="0 0 0" rpy="${radians(180)} ${radians(-90)} 0"/>
         <parent link="${prefix}link_6_t"/>
-        <child link="${prefix}tool0"/>
+        <child link="${prefix}flange"/>
     </joint>
     <!-- end of joint list -->
@@ -152,8 +149,22 @@
     <link name="${prefix}base" />
     <joint name="${prefix}base_link-base" type="fixed">
-        <origin xyz="0 0 0.650" rpy="0 0 0"/>
+        <origin xyz="0 0 0.450" rpy="0 0 0"/>
         <parent link="${prefix}base_link"/>
         <child link="${prefix}base"/>
     </joint>
+    <!-- ROS-Industrial 'flange' frame: attachment point for EEF models -->
+    <link name="${prefix}flange"/>
+    <joint name="${prefix}joint_6_t-flange" type="fixed">
+      <origin xyz="0 0 0" rpy="0 0 0"/>
+      <parent link="${prefix}link_6_t"/>
+      <child link="${prefix}flange"/>
+    </joint>
+    <!-- ROS-Industrial 'tool0' frame: all-zeros tool frame -->
+    <link name="${prefix}tool0"/>
+    <joint name="${prefix}flange-tool0" type="fixed">
+      <origin xyz="0 0 0" rpy="${radians(180)} ${radians(-90)} 0"/>
+      <parent link="${prefix}flange"/>
+      <child link="${prefix}tool0"/>
+    </joint>
 </xacro:macro>
 </robot>

Commit message: added ROS-I maintainer to list, removed extra joint_6_t-flange from macro_xacro

File: motoman_gp200r_support/urdf/gp200r_macro.xacro (robot description, xacro)
@@ -140,9 +140,4 @@
         <limit lower="${radians(-180)}" upper="${radians(180)}" effort="1765.19" velocity="${radians(190)}"/>
     </joint>
-    <joint name="${prefix}joint_6_t-tool0" type="fixed">
-        <origin xyz="0 0 0" rpy="${radians(180)} ${radians(-90)} 0"/>
-        <parent link="${prefix}link_6_t"/>
-        <child link="${prefix}flange"/>
-    </joint>
     <!-- end of joint list -->
     <!-- ROS base_link to Robot Manufacturer World Coordinates transform -->
