Commit message: use correct MH110 efforts instead of GP110 values

File: motoman_mh110_support/urdf/mh110_macro.xacro (robot description, xacro)
@@ -102,5 +102,5 @@
       <origin xyz="0 0 0.540" rpy="0 0 0" />
       <axis xyz="0 0 1" />
-      <limit lower="${radians(-180)}" upper="${radians(180)}" effort="4596.87" velocity="${radians(140)}"/>
+      <limit lower="${radians(-180)}" upper="${radians(180)}" effort="5516.24" velocity="${radians(140)}"/>
     </joint>
     <joint name="${prefix}joint_2_l" type="revolute">
@@ -109,5 +109,5 @@
       <origin xyz="0.320 0 0" rpy="0 0 0" />
       <axis xyz="0 1 0" />
-      <limit lower="${radians(-90)}" upper="${radians(155)}" effort="11032.48" velocity="${radians(110)}"/>
+      <limit lower="${radians(-90)}" upper="${radians(155)}" effort="11645.40" velocity="${radians(110)}"/>
     </joint>
     <joint name="${prefix}joint_3_u" type="revolute">
@@ -116,5 +116,5 @@
       <origin xyz="0 0 0.870" rpy="0 0 0" />
       <axis xyz="0 -1 0" />
-      <limit lower="${radians(-80)}" upper="${radians(90)}" effort="5148.49" velocity="${radians(130)}"/>
+      <limit lower="${radians(-80)}" upper="${radians(90)}" effort="4167.83" velocity="${radians(130)}"/>
     </joint>
     <joint name="${prefix}joint_4_r" type="revolute">
@@ -130,5 +130,5 @@
       <origin xyz="1.020 0 0" rpy="0 0 0" />
       <axis xyz="0 -1 0" />
-      <limit lower="${radians(-125)}" upper="${radians(125)}" effort="1323.90" velocity="${radians(175)}"/>
+      <limit lower="${radians(-125)}" upper="${radians(125)}" effort="1176.80" velocity="${radians(175)}"/>
     </joint>
     <joint name="${prefix}joint_6_t" type="revolute">
