Commit message: fix flange orientation, should be +X forward

File: motoman_gp110_support/urdf/gp110_macro.xacro (robot description, xacro)
@@ -143,5 +143,5 @@
     <link name="${prefix}flange"/>
     <joint name="${prefix}joint_6_t-flange" type="fixed">
-      <origin xyz="0.200 0 0" rpy="${radians(180)} ${radians(-90)} 0"/>
+      <origin xyz="0.200 0 0" rpy="0 0 0"/>
       <parent link="${prefix}link_6_t"/>
       <child link="${prefix}flange"/>
@@ -150,5 +150,5 @@
     <link name="${prefix}tool0"/>
     <joint name="${prefix}flange-tool0" type="fixed">
-      <origin xyz="0 0 0" rpy="0 0 0"/>
+      <origin xyz="0 0 0" rpy="${radians(180)} ${radians(-90)} 0"/>
       <parent link="${prefix}flange"/>
       <child link="${prefix}tool0"/>
