Commit message: gp4: move 'flange' down below regular links & joints

File: motoman_gp4_support/urdf/gp4_macro.xacro (robot description, xacro)
@@ -139,5 +139,6 @@
       <limit lower="${radians(-455)}" upper="${radians(455)}" effort="16.46" velocity="${radians(1000)}"/>
     </joint>
-     <link name="${prefix}flange"/>
+    <!-- end of joint list -->
+    <link name="${prefix}flange"/>
     <joint name="${prefix}joint_6_t-flange" type="fixed">
       <origin xyz="0.072 0 0" rpy="${radians(180)} ${radians(-90)} 0"/>
@@ -145,5 +146,4 @@
       <child link="${prefix}flange"/>
     </joint>
-    <!-- end of joint list -->
     <!-- default tool -->
     <link name="${prefix}tool0"/>

Commit message: apply flange orientation fix to gp4 as well

File: motoman_gp4_support/urdf/gp4_macro.xacro (robot description, xacro)
@@ -143,5 +143,5 @@
     <link name="${prefix}flange"/>
     <joint name="${prefix}joint_6_t-flange" type="fixed">
-      <origin xyz="0.072 0 0" rpy="${radians(180)} ${radians(-90)} 0"/>
+      <origin xyz="0.072 0 0" rpy="0 0 0"/>
       <parent link="${prefix}link_6_t"/>
       <child link="${prefix}flange"/>
@@ -150,5 +150,5 @@
     <link name="${prefix}tool0"/>
     <joint name="${prefix}flange-tool0" type="fixed">
-      <origin xyz="0 0 0" rpy="0 0 0"/>
+      <origin xyz="0 0 0" rpy="${radians(180)} ${radians(-90)} 0"/>
       <parent link="${prefix}flange"/>
       <child link="${prefix}tool0"/>
