Commit message: Rename package to remove hyphen in name
Rename 'motoman_gp215-250_support' to 'motoman_gp215_250_support'

File: motoman_gp215_250_support/urdf/gp215.xacro (robot description, xacro)
@@ -1,5 +1,5 @@
 <?xml version="1.0" ?>
 <robot name="motoman_gp215" xmlns:xacro="http://ros.org/wiki/xacro">
-  <xacro:include filename="$(find motoman_gp215-250_support)/urdf/gp215_macro.xacro" />
+  <xacro:include filename="$(find motoman_gp215_250_support)/urdf/gp215_macro.xacro" />
   <xacro:motoman_gp215 prefix=""/>
 </robot>

File: motoman_gp215_250_support/urdf/gp215_macro.xacro (robot description, xacro)
@@ -1,5 +1,5 @@
 <?xml version="1.0" ?>
 <robot xmlns:xacro="http://ros.org/wiki/xacro">
-  <xacro:macro name="motoman_gp250" params="prefix">
+  <xacro:macro name="motoman_gp215" params="prefix">
     <xacro:include filename="$(find motoman_resources)/urdf/common_materials.xacro"/>
     <!-- link list -->
@@ -7,5 +7,5 @@
       <visual>
         <geometry>
-          <mesh filename="package://motoman_gp215-250_support/meshes/gp215/visual/base_link.dae"/>
+          <mesh filename="package://motoman_gp215_250_support/meshes/gp215/visual/base_link.dae"/>
         </geometry>
         <xacro:material_yaskawa_blue/>
@@ -13,5 +13,5 @@
       <collision>
         <geometry>
-          <mesh filename="package://motoman_gp215-250_support/meshes/gp215/collision/base_link.stl"/>
+          <mesh filename="package://motoman_gp215_250_support/meshes/gp215/collision/base_link.stl"/>
         </geometry>
       </collision>
@@ -20,5 +20,5 @@
       <visual>
         <geometry>
-          <mesh filename="package://motoman_gp215-250_support/meshes/gp215/visual/link_1_s.dae"/>
+          <mesh filename="package://motoman_gp215_250_support/meshes/gp215/visual/link_1_s.dae"/>
         </geometry>
         <xacro:material_yaskawa_blue/>
@@ -26,5 +26,5 @@
       <collision>
         <geometry>
-          <mesh filename="package://motoman_gp215-250_support/meshes/gp215/collision/link_1_s.stl"/>
+          <mesh filename="package://motoman_gp215_250_support/meshes/gp215/collision/link_1_s.stl"/>
         </geometry>
       </collision>
@@ -33,5 +33,5 @@
       <visual>
         <geometry>
-          <mesh filename="package://motoman_gp215-250_support/meshes/gp215/visual/link_2_l.dae"/>
+          <mesh filename="package://motoman_gp215_250_support/meshes/gp215/visual/link_2_l.dae"/>
         </geometry>
         <xacro:material_yaskawa_blue/>
@@ -39,5 +39,5 @@
       <collision>
         <geometry>
-          <mesh filename="package://motoman_gp215-250_support/meshes/gp215/collision/link_2_l.stl"/>
+          <mesh filename="package://motoman_gp215_250_support/meshes/gp215/collision/link_2_l.stl"/>
         </geometry>
       </collision>
@@ -46,5 +46,5 @@
       <visual>
         <geometry>
-          <mesh filename="package://motoman_gp215-250_support/meshes/gp250/visual/link_3_u.dae"/>
+          <mesh filename="package://motoman_gp215_250_support/meshes/gp215/visual/link_3_u.dae"/>
         </geometry>
         <xacro:material_yaskawa_blue/>
@@ -52,5 +52,5 @@
       <collision>
         <geometry>
-          <mesh filename="package://motoman_gp215-250_support/meshes/gp250/collision/link_3_u.stl"/>
+          <mesh filename="package://motoman_gp215_250_support/meshes/gp215/collision/link_3_u.stl"/>
         </geometry>
       </collision>
@@ -59,5 +59,5 @@
       <visual>
         <geometry>
-          <mesh filename="package://motoman_gp215-250_support/meshes/gp215/visual/link_4_r.dae"/>
+          <mesh filename="package://motoman_gp215_250_support/meshes/gp215/visual/link_4_r.dae"/>
         </geometry>
         <xacro:material_yaskawa_blue/>
@@ -65,5 +65,5 @@
       <collision>
         <geometry>
-          <mesh filename="package://motoman_gp215-250_support/meshes/gp215/collision/link_4_r.stl"/>
+          <mesh filename="package://motoman_gp215_250_support/meshes/gp215/collision/link_4_r.stl"/>
         </geometry>
       </collision>
@@ -72,5 +72,5 @@
       <visual>
         <geometry>
-          <mesh filename="package://motoman_gp215-250_support/meshes/gp215/visual/link_5_b.dae"/>
+          <mesh filename="package://motoman_gp215_250_support/meshes/gp215/visual/link_5_b.dae"/>
         </geometry>
         <xacro:material_yaskawa_blue/>
@@ -78,5 +78,5 @@
       <collision>
         <geometry>
-          <mesh filename="package://motoman_gp215-250_support/meshes/gp215/collision/link_5_b.stl"/>
+          <mesh filename="package://motoman_gp215_250_support/meshes/gp215/collision/link_5_b.stl"/>
         </geometry>
       </collision>
@@ -85,5 +85,5 @@
       <visual>
         <geometry>
-          <mesh filename="package://motoman_gp215-250_support/meshes/gp215/visual/link_6_t.dae"/>
+          <mesh filename="package://motoman_gp215_250_support/meshes/gp215/visual/link_6_t.dae"/>
         </geometry>
         <xacro:material_yaskawa_silver/>
@@ -91,5 +91,5 @@
       <collision>
         <geometry>
-          <mesh filename="package://motoman_gp215-250_support/meshes/gp215/collision/link_6_t.stl"/>
+          <mesh filename="package://motoman_gp215_250_support/meshes/gp215/collision/link_6_t.stl"/>
         </geometry>
       </collision>
@@ -121,5 +121,5 @@
       <parent link="${prefix}link_3_u"/>
       <child link="${prefix}link_4_r"/>
-      <origin xyz="1.285 0 0.250" rpy="0 0 0" />
+      <origin xyz="1.490 0 0.250" rpy="0 0 0" />
       <axis xyz="-1 0 0" />
       <limit lower="${radians(-360)}" upper="${radians(360)}" effort="2758.0" velocity="${radians(120)}"/>

File: motoman_gp215_250_support/urdf/gp250.xacro (robot description, xacro)
@@ -1,5 +1,5 @@
 <?xml version="1.0" ?>
 <robot name="motoman_gp250" xmlns:xacro="http://ros.org/wiki/xacro">
-  <xacro:include filename="$(find motoman_gp215-250_support)/urdf/gp250_macro.xacro" />
+  <xacro:include filename="$(find motoman_gp215_250_support)/urdf/gp250_macro.xacro" />
   <xacro:motoman_gp250 prefix=""/>
 </robot>

File: motoman_gp215_250_support/urdf/gp250_macro.xacro (robot description, xacro)
@@ -1,5 +1,5 @@
 <?xml version="1.0" ?>
 <robot xmlns:xacro="http://ros.org/wiki/xacro">
-  <xacro:macro name="motoman_gp215" params="prefix">
+  <xacro:macro name="motoman_gp250" params="prefix">
     <xacro:include filename="$(find motoman_resources)/urdf/common_materials.xacro"/>
     <!-- link list -->
@@ -7,5 +7,5 @@
       <visual>
         <geometry>
-          <mesh filename="package://motoman_gp215-250_support/meshes/gp215/visual/base_link.dae"/>
+          <mesh filename="package://motoman_gp215_250_support/meshes/gp215/visual/base_link.dae"/>
         </geometry>
         <xacro:material_yaskawa_blue/>
@@ -13,5 +13,5 @@
       <collision>
         <geometry>
-          <mesh filename="package://motoman_gp215-250_support/meshes/gp215/collision/base_link.stl"/>
+          <mesh filename="package://motoman_gp215_250_support/meshes/gp215/collision/base_link.stl"/>
         </geometry>
       </collision>
@@ -20,5 +20,5 @@
       <visual>
         <geometry>
-          <mesh filename="package://motoman_gp215-250_support/meshes/gp215/visual/link_1_s.dae"/>
+          <mesh filename="package://motoman_gp215_250_support/meshes/gp215/visual/link_1_s.dae"/>
         </geometry>
         <xacro:material_yaskawa_blue/>
@@ -26,5 +26,5 @@
       <collision>
         <geometry>
-          <mesh filename="package://motoman_gp215-250_support/meshes/gp215/collision/link_1_s.stl"/>
+          <mesh filename="package://motoman_gp215_250_support/meshes/gp215/collision/link_1_s.stl"/>
         </geometry>
       </collision>
@@ -33,5 +33,5 @@
       <visual>
         <geometry>
-          <mesh filename="package://motoman_gp215-250_support/meshes/gp215/visual/link_2_l.dae"/>
+          <mesh filename="package://motoman_gp215_250_support/meshes/gp215/visual/link_2_l.dae"/>
         </geometry>
         <xacro:material_yaskawa_blue/>
@@ -39,5 +39,5 @@
       <collision>
         <geometry>
-          <mesh filename="package://motoman_gp215-250_support/meshes/gp215/collision/link_2_l.stl"/>
+          <mesh filename="package://motoman_gp215_250_support/meshes/gp215/collision/link_2_l.stl"/>
         </geometry>
       </collision>
@@ -46,5 +46,5 @@
       <visual>
         <geometry>
-          <mesh filename="package://motoman_gp215-250_support/meshes/gp215/visual/link_3_u.dae"/>
+          <mesh filename="package://motoman_gp215_250_support/meshes/gp250/visual/link_3_u.dae"/>
         </geometry>
         <xacro:material_yaskawa_blue/>
@@ -52,5 +52,5 @@
       <collision>
         <geometry>
-          <mesh filename="package://motoman_gp215-250_support/meshes/gp215/collision/link_3_u.stl"/>
+          <mesh filename="package://motoman_gp215_250_support/meshes/gp250/collision/link_3_u.stl"/>
         </geometry>
       </collision>
@@ -59,5 +59,5 @@
       <visual>
         <geometry>
-          <mesh filename="package://motoman_gp215-250_support/meshes/gp215/visual/link_4_r.dae"/>
+          <mesh filename="package://motoman_gp215_250_support/meshes/gp215/visual/link_4_r.dae"/>
         </geometry>
         <xacro:material_yaskawa_blue/>
@@ -65,5 +65,5 @@
       <collision>
         <geometry>
-          <mesh filename="package://motoman_gp215-250_support/meshes/gp215/collision/link_4_r.stl"/>
+          <mesh filename="package://motoman_gp215_250_support/meshes/gp215/collision/link_4_r.stl"/>
         </geometry>
       </collision>
@@ -72,5 +72,5 @@
       <visual>
         <geometry>
-          <mesh filename="package://motoman_gp215-250_support/meshes/gp215/visual/link_5_b.dae"/>
+          <mesh filename="package://motoman_gp215_250_support/meshes/gp215/visual/link_5_b.dae"/>
         </geometry>
         <xacro:material_yaskawa_blue/>
@@ -78,5 +78,5 @@
       <collision>
         <geometry>
-          <mesh filename="package://motoman_gp215-250_support/meshes/gp215/collision/link_5_b.stl"/>
+          <mesh filename="package://motoman_gp215_250_support/meshes/gp215/collision/link_5_b.stl"/>
         </geometry>
       </collision>
@@ -85,5 +85,5 @@
       <visual>
         <geometry>
-          <mesh filename="package://motoman_gp215-250_support/meshes/gp215/visual/link_6_t.dae"/>
+          <mesh filename="package://motoman_gp215_250_support/meshes/gp215/visual/link_6_t.dae"/>
         </geometry>
         <xacro:material_yaskawa_silver/>
@@ -91,5 +91,5 @@
       <collision>
         <geometry>
-          <mesh filename="package://motoman_gp215-250_support/meshes/gp215/collision/link_6_t.stl"/>
+          <mesh filename="package://motoman_gp215_250_support/meshes/gp215/collision/link_6_t.stl"/>
         </geometry>
       </collision>
@@ -121,5 +121,5 @@
       <parent link="${prefix}link_3_u"/>
       <child link="${prefix}link_4_r"/>
-      <origin xyz="1.490 0 0.250" rpy="0 0 0" />
+      <origin xyz="1.285 0 0.250" rpy="0 0 0" />
       <axis xyz="-1 0 0" />
       <limit lower="${radians(-360)}" upper="${radians(360)}" effort="2758.0" velocity="${radians(120)}"/>
