Commit message: Treat the 'equipped' variant as a proper variant
Needs some file duplication, but it's at least consistent with other packages.

File: motoman_gp165r_support/urdf/gp165r_equipped_macro.xacro (robot description, xacro)
@@ -1,5 +1,5 @@
 <?xml version="1.0" ?>
 <robot xmlns:xacro="http://ros.org/wiki/xacro">
-<xacro:macro name="motoman_gp165r" params="prefix">
+<xacro:macro name="motoman_gp165r_equipped" params="prefix">
     <!-- Properties -->
     <xacro:include filename="$(find motoman_resources)/urdf/common_materials.xacro"/>
