Commit message: Added collision model

File: motoman_up50n_support/urdf/up50n_35_macro.xacro (robot description, xacro)
@@ -13,5 +13,5 @@
         <collision>
             <geometry>
-                <mesh filename="package://motoman_up50n_support/meshes/up50n_35/visual/base_link.dae"/>
+                <mesh filename="package://motoman_up50n_support/meshes/up50n_35/collision/base_link.stl"/>
             </geometry>
         </collision>
@@ -26,5 +26,5 @@
         <collision>
             <geometry>
-                <mesh filename="package://motoman_up50n_support/meshes/up50n_35/visual/link_1_s.dae"/>
+                <mesh filename="package://motoman_up50n_support/meshes/up50n_35/collision/link_1_s.stl"/>
             </geometry>
         </collision>
@@ -39,5 +39,5 @@
         <collision>
             <geometry>
-                <mesh filename="package://motoman_up50n_support/meshes/up50n_35/visual/link_2_l.dae"/>
+                <mesh filename="package://motoman_up50n_support/meshes/up50n_35/collision/link_2_l.stl"/>
             </geometry>
         </collision>
@@ -52,5 +52,5 @@
         <collision>
             <geometry>
-                <mesh filename="package://motoman_up50n_support/meshes/up50n_35/visual/link_3_u.dae"/>
+                <mesh filename="package://motoman_up50n_support/meshes/up50n_35/collision/link_3_u.stl"/>
             </geometry>
         </collision>
@@ -65,5 +65,5 @@
         <collision>
             <geometry>
-                <mesh filename="package://motoman_up50n_support/meshes/up50n_35/visual/link_4_r.dae"/>
+                <mesh filename="package://motoman_up50n_support/meshes/up50n_35/collision/link_4_r.stl"/>
             </geometry>
         </collision>
@@ -78,5 +78,5 @@
         <collision>
             <geometry>
-                <mesh filename="package://motoman_up50n_support/meshes/up50n_35/visual/link_5_b.dae"/>
+                <mesh filename="package://motoman_up50n_support/meshes/up50n_35/collision/link_5_b.stl"/>
             </geometry>
         </collision>
@@ -91,5 +91,5 @@
         <collision>
             <geometry>
-                <mesh filename="package://motoman_up50n_support/meshes/up50n_35/visual/link_6_t.dae"/>
+                <mesh filename="package://motoman_up50n_support/meshes/up50n_35/collision/link_6_t.stl"/>
             </geometry>
         </collision>

Commit message: Formatting (xacro:macro)

File: motoman_up50n_support/urdf/up50n_35_macro.xacro (robot description, xacro)
@@ -143,14 +143,14 @@
     <link name="${prefix}flange"/>
     <joint name="${prefix}joint_6_t-flange" type="fixed">
-      <origin xyz="0.175 0 0" rpy="0 0 0"/>
-      <parent link="${prefix}link_6_t"/>
-      <child link="${prefix}flange"/>
+        <origin xyz="0.175 0 0" rpy="0 0 0"/>
+        <parent link="${prefix}link_6_t"/>
+        <child link="${prefix}flange"/>
     </joint>
     <!-- ROS-Industrial 'tool0' frame: all-zeros tool frame -->
     <link name="${prefix}tool0"/>
     <joint name="${prefix}flange-tool0" type="fixed">
-      <origin xyz="0 0 0" rpy="${radians(180)} ${radians(-90)} 0"/>
-      <parent link="${prefix}flange"/>
-      <child link="${prefix}tool0"/>
+        <origin xyz="0 0 0" rpy="${radians(180)} ${radians(-90)} 0"/>
+        <parent link="${prefix}flange"/>
+        <child link="${prefix}tool0"/>
     </joint>
     <!-- ROS base_link to Robot Manufacturer World Coordinates transform -->
